File: CANBuster/CANBuster.sch (KiCad schematic (older format))
At the start: 6 parts, among them U1 PIC18(L)F45K80-I/P, Y1 16MHz

Commit message: wip
Parts:
- added C1, C2, C6: 100nF, symbol C
- added U2: MCP2551-I/P, DIP-8, symbol MCP2551-I/P
- C5: renamed from C3; value CP -> 47uF
- renumbered C1 to C3, C2 to C4
Connections:
- net labels added: CANH, CANL, CANRX, CANTX, RxD, TxD
- wire segments 31 -> 45
- no-connect marks 31 -> 28
Changed lines of the file:
@@
 Wire Wire Line
 	8450 5450 9000 5450
-Wire Wire Line
-	8200 5550 9000 5550
 NoConn ~ 9000 5850
 $Comp
@@
 L PWR_FLAG #FLG05
 U 1 1 55B646CE
-P 8200 5250
-F 0 "#FLG05" H 8200 5345 50  0001 C CNN
-F 1 "PWR_FLAG" H 8200 5430 50  0000 C CNN
-F 2 "" H 8200 5250 60  0000 C CNN
-F 3 "" H 8200 5250 60  0000 C CNN
-	1    8200 5250
+P 5400 5950
+F 0 "#FLG05" H 5400 6045 50  0001 C CNN
+F 1 "PWR_FLAG" H 5400 6130 50  0000 C CNN
+F 2 "" H 5400 5950 60  0000 C CNN
+F 3 "" H 5400 5950 60  0000 C CNN
+	1    5400 5950
 	1    0    0    -1
 $EndComp
@@
 L PWR_FLAG #FLG07
 U 1 1 55B651E4
-P 8200 5550
-F 0 "#FLG07" H 8200 5645 50  0001 C CNN
-F 1 "PWR_FLAG" H 8200 5730 50  0000 C CNN
-F 2 "" H 8200 5550 60  0000 C CNN
-F 3 "" H 8200 5550 60  0000 C CNN
-	1    8200 5550
-	1    0    0    -1
-$EndComp
-Connection ~ 8450 5550
-Wire Wire Line
-	8450 5300 8200 5300
-Wire Wire Line
-	8200 5300 8200 5250
+P 5500 2900
+F 0 "#FLG07" H 5500 2995 50  0001 C CNN
+F 1 "PWR_FLAG" H 5500 3080 50  0000 C CNN
+F 2 "" H 5500 2900 60  0000 C CNN
+F 3 "" H 5500 2900 60  0000 C CNN
+	1    5500 2900
+	1    0    0    -1
+$EndComp
 Wire Wire Line
 	3950 3300 3750 3300
@@
 NoConn ~ 6350 4600
 NoConn ~ 6350 4700
-NoConn ~ 6350 4800
-NoConn ~ 6350 4900
 NoConn ~ 3950 4600
 NoConn ~ 3950 4500
-NoConn ~ 3950 4400
-NoConn ~ 3950 4300
 NoConn ~ 3950 4200
 NoConn ~ 3950 4100
@@
 Connection ~ 3500 5350
 $Comp
-L C C1
+L C C3
 U 1 1 55B65742
 P 2750 5500
-F 0 "C1" H 2775 5600 50  0000 L CNN
+F 0 "C3" H 2775 5600 50  0000 L CNN
 F 1 "22pf" H 2775 5400 50  0000 L CNN
 F 2 "" H 2788 5350 30  0001 C CNN
@@
 $EndComp
 $Comp
-L C C2
+L C C4
 U 1 1 55B65839
 P 3050 5500
-F 0 "C2" H 3075 5600 50  0000 L CNN
+F 0 "C4" H 3075 5600 50  0000 L CNN
 F 1 "22pf" H 3075 5400 50  0000 L CNN
 F 2 "" H 3088 5350 30  0001 C CNN
@@
 Connection ~ 2900 5650
 $Comp
-L CP C3
+L CP C5
 U 1 1 55B65D4C
 P 4750 2700
-F 0 "C3" H 4775 2800 50  0000 L CNN
-F 1 "CP" H 4775 2600 50  0000 L CNN
+F 0 "C5" H 4775 2800 50  0000 L CNN
+F 1 "47uF" H 4775 2600 50  0000 L CNN
 F 2 "" H 4788 2550 30  0001 C CNN
 F 3 "" H 4750 2700 60  0000 C CNN
@@
 Wire Wire Line
 	5050 2550 5050 3000
+Wire Wire Line
+	3600 4300 3950 4300
+Text Label 3600 4300 0    60   ~ 0
+CANTX
+Text Label 3600 4400 0    60   ~ 0
+CANRX
+Wire Wire Line
+	6350 4800 6650 4800
+Wire Wire Line
+	6350 4900 6650 4900
+Text Label 6500 4800 0    60   ~ 0
+TxD
+Text Label 56500 -4200 0    60   ~ 0
+RxD
+Text Label 6500 4900 0    60   ~ 0
+RxD
+$Comp
+L MCP2551-I/P U2
+U 1 1 55B65B4E
+P 8850 1800
+F 0 "U2" H 8450 2150 50  0000 L CNN
+F 1 "MCP2551-I/P" H 8950 2150 50  0000 L CNN
+F 2 "DIP-8" H 8850 1800 50  0000 C CIN
+F 3 "" H 8850 1800 60  0000 C CNN
+	1    8850 1800
+	1    0    0    -1
+$EndComp
+Wire Wire Line
+	8350 1700 8050 1700
+Text Label 8050 1700 0    60   ~ 0
+CANTX
+Text Label 8050 1600 0    60   ~ 0
+CANRX
+$Comp
+L VDD #PWR010
+U 1 1 55B662A2
+P 8850 1200
+F 0 "#PWR010" H 8850 1050 50  0001 C CNN
+F 1 "VDD" H 8850 1350 50  0000 C CNN
+F 2 "" H 8850 1200 60  0000 C CNN
+F 3 "" H 8850 1200 60  0000 C CNN
+	1    8850 1200
+	1    0    0    -1
+$EndComp
+$Comp
+L GND #PWR011
+U 1 1 55B663CC
+P 8850 2300
+F 0 "#PWR011" H 8850 2050 50  0001 C CNN
+F 1 "GND" H 8850 2150 50  0000 C CNN
+F 2 "" H 8850 2300 60  0000 C CNN
+F 3 "" H 8850 2300 60  0000 C CNN
+	1    8850 2300
+	1    0    0    -1
+$EndComp
+Wire Wire Line
+	8850 1200 8850 1400
+Wire Wire Line
+	8850 2200 8850 2300
+Wire Wire Line
+	8350 2000 8150 2000
+Wire Wire Line
+	8150 2000 8150 2300
+$Comp
+L GND #PWR012
+U 1 1 55B665FF
+P 8150 2300
+F 0 "#PWR012" H 8150 2050 50  0001 C CNN
+F 1 "GND" H 8150 2150 50  0000 C CNN
+F 2 "" H 8150 2300 60  0000 C CNN
+F 3 "" H 8150 2300 60  0000 C CNN
+	1    8150 2300
+	1    0    0    -1
+$EndComp
+Wire Wire Line
+	9350 1700 9800 1700
+Wire Wire Line
+	9350 1900 9800 1900
+Text Label 9500 1900 0    60   ~ 0
+CANL
+Text Label 9500 1700 0    60   ~ 0
+CANH
+$Comp
+L VDD #PWR013
+U 1 1 55B667BB
+P 10300 1600
+F 0 "#PWR013" H 10300 1450 50  0001 C CNN
+F 1 "VDD" H 10300 1750 50  0000 C CNN
+F 2 "" H 10300 1600 60  0000 C CNN
+F 3 "" H 10300 1600 60  0000 C CNN
+	1    10300 1600
+	1    0    0    -1
+$EndComp
+$Comp
+L GND #PWR014
+U 1 1 55B667DB
+P 10300 1900
+F 0 "#PWR014" H 10300 1650 50  0001 C CNN
+F 1 "GND" H 10300 1750 50  0000 C CNN
+F 2 "" H 10300 1900 60  0000 C CNN
+F 3 "" H 10300 1900 60  0000 C CNN
+	1    10300 1900
+	1    0    0    -1
+$EndComp
+$Comp
+L C C6
+U 1 1 55B667FD
+P 10300 1750
+F 0 "C6" H 10325 1850 50  0000 L CNN
+F 1 "100nF" H 10325 1650 50  0000 L CNN
+F 2 "" H 10338 1600 30  0000 C CNN
+F 3 "" H 10300 1750 60  0000 C CNN
+	1    10300 1750
+	1    0    0    -1
+$EndComp
+$Comp
+L VDD #PWR015
+U 1 1 55B672AA
+P 5750 2550
+F 0 "#PWR015" H 5750 2400 50  0001 C CNN
+F 1 "VDD" H 5750 2700 50  0000 C CNN
+F 2 "" H 5750 2550 60  0000 C CNN
+F 3 "" H 5750 2550 60  0000 C CNN
+	1    5750 2550
+	1    0    0    -1
+$EndComp
+$Comp
+L GND #PWR016
+U 1 1 55B672CD
+P 5750 2900
+F 0 "#PWR016" H 5750 2650 50  0001 C CNN
+F 1 "GND" H 5750 2750 50  0000 C CNN
+F 2 "" H 5750 2900 60  0000 C CNN
+F 3 "" H 5750 2900 60  0000 C CNN
+	1    5750 2900
+	1    0    0    -1
+$EndComp
+$Comp
+L GND #PWR017
+U 1 1 55B672F0
+P 6050 2900
+F 0 "#PWR017" H 6050 2650 50  0001 C CNN
+F 1 "GND" H 6050 2750 50  0000 C CNN
+F 2 "" H 6050 2900 60  0000 C CNN
+F 3 "" H 6050 2900 60  0000 C CNN
+	1    6050 2900
+	1    0    0    -1
+$EndComp
+$Comp
+L VDD #PWR018
+U 1 1 55B67313
+P 6050 2550
+F 0 "#PWR018" H 6050 2400 50  0001 C CNN
+F 1 "VDD" H 6050 2700 50  0000 C CNN
+F 2 "" H 6050 2550 60  0000 C CNN
+F 3 "" H 6050 2550 60  0000 C CNN
+	1    6050 2550
+	1    0    0    -1
+$EndComp
+$Comp
+L C C1
+U 1 1 55B67336
+P 5750 2750
+F 0 "C1" H 5775 2850 50  0000 L CNN
+F 1 "100nF" H 5775 2650 50  0000 L CNN
+F 2 "" H 5788 2600 30  0000 C CNN
+F 3 "" H 5750 2750 60  0000 C CNN
+	1    5750 2750
+	1    0    0    -1
+$EndComp
+$Comp
+L C C2
+U 1 1 55B67397
+P 6050 2750
+F 0 "C2" H 6075 2850 50  0000 L CNN
+F 1 "100nF" H 6075 2650 50  0000 L CNN
+F 2 "" H 6088 2600 30  0000 C CNN
+F 3 "" H 6050 2750 60  0000 C CNN
+	1    6050 2750
+	1    0    0    -1
+$EndComp
+Wire Wire Line
+	5750 2550 5750 2600
+Wire Wire Line
+	6050 2550 6050 2600
+NoConn ~ 8350 1900
+Wire Wire Line
+	8350 1600 8050 1600
+Wire Wire Line
+	5400 5950 5100 5950
+Connection ~ 5100 5950
+Wire Wire Line
+	5500 2900 5300 2900
+Wire Wire Line
+	9000 5550 8450 5550
+Wire Wire Line
+	3950 4400 3600 4400
+Connection ~ 5350 2900
 $EndSCHEMATC

Commit message: wip
Parts:
- added P1, P2: CONN_01X08, symbol CONN_01X08
- added P3, P4, P5, P6: CONN_01X03, symbol CONN_01X03
Connections:
- net labels added: IO1, IO10, IO11, IO12, IO13, IO14, IO15, IO16, IO2, IO3, IO4, IO5, IO6, IO7, IO8, IO9, PWM1, PWM2, PWM3, PWM4, SCL, SDA
- wire segments 45 -> 103
- no-connect marks 28 -> 6

Commit message: wip
Parts:
- C1, C2, C3, C4, C6: footprint (none) -> Capacitors_ThroughHole:C_Rect_L4_W2.5_P2.5
- C5: footprint (none) -> Capacitors_Elko_ThroughHole:Elko_vert_11x5mm_RM2.5
- JP1: footprint (none) -> CANBuster:ICSP
- P1, P2: footprint (none) -> Pin_Headers:Pin_Header_Straight_1x08
- P3, P4, P5, P6: footprint (none) -> Pin_Headers:Pin_Header_Angled_1x03
- U1: footprint (none) -> Housings_DIP:DIP-40_W15.24mm_LongPads; symbol PIC18(L)F45K80-I/P -> PIC18(L)F45K80-I/P-RESCUE-CANBuster
- U2: footprint DIP-8 -> Housings_DIP:DIP-8_W7.62mm_LongPads
- Y1: footprint (none) -> Crystals:Crystal_HC49-U_Vertical
Changed lines of the file:
@@
 EESchema Schematic File Version 2
+LIBS:CANBuster-rescue
 LIBS:power
 LIBS:device
@@
 $EndDescr
 $Comp
-L PIC18(L)F45K80-I/P U1
+L PIC18(L)F45K80-I/P-RESCUE-CANBuster U1
 U 1 1 55B62FE6
 P 5150 4300
 F 0 "U1" H 4150 5500 50  0000 C CNN
 F 1 "PIC18(L)F45K80-I/P" H 5800 3100 50  0000 C CNN
-F 2 "" H 5150 4300 50  0000 C CIN
+F 2 "Housings_DIP:DIP-40_W15.24mm_LongPads" H 5150 4300 50  0001 C CIN
 F 3 "" H 4000 5500 60  0000 C CNN
 	1    5150 4300
@@
 F 0 "JP1" H 9750 5500 50  0000 C CNN
 F 1 "ICSP" H 9750 5700 50  0000 C CNN
-F 2 "" H 9750 5600 50  0001 C CNN
+F 2 "CANBuster:ICSP" H 9750 5600 50  0001 C CNN
 F 3 "DOCUMENTATION" H 9750 5600 50  0001 C CNN
 	1    9750 5600
@@
 F 0 "Y1" H 3500 5350 50  0000 C CNN
 F 1 "16MHz" H 3500 5050 50  0000 C CNN
-F 2 "" H 3500 5200 60  0001 C CNN
+F 2 "Crystals:Crystal_HC49-U_Vertical" H 3500 5200 60  0001 C CNN
 F 3 "" H 3500 5200 60  0000 C CNN
 	1    3500 5200
@@
 F 0 "C3" H 2775 5600 50  0000 L CNN
 F 1 "22pf" H 2775 5400 50  0000 L CNN
-F 2 "" H 2788 5350 30  0001 C CNN
+F 2 "Capacitors_ThroughHole:C_Rect_L4_W2.5_P2.5" H 2788 5350 30  0001 C CNN
 F 3 "" H 2750 5500 60  0000 C CNN
 	1    2750 5500
@@
 F 0 "C4" H 3075 5600 50  0000 L CNN
 F 1 "22pf" H 3075 5400 50  0000 L CNN
-F 2 "" H 3088 5350 30  0001 C CNN
+F 2 "Capacitors_ThroughHole:C_Rect_L4_W2.5_P2.5" H 3088 5350 30  0001 C CNN
 F 3 "" H 3050 5500 60  0000 C CNN
 	1    3050 5500
@@
 F 0 "C5" H 4775 2800 50  0000 L CNN
 F 1 "47uF" H 4775 2600 50  0000 L CNN
-F 2 "" H 4788 2550 30  0001 C CNN
+F 2 "Capacitors_Elko_ThroughHole:Elko_vert_11x5mm_RM2.5" H 4788 2550 30  0001 C CNN
 F 3 "" H 4750 2700 60  0000 C CNN
 	1    4750 2700
@@
 F 0 "U2" H 8450 2150 50  0000 L CNN
 F 1 "MCP2551-I/P" H 8950 2150 50  0000 L CNN
-F 2 "DIP-8" H 8850 1800 50  0000 C CIN
+F 2 "Housings_DIP:DIP-8_W7.62mm_LongPads" H 8850 1800 50  0001 C CIN
 F 3 "" H 8850 1800 60  0000 C CNN
 	1    8850 1800
@@
 F 0 "C6" H 10325 1850 50  0000 L CNN
 F 1 "100nF" H 10325 1650 50  0000 L CNN
-F 2 "" H 10338 1600 30  0000 C CNN
+F 2 "Capacitors_ThroughHole:C_Rect_L4_W2.5_P2.5" H 10338 1600 30  0001 C CNN
 F 3 "" H 10300 1750 60  0000 C CNN
 	1    10300 1750
@@
 F 0 "C1" H 5775 2850 50  0000 L CNN
 F 1 "100nF" H 5775 2650 50  0000 L CNN
-F 2 "" H 5788 2600 30  0000 C CNN
+F 2 "Capacitors_ThroughHole:C_Rect_L4_W2.5_P2.5" H 5788 2600 30  0001 C CNN
 F 3 "" H 5750 2750 60  0000 C CNN
 	1    5750 2750
@@
 F 0 "C2" H 6075 2850 50  0000 L CNN
 F 1 "100nF" H 6075 2650 50  0000 L CNN
-F 2 "" H 6088 2600 30  0000 C CNN
+F 2 "Capacitors_ThroughHole:C_Rect_L4_W2.5_P2.5" H 6088 2600 30  0001 C CNN
 F 3 "" H 6050 2750 60  0000 C CNN
 	1    6050 2750
@@
 F 0 "P1" H 1500 2150 50  0000 C CNN
 F 1 "CONN_01X08" V 1600 1700 50  0000 C CNN
-F 2 "" H 1500 1700 60  0000 C CNN
+F 2 "Pin_Headers:Pin_Header_Straight_1x08" H 1500 1700 60  0001 C CNN
 F 3 "" H 1500 1700 60  0000 C CNN
 	1    1500 1700
@@
 F 0 "P2" H 1500 3050 50  0000 C CNN
 F 1 "CONN_01X08" V 1600 2600 50  0000 C CNN
-F 2 "" H 1500 2600 60  0000 C CNN
+F 2 "Pin_Headers:Pin_Header_Straight_1x08" H 1500 2600 60  0001 C CNN
 F 3 "" H 1500 2600 60  0000 C CNN
 	1    1500 2600
@@
 F 0 "P3" H 1550 4250 50  0000 C CNN
 F 1 "CONN_01X03" V 1650 4050 50  0000 C CNN
-F 2 "" H 1550 4050 60  0000 C CNN
+F 2 "Pin_Headers:Pin_Header_Angled_1x03" H 1550 4050 60  0001 C CNN
 F 3 "" H 1550 4050 60  0000 C CNN
 	1    1550 4050
@@
 F 0 "P4" H 1550 5050 50  0000 C CNN
 F 1 "CONN_01X03" V 1650 4850 50  0000 C CNN
-F 2 "" H 1550 4850 60  0000 C CNN
+F 2 "Pin_Headers:Pin_Header_Angled_1x03" H 1550 4850 60  0001 C CNN
 F 3 "" H 1550 4850 60  0000 C CNN
 	1    1550 4850
@@
 F 0 "P5" H 1550 6000 50  0000 C CNN
 F 1 "CONN_01X03" V 1650 5800 50  0000 C CNN
-F 2 "" H 1550 5800 60  0000 C CNN
+F 2 "Pin_Headers:Pin_Header_Angled_1x03" H 1550 5800 60  0001 C CNN
 F 3 "" H 1550 5800 60  0000 C CNN
 	1    1550 5800
@@
 F 0 "P6" H 1550 6900 50  0000 C CNN
 F 1 "CONN_01X03" V 1650 6700 50  0000 C CNN
-F 2 "" H 1550 6700 60  0000 C CNN
+F 2 "Pin_Headers:Pin_Header_Angled_1x03" H 1550 6700 60  0001 C CNN
 F 3 "" H 1550 6700 60  0000 C CNN
 	1    1550 6700

Commit message: wip
Parts:
- added D1, D2, D3: LED, symbol LED
- added J1, J2: RJ45, symbol RJ45
- added OK1, OK2, OK3: 6N137, DIP8, symbol 6N137
- added P10: CONN_02X04, symbol CONN_02X04
- added P7: CONN_01X02, symbol CONN_01X02
- added P8: CONN_01X06, symbol CONN_01X06
- added P9: CONN_01X04, symbol CONN_01X04
- added R1: 15k, symbol R
- added R10, R5, R6: 220, symbol R
- added R11, R7, R8: 1K, symbol R
- added R2, R3, R4: 1,5k, symbol R
Connections:
- net labels added: BOOT_LED, CTS, GNDA, VCC, _RxD, _TxD
- wire segments 103 -> 195
Other:
- note added: "CAN overflow"
- note added: "RS232 overflow"

Commit message: wip
Parts:
- D1, D2, D3: footprint (none) -> LEDs:LED-3MM
- U2: symbol MCP2551-I/P -> MCP2551-I/P-RESCUE-CANBuster
Changed lines of the file:
@@
 RxD
 $Comp
-L MCP2551-I/P U2
+L MCP2551-I/P-RESCUE-CANBuster U2
 U 1 1 55B65B4E
 P 7850 1450
@@
 F 0 "R1" V 3680 3000 50  0000 C CNN
 F 1 "15k" V 3600 3000 50  0000 C CNN
-F 2 "" V 3530 3000 30  0000 C CNN
+F 2 "" V 3530 3000 30  0001 C CNN
 F 3 "" H 3600 3000 30  0000 C CNN
 	1    3600 3000
@@
 F 0 "R2" V 4430 1050 50  0000 C CNN
 F 1 "1,5k" V 4350 1050 50  0000 C CNN
-F 2 "" V 4280 1050 30  0000 C CNN
+F 2 "" V 4280 1050 30  0001 C CNN
 F 3 "" H 4350 1050 30  0000 C CNN
 	1    4350 1050
@@
 F 0 "D1" H 4350 1500 50  0000 C CNN
 F 1 "LED" H 4350 1300 50  0000 C CNN
-F 2 "" H 4350 1400 60  0000 C CNN
+F 2 "LEDs:LED-3MM" H 4350 1400 60  0001 C CNN
 F 3 "" H 4350 1400 60  0000 C CNN
 	1    4350 1400
@@
 F 0 "R3" V 4930 1050 50  0000 C CNN
 F 1 "1,5k" V 4850 1050 50  0000 C CNN
-F 2 "" V 4780 1050 30  0000 C CNN
+F 2 "" V 4780 1050 30  0001 C CNN
 F 3 "" H 4850 1050 30  0000 C CNN
 	1    4850 1050
@@
 F 0 "D2" H 4850 1500 50  0000 C CNN
 F 1 "LED" H 4850 1300 50  0000 C CNN
-F 2 "" H 4850 1400 60  0000 C CNN
+F 2 "LEDs:LED-3MM" H 4850 1400 60  0001 C CNN
 F 3 "" H 4850 1400 60  0000 C CNN
 	1    4850 1400
@@
 F 0 "R4" V 5430 1050 50  0000 C CNN
 F 1 "1,5k" V 5350 1050 50  0000 C CNN
-F 2 "" V 5280 1050 30  0000 C CNN
+F 2 "" V 5280 1050 30  0001 C CNN
 F 3 "" H 5350 1050 30  0000 C CNN
 	1    5350 1050
@@
 F 0 "D3" H 5350 1500 50  0000 C CNN
 F 1 "LED" H 5350 1300 50  0000 C CNN
-F 2 "" H 5350 1400 60  0000 C CNN
+F 2 "LEDs:LED-3MM" H 5350 1400 60  0001 C CNN
 F 3 "" H 5350 1400 60  0000 C CNN
 	1    5350 1400
@@
 F 0 "R5" V 8880 3350 50  0000 C CNN
 F 1 "220" V 8800 3350 50  0000 C CNN
-F 2 "" V 8730 3350 30  0000 C CNN
+F 2 "" V 8730 3350 30  0001 C CNN
 F 3 "" H 8800 3350 30  0000 C CNN
 	1    8800 3350
@@
 F 0 "R6" V 8980 5250 50  0000 C CNN
 F 1 "220" V 8900 5250 50  0000 C CNN
-F 2 "" V 8830 5250 30  0000 C CNN
+F 2 "" V 8830 5250 30  0001 C CNN
 F 3 "" H 8900 5250 30  0000 C CNN
 	1    8900 5250
@@
 F 0 "R8" V 9930 3000 50  0000 C CNN
 F 1 "1K" V 9850 3000 50  0000 C CNN
-F 2 "" V 9780 3000 30  0000 C CNN
+F 2 "" V 9780 3000 30  0001 C CNN
 F 3 "" H 9850 3000 30  0000 C CNN
 	1    9850 3000
@@
 F 0 "R7" V 8930 4200 50  0000 C CNN
 F 1 "1K" V 8850 4200 50  0000 C CNN
-F 2 "" V 8780 4200 30  0000 C CNN
+F 2 "" V 8780 4200 30  0001 C CNN
 F 3 "" H 8850 4200 30  0000 C CNN
 	1    8850 4200
@@
 F 0 "R10" V 9980 4500 50  0000 C CNN
 F 1 "220" V 9900 4500 50  0000 C CNN
-F 2 "" V 9830 4500 30  0000 C CNN
+F 2 "" V 9830 4500 30  0001 C CNN
 F 3 "" H 9900 4500 30  0000 C CNN
 	1    9900 4500
@@
 F 0 "R11" V 9980 5750 50  0000 C CNN
 F 1 "1K" V 9900 5750 50  0000 C CNN
-F 2 "" V 9830 5750 30  0000 C CNN
+F 2 "" V 9830 5750 30  0001 C CNN
 F 3 "" H 9900 5750 30  0000 C CNN
 	1    9900 5750
@@
 F 0 "P7" H 7650 4000 50  0000 C CNN
 F 1 "CONN_01X02" V 7750 3850 50  0000 C CNN
-F 2 "" H 7650 3850 60  0000 C CNN
+F 2 "" H 7650 3850 60  0001 C CNN
 F 3 "" H 7650 3850 60  0000 C CNN
 	1    7650 3850
@@
 F 0 "P8" H 10450 2200 50  0000 C CNN
 F 1 "CONN_01X06" V 10550 1850 50  0000 C CNN
-F 2 "" H 10450 1850 60  0000 C CNN
+F 2 "" H 10450 1850 60  0001 C CNN
 F 3 "" H 10450 1850 60  0000 C CNN
 	1    10450 1850
@@
 F 0 "J1" H 2350 1700 60  0000 C CNN
 F 1 "RJ45" H 2000 1700 60  0000 C CNN
-F 2 "" H 2150 1200 60  0000 C CNN
+F 2 "" H 2150 1200 60  0001 C CNN
 F 3 "" H 2150 1200 60  0000 C CNN
 	1    2150 1200
@@
 F 0 "J2" H 3350 1700 60  0000 C CNN
 F 1 "RJ45" H 3000 1700 60  0000 C CNN
-F 2 "" H 3150 1200 60  0000 C CNN
+F 2 "" H 3150 1200 60  0001 C CNN
 F 3 "" H 3150 1200 60  0000 C CNN
 	1    3150 1200
@@
 F 0 "P10" H 2500 3550 50  0000 C CNN
 F 1 "CONN_02X04" H 2500 3050 50  0000 C CNN
-F 2 "" H 2500 2100 60  0000 C CNN
+F 2 "" H 2500 2100 60  0001 C CNN
 F 3 "" H 2500 2100 60  0000 C CNN
 	1    2500 3300
@@
 F 0 "P9" H 2450 2950 50  0000 C CNN
 F 1 "CONN_01X04" V 2550 2700 50  0000 C CNN
-F 2 "" H 2450 2700 60  0000 C CNN
+F 2 "" H 2450 2700 60  0001 C CNN
 F 3 "" H 2450 2700 60  0000 C CNN
 	1    2450 2700

Commit message: wip
Parts:
- added R12, R9: 3k3, symbol R
Connections:
- wire segments 195 -> 201
Changed lines of the file:
@@
 Connection ~ 5350 2900
 Wire Wire Line
-	6350 3600 6650 3600
-Wire Wire Line
-	6350 3700 6650 3700
+	6350 3600 7000 3600
+Wire Wire Line
+	6350 3700 7200 3700
 Wire Wire Line
 	1150 1300 1450 1300
@@
 Wire Wire Line
 	3950 4400 3600 4400
+$Comp
+L R R9
+U 1 1 55B7B8AA
+P 7000 3300
+F 0 "R9" V 7080 3300 50  0000 C CNN
+F 1 "3k3" V 7000 3300 50  0000 C CNN
+F 2 "" V 6930 3300 30  0001 C CNN
+F 3 "" H 7000 3300 30  0000 C CNN
+	1    7000 3300
+	-1   0    0    1
+$EndComp
+$Comp
+L R R12
+U 1 1 55B7B994
+P 7200 3300
+F 0 "R12" V 7280 3300 50  0000 C CNN
+F 1 "3k3" V 7200 3300 50  0000 C CNN
+F 2 "" V 7130 3300 30  0001 C CNN
+F 3 "" H 7200 3300 30  0000 C CNN
+	1    7200 3300
+	-1   0    0    1
+$EndComp
+Wire Wire Line
+	7000 3600 7000 3450
+Wire Wire Line
+	7200 3700 7200 3450
+$Comp
+L VDD #PWR046
+U 1 1 55B7BCC9
+P 7100 3000
+F 0 "#PWR046" H 7100 2850 50  0001 C CNN
+F 1 "VDD" H 7100 3150 50  0000 C CNN
+F 2 "" H 7100 3000 60  0000 C CNN
+F 3 "" H 7100 3000 60  0000 C CNN
+	1    7100 3000
+	1    0    0    -1
+$EndComp
+Wire Wire Line
+	7200 3150 7200 3050
+Wire Wire Line
+	7200 3050 7000 3050
+Wire Wire Line
+	7000 3050 7000 3150
+Wire Wire Line
+	7100 3050 7100 3000
+Connection ~ 7100 3050
 $EndSCHEMATC

Commit message: wip
Parts:
- added P11: CONN_01X06, symbol CONN_01X06
- added R13: 1K, symbol R
Connections:
- net labels added: PGD_IN
- wire segments 201 -> 202
Changed lines of the file:
@@
 	3950 4700 3700 4700
 Wire Wire Line
-	3950 4800 3700 4800
+	3550 4800 3950 4800
 Wire Wire Line
 	5050 7150 4850 7150
@@
 	3950 5300 3750 5300
 Wire Wire Line
-	3750 5300 3750 5350
-Wire Wire Line
-	3750 5350 3050 5350
+	3750 5350 3750 5300
+Wire Wire Line
+	3050 5350 3750 5350
 Wire Wire Line
 	2750 5050 3750 5050
@@
 	2000 1650 2000 2750
 Wire Wire Line
-	2000 1900 3000 1900
+	3000 1900 2000 1900
 Wire Wire Line
 	3000 1650 3000 3350
@@
 	2100 1650 2100 1950
 Wire Wire Line
-	2100 1950 3100 1950
-Wire Wire Line
-	3100 1950 3100 1650
+	3100 1950 2100 1950
+Wire Wire Line
+	3100 1650 3100 1950
 Wire Wire Line
 	2200 1650 2200 2000
 Wire Wire Line
-	2200 2000 3200 2000
-Wire Wire Line
-	3200 2000 3200 1650
+	3200 2000 2200 2000
+Wire Wire Line
+	3200 1650 3200 2000
 Wire Wire Line
 	2300 1650 2300 2050
 Wire Wire Line
-	2300 2050 3300 2050
-Wire Wire Line
-	3300 2050 3300 1650
+	3300 2050 2300 2050
+Wire Wire Line
+	3300 1650 3300 2050
 Wire Wire Line
 	2400 1650 2400 2100
@@
 $EndComp
 Wire Wire Line
-	7200 3150 7200 3050
-Wire Wire Line
-	7200 3050 7000 3050
+	7200 3050 7200 3150
+Wire Wire Line
+	7000 3050 7200 3050
 Wire Wire Line
 	7000 3050 7000 3150
@@
 	7100 3050 7100 3000
 Connection ~ 7100 3050
+$Comp
+L CONN_01X06 P11
+U 1 1 55B7C26E
+P 3450 7050
+F 0 "P11" H 3450 7400 50  0000 C CNN
+F 1 "CONN_01X06" V 3550 7050 50  0000 C CNN
+F 2 "" H 3450 7050 60  0001 C CNN
+F 3 "" H 3450 7050 60  0000 C CNN
+	1    3450 7050
+	1    0    0    -1
+$EndComp
+$Comp
+L R R13
+U 1 1 55B7E037
+P 3400 4800
+F 0 "R13" V 3480 4800 50  0000 C CNN
+F 1 "1K" V 3400 4800 50  0000 C CNN
+F 2 "" V 3330 4800 30  0001 C CNN
+F 3 "" H 3400 4800 30  0000 C CNN
+	1    3400 4800
+	0    1    1    0
+$EndComp
+Wire Wire Line
+	3250 4800 2950 4800
+Text Label 2950 4800 0    60   ~ 0
+PGD_IN
 $EndSCHEMATC
