File: CANBuster/CANBuster.sch (KiCad schematic (older format))
At the start: 42 parts, among them J1 RJ45, J2 RJ45, P1 CONN_01X08, P10 CONN_02X04, P11 CONN_01X06, P2 CONN_01X08, P3 CONN_01X03, P4 CONN_01X03, P5 CONN_01X03, P6 CONN_01X03, P7 CONN_01X02, P8 CONN_01X06, P9 CONN_01X04, U1 PIC18(L)F45K80-I/P, U2 MCP2551-I/P, Y1 16MHz

Commit message: wip
Parts:
- J1, J2: footprint (none) -> Connect:RJ45_8
- OK1, OK2, OK3: footprint DIP8 -> Housings_DIP:DIP-8_W7.62mm
- P10: footprint (none) -> Pin_Headers:Pin_Header_Straight_2x04
- P11, P8: footprint (none) -> Pin_Headers:Pin_Header_Straight_1x06
- P7: footprint (none) -> Pin_Headers:Pin_Header_Straight_1x02
- P9: footprint (none) -> Pin_Headers:Pin_Header_Straight_1x04
- R1, R10, R11, R12, R13, R2, R3, R4, R5, R6, R7, R8, R9: footprint (none) -> Resistors_ThroughHole:Resistor_Horizontal_RM10mm
Connections:
- net labels added: _CTS
- wire segments 202 -> 210
Changed lines of the file:
@@
 F 0 "OK1" H 9136 3479 40  0000 C CNN
 F 1 "6N137" H 9500 3010 40  0000 C CNN
-F 2 "DIP8" H 9185 3015 29  0000 C CNN
+F 2 "Housings_DIP:DIP-8_W7.62mm" H 9185 3015 29  0000 C CNN
 F 3 "" H 9350 3250 60  0000 C CNN
 	1    9350 3250
@@
 F 0 "OK2" H 9186 5579 40  0000 C CNN
 F 1 "6N137" H 9550 5110 40  0000 C CNN
-F 2 "DIP8" H 9235 5115 29  0000 C CNN
+F 2 "Housings_DIP:DIP-8_W7.62mm" H 9235 5115 29  0000 C CNN
 F 3 "" H 9400 5350 60  0000 C CNN
 	1    9400 5350
@@
 F 0 "OK3" H 9186 4629 40  0000 C CNN
 F 1 "6N137" H 9550 4160 40  0000 C CNN
-F 2 "DIP8" H 9235 4165 29  0000 C CNN
+F 2 "Housings_DIP:DIP-8_W7.62mm" H 9235 4165 29  0000 C CNN
 F 3 "" H 9400 4400 60  0000 C CNN
 	1    9400 4400
@@
 F 0 "R1" V 3680 3000 50  0000 C CNN
 F 1 "15k" V 3600 3000 50  0000 C CNN
-F 2 "" V 3530 3000 30  0001 C CNN
+F 2 "Resistors_ThroughHole:Resistor_Horizontal_RM10mm" V 3530 3000 30  0001 C CNN
 F 3 "" H 3600 3000 30  0000 C CNN
 	1    3600 3000
@@
 F 0 "R2" V 4430 1050 50  0000 C CNN
 F 1 "1,5k" V 4350 1050 50  0000 C CNN
-F 2 "" V 4280 1050 30  0001 C CNN
+F 2 "Resistors_ThroughHole:Resistor_Horizontal_RM10mm" V 4280 1050 30  0001 C CNN
 F 3 "" H 4350 1050 30  0000 C CNN
 	1    4350 1050
@@
 F 0 "R3" V 4930 1050 50  0000 C CNN
 F 1 "1,5k" V 4850 1050 50  0000 C CNN
-F 2 "" V 4780 1050 30  0001 C CNN
+F 2 "Resistors_ThroughHole:Resistor_Horizontal_RM10mm" V 4780 1050 30  0001 C CNN
 F 3 "" H 4850 1050 30  0000 C CNN
 	1    4850 1050
@@
 F 0 "R4" V 5430 1050 50  0000 C CNN
 F 1 "1,5k" V 5350 1050 50  0000 C CNN
-F 2 "" V 5280 1050 30  0001 C CNN
+F 2 "Resistors_ThroughHole:Resistor_Horizontal_RM10mm" V 5280 1050 30  0001 C CNN
 F 3 "" H 5350 1050 30  0000 C CNN
 	1    5350 1050
@@
 F 0 "R5" V 8880 3350 50  0000 C CNN
 F 1 "220" V 8800 3350 50  0000 C CNN
-F 2 "" V 8730 3350 30  0001 C CNN
+F 2 "Resistors_ThroughHole:Resistor_Horizontal_RM10mm" V 8730 3350 30  0001 C CNN
 F 3 "" H 8800 3350 30  0000 C CNN
 	1    8800 3350
@@
 F 0 "R6" V 8980 5250 50  0000 C CNN
 F 1 "220" V 8900 5250 50  0000 C CNN
-F 2 "" V 8830 5250 30  0001 C CNN
+F 2 "Resistors_ThroughHole:Resistor_Horizontal_RM10mm" V 8830 5250 30  0001 C CNN
 F 3 "" H 8900 5250 30  0000 C CNN
 	1    8900 5250
@@
 F 0 "R8" V 9930 3000 50  0000 C CNN
 F 1 "1K" V 9850 3000 50  0000 C CNN
-F 2 "" V 9780 3000 30  0001 C CNN
+F 2 "Resistors_ThroughHole:Resistor_Horizontal_RM10mm" V 9780 3000 30  0001 C CNN
 F 3 "" H 9850 3000 30  0000 C CNN
 	1    9850 3000
@@
 F 0 "R7" V 8930 4200 50  0000 C CNN
 F 1 "1K" V 8850 4200 50  0000 C CNN
-F 2 "" V 8780 4200 30  0001 C CNN
+F 2 "Resistors_ThroughHole:Resistor_Horizontal_RM10mm" V 8780 4200 30  0001 C CNN
 F 3 "" H 8850 4200 30  0000 C CNN
 	1    8850 4200
@@
 F 0 "R10" V 9980 4500 50  0000 C CNN
 F 1 "220" V 9900 4500 50  0000 C CNN
-F 2 "" V 9830 4500 30  0001 C CNN
+F 2 "Resistors_ThroughHole:Resistor_Horizontal_RM10mm" V 9830 4500 30  0001 C CNN
 F 3 "" H 9900 4500 30  0000 C CNN
 	1    9900 4500
@@
 F 0 "R11" V 9980 5750 50  0000 C CNN
 F 1 "1K" V 9900 5750 50  0000 C CNN
-F 2 "" V 9830 5750 30  0001 C CNN
+F 2 "Resistors_ThroughHole:Resistor_Horizontal_RM10mm" V 9830 5750 30  0001 C CNN
 F 3 "" H 9900 5750 30  0000 C CNN
 	1    9900 5750
@@
 $EndComp
 Text Label 9950 5500 0    60   ~ 0
-CTS
+_CTS
 $Comp
 L PWR_FLAG #FLG039
@@
 F 0 "P7" H 7650 4000 50  0000 C CNN
 F 1 "CONN_01X02" V 7750 3850 50  0000 C CNN
-F 2 "" H 7650 3850 60  0001 C CNN
+F 2 "Pin_Headers:Pin_Header_Straight_1x02" H 7650 3850 60  0001 C CNN
 F 3 "" H 7650 3850 60  0000 C CNN
 	1    7650 3850
@@
 F 0 "P8" H 10450 2200 50  0000 C CNN
 F 1 "CONN_01X06" V 10550 1850 50  0000 C CNN
-F 2 "" H 10450 1850 60  0001 C CNN
+F 2 "Pin_Headers:Pin_Header_Straight_1x06" H 10450 1850 60  0001 C CNN
 F 3 "" H 10450 1850 60  0000 C CNN
 	1    10450 1850
@@
 $EndComp
 Text Label 10100 2000 0    60   ~ 0
-CTS
+_CTS
 Text Label 10050 1800 0    60   ~ 0
 _TxD
@@
 F 0 "J1" H 2350 1700 60  0000 C CNN
 F 1 "RJ45" H 2000 1700 60  0000 C CNN
-F 2 "" H 2150 1200 60  0001 C CNN
+F 2 "Connect:RJ45_8" H 2150 1200 60  0001 C CNN
 F 3 "" H 2150 1200 60  0000 C CNN
 	1    2150 1200
@@
 F 0 "J2" H 3350 1700 60  0000 C CNN
 F 1 "RJ45" H 3000 1700 60  0000 C CNN
-F 2 "" H 3150 1200 60  0001 C CNN
+F 2 "Connect:RJ45_8" H 3150 1200 60  0001 C CNN
 F 3 "" H 3150 1200 60  0000 C CNN
 	1    3150 1200
@@
 F 0 "P10" H 2500 3550 50  0000 C CNN
 F 1 "CONN_02X04" H 2500 3050 50  0000 C CNN
-F 2 "" H 2500 2100 60  0001 C CNN
+F 2 "Pin_Headers:Pin_Header_Straight_2x04" H 2500 2100 60  0001 C CNN
 F 3 "" H 2500 2100 60  0000 C CNN
 	1    2500 3300
@@
 F 0 "P9" H 2450 2950 50  0000 C CNN
 F 1 "CONN_01X04" V 2550 2700 50  0000 C CNN
-F 2 "" H 2450 2700 60  0001 C CNN
+F 2 "Pin_Headers:Pin_Header_Straight_1x04" H 2450 2700 60  0001 C CNN
 F 3 "" H 2450 2700 60  0000 C CNN
 	1    2450 2700
@@
 	3950 5300 3750 5300
 Wire Wire Line
-	3750 5350 3750 5300
-Wire Wire Line
-	3050 5350 3750 5350
+	3750 5300 3750 5350
+Wire Wire Line
+	3750 5350 3050 5350
 Wire Wire Line
 	2750 5050 3750 5050
@@
 	2100 1650 2100 1950
 Wire Wire Line
-	3100 1950 2100 1950
-Wire Wire Line
-	3100 1650 3100 1950
+	2100 1950 3100 1950
+Wire Wire Line
+	3100 1950 3100 1650
 Wire Wire Line
 	2200 1650 2200 2000
 Wire Wire Line
-	3200 2000 2200 2000
-Wire Wire Line
-	3200 1650 3200 2000
+	2200 2000 3200 2000
+Wire Wire Line
+	3200 2000 3200 1650
 Wire Wire Line
 	2300 1650 2300 2050
 Wire Wire Line
-	3300 2050 2300 2050
-Wire Wire Line
-	3300 1650 3300 2050
+	2300 2050 3300 2050
+Wire Wire Line
+	3300 2050 3300 1650
 Wire Wire Line
 	2400 1650 2400 2100
@@
 F 0 "R9" V 7080 3300 50  0000 C CNN
 F 1 "3k3" V 7000 3300 50  0000 C CNN
-F 2 "" V 6930 3300 30  0001 C CNN
+F 2 "Resistors_ThroughHole:Resistor_Horizontal_RM10mm" V 6930 3300 30  0001 C CNN
 F 3 "" H 7000 3300 30  0000 C CNN
 	1    7000 3300
@@
 F 0 "R12" V 7280 3300 50  0000 C CNN
 F 1 "3k3" V 7200 3300 50  0000 C CNN
-F 2 "" V 7130 3300 30  0001 C CNN
+F 2 "Resistors_ThroughHole:Resistor_Horizontal_RM10mm" V 7130 3300 30  0001 C CNN
 F 3 "" H 7200 3300 30  0000 C CNN
 	1    7200 3300
@@
 F 0 "P11" H 3450 7400 50  0000 C CNN
 F 1 "CONN_01X06" V 3550 7050 50  0000 C CNN
-F 2 "" H 3450 7050 60  0001 C CNN
+F 2 "Pin_Headers:Pin_Header_Straight_1x06" H 3450 7050 60  0001 C CNN
 F 3 "" H 3450 7050 60  0000 C CNN
 	1    3450 7050
@@
 F 0 "R13" V 3480 4800 50  0000 C CNN
 F 1 "1K" V 3400 4800 50  0000 C CNN
-F 2 "" V 3330 4800 30  0001 C CNN
+F 2 "Resistors_ThroughHole:Resistor_Horizontal_RM10mm" V 3330 4800 30  0001 C CNN
 F 3 "" H 3400 4800 30  0000 C CNN
 	1    3400 4800
@@
 Text Label 2950 4800 0    60   ~ 0
 PGD_IN
+Wire Wire Line
+	3250 6800 2950 6800
+Wire Wire Line
+	3250 6900 2950 6900
+Wire Wire Line
+	3250 7000 2950 7000
+Wire Wire Line
+	2500 7100 3250 7100
+Wire Wire Line
+	3250 7200 2950 7200
+Wire Wire Line
+	3250 7300 3150 7300
+Wire Wire Line
+	3150 7300 3150 7450
+$Comp
+L GND #PWR047
+U 1 1 55B7D3A4
+P 3150 7450
+F 0 "#PWR047" H 3150 7200 50  0001 C CNN
+F 1 "GND" H 3150 7300 50  0000 C CNN
+F 2 "" H 3150 7450 60  0000 C CNN
+F 3 "" H 3150 7450 60  0000 C CNN
+	1    3150 7450
+	1    0    0    -1
+$EndComp
+$Comp
+L VDD #PWR048
+U 1 1 55B7D42D
+P 2500 7050
+F 0 "#PWR048" H 2500 6900 50  0001 C CNN
+F 1 "VDD" H 2500 7200 50  0000 C CNN
+F 2 "" H 2500 7050 60  0000 C CNN
+F 3 "" H 2500 7050 60  0000 C CNN
+	1    2500 7050
+	1    0    0    -1
+$EndComp
+Wire Wire Line
+	2500 7100 2500 7050
+Text Label 2950 6800 0    60   ~ 0
+PGD_IN
+Text Label 2950 6900 0    60   ~ 0
+PGC
+Text Label 2950 7000 0    60   ~ 0
+~MCLR
+Text Label 2950 7200 0    60   ~ 0
+PGD
 $EndSCHEMATC
