File: CANBuster/CANBuster.sch (KiCad schematic (older format))
At the start: 107 parts, among them CON1 BARREL_JACK, J1 RJ45, J2 RJ45, J3 RJ12, P1 CONN_01X10, P10 CONN_02X04, P11 CONN_01X06, P12 CONN_01X06, P13 CONN_01X10, P14 CONN_01X10, P2 CONN_01X10, P3 CONN_01X03, P4 CONN_01X03, P5 CONN_01X03, P6 CONN_01X03, P7 CONN_01X02, P8 CONN_01X06, P9 CONN_01X04, Q1 BC547, Q2 BC547, SW1 SW_PUSH, U1 PIC18(L)F45K80-I/P, U2 MCP2551-I/P, U3 7805, U4 LTV-844, U5 LTV-844, U6 LTV-844, U7 LTV-844, Y1 16MHz

Commit message: change footprints
Parts:
- OK1, OK2, OK3, OK4, OK5, OK6, OK7, OK8, OK9: footprint Housings_DIP:DIP-8_W7.62mm -> w_pth_circuits:dil_8-300_socket
- R10, R11, R12, R13, R14, R15, R16, R17, R18, R19, R20, R37, R38, R39, R40, R41, R42, R43, R44, R45, R6, R8, R9: footprint Resistors_ThroughHole:Resistor_Horizontal_RM10mm -> w_pth_resistors:RC03
- R21, R22, R23, R24, R25, R26, R27, R28, R29, R30, R31, R32, R33, R34, R35, R36: footprint Resistors_ThroughHole:Resistor_Horizontal_RM7.5mm -> w_pth_resistors:RC03
- R7: footprint Resistors_ThroughHole:Resistor_Horizontal_RM10mm -> w_pth_resistors:rc03_vert
- U1: footprint Housings_DIP:DIP-40_W15.24mm_LongPads -> w_pth_circuits:dil_40-600_socket
- U2: footprint Housings_DIP:DIP-8_W7.62mm_LongPads -> w_pth_circuits:dil_8-300_socket
- U4, U5: footprint Housings_DIP:DIP-16_W7.62mm_LongPads -> w_pth_circuits:dil_16-300_socket
- U6, U7: footprint Housings_DIP:DIP-18_W7.62mm_LongPads -> w_pth_circuits:dil_16-300_socket
Connections:
- wire segments 402 -> 401

Commit message: wip
Parts:
- P3, P4, P5, P6: footprint Pin_Headers:Pin_Header_Angled_1x03 -> Pin_Headers:Pin_Header_Straight_1x03
- R1, R2, R3, R4, R5: footprint Resistors_ThroughHole:Resistor_Horizontal_RM10mm -> w_pth_resistors:RC03
- R7: footprint w_pth_resistors:rc03_vert -> w_pth_resistors:RC03
- U1: value PIC18(L)F45K80-I/P -> PIC18F45K80
Changed lines of the file:
@@
 P 8850 5800
 F 0 "U1" H 7850 7000 50  0000 C CNN
-F 1 "PIC18(L)F45K80-I/P" H 9500 4600 50  0000 C CNN
+F 1 "PIC18F45K80" H 9500 4600 50  0000 C CNN
 F 2 "w_pth_circuits:dil_40-600_socket" H 8850 5800 50  0001 C CIN
 F 3 "" H 7700 7000 60  0000 C CNN
@@
 F 0 "P3" H 5700 8400 50  0000 C CNN
 F 1 "CONN_01X03" V 5800 8200 50  0000 C CNN
-F 2 "Pin_Headers:Pin_Header_Angled_1x03" H 5700 8200 60  0001 C CNN
+F 2 "Pin_Headers:Pin_Header_Straight_1x03" H 5700 8200 60  0001 C CNN
 F 3 "" H 5700 8200 60  0000 C CNN
 	1    5700 8200
@@
 F 0 "P4" H 5700 9300 50  0000 C CNN
 F 1 "CONN_01X03" V 5800 9100 50  0000 C CNN
-F 2 "Pin_Headers:Pin_Header_Angled_1x03" H 5700 9100 60  0001 C CNN
+F 2 "Pin_Headers:Pin_Header_Straight_1x03" H 5700 9100 60  0001 C CNN
 F 3 "" H 5700 9100 60  0000 C CNN
 	1    5700 9100
@@
 F 0 "P5" H 5700 10150 50  0000 C CNN
 F 1 "CONN_01X03" V 5800 9950 50  0000 C CNN
-F 2 "Pin_Headers:Pin_Header_Angled_1x03" H 5700 9950 60  0001 C CNN
+F 2 "Pin_Headers:Pin_Header_Straight_1x03" H 5700 9950 60  0001 C CNN
 F 3 "" H 5700 9950 60  0000 C CNN
 	1    5700 9950
@@
 F 0 "P6" H 5700 11000 50  0000 C CNN
 F 1 "CONN_01X03" V 5800 10800 50  0000 C CNN
-F 2 "Pin_Headers:Pin_Header_Angled_1x03" H 5700 10800 60  0001 C CNN
+F 2 "Pin_Headers:Pin_Header_Straight_1x03" H 5700 10800 60  0001 C CNN
 F 3 "" H 5700 10800 60  0000 C CNN
 	1    5700 10800
@@
 F 0 "R1" V 7380 3950 50  0000 C CNN
 F 1 "4k7" V 7300 3950 50  0000 C CNN
-F 2 "Resistors_ThroughHole:Resistor_Horizontal_RM10mm" V 7230 3950 30  0001 C CNN
+F 2 "w_pth_resistors:RC03" V 7230 3950 30  0001 C CNN
 F 3 "" H 7300 3950 30  0000 C CNN
 	1    7300 3950
@@
 F 0 "R2" V 5630 1050 50  0000 C CNN
 F 1 "1,5k" V 5550 1050 50  0000 C CNN
-F 2 "Resistors_ThroughHole:Resistor_Horizontal_RM10mm" V 5480 1050 30  0001 C CNN
+F 2 "w_pth_resistors:RC03" V 5480 1050 30  0001 C CNN
 F 3 "" H 5550 1050 30  0000 C CNN
 	1    5550 1050
@@
 F 0 "R3" V 6130 1050 50  0000 C CNN
 F 1 "1,5k" V 6050 1050 50  0000 C CNN
-F 2 "Resistors_ThroughHole:Resistor_Horizontal_RM10mm" V 5980 1050 30  0001 C CNN
+F 2 "w_pth_resistors:RC03" V 5980 1050 30  0001 C CNN
 F 3 "" H 6050 1050 30  0000 C CNN
 	1    6050 1050
@@
 F 0 "R4" V 6880 1050 50  0000 C CNN
 F 1 "1,5k" V 6800 1050 50  0000 C CNN
-F 2 "Resistors_ThroughHole:Resistor_Horizontal_RM10mm" V 6730 1050 30  0001 C CNN
+F 2 "w_pth_resistors:RC03" V 6730 1050 30  0001 C CNN
 F 3 "" H 6800 1050 30  0000 C CNN
 	1    6800 1050
@@
 F 0 "R5" V 14230 9350 50  0000 C CNN
 F 1 "330" V 14150 9350 50  0000 C CNN
-F 2 "Resistors_ThroughHole:Resistor_Horizontal_RM10mm" V 14080 9350 30  0001 C CNN
+F 2 "w_pth_resistors:RC03" V 14080 9350 30  0001 C CNN
 F 3 "" H 14150 9350 30  0000 C CNN
 	1    14150 9350
@@
 F 0 "R7" V 12830 6150 50  0000 C CNN
 F 1 "1K" V 12750 6150 50  0000 C CNN
-F 2 "w_pth_resistors:rc03_vert" V 12680 6150 30  0001 C CNN
+F 2 "w_pth_resistors:RC03" V 12680 6150 30  0001 C CNN
 F 3 "" H 12750 6150 30  0000 C CNN
 	1    12750 6150

Commit message: wip
Parts:
- added SW2: SW_PUSH, Buttons_Switches_ThroughHole:SW_PUSH_SMALL, symbol SW_PUSH
Connections:
- wire segments 401 -> 403

Commit message: wip
Parts:
- removed R4: 1,5k, w_pth_resistors:RC03, symbol R
- added C11, C12, C13, C14: 100nF, Capacitors_ThroughHole:C_Rect_L4_W2.5_P2.5, symbol C
- added D7: 1N4148, Discret:D3, symbol ZENER
- added OK10: 6N137, w_pth_circuits:dil_8-300_socket, symbol 6N137
- added P15: SNIFFER, w_conn_pt-1,5:pt_1,5-2-3,5-h, symbol CONN_01X02
- added P16: CONN_01X02, Pin_Headers:Pin_Header_Straight_1x02, symbol CONN_01X02
- added R46, R47: 1k5, w_pth_resistors:RC03, symbol R
- added R48: 390, w_pth_resistors:RC03, symbol R
- P11: value CONN_01X06 -> RS232-Programmer
- P12: value CONN_01X06 -> S88; footprint Pin_Headers:Pin_Header_Angled_1x06 -> Socket_Strips:Socket_Strip_Straight_1x06
Connections:
- net labels added: SNIFF
- net labels removed: S88
- wire segments 403 -> 427
- no-connect marks 7 -> 6

Commit message: wip
Parts:
- added C15: 100nF, w_capacitors:cnp_3mm_disc, symbol C
- added R4: 1,5k, w_pth_resistors:RC03, symbol R
- C1, C10, C11, C12, C13, C14, C2, C3, C4, C6, C7, C8, C9: footprint Capacitors_ThroughHole:C_Rect_L4_W2.5_P2.5 -> w_capacitors:cnp_3mm_disc
- P1, P2: footprint Socket_Strips:Socket_Strip_Straight_1x10 -> w_conn_pt-1,5:pt_1,5-10-3,5-h
- P13, P14: footprint Socket_Strips:Socket_Strip_Straight_1x10 -> Pin_Headers:Pin_Header_Straight_1x10
- P8: footprint Pin_Headers:Pin_Header_Straight_1x06 -> Socket_Strips:Socket_Strip_Angled_1x06
- Q1, Q2: footprint Housings_TO-92:TO-92_Inline_Narrow_Oval -> Housings_TO-92:TO-92_Molded_Narrow
- RR1, RR2: footprint Pin_Headers:Pin_Header_Straight_1x09 -> w_pth_resistors:r-sil_9
- U3: footprint Power_Integrations:TO-220 -> 78xx:TO-220
Connections:
- wire segments 427 -> 428

Commit message: wip
Parts:
- removed R21, R22, R23, R24, R25, R26, R27, R28, R29, R30, R31, R32, R33, R34, R35, R36: R, w_pth_resistors:RC03, symbol R
Connections:
- wire segments 428 -> 412
Changed lines of the file:
@@
 Text Label 10150 5200 0    60   ~ 0
 SDA
-Text Label 6850 5000 0    60   ~ 0
+Text Label 7300 5000 0    60   ~ 0
 IO1
-Text Label 6850 5100 0    60   ~ 0
+Text Label 7300 5100 0    60   ~ 0
 IO2
-Text Label 6850 5200 0    60   ~ 0
+Text Label 7300 5200 0    60   ~ 0
 IO3
-Text Label 6850 5300 0    60   ~ 0
+Text Label 7300 5300 0    60   ~ 0
 IO4
-Text Label 6850 5400 0    60   ~ 0
+Text Label 7300 5400 0    60   ~ 0
 IO5
-Text Label 10600 6600 0    60   ~ 0
+Text Label 10150 6600 0    60   ~ 0
 IO6
-Text Label 10600 6700 0    60   ~ 0
+Text Label 10150 6700 0    60   ~ 0
 IO7
-Text Label 10600 6800 0    60   ~ 0
+Text Label 10150 6800 0    60   ~ 0
 IO8
-Text Label 10600 5700 0    60   ~ 0
+Text Label 10150 5700 0    60   ~ 0
 IO9
-Text Label 10600 5800 0    60   ~ 0
+Text Label 10100 5800 0    60   ~ 0
 IO10
-Text Label 10600 5900 0    60   ~ 0
+Text Label 10100 5900 0    60   ~ 0
 IO11
-Text Label 10600 6000 0    60   ~ 0
+Text Label 10100 6000 0    60   ~ 0
 IO12
-Text Label 10600 6100 0    60   ~ 0
+Text Label 10100 6100 0    60   ~ 0
 IO13
-Text Label 10600 6200 0    60   ~ 0
+Text Label 10100 6200 0    60   ~ 0
 IO14
-Text Label 6800 5600 0    60   ~ 0
+Text Label 7300 5600 0    60   ~ 0
 IO15
-Text Label 6800 5700 0    60   ~ 0
+Text Label 7300 5700 0    60   ~ 0
 IO16
 $Comp
@@
 	1    4200 10850
 	1    0    0    -1
-$EndComp
-$Comp
-L R R21
-U 1 1 561B862E
-P 7150 5000
-F 0 "R21" V 7150 4550 50  0000 C CNN
-F 1 "R" V 7150 5000 50  0000 C CNN
-F 2 "w_pth_resistors:RC03" V 7080 5000 30  0001 C CNN
-F 3 "" H 7150 5000 30  0000 C CNN
-	1    7150 5000
-	0    1    1    0
-$EndComp
-$Comp
-L R R22
-U 1 1 561BA02A
-P 7150 5100
-F 0 "R22" V 7150 4650 50  0000 C CNN
-F 1 "R" V 7150 5100 50  0000 C CNN
-F 2 "w_pth_resistors:RC03" V 7080 5100 30  0001 C CNN
-F 3 "" H 7150 5100 30  0000 C CNN
-	1    7150 5100
-	0    1    1    0
-$EndComp
-$Comp
-L R R23
-U 1 1 561BA1AA
-P 7150 5200
-F 0 "R23" V 7150 4750 50  0000 C CNN
-F 1 "R" V 7150 5200 50  0000 C CNN
-F 2 "w_pth_resistors:RC03" V 7080 5200 30  0001 C CNN
-F 3 "" H 7150 5200 30  0000 C CNN
-	1    7150 5200
-	0    1    1    0
-$EndComp
-$Comp
-L R R24
-U 1 1 561BA3C4
-P 7150 5300
-F 0 "R24" V 7150 4850 50  0000 C CNN
-F 1 "R" V 7150 5300 50  0000 C CNN
-F 2 "w_pth_resistors:RC03" V 7080 5300 30  0001 C CNN
-F 3 "" H 7150 5300 30  0000 C CNN
-	1    7150 5300
-	0    1    1    0
-$EndComp
-$Comp
-L R R25
-U 1 1 561BA53C
-P 7150 5400
-F 0 "R25" V 7150 4950 50  0000 C CNN
-F 1 "R" V 7150 5400 50  0000 C CNN
-F 2 "w_pth_resistors:RC03" V 7080 5400 30  0001 C CNN
-F 3 "" H 7150 5400 30  0000 C CNN
-	1    7150 5400
-	0    1    1    0
-$EndComp
-$Comp
-L R R34
-U 1 1 561BA6B4
-P 10450 6600
-F 0 "R34" V 10450 6150 50  0000 C CNN
-F 1 "R" V 10450 6600 50  0000 C CNN
-F 2 "w_pth_resistors:RC03" V 10380 6600 30  0001 C CNN
-F 3 "" H 10450 6600 30  0000 C CNN
-	1    10450 6600
-	0    -1   -1   0
-$EndComp
-$Comp
-L R R35
-U 1 1 561BC266
-P 10450 6700
-F 0 "R35" V 10450 6250 50  0000 C CNN
-F 1 "R" V 10450 6700 50  0000 C CNN
-F 2 "w_pth_resistors:RC03" V 10380 6700 30  0001 C CNN
-F 3 "" H 10450 6700 30  0000 C CNN
-	1    10450 6700
-	0    -1   -1   0
-$EndComp
-$Comp
-L R R36
-U 1 1 561BC38B
-P 10450 6800
-F 0 "R36" V 10450 6350 50  0000 C CNN
-F 1 "R" V 10450 6800 50  0000 C CNN
-F 2 "w_pth_resistors:RC03" V 10380 6800 30  0001 C CNN
-F 3 "" H 10450 6800 30  0000 C CNN
-	1    10450 6800
-	0    -1   -1   0
-$EndComp
-$Comp
-L R R28
-U 1 1 561BCFDB
-P 10450 5700
-F 0 "R28" V 10450 5250 50  0000 C CNN
-F 1 "R" V 10450 5700 50  0000 C CNN
-F 2 "w_pth_resistors:RC03" V 10380 5700 30  0001 C CNN
-F 3 "" H 10450 5700 30  0000 C CNN
-	1    10450 5700
-	0    -1   -1   0
-$EndComp
-$Comp
-L R R29
-U 1 1 561BD239
-P 10450 5800
-F 0 "R29" V 10450 5350 50  0000 C CNN
-F 1 "R" V 10450 5800 50  0000 C CNN
-F 2 "w_pth_resistors:RC03" V 10380 5800 30  0001 C CNN
-F 3 "" H 10450 5800 30  0000 C CNN
-	1    10450 5800
-	0    -1   -1   0
-$EndComp
-$Comp
-L R R30
-U 1 1 561BD3C5
-P 10450 5900
-F 0 "R30" V 10450 5450 50  0000 C CNN
-F 1 "R" V 10450 5900 50  0000 C CNN
-F 2 "w_pth_resistors:RC03" V 10380 5900 30  0001 C CNN
-F 3 "" H 10450 5900 30  0000 C CNN
-	1    10450 5900
-	0    -1   -1   0
-$EndComp
-$Comp
-L R R31
-U 1 1 561BD611
-P 10450 6000
-F 0 "R31" V 10450 5550 50  0000 C CNN
-F 1 "R" V 10450 6000 50  0000 C CNN
-F 2 "w_pth_resistors:RC03" V 10380 6000 30  0001 C CNN
-F 3 "" H 10450 6000 30  0000 C CNN
-	1    10450 6000
-	0    -1   -1   0
-$EndComp
-$Comp
-L R R32
-U 1 1 561BD7AD
-P 10450 6100
-F 0 "R32" V 10450 5650 50  0000 C CNN
-F 1 "R" V 10450 6100 50  0000 C CNN
-F 2 "w_pth_resistors:RC03" V 10380 6100 30  0001 C CNN
-F 3 "" H 10450 6100 30  0000 C CNN
-	1    10450 6100
-	0    -1   -1   0
-$EndComp
-$Comp
-L R R33
-U 1 1 561BD9AA
-P 10450 6200
-F 0 "R33" V 10450 5750 50  0000 C CNN
-F 1 "R" V 10450 6200 50  0000 C CNN
-F 2 "w_pth_resistors:RC03" V 10380 6200 30  0001 C CNN
-F 3 "" H 10450 6200 30  0000 C CNN
-	1    10450 6200
-	0    -1   -1   0
-$EndComp
-$Comp
-L R R26
-U 1 1 561BFCFA
-P 7150 5600
-F 0 "R26" V 7150 5150 50  0000 C CNN
-F 1 "R" V 7150 5600 50  0000 C CNN
-F 2 "w_pth_resistors:RC03" V 7080 5600 30  0001 C CNN
-F 3 "" H 7150 5600 30  0000 C CNN
-	1    7150 5600
-	0    1    1    0
-$EndComp
-$Comp
-L R R27
-U 1 1 561BFF0D
-P 7150 5700
-F 0 "R27" V 7150 5250 50  0000 C CNN
-F 1 "R" V 7150 5700 50  0000 C CNN
-F 2 "w_pth_resistors:RC03" V 7080 5700 30  0001 C CNN
-F 3 "" H 7150 5700 30  0000 C CNN
-	1    7150 5700
-	0    1    1    0
 $EndComp
 $Comp
@@
 Connection ~ 4200 10400
 Wire Wire Line
-	7000 5700 6800 5700
-Wire Wire Line
-	7000 5600 6800 5600
-Wire Wire Line
-	7000 5400 6800 5400
-Wire Wire Line
-	7000 5300 6800 5300
-Wire Wire Line
-	7000 5200 6800 5200
-Wire Wire Line
-	7000 5100 6800 5100
-Wire Wire Line
-	7000 5000 6800 5000
-Wire Wire Line
-	10600 5700 10800 5700
-Wire Wire Line
-	10600 5800 10800 5800
-Wire Wire Line
-	10600 5900 10800 5900
-Wire Wire Line
-	10600 6000 10800 6000
-Wire Wire Line
-	10600 6100 10800 6100
-Wire Wire Line
-	10600 6200 10800 6200
-Wire Wire Line
-	10600 6600 10800 6600
-Wire Wire Line
-	10600 6700 10800 6700
-Wire Wire Line
-	10600 6800 10800 6800
-Wire Wire Line
 	5850 7250 6050 7250

Commit message: wip
Parts:
- added C16, C17, C18: 100nF, w_capacitors:cnp_3mm_disc, symbol C
Connections:
- wire segments 412 -> 415
Changed lines of the file:
@@
 L VDD #PWR091
 U 1 1 56B42640
-P 6600 8800
-F 0 "#PWR091" H 6600 8650 50  0001 C CNN
-F 1 "VDD" H 6600 8950 50  0000 C CNN
-F 2 "" H 6600 8800 60  0000 C CNN
-F 3 "" H 6600 8800 60  0000 C CNN
-	1    6600 8800
+P 6950 9550
+F 0 "#PWR091" H 6950 9400 50  0001 C CNN
+F 1 "VDD" H 6950 9700 50  0000 C CNN
+F 2 "" H 6950 9550 60  0000 C CNN
+F 3 "" H 6950 9550 60  0000 C CNN
+	1    6950 9550
 	1    0    0    -1
 $EndComp
@@
 L GND-RESCUE-CANBuster #PWR092
 U 1 1 56B42646
-P 6600 9150
-F 0 "#PWR092" H 6600 8900 50  0001 C CNN
-F 1 "GND" H 6600 9000 50  0000 C CNN
-F 2 "" H 6600 9150 60  0000 C CNN
-F 3 "" H 6600 9150 60  0000 C CNN
-	1    6600 9150
+P 6950 9900
+F 0 "#PWR092" H 6950 9650 50  0001 C CNN
+F 1 "GND" H 6950 9750 50  0000 C CNN
+F 2 "" H 6950 9900 60  0000 C CNN
+F 3 "" H 6950 9900 60  0000 C CNN
+	1    6950 9900
 	1    0    0    -1
 $EndComp
@@
 L C C11
 U 1 1 56B4264C
-P 6600 9000
-F 0 "C11" H 6625 9100 50  0000 L CNN
-F 1 "100nF" H 6625 8900 50  0000 L CNN
-F 2 "w_capacitors:cnp_3mm_disc" H 6638 8850 30  0001 C CNN
-F 3 "" H 6600 9000 60  0000 C CNN
-	1    6600 9000
-	1    0    0    -1
-$EndComp
-Wire Wire Line
-	6600 8800 6600 8850
+P 6950 9750
+F 0 "C11" H 6975 9850 50  0000 L CNN
+F 1 "100nF" H 6975 9650 50  0000 L CNN
+F 2 "w_capacitors:cnp_3mm_disc" H 6988 9600 30  0001 C CNN
+F 3 "" H 6950 9750 60  0000 C CNN
+	1    6950 9750
+	1    0    0    -1
+$EndComp
+Wire Wire Line
+	6950 9550 6950 9600
 $Comp
 L GND-RESCUE-CANBuster #PWR093
@@
 	1    0    0    -1
 $EndComp
+$Comp
+L C C16
+U 1 1 56C43D8D
+P 6450 8550
+F 0 "C16" H 6475 8650 50  0000 L CNN
+F 1 "100nF" H 6475 8450 50  0000 L CNN
+F 2 "w_capacitors:cnp_3mm_disc" H 6488 8400 30  0001 C CNN
+F 3 "" H 6450 8550 60  0000 C CNN
+	1    6450 8550
+	1    0    0    -1
+$EndComp
+Wire Wire Line
+	6450 8350 6450 8400
+$Comp
+L VCC #PWR0101
+U 1 1 56C441A8
+P 6450 8350
+F 0 "#PWR0101" H 6450 8200 50  0001 C CNN
+F 1 "VCC" H 6450 8500 50  0000 C CNN
+F 2 "" H 6450 8350 60  0000 C CNN
+F 3 "" H 6450 8350 60  0000 C CNN
+	1    6450 8350
+	1    0    0    -1
+$EndComp
+$Comp
+L C C17
+U 1 1 56C4466D
+P 6750 8550
+F 0 "C17" H 6775 8650 50  0000 L CNN
+F 1 "100nF" H 6775 8450 50  0000 L CNN
+F 2 "w_capacitors:cnp_3mm_disc" H 6788 8400 30  0001 C CNN
+F 3 "" H 6750 8550 60  0000 C CNN
+	1    6750 8550
+	1    0    0    -1
+$EndComp
+Wire Wire Line
+	6750 8350 6750 8400
+$Comp
+L VCC #PWR0102
+U 1 1 56C44674
+P 6750 8350
+F 0 "#PWR0102" H 6750 8200 50  0001 C CNN
+F 1 "VCC" H 6750 8500 50  0000 C CNN
+F 2 "" H 6750 8350 60  0000 C CNN
+F 3 "" H 6750 8350 60  0000 C CNN
+	1    6750 8350
+	1    0    0    -1
+$EndComp
+$Comp
+L C C18
+U 1 1 56C44780
+P 7050 8550
+F 0 "C18" H 7075 8650 50  0000 L CNN
+F 1 "100nF" H 7075 8450 50  0000 L CNN
+F 2 "w_capacitors:cnp_3mm_disc" H 7088 8400 30  0001 C CNN
+F 3 "" H 7050 8550 60  0000 C CNN
+	1    7050 8550
+	1    0    0    -1
+$EndComp
+Wire Wire Line
+	7050 8350 7050 8400
+$Comp
+L VCC #PWR0103
+U 1 1 56C44787
+P 7050 8350
+F 0 "#PWR0103" H 7050 8200 50  0001 C CNN
+F 1 "VCC" H 7050 8500 50  0000 C CNN
+F 2 "" H 7050 8350 60  0000 C CNN
+F 3 "" H 7050 8350 60  0000 C CNN
+	1    7050 8350
+	1    0    0    -1
+$EndComp
+$Comp
+L GNDA-RESCUE-CANBuster #PWR0104
+U 1 1 56C44FDC
+P 7050 8700
+F 0 "#PWR0104" H 7050 8450 50  0001 C CNN
+F 1 "GNDA" H 7050 8550 50  0000 C CNN
+F 2 "" H 7050 8700 60  0000 C CNN
+F 3 "" H 7050 8700 60  0000 C CNN
+	1    7050 8700
+	1    0    0    -1
+$EndComp
+$Comp
+L GNDA-RESCUE-CANBuster #PWR0105
+U 1 1 56C4514C
+P 6750 8700
+F 0 "#PWR0105" H 6750 8450 50  0001 C CNN
+F 1 "GNDA" H 6750 8550 50  0000 C CNN
+F 2 "" H 6750 8700 60  0000 C CNN
+F 3 "" H 6750 8700 60  0000 C CNN
+	1    6750 8700
+	1    0    0    -1
+$EndComp
+$Comp
+L GNDA-RESCUE-CANBuster #PWR0106
+U 1 1 56C452BC
+P 6450 8700
+F 0 "#PWR0106" H 6450 8450 50  0001 C CNN
+F 1 "GNDA" H 6450 8550 50  0000 C CNN
+F 2 "" H 6450 8700 60  0000 C CNN
+F 3 "" H 6450 8700 60  0000 C CNN
+	1    6450 8700
+	1    0    0    -1
+$EndComp

Commit message: wip
Parts:
- added R21, R22, R23, R24: R-SIL_8NB, w_pth_resistors:r-sil_8, symbol R-SIL_8NB
- P12: footprint Socket_Strips:Socket_Strip_Straight_1x06 -> w_conn_kk100:kk100_22-23-2061
- P13, P14: footprint Pin_Headers:Pin_Header_Straight_1x10 -> w_conn_kk100:kk100_22-23-2101
Connections:
- wire segments 415 -> 431
Changed lines of the file:
@@
 LIBS:microchip_pic18mcu
 LIBS:icsp
+LIBS:w_device
 LIBS:CANBuster-cache
 EELAYER 25 0
@@
 F 0 "P12" H 12650 9450 50  0000 C CNN
 F 1 "S88" V 12750 9100 50  0000 C CNN
-F 2 "Socket_Strips:Socket_Strip_Straight_1x06" H 12650 9100 60  0001 C CNN
+F 2 "w_conn_kk100:kk100_22-23-2061" H 12650 9100 60  0001 C CNN
 F 3 "" H 12650 9100 60  0000 C CNN
 	1    12650 9100
@@
 F 0 "P13" H 5600 6100 50  0000 C CNN
 F 1 "CONN_01X10" V 5700 5550 50  0000 C CNN
-F 2 "Pin_Headers:Pin_Header_Straight_1x10" H 5600 5550 60  0001 C CNN
+F 2 "w_conn_kk100:kk100_22-23-2101" H 5600 5550 60  0001 C CNN
 F 3 "" H 5600 5550 60  0000 C CNN
 	1    5600 5550
@@
 F 0 "P14" H 5650 7450 50  0000 C CNN
 F 1 "CONN_01X10" V 5750 6900 50  0000 C CNN
-F 2 "Pin_Headers:Pin_Header_Straight_1x10" H 5650 6900 60  0001 C CNN
+F 2 "w_conn_kk100:kk100_22-23-2101" H 5650 6900 60  0001 C CNN
 F 3 "" H 5650 6900 60  0000 C CNN
 	1    5650 6900
@@
 	1    0    0    -1
 $EndComp
+$Comp
+L R-SIL_8NB R21
+U 1 1 56C3A6E8
+P 3000 1250
+F 0 "R21" V 2945 1255 50  0000 C CNN
+F 1 "R-SIL_8NB" V 3065 1250 50  0000 C CNN
+F 2 "w_pth_resistors:r-sil_8" H 3000 1250 60  0001 C CNN
+F 3 "" H 3000 1250 60  0000 C CNN
+	1    3000 1250
+	0    1    1    0
+$EndComp
+$Comp
+L R-SIL_8NB R21
+U 2 1 56C3B4D0
+P 3000 1750
+F 0 "R21" V 2945 1755 50  0000 C CNN
+F 1 "R-SIL_8NB" V 3065 1750 50  0000 C CNN
+F 2 "w_pth_resistors:r-sil_8" H 3000 1750 60  0001 C CNN
+F 3 "" H 3000 1750 60  0000 C CNN
+	2    3000 1750
+	0    1    1    0
+$EndComp
+$Comp
+L R-SIL_8NB R21
+U 3 1 56C3B65F
+P 3000 2250
+F 0 "R21" V 2945 2255 50  0000 C CNN
+F 1 "R-SIL_8NB" V 3065 2250 50  0000 C CNN
+F 2 "w_pth_resistors:r-sil_8" H 3000 2250 60  0001 C CNN
+F 3 "" H 3000 2250 60  0000 C CNN
+	3    3000 2250
+	0    1    1    0
+$EndComp
+$Comp
+L R-SIL_8NB R21
+U 4 1 56C3B7F0
+P 3000 2750
+F 0 "R21" V 2945 2755 50  0000 C CNN
+F 1 "R-SIL_8NB" V 3065 2750 50  0000 C CNN
+F 2 "w_pth_resistors:r-sil_8" H 3000 2750 60  0001 C CNN
+F 3 "" H 3000 2750 60  0000 C CNN
+	4    3000 2750
+	0    1    1    0
+$EndComp
+Wire Wire Line
+	3100 1250 3400 1250
+Wire Wire Line
+	3100 1750 3400 1750
+Wire Wire Line
+	3100 2250 3400 2250
+Wire Wire Line
+	3100 2750 3400 2750
+$Comp
+L R-SIL_8NB R22
+U 1 1 56C3E0A4
+P 3000 3400
+F 0 "R22" V 2945 3405 50  0000 C CNN
+F 1 "R-SIL_8NB" V 3065 3400 50  0000 C CNN
+F 2 "w_pth_resistors:r-sil_8" H 3000 3400 60  0001 C CNN
+F 3 "" H 3000 3400 60  0000 C CNN
+	1    3000 3400
+	0    1    1    0
+$EndComp
+$Comp
+L R-SIL_8NB R23
+U 1 1 56C3E5BA
+P 3000 5900
+F 0 "R23" V 2945 5905 50  0000 C CNN
+F 1 "R-SIL_8NB" V 3065 5900 50  0000 C CNN
+F 2 "w_pth_resistors:r-sil_8" H 3000 5900 60  0001 C CNN
+F 3 "" H 3000 5900 60  0000 C CNN
+	1    3000 5900
+	0    1    1    0
+$EndComp
+$Comp
+L R-SIL_8NB R24
+U 1 1 56C3E753
+P 3000 8400
+F 0 "R24" V 2945 8405 50  0000 C CNN
+F 1 "R-SIL_8NB" V 3065 8400 50  0000 C CNN
+F 2 "w_pth_resistors:r-sil_8" H 3000 8400 60  0001 C CNN
+F 3 "" H 3000 8400 60  0000 C CNN
+	1    3000 8400
+	0    1    1    0
+$EndComp
+Wire Wire Line
+	3100 3400 3400 3400
+Wire Wire Line
+	3100 3900 3400 3900
+Wire Wire Line
+	3100 4400 3400 4400
+Wire Wire Line
+	3100 4900 3400 4900
+$Comp
+L R-SIL_8NB R22
+U 2 1 56C41F61
+P 3000 3900
+F 0 "R22" V 2945 3905 50  0000 C CNN
+F 1 "R-SIL_8NB" V 3065 3900 50  0000 C CNN
+F 2 "w_pth_resistors:r-sil_8" H 3000 3900 60  0001 C CNN
+F 3 "" H 3000 3900 60  0000 C CNN
+	2    3000 3900
+	0    1    1    0
+$EndComp
+$Comp
+L R-SIL_8NB R23
+U 2 1 56C4243D
+P 3000 6450
+F 0 "R23" V 2945 6455 50  0000 C CNN
+F 1 "R-SIL_8NB" V 3065 6450 50  0000 C CNN
+F 2 "w_pth_resistors:r-sil_8" H 3000 6450 60  0001 C CNN
+F 3 "" H 3000 6450 60  0000 C CNN
+	2    3000 6450
+	0    1    1    0
+$EndComp
+$Comp
+L R-SIL_8NB R22
+U 3 1 56C425F6
+P 3000 4400
+F 0 "R22" V 2945 4405 50  0000 C CNN
+F 1 "R-SIL_8NB" V 3065 4400 50  0000 C CNN
+F 2 "w_pth_resistors:r-sil_8" H 3000 4400 60  0001 C CNN
+F 3 "" H 3000 4400 60  0000 C CNN
+	3    3000 4400
+	0    1    1    0
+$EndComp
+$Comp
+L R-SIL_8NB R22
+U 4 1 56C427B3
+P 3000 4900
+F 0 "R22" V 2945 4905 50  0000 C CNN
+F 1 "R-SIL_8NB" V 3065 4900 50  0000 C CNN
+F 2 "w_pth_resistors:r-sil_8" H 3000 4900 60  0001 C CNN
+F 3 "" H 3000 4900 60  0000 C CNN
+	4    3000 4900
+	0    1    1    0
+$EndComp
+Wire Wire Line
+	3100 5900 3400 5900
+Wire Wire Line
+	3100 6450 3400 6450
+$Comp
+L R-SIL_8NB R23
+U 3 1 56C43704
+P 3000 7000
+F 0 "R23" V 2945 7005 50  0000 C CNN
+F 1 "R-SIL_8NB" V 3065 7000 50  0000 C CNN
+F 2 "w_pth_resistors:r-sil_8" H 3000 7000 60  0001 C CNN
+F 3 "" H 3000 7000 60  0000 C CNN
+	3    3000 7000
+	0    1    1    0
+$EndComp
+$Comp
+L R-SIL_8NB R23
+U 4 1 56C438C1
+P 3000 7600
+F 0 "R23" V 2945 7605 50  0000 C CNN
+F 1 "R-SIL_8NB" V 3065 7600 50  0000 C CNN
+F 2 "w_pth_resistors:r-sil_8" H 3000 7600 60  0001 C CNN
+F 3 "" H 3000 7600 60  0000 C CNN
+	4    3000 7600
+	0    1    1    0
+$EndComp
+$Comp
+L R-SIL_8NB R24
+U 2 1 56C43B7B
+P 3000 9000
+F 0 "R24" V 2945 9005 50  0000 C CNN
+F 1 "R-SIL_8NB" V 3065 9000 50  0000 C CNN
+F 2 "w_pth_resistors:r-sil_8" H 3000 9000 60  0001 C CNN
+F 3 "" H 3000 9000 60  0000 C CNN
+	2    3000 9000
+	0    1    1    0
+$EndComp
+$Comp
+L R-SIL_8NB R24
+U 3 1 56C43D3B
+P 3000 9600
+F 0 "R24" V 2945 9605 50  0000 C CNN
+F 1 "R-SIL_8NB" V 3065 9600 50  0000 C CNN
+F 2 "w_pth_resistors:r-sil_8" H 3000 9600 60  0001 C CNN
+F 3 "" H 3000 9600 60  0000 C CNN
+	3    3000 9600
+	0    1    1    0
+$EndComp
+$Comp
+L R-SIL_8NB R24
+U 4 1 56C43EFA
+P 3000 10200
+F 0 "R24" V 2945 10205 50  0000 C CNN
+F 1 "R-SIL_8NB" V 3065 10200 50  0000 C CNN
+F 2 "w_pth_resistors:r-sil_8" H 3000 10200 60  0001 C CNN
+F 3 "" H 3000 10200 60  0000 C CNN
+	4    3000 10200
+	0    1    1    0
+$EndComp
+Wire Wire Line
+	3100 8400 3400 8400
+Wire Wire Line
+	3100 7000 3400 7000
+Wire Wire Line
+	3400 7600 3100 7600
+Wire Wire Line
+	3100 9000 3400 9000
+Wire Wire Line
+	3100 9600 3400 9600
+Wire Wire Line
+	3100 10200 3400 10200
 $EndSCHEMATC
