File: can-can-rpi/RPi_Hat.kicad_pcb (KiCad board)
At the start: 2 copper layers, 65 x 56 mm, 5 parts, among them J2 RPi_GPIO

Commit message: wip
Parts:
- removed J2: RPi_GPIO, RPi_Hat:Pin_Header_Straight_2x20
- added C1: 100nF, Capacitors_ThroughHole:C_Disc_D3_P2.5, F.Cu at (112.8, 87.6)
- added C2: 100nF, Capacitors_ThroughHole:C_Disc_D3_P2.5, F.Cu at (129.0, 87.9)
- added C3: 27pF, Capacitors_ThroughHole:C_Disc_D3_P2.5, F.Cu at (118.4, 112.0)
- added C4: 27pF, Capacitors_ThroughHole:C_Disc_D3_P2.5, F.Cu at (126.0, 98.0)
- added C5: 100nF, Capacitors_ThroughHole:C_Disc_D3_P2.5, F.Cu at (117.9, 125.7)
- added C6: 100nF, Capacitors_ThroughHole:C_Disc_D3_P2.5, F.Cu at (117.9, 122.2)
- added C7: 100nF, Capacitors_ThroughHole:C_Disc_D3_P2.5, F.Cu at (117.9, 118.4)
- added CON1: BARREL_JACK, Connect:BARREL_JACK, F.Cu at (147.3, 91.4)
- added J1: RPi_GPIO, Socket_Strips:Socket_Strip_Straight_2x20, B.Cu at (94.7, 76.5)
- added JP1: ICSP, ICSP:ICSP, F.Cu at (93.5, 91.2)
- added JP2: JUMPER, Wire_Pads:SolderWirePad_2x_1mmDrill, F.Cu at (127.0, 101.6)
- added JP3: JUMPER, Wire_Pads:SolderWirePad_2x_1mmDrill, F.Cu at (127.0, 105.4)
- added JP4: JUMPER, Wire_Pads:SolderWirePad_2x_1mmDrill, F.Cu at (127.0, 108.7)
- added JP5: JUMPER, Wire_Pads:SolderWirePad_2x_1mmDrill, F.Cu at (127.0, 112.0)
- added JP6: JUMPER, Wire_Pads:SolderWirePad_2x_1mmDrill, F.Cu at (127.3, 115.1)
- added OC1: 6N137, Housings_DIP:DIP-8_W7.62mm, F.Cu at (107.4, 115.8)
- added OC2: 6N137, Housings_DIP:DIP-8_W7.62mm, F.Cu at (107.4, 101.6)
- added P1: CONN_02X02, Pin_Headers:Pin_Header_Straight_2x02, F.Cu at (90.9, 81.5)
- added P2: CONN_01X14, Socket_Strips:Socket_Strip_Straight_1x14, F.Cu at (101.1, 94.7)
- added P3: CONN_01X14, Socket_Strips:Socket_Strip_Straight_1x14, F.Cu at (134.4, 80.8)
- added P5: CONN_01X03, Pin_Headers:Pin_Header_Straight_1x03, F.Cu at (96.5, 124.2)
- added R1: 15k, Resistors_ThroughHole:Resistor_Horizontal_RM10mm, F.Cu at (106.4, 97.8)
- added R10: 390, Resistors_ThroughHole:Resistor_Horizontal_RM10mm, F.Cu at (100.3, 111.3)
- added R3: 3k3, Resistors_ThroughHole:Resistor_Horizontal_RM10mm, F.Cu at (143.0, 83.3)
- added R4: 3k3, Resistors_ThroughHole:Resistor_Horizontal_RM10mm, F.Cu at (143.0, 80.5)
- added R5: 470, Resistors_ThroughHole:Resistor_Horizontal_RM10mm, F.Cu at (96.3, 95.5)
- added R6: 470, Resistors_ThroughHole:Resistor_Horizontal_RM10mm, F.Cu at (101.9, 87.1)
- added R7: 390, Resistors_ThroughHole:Resistor_Horizontal_RM10mm, F.Cu at (104.1, 115.6)
- added R8: 390, Resistors_ThroughHole:Resistor_Horizontal_RM10mm, F.Cu at (121.2, 105.4)
- added R9: 390, Resistors_ThroughHole:Resistor_Horizontal_RM10mm, F.Cu at (122.7, 120.4)
- added U1: PIC18F25K80, Housings_DIP:DIP-28_W7.62mm, F.Cu at (101.3, 90.9)
- added U2: MCP2562-I/P, Housings_DIP:DIP-8_W7.62mm_LongPads, F.Cu at (96.0, 118.4)
- added Y1: 16MHz, Crystals:Crystal_HC49-U_Vertical, F.Cu at (121.9, 87.4)

Commit message: update schematic and board
Parts:
- added D1: LED, LEDs:LED-3MM, F.Cu at (87.6, 100.3)
- added D2: LED, LEDs:LED-3MM, F.Cu at (81.3, 100.3)
- added D3: LED, LEDs:LED-3MM, F.Cu at (74.9, 100.3)
- added P4: CONN_01X02, Pin_Headers:Pin_Header_Straight_1x02, F.Cu at (103.1, 133.3)
- added R11: 560, Resistors_ThroughHole:Resistor_Horizontal_RM10mm, F.Cu at (81.3, 111.8)
- added R12: 560, Resistors_ThroughHole:Resistor_Horizontal_RM10mm, F.Cu at (74.9, 111.8)
- added R13: 120, Resistors_ThroughHole:Resistor_Horizontal_RM10mm, F.Cu at (102.1, 129.8)
- added R14: 680, Resistors_ThroughHole:Resistor_Horizontal_RM10mm, F.Cu at (120.9, 132.6)
- added R2: 560, Resistors_ThroughHole:Resistor_Horizontal_RM10mm, F.Cu at (87.6, 91.4)
- moved C6 22.2 mm to (104.9, 104.1), turned to 180 degrees
- moved C5 21.4 mm to (102.9, 110.5)
- moved R9 18.4 mm to (104.4, 118.4), turned to 270 degrees
- moved R7 18.2 mm to (121.9, 119.4)
- moved OC1 11.9 mm to (115.1, 125.0), turned to 180 degrees
- moved P2 1.05 mm to (101.3, 93.7)
- moved P3 0.25 mm to (134.4, 80.5)
Connections:
- J1 pad 36: Net-(J1-Pad36) -> /RPi_GPIO/CTS
- P1 pad 2: /RPi_GPIO/RxD -> Net-(P1-Pad2)
- P1 pad 4: /RPi_GPIO/TxD -> Net-(P1-Pad4)
- P3 pad 2: /RPi_GPIO/RC5 -> /RPi_GPIO/CTS
- R5 pad 2: Net-(J1-Pad18) -> Net-(P1-Pad2)
- R6 pad 2: Net-(J1-Pad22) -> Net-(P1-Pad4)
- U1 pad 16: /RPi_GPIO/RC5 -> /RPi_GPIO/CTS
Other:
- board text removed: "Camera Flex Slot (Optional)"
- board text removed: "Dimensions taken from https://github.com/raspberrypi/hats/blob/master/hat-board-mechanical.pdf"

Commit message: change footprints and layout - wip
Parts:
- C3, C4: value 27pF -> 22pF
- JP2, JP3, JP4, JP5, JP6: footprint Wire_Pads:SolderWirePad_2x_1mmDrill -> Wire_Pads:SolderWirePad_2x_0-2.54mmDrill
- R1: value 15k -> 4.7k; footprint Resistors_ThroughHole:Resistor_Horizontal_RM10mm -> Resistors_ThroughHole:Resistor_Horizontal_RM7.5mm
- R10, R11, R12, R13, R14, R2, R3, R4, R7, R8, R9: footprint Resistors_ThroughHole:Resistor_Horizontal_RM10mm -> Resistors_ThroughHole:Resistor_Horizontal_RM7.5mm
- R5, R6: value 470 -> 390; footprint Resistors_ThroughHole:Resistor_Horizontal_RM10mm -> Resistors_ThroughHole:Resistor_Horizontal_RM7.5mm
- moved R12 68.1 mm to (141.0, 95.2), turned to 180 degrees
- moved D2 66.8 mm to (147.3, 90.2)
- moved D3 66.8 mm to (141.0, 90.2)
- moved R11 66.3 mm to (146.1, 97.8), turned to 0 degrees
- moved D1 57.8 mm to (142.9, 83.2), turned to 90 degrees
- moved P1 56.4 mm to (147.3, 83.8)
- moved R4 51.0 mm to (92.1, 82.5), turned to 0 degrees
- moved R3 50.4 mm to (92.7, 80.0), turned to 0 degrees
- moved CON1 47.2 mm to (101.0, 100.3), turned to 0 degrees
- moved JP1 44.5 mm to (136.5, 80.0)
- moved P3 37.2 mm to (99.7, 94.0), turned to 0 degrees
- moved P2 34.2 mm to (132.7, 80.0), turned to 180 degrees
- moved R5 33.4 mm to (128.9, 88.3), turned to 180 degrees
- moved U1 32.3 mm to (132.7, 83.2), turned to 270 degrees
- moved C4 29.0 mm to (99.7, 85.7)
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Connections:
- D1 pad 1: /RPi_GPIO/RA2 -> /RPi_GPIO/RA0
- D3 pad 1: /RPi_GPIO/RA0 -> /RPi_GPIO/RA2
- OC1 pad 2: VCC -> Net-(OC1-Pad2)
- OC1 pad 3: Net-(OC1-Pad3) -> /RPi_GPIO/CANTX
- OC2 pad 2: +5V -> Net-(OC2-Pad2)
- OC2 pad 3: Net-(OC2-Pad3) -> /RPi_GPIO/_CANRX
- OC2 pad 6: /RPi_GPIO/CANTX -> /RPi_GPIO/CANRX
- R10 pad 1: /RPi_GPIO/_CANRX -> Net-(OC2-Pad2)
- R10 pad 2: Net-(OC2-Pad3) -> +5V
- R12 pad 2: Net-(D1-Pad2) -> Net-(D3-Pad2)
- R14 pad 2: /RPi_GPIO/CANTX -> /RPi_GPIO/CANRX
- R2 pad 2: Net-(D3-Pad2) -> Net-(D1-Pad2)
- R7 pad 1: Net-(OC1-Pad3) -> Net-(OC1-Pad2)
- R7 pad 2: /RPi_GPIO/CANTX -> VCC
- R8 pad 1: /RPi_GPIO/CANTX -> /RPi_GPIO/CANRX
