File: BPi-CAN/BPi-CAN.sch (KiCad schematic (older format))
At the start: 83 parts, among them J1 RJ45, J2 RJ45, J3 RJ45, J4 RJ45, P1 CONN_02X13, P10 SPI, P11 CONN_01X02, P12 CAN-Bus, P13 CONN_01X04, P14 CAN-Bus, P15 CONN_01X02, P16 CAN, P17 CAN, P18 CAN, P19 TERM, P2 S88, P20 S88 CONN, P3 CONN_02X04, P4 CONN_01X02, P5 CONN_01X02, P6 S88, P7 I2C-Bus, P8 CONN_01X03, P9 CONN_01X05, U1 MCP2562, U10 MCP2562, U11 6N137, U12 ISO1050, U13 FT230XS, U2 LM7805, U3 6N137, U4 6N137, U5 6N137, U6 6N137, U7 ADuM1251BR, U8 MAX3072E, U9 MAX3232

Commit message: more S88 parts
Connections:
- wire segments 322 -> 386
- no-connect marks 46 -> 34
Other:
- note added: "CLOCK"
- note added: "DATA"
- note added: "LOAD"
- note added: "RESET"
- moved on the sheet: P2

Commit message: S88 wip
Parts:
- P2, P6: footprint Pin_Headers:Pin_Header_Straight_1x06 -> w_conn_pt-1,5:pt_1,5-6-3,5-h
Connections:
- wire segments 386 -> 338

Commit message: wip
Parts:
- added P21: RS232 Con, Pin_Headers:Pin_Header_Straight_1x03, symbol CONN_01X03
- P11: value CONN_01X02 -> SNIFFER; footprint Pin_Headers:Pin_Header_Straight_1x02 -> w_conn_pt-1,5:pt_1,5-2-3,5-h
- P8: value CONN_01X03 -> RS485
- P9: value CONN_01X05 -> RS232
Connections:
- wire segments 338 -> 342
Changed lines of the file:
@@
 P 1050 5100
 F 0 "P3" H 1050 5350 50  0000 C CNN
-F 1 "CONN_02X04" H 1050 4850 50  0000 C CNN
+F 1 "CONN_02X04" H 1050 4850 50  0001 C CNN
 F 2 "Socket_Strips:Socket_Strip_Straight_2x04" H 1050 3900 50  0001 C CNN
 F 3 "" H 1050 3900 50  0000 C CNN
@@
 P 10950 3200
 F 0 "P8" H 10950 3400 50  0000 C CNN
-F 1 "CONN_01X03" V 11050 3200 50  0000 C CNN
+F 1 "RS485" V 11050 3200 50  0000 C CNN
 F 2 "Pin_Headers:Pin_Header_Straight_1x03" H 10950 3200 50  0001 C CNN
 F 3 "" H 10950 3200 50  0000 C CNN
@@
 P 10900 2150
 F 0 "P9" H 10900 2450 50  0000 C CNN
-F 1 "CONN_01X05" V 11000 2150 50  0000 C CNN
+F 1 "RS232" V 11000 2150 50  0000 C CNN
 F 2 "Pin_Headers:Pin_Header_Straight_1x05" H 10900 2150 50  0001 C CNN
 F 3 "" H 10900 2150 50  0000 C CNN
@@
 P 2700 4100
 F 0 "P11" H 2700 4250 50  0000 C CNN
-F 1 "CONN_01X02" V 2800 4100 50  0000 C CNN
-F 2 "Pin_Headers:Pin_Header_Straight_1x02" H 2700 4100 50  0001 C CNN
+F 1 "SNIFFER" V 2800 4100 50  0000 C CNN
+F 2 "w_conn_pt-1,5:pt_1,5-2-3,5-h" H 2700 4100 50  0001 C CNN
 F 3 "" H 2700 4100 50  0000 C CNN
 	1    2700 4100
@@
 Text Notes 5250 7100 0    60   ~ 0
 DATA
+$Comp
+L CONN_01X03 P21
+U 1 1 568C085A
+P 4600 3800
+F 0 "P21" H 4600 4000 50  0000 C CNN
+F 1 "RS232 Con" V 4700 3800 50  0000 C CNN
+F 2 "Pin_Headers:Pin_Header_Straight_1x03" H 4600 3800 50  0001 C CNN
+F 3 "" H 4600 3800 50  0000 C CNN
+	1    4600 3800
+	-1   0    0    1
+$EndComp
+Wire Wire Line
+	4800 3700 5100 3700
+Wire Wire Line
+	4800 3800 5100 3800
+Wire Wire Line
+	4800 3900 5050 3900
+Wire Wire Line
+	5050 3900 5050 4100
+$Comp
+L GND #PWR077
+U 1 1 568C12AA
+P 5050 4100
+F 0 "#PWR077" H 5050 3850 50  0001 C CNN
+F 1 "GND" H 5050 3950 50  0000 C CNN
+F 2 "" H 5050 4100 50  0000 C CNN
+F 3 "" H 5050 4100 50  0000 C CNN
+	1    5050 4100
+	1    0    0    -1
+$EndComp
+Text Label 4900 3700 0    60   ~ 0
+RxD
+Text Label 4900 3800 0    60   ~ 0
+TxD
 $EndSCHEMATC

Commit message: wip
Parts:
- added P22: S88, Pin_Headers:Pin_Header_Straight_1x06, symbol CONN_01X06
- U2: footprint Transistors_TO-220:TO-220_Neutral123_Horizontal -> 78xx:TO-220-78xx
Connections:
- wire segments 342 -> 348
Other:
- moved on the sheet: P2

Commit message: wip
Parts:
- P8: footprint Pin_Headers:Pin_Header_Straight_1x03 -> w_conn_pt-1,5:pt_1,5-3-3,5-h
- R10, R11, R12, R13, R14, R15, R2, R3, R4, R5, R6, R7, R8, R9: footprint Resistors_ThroughHole:Resistor_Horizontal_RM10mm -> w_pth_resistors:RC03
- U11, U3, U4, U5, U6: footprint Housings_DIP:DIP-8_W7.62mm -> w_pth_circuits:dil_8-300_socket; symbol 6N136 -> 6N136-RESCUE-BPi-CAN
- U7: symbol ADuM1201BR -> ADuM1201BR-RESCUE-BPi-CAN
- U8: footprint Housings_DIP:DIP-8_W7.62mm -> w_pth_circuits:dil_8-300_socket; symbol SP3485EP -> SP3485EP-RESCUE-BPi-CAN
- U9: symbol MAX232 -> MAX232-RESCUE-BPi-CAN
Changed lines of the file:
@@
 $EndComp
 $Comp
-L 6N136 U3
+L 6N136-RESCUE-BPi-CAN U3
 U 1 1 567EBDE8
 P 3350 5950
 F 0 "U3" H 3150 6250 50  0000 L CNN
 F 1 "6N137" H 3350 6250 50  0000 L CNN
-F 2 "Housings_DIP:DIP-8_W7.62mm" H 3150 5650 50  0001 L CIN
+F 2 "w_pth_circuits:dil_8-300_socket" H 3150 5650 50  0001 L CIN
 F 3 "" H 3350 5950 50  0000 L CNN
 	1    3350 5950
@@
 $EndComp
 $Comp
-L 6N136 U4
+L 6N136-RESCUE-BPi-CAN U4
 U 1 1 567EBE6F
 P 3350 6700
 F 0 "U4" H 3150 7000 50  0000 L CNN
 F 1 "6N137" H 3350 7000 50  0000 L CNN
-F 2 "Housings_DIP:DIP-8_W7.62mm" H 3150 6400 50  0001 L CIN
+F 2 "w_pth_circuits:dil_8-300_socket" H 3150 6400 50  0001 L CIN
 F 3 "" H 3350 6700 50  0000 L CNN
 	1    3350 6700
@@
 $EndComp
 $Comp
-L 6N136 U5
+L 6N136-RESCUE-BPi-CAN U5
 U 1 1 567EBEC9
 P 3350 7450
 F 0 "U5" H 3150 7750 50  0000 L CNN
 F 1 "6N137" H 3350 7750 50  0000 L CNN
-F 2 "Housings_DIP:DIP-8_W7.62mm" H 3150 7150 50  0001 L CIN
+F 2 "w_pth_circuits:dil_8-300_socket" H 3150 7150 50  0001 L CIN
 F 3 "" H 3350 7450 50  0000 L CNN
 	1    3350 7450
@@
 $EndComp
 $Comp
-L 6N136 U6
+L 6N136-RESCUE-BPi-CAN U6
 U 1 1 567EBF15
 P 1650 7050
 F 0 "U6" H 1450 7350 50  0000 L CNN
 F 1 "6N137" H 1650 7350 50  0000 L CNN
-F 2 "Housings_DIP:DIP-8_W7.62mm" H 1450 6750 50  0001 L CIN
+F 2 "w_pth_circuits:dil_8-300_socket" H 1450 6750 50  0001 L CIN
 F 3 "" H 1650 7050 50  0000 L CNN
 	1    1650 7050
@@
 F 0 "R2" V 2980 5850 50  0000 C CNN
 F 1 "270" V 2900 5850 50  0000 C CNN
-F 2 "Resistors_ThroughHole:Resistor_Horizontal_RM10mm" H 2830 5850 50  0001 C CNN
+F 2 "w_pth_resistors:RC03" H 2830 5850 50  0001 C CNN
 F 3 "" H 2900 5850 50  0000 C CNN
 	1    2900 5850
@@
 F 0 "R3" V 2980 6600 50  0000 C CNN
 F 1 "270" V 2900 6600 50  0000 C CNN
-F 2 "Resistors_ThroughHole:Resistor_Horizontal_RM10mm" V 2830 6600 50  0001 C CNN
+F 2 "w_pth_resistors:RC03" V 2830 6600 50  0001 C CNN
 F 3 "" H 2900 6600 50  0000 C CNN
 	1    2900 6600
@@
 F 0 "R4" V 2980 7350 50  0000 C CNN
 F 1 "270" V 2900 7350 50  0000 C CNN
-F 2 "Resistors_ThroughHole:Resistor_Horizontal_RM10mm" V 2830 7350 50  0001 C CNN
+F 2 "w_pth_resistors:RC03" V 2830 7350 50  0001 C CNN
 F 3 "" H 2900 7350 50  0000 C CNN
 	1    2900 7350
@@
 F 0 "R5" V 1100 7150 50  0000 C CNN
 F 1 "390" V 1200 7150 50  0000 C CNN
-F 2 "Resistors_ThroughHole:Resistor_Horizontal_RM10mm" V 1130 7150 50  0001 C CNN
+F 2 "w_pth_resistors:RC03" V 1130 7150 50  0001 C CNN
 F 3 "" H 1200 7150 50  0000 C CNN
 	1    1200 7150
@@
 F 0 "R6" V 2180 7150 50  0000 C CNN
 F 1 "390" V 2100 7150 50  0000 C CNN
-F 2 "Resistors_ThroughHole:Resistor_Horizontal_RM10mm" V 2030 7150 50  0001 C CNN
+F 2 "w_pth_resistors:RC03" V 2030 7150 50  0001 C CNN
 F 3 "" H 2100 7150 50  0000 C CNN
 	1    2100 7150
@@
 F 0 "R7" V 3880 6050 50  0000 C CNN
 F 1 "1k5" V 3800 6050 50  0000 C CNN
-F 2 "Resistors_ThroughHole:Resistor_Horizontal_RM10mm" H 3730 6050 50  0001 C CNN
+F 2 "w_pth_resistors:RC03" H 3730 6050 50  0001 C CNN
 F 3 "" H 3800 6050 50  0000 C CNN
 	1    3800 6050
@@
 F 0 "R8" V 3880 6800 50  0000 C CNN
 F 1 "1k5" V 3800 6800 50  0000 C CNN
-F 2 "Resistors_ThroughHole:Resistor_Horizontal_RM10mm" H 3730 6800 50  0001 C CNN
+F 2 "w_pth_resistors:RC03" H 3730 6800 50  0001 C CNN
 F 3 "" H 3800 6800 50  0000 C CNN
 	1    3800 6800
@@
 F 0 "R9" V 3880 7550 50  0000 C CNN
 F 1 "1k5" V 3800 7550 50  0000 C CNN
-F 2 "Resistors_ThroughHole:Resistor_Horizontal_RM10mm" H 3730 7550 50  0001 C CNN
+F 2 "w_pth_resistors:RC03" H 3730 7550 50  0001 C CNN
 F 3 "" H 3800 7550 50  0000 C CNN
 	1    3800 7550
@@
 F 0 "R11" V 1280 7250 50  0000 C CNN
 F 1 "1k" V 1200 7250 50  0000 C CNN
-F 2 "Resistors_ThroughHole:Resistor_Horizontal_RM10mm" V 1130 7250 50  0001 C CNN
+F 2 "w_pth_resistors:RC03" V 1130 7250 50  0001 C CNN
 F 3 "" H 1200 7250 50  0000 C CNN
 	1    1200 7250
@@
 F 0 "R10" V 1080 7450 50  0000 C CNN
 F 1 "1k8" V 1000 7450 50  0000 C CNN
-F 2 "Resistors_ThroughHole:Resistor_Horizontal_RM10mm" V 930 7450 50  0001 C CNN
+F 2 "w_pth_resistors:RC03" V 930 7450 50  0001 C CNN
 F 3 "" H 1000 7450 50  0000 C CNN
 	1    1000 7450
@@
 GPIO4
 $Comp
-L ADuM1201BR U7
+L ADuM1201BR-RESCUE-BPi-CAN U7
 U 1 1 5681379B
 P 2850 5000
@@
 $EndComp
 $Comp
-L SP3485EP U8
+L SP3485EP-RESCUE-BPi-CAN U8
 U 1 1 56818005
 P 9550 3200
 F 0 "U8" H 9250 3550 50  0000 L CNN
 F 1 "MAX3072E" H 9650 3550 50  0000 L CNN
-F 2 "Housings_DIP:DIP-8_W7.62mm" H 9550 3200 50  0001 C CIN
+F 2 "w_pth_circuits:dil_8-300_socket" H 9550 3200 50  0001 C CIN
 F 3 "" H 9550 3200 50  0000 C CNN
 	1    9550 3200
@@
 F 0 "P8" H 10950 3400 50  0000 C CNN
 F 1 "RS485" V 11050 3200 50  0000 C CNN
-F 2 "Pin_Headers:Pin_Header_Straight_1x03" H 10950 3200 50  0001 C CNN
+F 2 "w_conn_pt-1,5:pt_1,5-3-3,5-h" H 10950 3200 50  0001 C CNN
 F 3 "" H 10950 3200 50  0000 C CNN
 	1    10950 3200
@@
 $EndComp
 $Comp
-L MAX232 U9
+L MAX232-RESCUE-BPi-CAN U9
 U 1 1 5681D402
 P 9650 1550
@@
 PI14
 $Comp
-L 6N136 U11
+L 6N136-RESCUE-BPi-CAN U11
 U 1 1 5684F13B
 P 1550 4100
 F 0 "U11" H 1350 4400 50  0000 L CNN
 F 1 "6N137" H 1550 4400 50  0000 L CNN
-F 2 "Housings_DIP:DIP-8_W7.62mm" H 1350 3800 50  0001 L CIN
+F 2 "w_pth_circuits:dil_8-300_socket" H 1350 3800 50  0001 L CIN
 F 3 "" H 1550 4100 50  0000 L CNN
 	1    1550 4100
@@
 F 0 "R13" V 1000 4200 50  0000 C CNN
 F 1 "390" V 1100 4200 50  0000 C CNN
-F 2 "Resistors_ThroughHole:Resistor_Horizontal_RM10mm" V 1030 4200 50  0001 C CNN
+F 2 "w_pth_resistors:RC03" V 1030 4200 50  0001 C CNN
 F 3 "" H 1100 4200 50  0000 C CNN
 	1    1100 4200
@@
 F 0 "R15" V 2330 4000 50  0000 C CNN
 F 1 "1K5" V 2250 4000 50  0000 C CNN
-F 2 "Resistors_ThroughHole:Resistor_Horizontal_RM10mm" V 2180 4000 50  0001 C CNN
+F 2 "w_pth_resistors:RC03" V 2180 4000 50  0001 C CNN
 F 3 "" H 2250 4000 50  0000 C CNN
 	1    2250 4000
@@
 F 0 "R14" V 1180 4300 50  0000 C CNN
 F 1 "1k" V 1100 4300 50  0000 C CNN
-F 2 "Resistors_ThroughHole:Resistor_Horizontal_RM10mm" V 1030 4300 50  0001 C CNN
+F 2 "w_pth_resistors:RC03" V 1030 4300 50  0001 C CNN
 F 3 "" H 1100 4300 50  0000 C CNN
 	1    1100 4300
@@
 F 0 "R12" V 980 4500 50  0000 C CNN
 F 1 "1k8" V 900 4500 50  0000 C CNN
-F 2 "Resistors_ThroughHole:Resistor_Horizontal_RM10mm" V 830 4500 50  0001 C CNN
+F 2 "w_pth_resistors:RC03" V 830 4500 50  0001 C CNN
 F 3 "" H 900 4500 50  0000 C CNN
 	1    900  4500
@@
 S88_7
 Text Label 6650 7300 2    60   ~ 0
-S88_6
+S88_8
 NoConn ~ 6850 5350
 NoConn ~ 5700 5350

Commit message: wip
Parts:
- removed R10, R12: 1k8, w_pth_resistors:RC03, symbol R
- removed R11, R14: 1k, w_pth_resistors:RC03, symbol R
- added C21: 100nF, Capacitors_ThroughHole:C_Disc_D3_P2.5, symbol C
- P13: value CONN_01X04 -> USB
- R13, R5: value 390 -> 1k8
- R20: value 220 -> 120
Connections:
- net labels added: +5VA
- wire segments 348 -> 346
- no-connect marks 34 -> 33
Other:
- moved on the sheet: C8
Changed lines of the file:
@@
 $EndComp
 $Comp
-L +5VD #PWR015
+L +5VA #PWR015
 U 1 1 567EB708
 P 6450 850
 F 0 "#PWR015" H 6450 700 50  0001 C CNN
-F 1 "+5VD" H 6450 990 50  0000 C CNN
+F 1 "+5VA" H 6450 990 50  0000 C CNN
 F 2 "" H 6450 850 50  0000 C CNN
 F 3 "" H 6450 850 50  0000 C CNN
@@
 P 1200 7150
 F 0 "R5" V 1100 7150 50  0000 C CNN
-F 1 "390" V 1200 7150 50  0000 C CNN
+F 1 "1k8" V 1200 7150 50  0000 C CNN
 F 2 "w_pth_resistors:RC03" V 1130 7150 50  0001 C CNN
 F 3 "" H 1200 7150 50  0000 C CNN
@@
 CLOCK
 $Comp
-L GNDA #PWR024
+L GNDD #PWR024
 U 1 1 567ECC49
 P 1650 6300
 F 0 "#PWR024" H 1650 6050 50  0001 C CNN
-F 1 "GNDA" H 1650 6150 50  0000 C CNN
+F 1 "GNDD" H 1650 6150 50  0000 C CNN
 F 2 "" H 1650 6300 50  0000 C CNN
 F 3 "" H 1650 6300 50  0000 C CNN
@@
 L C C8
 U 1 1 567EC8AA
-P 600 7500
-F 0 "C8" H 625 7600 50  0000 L CNN
-F 1 "100nF" H 625 7400 50  0000 L CNN
-F 2 "Capacitors_ThroughHole:C_Disc_D3_P2.5" H 638 7350 50  0001 C CNN
-F 3 "" H 600 7500 50  0000 C CNN
-	1    600  7500
+P 600 7450
+F 0 "C8" H 625 7550 50  0000 L CNN
+F 1 "100nF" H 625 7350 50  0000 L CNN
+F 2 "Capacitors_ThroughHole:C_Disc_D3_P2.5" H 638 7300 50  0001 C CNN
+F 3 "" H 600 7450 50  0000 C CNN
+	1    600  7450
 	1    0    0    -1
 $EndComp
@@
 $EndComp
 $Comp
-L GNDA #PWR027
+L GNDD #PWR027
 U 1 1 567ECBAB
 P 2050 6200
 F 0 "#PWR027" H 2050 5950 50  0001 C CNN
-F 1 "GNDA" H 2050 6050 50  0000 C CNN
+F 1 "GNDD" H 2050 6050 50  0000 C CNN
 F 2 "" H 2050 6200 50  0000 C CNN
 F 3 "" H 2050 6200 50  0000 C CNN
@@
 	1    0    0    -1
 $EndComp
-Entry Wire Line
-	-5550 8000 -5450 8100
-$Comp
-L GNDA #PWR028
+$Comp
+L GNDD #PWR028
 U 1 1 5681215E
 P 2300 7200
 F 0 "#PWR028" H 2300 6950 50  0001 C CNN
-F 1 "GNDA" H 2300 7050 50  0000 C CNN
+F 1 "GNDD" H 2300 7050 50  0000 C CNN
 F 2 "" H 2300 7200 50  0000 C CNN
 F 3 "" H 2300 7200 50  0000 C CNN
 	1    2300 7200
-	1    0    0    -1
-$EndComp
-$Comp
-L R R11
-U 1 1 56812349
-P 1200 7250
-F 0 "R11" V 1280 7250 50  0000 C CNN
-F 1 "1k" V 1200 7250 50  0000 C CNN
-F 2 "w_pth_resistors:RC03" V 1130 7250 50  0001 C CNN
-F 3 "" H 1200 7250 50  0000 C CNN
-	1    1200 7250
-	0    1    1    0
-$EndComp
-$Comp
-L R R10
-U 1 1 56812D60
-P 1000 7450
-F 0 "R10" V 1080 7450 50  0000 C CNN
-F 1 "1k8" V 1000 7450 50  0000 C CNN
-F 2 "w_pth_resistors:RC03" V 930 7450 50  0001 C CNN
-F 3 "" H 1000 7450 50  0000 C CNN
-	1    1000 7450
 	1    0    0    -1
 $EndComp
@@
 L +5V #PWR044
 U 1 1 5681B4FE
-P 950 6800
-F 0 "#PWR044" H 950 6650 50  0001 C CNN
-F 1 "+5V" H 950 6940 50  0000 C CNN
-F 2 "" H 950 6800 50  0000 C CNN
-F 3 "" H 950 6800 50  0000 C CNN
-	1    950  6800
+P 1200 6800
+F 0 "#PWR044" H 1200 6650 50  0001 C CNN
+F 1 "+5V" H 1200 6940 50  0000 C CNN
+F 2 "" H 1200 6800 50  0000 C CNN
+F 3 "" H 1200 6800 50  0000 C CNN
+	1    1200 6800
 	1    0    0    -1
 $EndComp
@@
 P 1100 4200
 F 0 "R13" V 1000 4200 50  0000 C CNN
-F 1 "390" V 1100 4200 50  0000 C CNN
+F 1 "1k8" V 1100 4200 50  0000 C CNN
 F 2 "w_pth_resistors:RC03" V 1030 4200 50  0001 C CNN
 F 3 "" H 1100 4200 50  0000 C CNN
@@
 	0    1    1    0
 $EndComp
-$Comp
-L R R14
-U 1 1 5684F15A
-P 1100 4300
-F 0 "R14" V 1180 4300 50  0000 C CNN
-F 1 "1k" V 1100 4300 50  0000 C CNN
-F 2 "w_pth_resistors:RC03" V 1030 4300 50  0001 C CNN
-F 3 "" H 1100 4300 50  0000 C CNN
-	1    1100 4300
-	0    1    1    0
-$EndComp
-$Comp
-L R R12
-U 1 1 5684F160
-P 900 4500
-F 0 "R12" V 980 4500 50  0000 C CNN
-F 1 "1k8" V 900 4500 50  0000 C CNN
-F 2 "w_pth_resistors:RC03" V 830 4500 50  0001 C CNN
-F 3 "" H 900 4500 50  0000 C CNN
-	1    900  4500
-	1    0    0    -1
-$EndComp
 Text Label 550  4300 0    60   ~ 0
 PI3
@@
 L +5V #PWR059
 U 1 1 5684F16D
-P 850 3850
-F 0 "#PWR059" H 850 3700 50  0001 C CNN
-F 1 "+5V" H 850 3990 50  0000 C CNN
-F 2 "" H 850 3850 50  0000 C CNN
-F 3 "" H 850 3850 50  0000 C CNN
-	1    850  3850
+P 1150 3700
+F 0 "#PWR059" H 1150 3550 50  0001 C CNN
+F 1 "+5V" H 1150 3840 50  0000 C CNN
+F 2 "" H 1150 3700 50  0000 C CNN
+F 3 "" H 1150 3700 50  0000 C CNN
+	1    1150 3700
 	1    0    0    -1
 $EndComp
@@
 L GND #PWR060
 U 1 1 5685E5B0
-P 1000 7600
-F 0 "#PWR060" H 1000 7350 50  0001 C CNN
-F 1 "GND" H 1000 7450 50  0000 C CNN
-F 2 "" H 1000 7600 50  0000 C CNN
-F 3 "" H 1000 7600 50  0000 C CNN
-	1    1000 7600
+P 600 7600
+F 0 "#PWR060" H 600 7350 50  0001 C CNN
+F 1 "GND" H 600 7450 50  0000 C CNN
+F 2 "" H 600 7600 50  0000 C CNN
+F 3 "" H 600 7600 50  0000 C CNN
+	1    600  7600
 	1    0    0    -1
 $EndComp
@@
 L GND #PWR061
 U 1 1 5685F0B3
-P 900 4650
-F 0 "#PWR061" H 900 4400 50  0001 C CNN
-F 1 "GND" H 900 4500 50  0000 C CNN
-F 2 "" H 900 4650 50  0000 C CNN
-F 3 "" H 900 4650 50  0000 C CNN
-	1    900  4650
+P 850 4650
+F 0 "#PWR061" H 850 4400 50  0001 C CNN
+F 1 "GND" H 850 4500 50  0000 C CNN
+F 2 "" H 850 4650 50  0000 C CNN
+F 3 "" H 850 4650 50  0000 C CNN
+	1    850  4650
 	1    0    0    -1
 $EndComp
@@
 NoConn ~ 10000 5200
 NoConn ~ 11050 5200
-NoConn ~ 5550 -1900
 $Comp
 L ISO1050 U12
@@
 $EndComp
 $Comp
-L +5VD #PWR065
+L +5VA #PWR065
 U 1 1 568528D1
 P 7000 800
 F 0 "#PWR065" H 7000 650 50  0001 C CNN
-F 1 "+5VD" H 7000 940 50  0000 C CNN
+F 1 "+5VA" H 7000 940 50  0000 C CNN
 F 2 "" H 7000 800 50  0000 C CNN
 F 3 "" H 7000 800 50  0000 C CNN
@@
 $EndComp
 $Comp
-L +5VD #PWR069
+L +5VA #PWR069
 U 1 1 56856422
 P 7450 1700
 F 0 "#PWR069" H 7450 1550 50  0001 C CNN
-F 1 "+5VD" H 7450 1840 50  0000 C CNN
+F 1 "+5VA" H 7450 1840 50  0000 C CNN
 F 2 "" H 7450 1700 50  0000 C CNN
 F 3 "" H 7450 1700 50  0000 C CNN
@@
 P 4750 3200
 F 0 "P13" H 4750 3450 50  0000 C CNN
-F 1 "CONN_01X04" V 4850 3200 50  0000 C CNN
+F 1 "USB" V 4850 3200 50  0000 C CNN
 F 2 "w_conn_pc:conn_usb_B" H 4750 3200 50  0001 C CNN
 F 3 "" H 4750 3200 50  0000 C CNN
@@
 P 7600 2350
 F 0 "R20" V 7500 2350 50  0000 C CNN
-F 1 "220" V 7600 2350 50  0000 C CNN
+F 1 "120" V 7600 2350 50  0000 C CNN
 F 2 "Resistors_SMD:R_0805_HandSoldering" V 7530 2350 50  0001 C CNN
 F 3 "" H 7600 2350 50  0000 C CNN
@@
 	0    1    1    0
 $EndComp
+$Comp
+L +3V3 #PWR078
+U 1 1 569243DE
+P 950 6800
+F 0 "#PWR078" H 950 6650 50  0001 C CNN
+F 1 "+3V3" H 950 6940 50  0000 C CNN
+F 2 "" H 950 6800 50  0000 C CNN
+F 3 "" H 950 6800 50  0000 C CNN
+	1    950  6800
+	1    0    0    -1
+$EndComp
+$Comp
+L +3V3 #PWR079
+U 1 1 5692E2E3
+P 750 4000
+F 0 "#PWR079" H 750 3850 50  0001 C CNN
+F 1 "+3V3" H 750 4140 50  0000 C CNN
+F 2 "" H 750 4000 50  0000 C CNN
+F 3 "" H 750 4000 50  0000 C CNN
+	1    750  4000
+	1    0    0    -1
+$EndComp
+$Comp
+L C C21
+U 1 1 5692EB2B
+P 850 4500
+F 0 "C21" H 875 4600 50  0000 L CNN
+F 1 "100nF" H 875 4400 50  0000 L CNN
+F 2 "Capacitors_ThroughHole:C_Disc_D3_P2.5" H 888 4350 50  0001 C CNN
+F 3 "" H 850 4500 50  0000 C CNN
+	1    850  4500
+	1    0    0    -1
+$EndComp
 Wire Wire Line
 	1250 1250 1400 1250
@@
 	600  6950 1350 6950
 Wire Wire Line
-	950  6800 950  7150
-Wire Wire Line
-	1350 6850 950  6850
-Connection ~ 950  6850
+	1350 6850 1200 6850
+Connection ~ 1200 6850
 Wire Wire Line
 	2650 7300 2650 7350
@@
 Wire Wire Line
 	950  7150 1050 7150
-Connection ~ 950  6950
+Connection ~ 1200 6950
 Wire Wire Line
 	3950 5750 3950 6050
@@
 	2300 7150 2300 7200
 Wire Wire Line
-	650  7250 1050 7250
-Wire Wire Line
-	1000 7250 1000 7300
-Connection ~ 1000 7250
+	650  7250 1350 7250
 Wire Wire Line
 	2400 5250 2300 5250
@@
 	850  4000 1250 4000
 Wire Wire Line
-	850  3850 850  4200
-Wire Wire Line
-	1250 3900 850  3900
-Connection ~ 850  3900
-Wire Wire Line
-	850  4200 950  4200
-Connection ~ 850  4000
-Wire Wire Line
-	550  4300 950  4300
-Wire Wire Line
-	900  4300 900  4350
-Connection ~ 900  4300
+	1250 3900 1150 3900
+Connection ~ 1150 3900
+Wire Wire Line
+	750  4200 950  4200
 Wire Wire Line
 	2400 4000 2400 4050
@@
 Wire Wire Line
 	1750 6050 2350 6050
-Wire Wire Line
-	600  6950 600  7350
-Wire Wire Line
-	1000 7600 850  7600
-Wire Wire Line
-	850  7600 850  7650
-Wire Wire Line
-	850  7650 600  7650
 Wire Wire Line
 	6500 1300 6500 1250
@@
 	7850 2000 7850 2400
 Connection ~ 7850 2000
-Connection ~ -550 4200
 Wire Wire Line
 	7500 1750 7700 1750
@@
 Connection ~ 5300 7100
 Connection ~ 4800 6600
+Wire Wire Line
+	1200 6800 1200 6950
+Wire Wire Line
+	950  7150 950  6800
+Wire Wire Line
+	1150 3700 1150 4000
+Wire Wire Line
+	550  4300 1250 4300
+Wire Wire Line
+	750  4200 750  4000
+Wire Wire Line
+	850  4000 850  4350
+Connection ~ 1150 4000
+Wire Wire Line
+	600  6950 600  7300
 $EndSCHEMATC

Commit message: start routing the PCB
Parts:
- P1: value CONN_02X13 -> BPi
- P15: value CONN_01X02 -> POWER
- P5: value CONN_01X02 -> TERM
Connections:
- net labels added: VCOM
- wire segments 346 -> 347
