File: BPi-CAN/BPi-CAN.sch (KiCad schematic (older format))
At the start: 97 parts, among them J1 RJ45, J2 RJ45, J3 RJ45, J4 RJ45, J5 RJ45, P1 BPi, P10 SPI, P11 SNIFFER, P12 CAN-Bus, P13 USB, P14 CAN-Bus, P15 POWER, P16 CAN, P17 CAN, P18 CAN, P19 TERM, P2 S88, P20 S88 CONN, P21 RS232 Con, P22 S88, P23 CONN_01X08, P24 CONN_01X03, P25 I2C-Bus, P26 CONN_01X02, P27 POWER, P28 POWER, P29 POWER, P3 CONN_02X04, P30 CONN_01X02, P32 CONN_01X06, P33 CONN_01X05, P4 BPi Con, P6 S88, P7 I2C-Bus, P8 RS485, P9 RS232, U12 ISO1050, U13 FT230XS, U2 LM7805, U3 6N137, U4 6N137, U5 6N137, U6 6N137, U7 ADuM1251BR, U8 MAX3072E, U9 MAX3232

Commit message: V2.0 wip
Parts:
- removed C18, C19: 100nF, Resistors_SMD:R_0805_HandSoldering_II, symbol C
- removed D4: LED, LEDs:LED-0805, symbol LED
- removed R11: 220, Resistors_SMD:R_0805_HandSoldering_II, symbol R
- removed R20: 120, Resistors_SMD:R_1206, symbol R
- added C?: 100nF, Resistors_SMD:R_0805_HandSoldering_II, symbol C
- added D1: 1N4148, symbol D_Small
- added P?: CONN_01X03, symbol CONN_01X03
- added R13: 1k, w_pth_resistors:RC03, symbol R
- added R15: 1K5, w_pth_resistors:RC03, symbol R
- added R31, R32: 470, Resistors_SMD:R_0805_HandSoldering_II, symbol R
- added R?: 4k7, Resistors_SMD:R_0805_HandSoldering_II, symbol R
- added R?: 3k3, Resistors_SMD:R_0805_HandSoldering_II, symbol R
- added U1: PIC16F15325-I/P, w_pth_circuits:dil_14-300, symbol PIC16F15325-I/P
- added U11: 6N137, w_pth_circuits:dil_8-300_socket, symbol 6N136-RESCUE-BPi-CAN
- added U?: LM393, symbol LM393
Connections:
- net labels added: A, B, LNET_IN, LNET_OUT, RC2, RS485_DE, RS485_EN, RS485_RX, RS485_TX
- wire segments 450 -> 487
Other:
- note added: "BananaPi Modellbahn Adapter Board\nV2.0"
- note removed: "BananaPi Modellbahn Adapter Board\nV1.5"
- moved on the sheet: C12, C13, C14, C15, C20, C22, C23, C24, C25, C26, C27, C28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

Commit message: add LNET
Parts:
- removed P?: CONN_01X03, symbol CONN_01X03
- removed U?: LM393, symbol LM393
- added C?: 1nF, w_capacitors:cnp_3mm_disc, symbol C
- added C? (x3): 100nF, w_capacitors:cnp_3mm_disc, symbol C
- added C?: 47pF, w_capacitors:cnp_3mm_disc, symbol C
- added D? (x2): LED, LEDs:LED-3MM, symbol LED
- added P19: GROVE, w_conn_jst-ph:s4b-ph-kl, symbol CONN_01X04
- added P?: CONN_01X06, symbol CONN_01X06
- added P?: CONN_01X04, symbol CONN_01X04
- added Q?: BC337, TO-92, symbol BC237
- added R?: 240k, w_pth_resistors:RC03, symbol R
- added R?: 10k, w_pth_resistors:RC03, symbol R
- added R? (x2): 470, w_pth_resistors:RC03, symbol R
- added R?: 1k8, w_pth_resistors:RC03, symbol R
- added R?: 39k, w_pth_resistors:RC03, symbol R
- added R? (x2): 12, w_pth_resistors:RC03, symbol R
- added R?: 150k, w_pth_resistors:RC03, symbol R
- added R?: 47k, w_pth_resistors:RC03, symbol R
- added U? (x2): LM393, symbol LM393
- R?: value 3k3 -> 27k; footprint Resistors_SMD:R_0805_HandSoldering_II -> w_pth_resistors:RC03
Connections:
- wire segments 487 -> 564
Other:
- note added: "S88"
- note added: "ext\nCAN"
- moved on the sheet: C11, C5, C6, C7, C8, C9, C?, D1, J5, P10, P11, P25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

Commit message: wip
Parts:
- added U?: 4504, symbol 4504
Connections:
- net labels added: 8CLK, 8DAT, 8GND, 8LD, 8PWR, 8RST
- wire segments 564 -> 565
Other:
- note removed: "CLOCK"
- note removed: "DATA"
- note removed: "LOAD"
- note removed: "RESET"
- moved on the sheet: C10, C11, C20, C22, C23, C24, C25, C26, C27, C28, C3, C4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

Commit message: add schematic
Connections:
- wire segments 565 -> 474

Commit message: wip
Parts:
- D2, D3, D5, D6, D? (x2): symbol LED -> LED-RESCUE-BPi-CAN
- U?: symbol 4504 -> 4504-RESCUE-BPi-CAN
Connections:
- wire segments 474 -> 571

Commit message: testing
Parts:
- removed P20: S88 CONN, Pin_Headers:Pin_Header_Straight_2x08, symbol CONN_02X08
- P2: footprint w_conn_pt-1,5:pt_1,5-6-3,5-h -> Pin_Headers:Pin_Header_Straight_1x06
Connections:
- net S88_1 is gone; now on net 8PWR: J3.1, J4.1
- net S88_2 is gone; now on net 8CLK: J3.2, J4.2
- net S88_3 is gone; now on net 8CLK: J3.3, J4.3
- net S88_4 is gone; now on net 8CLK: J3.4, J4.4
- net S88_6 is gone; now on net 8CLK: J3.6, J4.6
- net S88_7 is gone; now on net 8CLK: J3.7, J4.7
Changed lines of the file:
@@
 F 0 "P2" H 3875 7550 50  0000 C CNN
 F 1 "S88" V 3900 6825 50  0000 C CNN
-F 2 "w_conn_pt-1,5:pt_1,5-6-3,5-h" H 3875 7200 50  0001 C CNN
+F 2 "Pin_Headers:Pin_Header_Straight_1x06" H 3875 7200 50  0001 C CNN
 F 3 "" H 3875 7200 50  0000 C CNN
 	1    3875 7200
@@
 Entry Wire Line
 	5625 7650 5725 7750
-$Comp
-L CONN_02X08 P20
-U 1 1 568C5586
-P 5125 7300
-F 0 "P20" H 5125 7750 50  0000 C CNN
-F 1 "S88 CONN" V 5125 7300 50  0000 C CNN
-F 2 "Pin_Headers:Pin_Header_Straight_2x08" H 5125 6100 50  0001 C CNN
-F 3 "" H 5125 6100 50  0000 C CNN
-	1    5125 7300
-	-1   0    0    -1
-$EndComp
 Entry Wire Line
 	5625 7450 5725 7550
@@
 Text Label 8175 3325 0    60   ~ 0
 TxD
-NoConn ~ 4875 7350
-NoConn ~ 4875 7650
+NoConn ~ 5050 7350
+NoConn ~ 5050 7650
 $Comp
 L CONN_01X06 P22
@@
 P 2900 3000
 F 0 "U?" H 3050 3150 50  0000 C CNN
-F 1 "LM393" H 3150 2850 50  0000 C CNN
+F 1 "LM393" H 3025 2850 50  0000 C CNN
 F 2 "" H 2900 3000 50  0000 C CNN
 F 3 "" H 2900 3000 50  0000 C CNN
@@
 U 1 1 5A8490D6
 P 2400 3350
-F 0 "C?" H 2525 3425 50  0000 L CNN
-F 1 "100nF" H 2525 3350 50  0000 L CNN
+F 0 "C?" H 2300 3425 50  0000 L CNN
+F 1 "100nF" H 2250 3250 50  0000 L CNN
 F 2 "w_capacitors:cnp_3mm_disc" H 2438 3200 50  0001 C CNN
 F 3 "" H 2400 3350 50  0000 C CNN
@@
 P 3250 3600
 F 0 "U?" H 3400 3750 50  0000 C CNN
-F 1 "LM393" H 3500 3450 50  0000 C CNN
+F 1 "LM393" H 3400 3450 50  0000 C CNN
 F 2 "" H 3250 3600 50  0000 C CNN
 F 3 "" H 3250 3600 50  0000 C CNN
@@
 	4625 6500 4625 6700
 Wire Wire Line
-	5375 6950 5625 6950
-Wire Wire Line
-	5375 7050 5625 7050
-Wire Wire Line
-	5375 7150 5625 7150
-Wire Wire Line
-	5375 7250 5625 7250
-Wire Wire Line
-	5375 7350 5625 7350
-Wire Wire Line
-	5375 7450 5625 7450
-Wire Wire Line
-	5375 7550 5625 7550
-Wire Wire Line
-	5375 7650 5625 7650
-Wire Wire Line
 	4075 6950 4125 6950
 Wire Wire Line
-	4125 6950 4875 6950
-Wire Wire Line
-	4875 7550 4725 7550
-Wire Wire Line
-	4725 7550 4725 7050
-Wire Wire Line
-	4725 7050 4225 7050
+	4125 6950 5625 6950
+Wire Wire Line
+	4900 7050 5625 7050
+Wire Wire Line
+	4950 7150 5625 7150
+Wire Wire Line
+	4075 7250 4425 7250
+Wire Wire Line
+	4425 7250 5625 7250
+Wire Wire Line
+	5050 7350 5625 7350
+Wire Wire Line
+	4850 7450 5625 7450
+Wire Wire Line
+	4750 7550 5625 7550
+Wire Wire Line
+	5050 7650 5625 7650
+Wire Wire Line
+	4750 7550 4750 7050
+Wire Wire Line
+	4750 7050 4225 7050
 Wire Wire Line
 	4225 7050 4075 7050
 Wire Wire Line
-	4875 7450 4775 7450
-Wire Wire Line
-	4775 7450 4775 7150
-Wire Wire Line
-	4775 7150 4325 7150
+	4850 7450 4850 7150
+Wire Wire Line
+	4850 7150 4325 7150
 Wire Wire Line
 	4325 7150 4075 7150
 Wire Wire Line
-	4075 7250 4425 7250
-Wire Wire Line
-	4425 7250 4875 7250
-Wire Wire Line
 	4075 7350 4525 7350
 Wire Wire Line
-	4525 7350 4825 7350
-Wire Wire Line
-	4825 7350 4825 7150
-Wire Wire Line
-	4825 7150 4875 7150
+	4525 7350 4950 7350
+Wire Wire Line
+	4950 7350 4950 7150
 Wire Wire Line
 	4075 7450 4625 7450
@@
 	4625 7450 4625 7500
 Wire Wire Line
-	4625 7100 4825 7100
-Wire Wire Line
-	4825 7100 4825 7050
-Wire Wire Line
-	4825 7050 4875 7050
+	4625 7100 4900 7100
+Wire Wire Line
+	4900 7100 4900 7050
 Wire Wire Line
 	8175 3225 8325 3225
@@
 	2175 3100 2400 3100
 Wire Wire Line
-	2400 3100 2500 3100
-Wire Wire Line
-	2500 3100 2600 3100
-Connection ~ 2500 3100
+	2400 3100 2550 3100
+Wire Wire Line
+	2550 3100 2600 3100
+Connection ~ 2550 3100
 Wire Wire Line
 	1900 975  1900 1375
@@
 Connection ~ 2400 3100
 Wire Wire Line
-	2500 3100 2500 3500
-Wire Wire Line
-	2500 3500 2950 3500
+	2550 3100 2550 3500
+Wire Wire Line
+	2550 3500 2950 3500
 Wire Wire Line
 	2850 3700 2900 3700

Commit message: fix values for S88
Parts:
- R5: value 1k -> 390
- R6: value 390 -> 330
Changed lines of the file:
@@
 P 900 6150
 F 0 "R5" V 800 6150 50  0000 C CNN
-F 1 "1k" V 900 6150 50  0000 C CNN
+F 1 "390" V 900 6150 50  0000 C CNN
 F 2 "w_pth_resistors:RC03" V 830 6150 50  0001 C CNN
 F 3 "" H 900 6150 50  0000 C CNN
@@
 P 1950 5950
 F 0 "R6" V 1850 5950 50  0000 C CNN
-F 1 "390" V 1950 5950 50  0000 C CNN
+F 1 "330" V 1950 5950 50  0000 C CNN
 F 2 "w_pth_resistors:RC03" V 1880 5950 50  0001 C CNN
 F 3 "" H 1950 5950 50  0000 C CNN

Commit message: wip
Parts:
- removed J4: RJ45, w_conn_pc:megb8-8, symbol RJ45
- added C61, C62: 100nF, Capacitors_ThroughHole:C_Disc_D3_P2.5, symbol C
- added CON1: BARREL_JACK, symbol BARREL_JACK
- added P62: TERM, Pin_Headers:Pin_Header_Straight_1x02, symbol CONN_01X02
- added Q61: BC547, TO-92, symbol BC237
- added R61: 4k7, w_pth_resistors:RC03, symbol R
- added R63: 120, Resistors_SMD:R_0805_HandSoldering_II, symbol R
- added U61: LM7805, 78xx:TO-220-78xx, symbol LM7805
- P6: footprint w_conn_pt-1,5:pt_1,5-6-3,5-h -> Pin_Headers:Pin_Header_Straight_1x06
- U1: value PIC16F15325-I/P -> PIC16F15325
- gave numbers to parts that had none: 25
- renumbered P8 to P61, R31 to R61, R32 to R62
Connections:
- net labels added: +12L, RC0, RC1
- wire segments 565 -> 588
- no-connect marks 34 -> 37
Other:
- note added: "CAN\nEXT"
- note added: "S88 EXT"
- note removed: "ext\nCAN"
- moved on the sheet: C11, D5, P2, P21, P22, P25, P61, R12, R61, R62, U62, U8
