File: srse/Domino-CAN/Domino-CAN.kicad_pcb (KiCad board)
At the start: 2 copper layers, 1 part, among them U1 DOMINO_DOMINO

Commit message: Domino-CAN wip
Parts:
- added P1: UART, Pin_Headers:Pin_Header_Straight_1x03, F.Cu at (156.5, 138.8)
- added RF1: 1pin, Connect:1pin, F.Cu at (108.0, 90.0)
- added RF2: 1pin, Connect:1pin, F.Cu at (107.0, 130.0)
- added RF3: 1pin, Connect:1pin, F.Cu at (174.0, 130.0)
- added RF4: 1pin, Connect:1pin, F.Cu at (174.0, 90.0)
- added U2: PIC18F25K80_I/SS, w_smd_dil:soic-28, F.Cu at (118.0, 115.0)
- added U3: FT230XS, w_smd_dil:ssop-16, F.Cu at (123.0, 101.0)
- U1: value DOMINO_DOMINO -> DOMINO_CORE
- moved U1 3.50 mm to (145.0, 105.0)
Connections:
- U1 pad 1: Net-(U1-Pad1) -> GND
- U1 pad 10: Net-(U1-Pad10) -> GND
- U1 pad 2: Net-(U1-Pad2) -> GND
- U1 pad 3: Net-(U1-Pad3) -> GND
- U1 pad 35: Net-(U1-Pad35) -> GND
- U1 pad 45: Net-(U1-Pad45) -> GND
- U1 pad 51: Net-(U1-Pad51) -> GND
- U1 pad 57: Net-(U1-Pad57) -> GND
- U1 pad 58: Net-(U1-Pad58) -> GND
- U1 pad 60: Net-(U1-Pad60) -> GND
Other:
- board outline added: 82 x 72 mm

Commit message: wip
Parts:
- added C1: 47pF, Resistors_SMD:R_0805_HandSoldering_II, F.Cu at (117.0, 90.2)
- added C2: 47pF, Resistors_SMD:R_0805_HandSoldering_II, F.Cu at (115.6, 100.2)
- added C4: 100nF, Resistors_SMD:R_0805_HandSoldering_II, F.Cu at (119.1, 97.4)
- added C5: 100nF, Resistors_SMD:R_0805_HandSoldering_II, F.Cu at (124.5, 89.9)
- added C6: 4.7uF, Resistors_SMD:R_0805_HandSoldering_II, F.Cu at (118.6, 104.8)
- added R1: 27, Resistors_SMD:R_0805_HandSoldering_II, F.Cu at (119.9, 93.9)
- added R2: 27, Resistors_SMD:R_0805_HandSoldering_II, F.Cu at (127.8, 85.9)
- added R3: 220, Resistors_SMD:R_0805_HandSoldering_II, F.Cu at (126.9, 94.4)
- added R4: 220, Resistors_SMD:R_0805_HandSoldering_II, F.Cu at (121.0, 85.3)
- added U4: HR911105A, RJ45ALED_1PRIMARY, F.Cu at (154.2, 150.4)
- added U5: HR911105A, RJ45ALED_1PRIMARY, F.Cu at (137.9, 150.4)
- U2: value PIC18F25K80_I/SS -> PIC18F25K80
- moved P1 31.4 mm to (128.0, 125.6)
- moved U1 11.8 mm to (156.5, 107.7), turned to 270 degrees
- moved U3 1.46 mm to (124.5, 101.1)
Connections:
- net Net-(U3-Pad15) renamed /CBUS0
- net Net-(U3-Pad16) renamed /CBUS3
- net Net-(U3-Pad2) renamed /RTS
- net Net-(U3-Pad6) renamed /CTS
- U1 pad 52: Net-(U1-Pad52) -> /USBDM
- U1 pad 53: Net-(U1-Pad53) -> /USBDP
- U2 pad 19: Net-(U2-Pad19) -> GND
- U2 pad 27: Net-(U2-Pad27) -> /RxD
- U2 pad 28: Net-(U2-Pad28) -> /TxD
- U2 pad 8: Net-(U2-Pad8) -> GND
- U3 pad 1: Net-(U3-Pad1) -> /TxD
- U3 pad 10: Net-(U3-Pad10) -> Net-(C3-Pad1)
- U3 pad 11: Net-(U3-Pad11) -> Net-(C3-Pad1)
- U3 pad 12: Net-(U3-Pad12) -> VCC
- U3 pad 13: Net-(U3-Pad13) -> GND
- U3 pad 3: Net-(U3-Pad3) -> Net-(C3-Pad1)
- U3 pad 4: Net-(U3-Pad4) -> /RxD
- U3 pad 5: Net-(U3-Pad5) -> GND

Commit message: working on LAN/WAN
Parts:
- moved P1 51.3 mm to (179.1, 130.6), turned to 180 degrees
- moved U3 15.4 mm to (109.1, 100.2)
- moved C2 6.54 mm to (112.0, 105.7), turned to 180 degrees
- moved U1 0.98 mm to (155.5, 108.1)
