File: BPI-AddOn/BPI-AddOn.sch (KiCad schematic (older format))
At the start: 14 parts, among them J1 RJ45, J2 RJ45, P1 CONN_01X13, P10 CONN_01X03, P11 CONN_01X05, P12 CONN_01X05, P2 CONN_01X13, P3 CONN_01X13, P4 CONN_01X13, P5 CONN_01X13, P6 CONN_01X13, P7 CONN_01X10, P8 CONN_01X10, P9 CONN_01X03

Commit message: wip
Parts:
- added J3: RJ45, w_conn_pc:megb8-8, symbol RJ45
- added P13: CONN_01X08, Pin_Headers:Pin_Header_Straight_1x08, symbol CONN_01X08
- added P?: CONN_02X11, symbol CONN_02X11
- added U?: MC34063, w_smd_dil:so-8, symbol MC34063
- P1, P2, P3, P4, P5, P6: value CONN_01X13 -> DIN10
- P7, P8: value CONN_01X10 -> DIN7
Connections:
- wire segments 140 -> 148
- no-connect marks 2 -> 3
Changed lines of the file:
@@
 P 1250 3100
 F 0 "P2" H 1250 3800 50  0000 C CNN
-F 1 "CONN_01X13" V 1350 3100 50  0000 C CNN
+F 1 "DIN10" V 1350 3100 50  0000 C CNN
 F 2 "maerklin:minidin-10" H 1250 3100 50  0001 C CNN
 F 3 "" H 1250 3100 50  0000 C CNN
@@
 P 1250 1400
 F 0 "P1" H 1250 2100 50  0000 C CNN
-F 1 "CONN_01X13" V 1350 1400 50  0000 C CNN
+F 1 "DIN10" V 1350 1400 50  0000 C CNN
 F 2 "maerklin:minidin-10" H 1250 1400 50  0001 C CNN
 F 3 "" H 1250 1400 50  0000 C CNN
@@
 P 2200 1400
 F 0 "P4" H 2200 2100 50  0000 C CNN
-F 1 "CONN_01X13" V 2300 1400 50  0000 C CNN
+F 1 "DIN10" V 2300 1400 50  0000 C CNN
 F 2 "maerklin:minidin-10" H 2200 1400 50  0001 C CNN
 F 3 "" H 2200 1400 50  0000 C CNN
@@
 P 2200 3100
 F 0 "P5" H 2200 3800 50  0000 C CNN
-F 1 "CONN_01X13" V 2300 3100 50  0000 C CNN
+F 1 "DIN10" V 2300 3100 50  0000 C CNN
 F 2 "maerklin:minidin-10" H 2200 3100 50  0001 C CNN
 F 3 "" H 2200 3100 50  0000 C CNN
@@
 P 2200 4750
 F 0 "P6" H 2200 5450 50  0000 C CNN
-F 1 "CONN_01X13" V 2300 4750 50  0000 C CNN
+F 1 "DIN10" V 2300 4750 50  0000 C CNN
 F 2 "maerklin:minidin-10" H 2200 4750 50  0001 C CNN
 F 3 "" H 2200 4750 50  0000 C CNN
@@
 P 1250 4750
 F 0 "P3" H 1250 5450 50  0000 C CNN
-F 1 "CONN_01X13" V 1350 4750 50  0000 C CNN
+F 1 "DIN10" V 1350 4750 50  0000 C CNN
 F 2 "maerklin:minidin-10" H 1250 4750 50  0001 C CNN
 F 3 "" H 1250 4750 50  0000 C CNN
@@
 P 3150 1250
 F 0 "P7" H 3150 1800 50  0000 C CNN
-F 1 "CONN_01X10" V 3250 1250 50  0000 C CNN
+F 1 "DIN7" V 3250 1250 50  0000 C CNN
 F 2 "maerklin:minidin-7" H 3150 1250 50  0001 C CNN
 F 3 "" H 3150 1250 50  0000 C CNN
@@
 P 3150 2950
 F 0 "P8" H 3150 3500 50  0000 C CNN
-F 1 "CONN_01X10" V 3250 2950 50  0000 C CNN
+F 1 "DIN7" V 3250 2950 50  0000 C CNN
 F 2 "maerklin:minidin-7" H 3150 2950 50  0001 C CNN
 F 3 "" H 3150 2950 50  0000 C CNN
@@
 Wire Wire Line
 	3800 3350 4050 3350
-Text Label 3850 2150 0    60   ~ 0
+Text Label 3850 2350 0    60   ~ 0
 5V
 Text Label 3850 2250 0    60   ~ 0
@@
 	1    0    0    -1
 $EndComp
-Text Label 3850 2950 0    60   ~ 0
+Text Label 3850 3150 0    60   ~ 0
 5V
 Text Label 3850 3050 0    60   ~ 0
 GND
-Text Label 3850 3150 0    60   ~ 0
-Vcc
-Text Label 3850 2350 0    60   ~ 0
+Text Label 3850 2950 0    60   ~ 0
+Vcc
+Text Label 3850 2150 0    60   ~ 0
 Vcc
 Text Label 3850 2450 0    60   ~ 0
@@
 Text Label 3850 3350 0    60   ~ 0
 CANH
+$Comp
+L RJ45 J3
+U 1 1 5759CFBF
+P 1600 6650
+F 0 "J3" H 1800 7150 50  0000 C CNN
+F 1 "RJ45" H 1450 7150 50  0000 C CNN
+F 2 "w_conn_pc:megb8-8" H 1600 6650 50  0001 C CNN
+F 3 "" H 1600 6650 50  0000 C CNN
+	1    1600 6650
+	1    0    0    -1
+$EndComp
+$Comp
+L CONN_01X08 P13
+U 1 1 5759D031
+P 1600 7600
+F 0 "P13" H 1600 8050 50  0000 C CNN
+F 1 "CONN_01X08" V 1700 7600 50  0001 C CNN
+F 2 "Pin_Headers:Pin_Header_Straight_1x08" V 1600 7600 50  0001 C CNN
+F 3 "" H 1600 7600 50  0000 C CNN
+	1    1600 7600
+	0    -1   1    0
+$EndComp
+Wire Wire Line
+	1250 7100 1250 7400
+Wire Wire Line
+	1350 7400 1350 7100
+Wire Wire Line
+	1450 7100 1450 7400
+Wire Wire Line
+	1550 7400 1550 7100
+Wire Wire Line
+	1650 7100 1650 7400
+Wire Wire Line
+	1750 7100 1750 7400
+Wire Wire Line
+	1850 7100 1850 7400
+Wire Wire Line
+	1950 7100 1950 7400
+NoConn ~ 2150 6300
+Wire Notes Line
+	2600 7650 2600 5950
+Wire Notes Line
+	2600 5950 600  5950
+Wire Notes Line
+	600  5950 600  6000
+$Comp
+L MC34063 U?
+U 1 1 5759E1D1
+P 7900 2350
+F 0 "U?" H 8050 2700 50  0000 L CNN
+F 1 "MC34063" H 8000 2000 50  0000 L CNN
+F 2 "w_smd_dil:so-8" H 7900 2350 50  0000 C CNN
+F 3 "" H 7900 2350 50  0000 C CNN
+	1    7900 2350
+	1    0    0    -1
+$EndComp
+$Comp
+L CONN_02X11 P?
+U 1 1 5759E2E8
+P 9550 3850
+F 0 "P?" H 9550 4450 50  0000 C CNN
+F 1 "CONN_02X11" V 9550 3850 50  0000 C CNN
+F 2 "" H 9550 2650 50  0000 C CNN
+F 3 "" H 9550 2650 50  0000 C CNN
+	1    9550 3850
+	-1   0    0    1
+$EndComp
 $EndSCHEMATC

Commit message: wip
Parts:
- added C1: 680pF, w_capacitors:cnp_3mm_disc, symbol C
- added CON1: BARREL_JACK, w_conn_misc:dc_socket, symbol BARREL_JACK
- added F1, F2: FUSE, Fuse_Holders_and_Fuses:BladeFuse-Mini, symbol FUSE
- added P14: DCDC-Conevrter, 78xx:DCDC, symbol CONN_01X08
- added P16: USB_B, w_conn_pc:conn_usb_B, symbol USB_B
- added P17, P18: CONN_01X05, Pin_Headers:Pin_Header_Straight_1x05, symbol CONN_01X05
- added P19: V, Pin_Headers:Pin_Header_Straight_1x03, symbol CONN_01X03
- added P20: - +, w_conn_pt-1,5:pt_1,5-2-3,5-h, symbol CONN_01X02
- added R1: 0, Resistors_SMD:R_0805_HandSoldering, symbol R
- P15: renamed from P?; footprint (none) -> w_conn_ftsh:ftsh-2211-01-l-dv
- gave numbers to parts that had none: 1
Connections:
- net labels added: GNDD, VCC, Vdd
- wire segments 148 -> 195
- no-connect marks 3 -> 32
Other:
- moved on the sheet: J3, P10, P11, P12, P13, P9

Commit message: working on stepup
Parts:
- added C2, C3: 100uF, w_capacitors:CP_5x11mm, symbol CP
- added D1: D_Schottky, Diodes_ThroughHole:Diode_DO-35_SOD27_Horizontal_RM10, symbol D_Schottky
- added L1: 68uH, Choke_Radial_ThroughHole:Choke_Radial_27mm_2,8mm-Drills_CD_Bobin_Type_No1410311, symbol INDUCTOR
- added R2, R3: R, w_pth_resistors:RC03, symbol R
- added R4: 1k, w_pth_resistors:RC03, symbol R
- added R5: 11k, w_pth_resistors:RC03, symbol R
Connections:
- net labels added: Vin, Vout
- wire segments 195 -> 221
- no-connect marks 32 -> 27
Other:
- moved on the sheet: P15

Commit message: BPi AddOn wip
Parts:
- removed P6: DIN10, maerklin:minidin-10, symbol CONN_01X13
- added P8: DIN7, maerklin:minidin-7, symbol CONN_01X10
- L1: footprint Choke_Radial_ThroughHole:Choke_Radial_27mm_2,8mm-Drills_CD_Bobin_Type_No1410311 -> Choke_Toroid_ThroughHole:Choke_Toroid_8x16mm_Vertical
- renumbered P7 to P6, P8 to P7
Connections:
- wire segments 221 -> 218
Other:
- moved on the sheet: CON1, F1, F2, J1, J2, P10, P16, P19, P20, P9, R1

Commit message: wip
Parts:
- added C4, C5, C8: 10nF, Resistors_SMD:R_0805_HandSoldering, symbol C
- added C6, C7: 47pF, Resistors_SMD:R_0805_HandSoldering, symbol C
- added C9: 100nF, Resistors_SMD:R_0805_HandSoldering, symbol C
- added D2: TxD, LEDs:LED_0805, symbol LED
- added D3: RxD, LEDs:LED_0805, symbol LED
- added F3: Ferrit, Resistors_SMD:R_0805_HandSoldering, symbol R
- added P21: USB_OTG, w_conn_pc:conn_usb_B_mini_smd, symbol USB_OTG
- added P22: CONN_01X06, Pin_Headers:Pin_Header_Straight_1x06, symbol CONN_01X06
- added P23: CONN_01X06, w_conn_pt-1,5:pt_1,5-6-3,5-h, symbol CONN_01X06
- added P24: CONN_02X02, Pin_Headers:Pin_Header_Straight_2x02, symbol CONN_02X02
- added R10, R8: 220, Resistors_SMD:R_0805_HandSoldering, symbol R
- added R6, R7: 27, Resistors_SMD:R_0805_HandSoldering, symbol R
- added R9: 0, Resistors_SMD:R_0805_HandSoldering, symbol R
- added U2: FT230XS, w_smd_dil:ssop-16, symbol FT230XS
- L1: footprint Choke_Toroid_ThroughHole:Choke_Toroid_8x16mm_Vertical -> Inductors_NEOSID:Neosid_Inductor_Sd14
Connections:
- net labels added: CTS, RTS, RxD, TxD
- wire segments 218 -> 297
- no-connect marks 27 -> 23
Other:
- moved on the sheet: P15

Commit message: wip
Parts:
- added D4: LED, LEDs:LED-5MM, symbol LED
- added P25: CONN_01X02, Pin_Headers:Pin_Header_Straight_1x02, symbol CONN_01X02
- added R13, R3: 120, w_pth_resistors:RC03, symbol R
- added R2: 120, Resistors_SMD:R_1206_HandSoldering, symbol R
- P1: value DIN10 -> DIN10-1
- P2: value DIN10 -> DIN10-2
- P3: value DIN10 -> DIN10-3
- P4: value DIN10 -> DIN10-4
- P5: value DIN10 -> DIN10-5
- P6: value DIN7 -> DIN7-1
- P7: value DIN7 -> DIN7-2
- P8: value DIN7 -> DIN7-3
- renumbered P14 to DCDC1, R8 to R10, R10 to R11, R9 to R12, R2 to R4, R3 to R5, R4 to R6, R5 to R7, R6 to R8, R7 to R9
Connections:
- wire segments 297 -> 308

Commit message: wip
Parts:
- F1, F2: footprint Fuse_Holders_and_Fuses:BladeFuse-Mini -> w_capacitors:cnp_6mm_disc
Changed lines of the file:
@@
 F 0 "F1" H 1250 7500 50  0000 C CNN
 F 1 "FUSE" H 1050 7400 50  0000 C CNN
-F 2 "Fuse_Holders_and_Fuses:BladeFuse-Mini" H 1150 7450 50  0001 C CNN
+F 2 "w_capacitors:cnp_6mm_disc" H 1150 7450 50  0001 C CNN
 F 3 "" H 1150 7450 50  0000 C CNN
 	1    1150 7450
@@
 F 0 "F2" H 2650 6200 50  0000 C CNN
 F 1 "FUSE" H 2450 6100 50  0000 C CNN
-F 2 "Fuse_Holders_and_Fuses:BladeFuse-Mini" H 2550 6150 50  0001 C CNN
+F 2 "w_capacitors:cnp_6mm_disc" H 2550 6150 50  0001 C CNN
 F 3 "" H 2550 6150 50  0000 C CNN
 	1    2550 6150

Commit message: routing ...
Connections:
- net labels added: GNDB
Changed lines of the file:
@@
 Wire Wire Line
 	3500 3950 3500 4050
+Text Label 4900 7350 1    60   ~ 0
+GNDB
 $EndSCHEMATC
