File: BPI-AddOn/BPI-AddOn.sch (KiCad schematic (older format))
At the start: 79 parts, among them CON1 BARREL_JACK, J1 RJ45, J2 RJ45, J3 RJ45, P1 DIN10-1, P10 CONN_01X03, P11 CONN_01X05, P12 CONN_01X05, P13 CONN_01X08, P14 CONN_02X11, P15 CONN_02X11, P16 USB_B, P17 CONN_01X05, P18 CONN_01X05, P19 V, P2 DIN10-2, P20 - +, P21 USB_OTG, P22 CONN_01X06, P23 CONN_01X06, P24 CONN_02X02, P25 CONN_01X02, P26 CONN_01X03, P27 CONN_01X04, P28 CONN_01X03, P3 DIN10-3, P4 DIN10-4, P5 DIN10-5, P6 DIN7-1, P7 DIN7-2, P8 DIN7-3, P9 CONN_01X03, Q1 BS170, Q2 BS170, Q3 BS170, Q4 BS170, U1 MC34063, U2 FT230XS

Commit message: wip
Parts:
- added P29: CONN_01X01, Pin_Headers:Pin_Header_Straight_1x01, symbol CONN_01X01
- added R23, R24, R25: R, w_pth_resistors:RC03, symbol R
- R15, R16, R17, R18, R19, R20, R21, R22: footprint w_pth_resistors:RC03 -> Resistors_SMD:R_0805_HandSoldering
Connections:
- wire segments 401 -> 404
Changed lines of the file:
@@
 	0    1    1    0
 $EndComp
-Text Label 10750 4700 1    60   ~ 0
-_TxD
-Text Label 10850 5450 1    60   ~ 0
-_RxD
+Text Label 10850 5950 1    60   ~ 0
+TxD
+Text Label 10750 4350 1    60   ~ 0
+RxD
 $Comp
 L GNDD #PWR029
@@
 F 0 "R15" V 5580 900 50  0000 C CNN
 F 1 "4k7" V 5500 900 50  0000 C CNN
-F 2 "w_pth_resistors:RC03" V 5430 900 50  0001 C CNN
+F 2 "Resistors_SMD:R_0805_HandSoldering" V 5430 900 50  0001 C CNN
 F 3 "" H 5500 900 50  0000 C CNN
 	1    5500 900
@@
 F 0 "R17" V 6180 900 50  0000 C CNN
 F 1 "4k7" V 6100 900 50  0000 C CNN
-F 2 "w_pth_resistors:RC03" V 6030 900 50  0001 C CNN
+F 2 "Resistors_SMD:R_0805_HandSoldering" V 6030 900 50  0001 C CNN
 F 3 "" H 6100 900 50  0000 C CNN
 	1    6100 900
@@
 F 0 "R16" V 5580 1750 50  0000 C CNN
 F 1 "4k7" V 5500 1750 50  0000 C CNN
-F 2 "w_pth_resistors:RC03" V 5430 1750 50  0001 C CNN
+F 2 "Resistors_SMD:R_0805_HandSoldering" V 5430 1750 50  0001 C CNN
 F 3 "" H 5500 1750 50  0000 C CNN
 	1    5500 1750
@@
 F 0 "R18" V 6180 1750 50  0000 C CNN
 F 1 "4k7" V 6100 1750 50  0000 C CNN
-F 2 "w_pth_resistors:RC03" V 6030 1750 50  0001 C CNN
+F 2 "Resistors_SMD:R_0805_HandSoldering" V 6030 1750 50  0001 C CNN
 F 3 "" H 6100 1750 50  0000 C CNN
 	1    6100 1750
@@
 F 0 "R19" V 5580 2600 50  0000 C CNN
 F 1 "4k7" V 5500 2600 50  0000 C CNN
-F 2 "w_pth_resistors:RC03" V 5430 2600 50  0001 C CNN
+F 2 "Resistors_SMD:R_0805_HandSoldering" V 5430 2600 50  0001 C CNN
 F 3 "" H 5500 2600 50  0000 C CNN
 	1    5500 2600
@@
 F 0 "R21" V 6180 2600 50  0000 C CNN
 F 1 "4k7" V 6100 2600 50  0000 C CNN
-F 2 "w_pth_resistors:RC03" V 6030 2600 50  0001 C CNN
+F 2 "Resistors_SMD:R_0805_HandSoldering" V 6030 2600 50  0001 C CNN
 F 3 "" H 6100 2600 50  0000 C CNN
 	1    6100 2600
@@
 F 0 "R20" V 5580 3450 50  0000 C CNN
 F 1 "4k7" V 5500 3450 50  0000 C CNN
-F 2 "w_pth_resistors:RC03" V 5430 3450 50  0001 C CNN
+F 2 "Resistors_SMD:R_0805_HandSoldering" V 5430 3450 50  0001 C CNN
 F 3 "" H 5500 3450 50  0000 C CNN
 	1    5500 3450
@@
 F 0 "R22" V 6180 3450 50  0000 C CNN
 F 1 "4k7" V 6100 3450 50  0000 C CNN
-F 2 "w_pth_resistors:RC03" V 6030 3450 50  0001 C CNN
+F 2 "Resistors_SMD:R_0805_HandSoldering" V 6030 3450 50  0001 C CNN
 F 3 "" H 6100 3450 50  0000 C CNN
 	1    6100 3450
@@
 	11050 3950 10700 3950
 Wire Wire Line
-	10850 5250 10850 5550
-Wire Wire Line
-	10750 4750 10750 4500
-Wire Wire Line
 	10200 3450 9700 3450
 Wire Wire Line
@@
 Wire Wire Line
 	4600 1200 4600 1300
+$Comp
+L R R25
+U 1 1 576AF154
+P 10850 5400
+F 0 "R25" V 10930 5400 50  0000 C CNN
+F 1 "R" V 10850 5400 50  0000 C CNN
+F 2 "w_pth_resistors:RC03" V 10780 5400 50  0001 C CNN
+F 3 "" H 10850 5400 50  0000 C CNN
+	1    10850 5400
+	-1   0    0    1
+$EndComp
+$Comp
+L R R24
+U 1 1 576B0FAC
+P 10750 4500
+F 0 "R24" V 10830 4500 50  0000 C CNN
+F 1 "R" V 10750 4500 50  0000 C CNN
+F 2 "w_pth_resistors:RC03" V 10680 4500 50  0001 C CNN
+F 3 "" H 10750 4500 50  0000 C CNN
+	1    10750 4500
+	-1   0    0    1
+$EndComp
+$Comp
+L R R23
+U 1 1 576B139B
+P 10450 4350
+F 0 "R23" V 10530 4350 50  0000 C CNN
+F 1 "R" V 10450 4350 50  0000 C CNN
+F 2 "w_pth_resistors:RC03" V 10380 4350 50  0001 C CNN
+F 3 "" H 10450 4350 50  0000 C CNN
+	1    10450 4350
+	0    -1   -1   0
+$EndComp
+Wire Wire Line
+	10600 4350 10750 4350
+Wire Wire Line
+	10750 4650 10750 4750
+Wire Wire Line
+	10750 4350 10750 4200
+Connection ~ 10750 4350
+Wire Wire Line
+	10850 5550 10850 6100
+$Comp
+L CONN_01X01 P29
+U 1 1 576B2E5C
+P 10300 4650
+F 0 "P29" H 10300 4750 50  0000 C CNN
+F 1 "CONN_01X01" V 10400 4650 50  0001 C CNN
+F 2 "Pin_Headers:Pin_Header_Straight_1x01" H 10300 4650 50  0001 C CNN
+F 3 "" H 10300 4650 50  0000 C CNN
+	1    10300 4650
+	0    1    1    0
+$EndComp
+Wire Wire Line
+	10300 4350 10300 4450
 $EndSCHEMATC

Commit message: wip
Parts:
- added P30, P31: CONN_01X04, Pin_Headers:Pin_Header_Straight_1x04, symbol CONN_01X04
Connections:
- net labels added: hCTS, hRTS, hRxD, hTxD, lCTS, lRTS, lRxD, lTxD
- net labels removed: _CTS, _RTS, _RxD, _TxD
- wire segments 404 -> 412
Other:
- moved on the sheet: P29, R23
