File: BPI-AddOn/BPI-AddOn.kicad_pcb (KiCad board)
At the start: 2 copper layers, 100 x 100 mm, 81 parts, among them CON1 BARREL_JACK, J1 RJ45, J2 RJ45, J3 RJ45, P1 DIN10-1, P10 CONN_01X03, P11 CONN_01X05, P12 CONN_01X05, P13 CONN_01X08, P15 CONN_02X11, P16 USB_B, P17 CONN_01X05, P18 CONN_01X05, P19 V, P2 DIN10-2, P20 - +, P21 USB_OTG, P22 CONN_01X06, P23 CONN_01X06, P24 CONN_02X02, P25 CONN_01X02, P3 DIN10-3, P4 DIN10-4, P5 DIN10-5, P6 DIN7-1, P7 DIN7-2, P8 DIN7-3, P9 CONN_01X03, U1 MC34063, U2 FT230XS

Commit message: routing ...
Parts:
- removed F: Ferrit, Resistors_SMD:R_0805_HandSoldering
- added Fe1: Ferrit, Resistors_SMD:R_0805_HandSoldering, F.Cu at (140.8, 105.8)
- R3: footprint w_pth_resistors:RC03 -> w_pth_resistors:RC05
- moved R2 9.54 mm to (84.6, 130.7)
- moved R3 6.29 mm to (84.6, 130.5)
- moved P25 5.48 mm to (84.5, 122.2), turned to 180 degrees
Changed lines of the file:
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@@
-(kicad_pcb (version 4) (host pcbnew 4.0.2-stable)
+(kicad_pcb (version 4) (host pcbnew 4.0.2+e4-6225~38~ubuntu14.04.1-stable)
   (general
     (links 234)
-    (no_connects 215)
+    (no_connects 202)
     (area 66.924999 48.924999 167.075001 149.075001)
     (thickness 1.6)
@@
     )
   )
-  (module Resistors_SMD:R_0805_HandSoldering (layer F.Cu)
-    (at 141.34 105.77 270)
-    (descr "Resistor SMD 0805, hand soldering")
-    (tags "resistor 0805")
-    (attr smd)
-    (fp_text reference F (at -3.28 -0.08 270) (layer F.SilkS)
-      (effects (font (size 1 1) (thickness 0.15)))
-    )
-    (fp_text value Ferrit (at 0 2.1 270) (layer F.Fab)
-      (effects (font (size 1 1) (thickness 0.15)))
-    )
-    (fp_line (start -2.4 -1) (end 2.4 -1) (layer F.CrtYd) (width 0.05))
-    (fp_line (start -2.4 1) (end 2.4 1) (layer F.CrtYd) (width 0.05))
-    (fp_line (start -2.4 -1) (end -2.4 1) (layer F.CrtYd) (width 0.05))
-    (fp_line (start 2.4 -1) (end 2.4 1) (layer F.CrtYd) (width 0.05))
-    (fp_line (start 0.6 0.875) (end -0.6 0.875) (layer F.SilkS) (width 0.15))
-    (fp_line (start -0.6 -0.875) (end 0.6 -0.875) (layer F.SilkS) (width 0.15))
-    (pad 1 smd rect (at -1.35 0 270) (size 1.5 1.3) (layers F.Cu F.Paste F.Mask)
-      (net 53 "Net-(C5-Pad1)"))
-    (pad 2 smd rect (at 1.35 0 270) (size 1.5 1.3) (layers F.Cu F.Paste F.Mask)
-      (net 52 "Net-(C4-Pad1)"))
-    (model Resistors_SMD.3dshapes/R_0805_HandSoldering.wrl
-      (at (xyz 0 0 0))
-      (scale (xyz 1 1 1))
-      (rotate (xyz 0 0 0))
-    )
-  )
   (module w_conn_pc:conn_usb_B_mini_smd (layer F.Cu)
     (at 144 118)
@@
   )
   (module Pin_Headers:Pin_Header_Straight_1x02 (layer F.Cu)
-    (at 81.99 127.1)
+    (at 84.5185 122.2375 180)
     (descr "Through hole pin header")
     (tags "pin header")
-    (fp_text reference P25 (at 3.25 1.5) (layer F.SilkS)
-      (effects (font (size 1 1) (thickness 0.15)))
-    )
-    (fp_text value CONN_01X02 (at 0 -3.1) (layer F.Fab) hide
+    (fp_text reference P25 (at 3.25 1.5 180) (layer F.SilkS)
+      (effects (font (size 1 1) (thickness 0.15)))
+    )
+    (fp_text value CONN_01X02 (at 0 -3.1 180) (layer F.Fab) hide
       (effects (font (size 1 1) (thickness 0.15)))
     )
@@
     (fp_line (start -1.27 1.27) (end -1.27 3.81) (layer F.SilkS) (width 0.15))
     (fp_line (start -1.27 3.81) (end 1.27 3.81) (layer F.SilkS) (width 0.15))
-    (pad 1 thru_hole rect (at 0 0) (size 2.032 2.032) (drill 1.016) (layers *.Cu *.Mask F.SilkS)
+    (pad 1 thru_hole rect (at 0 0 180) (size 2.032 2.032) (drill 1.016) (layers *.Cu *.Mask F.SilkS)
       (net 68 "Net-(P25-Pad1)"))
-    (pad 2 thru_hole oval (at 0 2.54) (size 2.032 2.032) (drill 1.016) (layers *.Cu *.Mask F.SilkS)
+    (pad 2 thru_hole oval (at 0 2.54 180) (size 2.032 2.032) (drill 1.016) (layers *.Cu *.Mask F.SilkS)
       (net 3 /CANL))
     (model Pin_Headers.3dshapes/Pin_Header_Straight_1x02.wrl
@@
   )
   (module Resistors_SMD:R_1206_HandSoldering (layer F.Cu)
-    (at 81.95 121.58 90)
+    (at 84.582 130.7465 90)
     (descr "Resistor SMD 1206, hand soldering")
     (tags "resistor 1206")
@@
       (effects (font (size 1 1) (thickness 0.15)))
     )
-    (fp_text value 120 (at 0 2.3 90) (layer F.Fab) hide
+    (fp_text value 120 (at 4.191 2.159 90) (layer F.Fab) hide
       (effects (font (size 1 1) (thickness 0.15)))
     )
@@
   )
   (module w_pth_resistors:RC03 (layer F.Cu)
-    (at 84.77 124.21 90)
-    (descr "Resistor, RC03")
-    (tags R)
-    (autoplace_cost180 10)
-    (fp_text reference R3 (at 6.35 -0.05 90) (layer F.SilkS)
-      (effects (font (size 1.397 1.27) (thickness 0.2032)))
-    )
-    (fp_text value 120 (at 0 2.032 90) (layer F.SilkS) hide
-      (effects (font (size 1.397 1.27) (thickness 0.2032)))
-    )
-    (fp_line (start 2.159 0) (end 3.81 0) (layer F.SilkS) (width 0.254))
-    (fp_line (start -2.159 0) (end -3.81 0) (layer F.SilkS) (width 0.254))
-    (fp_line (start -2.159 -0.889) (end -2.159 0.889) (layer F.SilkS) (width 0.254))
-    (fp_line (start -2.159 0.889) (end 2.159 0.889) (layer F.SilkS) (width 0.254))
-    (fp_line (start 2.159 0.889) (end 2.159 -0.889) (layer F.SilkS) (width 0.254))
-    (fp_line (start 2.159 -0.889) (end -2.159 -0.889) (layer F.SilkS) (width 0.254))
-    (pad 1 thru_hole circle (at -3.81 0 90) (size 1.99898 1.99898) (drill 0.8001) (layers *.Cu *.Mask F.SilkS)
-      (net 2 /CANH))
-    (pad 2 thru_hole circle (at 3.81 0 90) (size 1.99898 1.99898) (drill 0.8001) (layers *.Cu *.Mask F.SilkS)
-      (net 68 "Net-(P25-Pad1)"))
-    (model walter/pth_resistors/rc03.wrl
-      (at (xyz 0 0 0))
-      (scale (xyz 1 1 1))
-      (rotate (xyz 0 0 0))
-    )
-  )
-  (module w_pth_resistors:RC03 (layer F.Cu)
     (at 135.75 71.75 180)
     (descr "Resistor, RC03")
@@
     (pad "" np_thru_hole circle (at -1.5 1.25 90) (size 0.5 0.5) (drill 0.5) (layers *.Cu *.Mask F.SilkS))
   )
+  (module w_pth_resistors:RC05 (layer F.Cu)
+    (at 84.582 130.4925 90)
+    (descr "Resistor, RC05")
+    (tags R)
+    (autoplace_cost180 10)
+    (fp_text reference R3 (at 0 0 90) (layer F.SilkS)
+      (effects (font (size 1.397 1.27) (thickness 0.2032)))
+    )
+    (fp_text value 120 (at 0 2.032 90) (layer F.SilkS) hide
+      (effects (font (size 1.397 1.27) (thickness 0.2032)))
+    )
+    (fp_line (start 4.572 1.27) (end -4.572 1.27) (layer F.SilkS) (width 0.254))
+    (fp_line (start -4.572 1.27) (end -4.572 -1.27) (layer F.SilkS) (width 0.254))
+    (fp_line (start -4.572 -1.27) (end 4.572 -1.27) (layer F.SilkS) (width 0.254))
+    (fp_line (start 4.572 -1.27) (end 4.572 1.27) (layer F.SilkS) (width 0.254))
+    (fp_line (start -5.08 0) (end -4.572 0) (layer F.SilkS) (width 0.3048))
+    (fp_line (start 5.08 0) (end 4.572 0) (layer F.SilkS) (width 0.3048))
+    (pad 1 thru_hole circle (at -5.08 0 90) (size 1.99898 1.99898) (drill 0.8001) (layers *.Cu *.Mask F.SilkS)
+      (net 2 /CANH))
+    (pad 2 thru_hole circle (at 5.08 0 90) (size 1.99898 1.99898) (drill 0.8001) (layers *.Cu *.Mask F.SilkS)
+      (net 68 "Net-(P25-Pad1)"))
+    (model walter/pth_resistors/rc05.wrl
+      (at (xyz 0 0 0))
+      (scale (xyz 1 1 1))
+      (rotate (xyz 0 0 0))
+    )
+  )
+  (module Resistors_SMD:R_0805_HandSoldering (layer F.Cu)
+    (at 140.843 105.791 270)
+    (descr "Resistor SMD 0805, hand soldering")
+    (tags "resistor 0805")
+    (attr smd)
+    (fp_text reference Fe1 (at 0 -2.1 270) (layer F.SilkS)
+      (effects (font (size 1 1) (thickness 0.15)))
+    )
+    (fp_text value Ferrit (at 0 2.1 270) (layer F.Fab)
+      (effects (font (size 1 1) (thickness 0.15)))
+    )
+    (fp_line (start -2.4 -1) (end 2.4 -1) (layer F.CrtYd) (width 0.05))
+    (fp_line (start -2.4 1) (end 2.4 1) (layer F.CrtYd) (width 0.05))
+    (fp_line (start -2.4 -1) (end -2.4 1) (layer F.CrtYd) (width 0.05))
+    (fp_line (start 2.4 -1) (end 2.4 1) (layer F.CrtYd) (width 0.05))
+    (fp_line (start 0.6 0.875) (end -0.6 0.875) (layer F.SilkS) (width 0.15))
+    (fp_line (start -0.6 -0.875) (end 0.6 -0.875) (layer F.SilkS) (width 0.15))
+    (pad 1 smd rect (at -1.35 0 270) (size 1.5 1.3) (layers F.Cu F.Paste F.Mask)
+      (net 53 "Net-(C5-Pad1)"))
+    (pad 2 smd rect (at 1.35 0 270) (size 1.5 1.3) (layers F.Cu F.Paste F.Mask)
+      (net 52 "Net-(C4-Pad1)"))
+    (model Resistors_SMD.3dshapes/R_0805_HandSoldering.wrl
+      (at (xyz 0 0 0))
+      (scale (xyz 1 1 1))
+      (rotate (xyz 0 0 0))
+    )
+  )
   (gr_line (start 117 69.8) (end 117 102.5) (angle 90) (layer Edge.Cuts) (width 0.15))

Commit message: wip
Parts:
- C5: value 10nF -> 100nF
- C8: value 10nF -> 4.7uF
- moved C5 13.1 mm to (139.5, 102.0), turned to 180 degrees
- moved R1 12.0 mm to (94.7, 56.1), turned to 270 degrees
- moved C9 11.8 mm to (130.2, 106.0), turned to 270 degrees
- moved C8 8.46 mm to (127.9, 106.1), turned to 270 degrees
- moved U2 0.65 mm to (135.2, 105.9), turned to 90 degrees
- moved P16 0.55 mm to (101.9, 49.1)
Connections:
- C8 pad 1: Net-(C5-Pad1) -> Net-(C8-Pad1)
- C9 pad 1: Net-(C9-Pad1) -> Net-(C8-Pad1)
- CON1 pad 2: Net-(CON1-Pad2) -> GNDA
- CON1 pad 3: GNDA -> Net-(CON1-Pad3)
- D2 pad 2: Net-(C9-Pad1) -> Net-(C5-Pad1)
- D3 pad 2: Net-(C9-Pad1) -> Net-(C5-Pad1)
- Fe1 pad 1: Net-(C5-Pad1) -> Net-(C8-Pad1)
- J1 pad 3: /GND -> Net-(J1-Pad3)
- J1 pad 5: /J1_V -> Net-(J1-Pad5)
- J2 pad 3: /GND -> Net-(J2-Pad3)
- J2 pad 5: /J2_V -> Net-(J2-Pad5)
- P19 pad 1: Net-(CON1-Pad2) -> Net-(CON1-Pad3)
- U2 pad 10: Net-(C9-Pad1) -> Net-(C5-Pad1)
- U2 pad 11: Net-(C9-Pad1) -> Net-(C5-Pad1)
- U2 pad 12: Net-(C5-Pad1) -> Net-(C8-Pad1)
- U2 pad 3: Net-(C9-Pad1) -> Net-(C5-Pad1)
Routing:
- net /J1_V: track 10.4 -> 8.56 mm
- net Net-(J2-Pad5): track 0.00 -> 1.80 mm
- net Net-(J1-Pad5): track 0.00 -> 1.80 mm
- net /J2_V: track 10.8 -> 8.99 mm

Commit message: wip
Parts:
- moved F1 9.69 mm to (92.0, 67.1)
- moved F2 7.69 mm to (88.0, 87.1)
- moved D4 6.23 mm to (98.2, 83.2)
- moved DCDC1 5.06 mm to (91.8, 101.2)
- moved R13 4.57 mm to (93.6, 84.5), turned to 270 degrees
Connections:
- J1 pad 4: /GND -> GNDA
- J2 pad 4: /GND -> GNDA
- P1 pad 2: /GND -> GNDA
- P1 pad 6: /GND -> GNDA
- P11 pad 2: /GND -> GNDA
- P12 pad 2: /GND -> GNDA
- P17 pad 2: /GND -> GNDA
- P18 pad 2: /GND -> GNDA
- P2 pad 2: /GND -> GNDA
- P2 pad 6: /GND -> GNDA
- P3 pad 2: /GND -> GNDA
- P3 pad 6: /GND -> GNDA
- P4 pad 2: /GND -> GNDA
- P4 pad 6: /GND -> GNDA
- P5 pad 2: /GND -> GNDA
- P5 pad 6: /GND -> GNDA
- P6 pad 2: /GND -> GNDA
- P6 pad 6: /GND -> GNDA
- P7 pad 2: /GND -> GNDA
- P7 pad 6: /GND -> GNDA
- P8 pad 2: /GND -> GNDA
- P8 pad 6: /GND -> GNDA
Routing:
- net /5V: track 77.9 -> 25.7 mm
- net /CANH: track 149.1 -> 133.9 mm, vias 3 -> 2
- net /CANL: track 146.0 -> 131.3 mm, vias 3 -> 2

Commit message: wip
Routing:
- net /GS0: track 0.00 -> 45.8 mm
Other:
- net class Vcc: via_dia 2 -> 1.3; via_drill 1.6 -> 1
Changed lines of the file:
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@@
-(kicad_pcb (version 4) (host pcbnew 4.0.2+e4-6225~38~ubuntu14.04.1-stable)
+(kicad_pcb (version 4) (host pcbnew 4.0.1-stable)
   (general
     (links 233)
     (no_connects 208)
-    (area 51.400001 38.02446 212.661501 154.700001)
+    (area 66.924999 48.924999 167.075001 149.075001)
     (thickness 1.6)
     (drawings 80)
-    (tracks 100)
+    (tracks 108)
     (zones 0)
     (modules 81)
@@
     (clearance 0.2)
     (trace_width 1.2)
-    (via_dia 2)
-    (via_drill 1.6)
-    (uvia_dia 1.3)
-    (uvia_drill 0.9)
+    (via_dia 1.3)
+    (via_drill 1)
+    (uvia_dia 0.6)
+    (uvia_drill 0.4)
     (add_net /5V)
     (add_net /J1_V)
@@
   (gr_line (start 69.5 149) (end 114.5 149) (angle 90) (layer Edge.Cuts) (width 0.15))
   (gr_line (start 69.5 49) (end 114.5 49) (angle 90) (layer Edge.Cuts) (width 0.15))
+  (segment (start 105.0925 142.494) (end 105.0925 105.156) (width 0.6) (layer B.Cu) (net 1))
+  (segment (start 108.0135 145.415) (end 105.0925 142.494) (width 0.6) (layer B.Cu) (net 1))
+  (segment (start 109.34566 145.415) (end 108.0135 145.415) (width 0.6) (layer B.Cu) (net 1))
+  (segment (start 110.75 142.95) (end 110.75 144.01066) (width 0.6) (layer B.Cu) (net 1))
+  (segment (start 110.75 144.01066) (end 109.34566 145.415) (width 0.6) (layer B.Cu) (net 1))
+  (segment (start 97.917 73.406) (end 84.201 73.406) (width 0.6) (layer B.Cu) (net 2))
   (segment (start 99.06 73.406) (end 97.917 73.406) (width 0.6) (layer B.Cu) (net 2))
-  (segment (start 97.917 73.406) (end 84.201 73.406) (width 0.6) (layer B.Cu) (net 2))
+  (segment (start 100.965 75.311) (end 99.06 73.406) (width 0.6) (layer B.Cu) (net 2))
+  (segment (start 84.201 73.406) (end 81.915 75.692) (width 0.6) (layer B.Cu) (net 2))
+  (segment (start 100.965 133.731) (end 100.965 75.311) (width 0.6) (layer B.Cu) (net 2))
   (segment (start 100.965 136.017) (end 100.965 133.731) (width 0.6) (layer B.Cu) (net 2))
-  (segment (start 100.965 133.731) (end 100.965 75.311) (width 0.6) (layer B.Cu) (net 2))
   (via (at 100.965 133.731) (size 1) (drill 0.8) (layers F.Cu B.Cu) (net 2))
   (segment (start 110.75 135.05) (end 110.75 134.84) (width 0.6) (layer F.Cu) (net 2))
@@
   (segment (start 109.64 133.73) (end 100.966 133.73) (width 0.6) (layer F.Cu) (net 2))
   (segment (start 100.966 133.73) (end 100.965 133.731) (width 0.6) (layer F.Cu) (net 2))
-  (segment (start 84.201 73.406) (end 81.915 75.692) (width 0.6) (layer B.Cu) (net 2))
-  (segment (start 100.965 75.311) (end 99.06 73.406) (width 0.6) (layer B.Cu) (net 2))
   (segment (start 97.932 139.05) (end 100.965 136.017) (width 0.6) (layer B.Cu) (net 2))
   (segment (start 87.99 139.05) (end 97.932 139.05) (width 0.6) (layer B.Cu) (net 2))
@@
   (segment (start 88.09 129.75) (end 88.09 120) (width 0.6) (layer B.Cu) (net 2))
   (segment (start 88.09 133.25) (end 88.09 129.75) (width 0.6) (layer B.Cu) (net 2))
+  (segment (start 83.947 72.39) (end 80.645 75.692) (width 0.6) (layer B.Cu) (net 3))
+  (segment (start 99.568 72.39) (end 83.947 72.39) (width 0.6) (layer B.Cu) (net 3))
+  (segment (start 99.822 72.644) (end 99.568 72.39) (width 0.6) (layer B.Cu) (net 3))
   (segment (start 101.981 74.803) (end 99.822 72.644) (width 0.6) (layer B.Cu) (net 3))
-  (segment (start 99.822 72.644) (end 99.568 72.39) (width 0.6) (layer B.Cu) (net 3))
+  (segment (start 101.981 125.095) (end 101.981 76.409612) (width 0.6) (layer B.Cu) (net 3))
+  (segment (start 101.981 135.001) (end 101.981 125.095) (width 0.6) (layer B.Cu) (net 3))
+  (segment (start 101.981 76.409612) (end 101.981 74.803) (width 0.6) (layer B.Cu) (net 3))
   (segment (start 101.981 135.708106) (end 101.981 135.001) (width 0.6) (layer B.Cu) (net 3))
   (segment (start 101.981 136.209998) (end 101.981 135.708106) (width 0.6) (layer B.Cu) (net 3))
   (segment (start 90.63 140.2) (end 97.990998 140.2) (width 0.6) (layer B.Cu) (net 3))
   (segment (start 97.990998 140.2) (end 101.981 136.209998) (width 0.6) (layer B.Cu) (net 3))
-  (segment (start 101.981 135.001) (end 101.981 125.095) (width 0.6) (layer B.Cu) (net 3))
   (via (at 101.981 135.001) (size 1) (drill 0.8) (layers F.Cu B.Cu) (net 3))
   (segment (start 108.25 135.05) (end 102.03 135.05) (width 0.6) (layer F.Cu) (net 3))
   (segment (start 102.03 135.05) (end 101.981 135.001) (width 0.6) (layer F.Cu) (net 3))
-  (segment (start 83.947 72.39) (end 80.645 75.692) (width 0.6) (layer B.Cu) (net 3))
-  (segment (start 99.568 72.39) (end 83.947 72.39) (width 0.6) (layer B.Cu) (net 3))
-  (segment (start 101.981 76.409612) (end 101.981 74.803) (width 0.6) (layer B.Cu) (net 3))
-  (segment (start 101.981 125.095) (end 101.981 76.409612) (width 0.6) (layer B.Cu) (net 3))
   (segment (start 90.63 133.25) (end 90.63 140.2) (width 0.6) (layer F.Cu) (net 3))
   (via (at 90.63 140.2) (size 1) (drill 0.8) (layers F.Cu B.Cu) (net 3))
@@
   (segment (start 152.78 134.72) (end 152.78 126.5) (width 0.6) (layer B.Cu) (net 20))
   (segment (start 150.38 137.12) (end 152.78 134.72) (width 0.6) (layer B.Cu) (net 20))
-  (segment (start 99.314 137.033) (end 98.25 135.969) (width 1.2) (layer F.Cu) (net 22))
-  (segment (start 98.25 135.969) (end 98.25 133.25) (width 1.2) (layer F.Cu) (net 22))
-  (segment (start 103.378 137.033) (end 99.314 137.033) (width 1.2) (layer F.Cu) (net 22))
-  (segment (start 103.411 137) (end 103.378 137.033) (width 1.2) (layer F.Cu) (net 22))
-  (segment (start 108.25 137) (end 103.411 137) (width 1.2) (layer F.Cu) (net 22))
-  (via (at 103.378 137.033) (size 2) (drill 1.6) (layers F.Cu B.Cu) (net 22))
   (segment (start 82.482999 71.695001) (end 79.248 74.93) (width 1.2) (layer B.Cu) (net 22))
+  (segment (start 103.378 73.914) (end 100.33 70.866) (width 1.2) (layer B.Cu) (net 22))
   (segment (start 83.312 70.866) (end 82.482999 71.695001) (width 1.2) (layer B.Cu) (net 22))
   (segment (start 100.33 70.866) (end 83.312 70.866) (width 1.2) (layer B.Cu) (net 22))
-  (segment (start 103.378 73.914) (end 100.33 70.866) (width 1.2) (layer B.Cu) (net 22))
-  (segment (start 103.378 137.795) (end 103.378 73.914) (width 1.2) (layer B.Cu) (net 22))
+  (segment (start 103.378 137.033) (end 103.378 73.914) (width 1.2) (layer B.Cu) (net 22))
+  (segment (start 103.378 136.9695) (end 99.568 136.9695) (width 1.2) (layer F.Cu) (net 22))
+  (segment (start 98.25 135.6515) (end 98.25 133.25) (width 1.2) (layer F.Cu) (net 22) (status 800000))
+  (segment (start 99.568 136.9695) (end 98.25 135.6515) (width 1.2) (layer F.Cu) (net 22))
+  (segment (start 108.25 137) (end 103.4085 137) (width 1.2) (layer F.Cu) (net 22) (status 400000))
+  (segment (start 103.4415 137.033) (end 103.378 137.033) (width 1.2) (layer B.Cu) (net 22))
+  (segment (start 103.378 136.9695) (end 103.4415 137.033) (width 1.2) (layer B.Cu) (net 22))
+  (via (at 103.378 136.9695) (size 1.3) (drill 1) (layers F.Cu B.Cu) (net 22))
+  (segment (start 103.4085 137) (end 103.378 136.9695) (width 1.2) (layer F.Cu) (net 22))
+  (segment (start 103.378 137.795) (end 103.378 137.033) (width 1.2) (layer B.Cu) (net 22))
   (segment (start 99.568 141.605) (end 103.378 137.795) (width 1.2) (layer B.Cu) (net 22))
   (segment (start 98.795 141.605) (end 99.568 141.605) (width 1.2) (layer B.Cu) (net 22))
+  (segment (start 98 144.8) (end 98 142.4) (width 1.2) (layer B.Cu) (net 22))
+  (segment (start 98 142.4) (end 98.795 141.605) (width 1.2) (layer B.Cu) (net 22))
   (segment (start 110.75 136.7) (end 108.55 136.7) (width 1.2) (layer F.Cu) (net 22))
   (segment (start 108.55 136.7) (end 108.25 137) (width 1.2) (layer F.Cu) (net 22))
@@
   (segment (start 98.25 133.25) (end 98.25 129.75) (width 1.2) (layer B.Cu) (net 22))
   (segment (start 108.6 118.5) (end 108.3 118.8) (width 1.2) (layer B.Cu) (net 22))
-  (segment (start 98 144.8) (end 98 142.4) (width 1.2) (layer B.Cu) (net 22))
-  (segment (start 98 142.4) (end 98.795 141.605) (width 1.2) (layer B.Cu) (net 22))
   (segment (start 98.9024 68.58) (end 98.75 68.58) (width 1.2) (layer B.Cu) (net 22))
   (segment (start 98 133.5) (end 98.25 133.25) (width 0.6) (layer B.Cu) (net 22))
