File: mcan-emergency-stop/doc/Emergengy-Stop.sch (KiCad schematic (older format))
At the start: 16 parts, among them Q1 BC547, Q2 BC547, Q3 BC547, SW1 SW_PUSH, SW2 SW_PUSH, U1 MCP2562, U2 STM32-BARE

Commit message: schematic wip
Parts:
- removed Q1, Q2, Q3: BC547, TO-92, symbol BC547
- removed R1: 1k, w_pth_resistors:RC03, symbol R
- removed R3, R5: 1k, w_pth_resistors:rc03_vert, symbol R
- added C1: 10uF, symbol CP
- added P1: CAN, symbol CONN_01X03
- added P2: Terminierung, symbol CONN_01X02
- added R7, R8: 1k5, w_pth_resistors:rc03_vert, symbol R
- added R9: 120, w_pth_resistors:rc03_vert, symbol R
- added SW3: Oeffner, symbol SW_PUSH
- D1: value Status LED -> Off LED
- D2: value LED -> Off LED
- D3: value LED -> ON LED
- R2: value 470 -> 1k5
- R4, R6: value 100 -> 1k5
- SW1: value SW_PUSH -> Oeffner
- SW2: value SW_PUSH -> Schliesser
Connections:
- net labels added: +3V3, 3V3
- wire segments 40 -> 61
- no-connect marks 26 -> 27
Other:
- moved on the sheet: D2, D3, R2, R4, R6, SW2
