File: srse2/SRSE2.kicad_pcb (KiCad board)
At the start: 2 copper layers, 82 x 72 mm, 18 parts, among them P1 UART, U2 PIC18F25K80, U3 FT230XS, U4 HR911105A, U5 HR911105A

Commit message: wip
Parts:
- removed P1: UART, Pin_Headers:Pin_Header_Straight_1x03
- removed R1: 27, Resistors_SMD:R_0805_HandSoldering_II
- removed REF**: Omega2, Onion2:DIP-32_1_ELL
- removed U2: PIC18F25K80, w_smd_dil:soic-28
- added C10, C7, C8: 100nF, Capacitors_SMD:C_0805_HandSoldering, F.Cu at (141.0, 156.1)
- added C3: 4.7uF, Capacitors_SMD:C_0805_HandSoldering, F.Cu at (141.0, 156.1)
- added C5: 22pF, Capacitors_SMD:C_0805_HandSoldering, F.Cu at (118.2, 106.0)
- added C9: 100nF, Capacitors_SMD:C_0805_HandSoldering, F.Cu at (146.1, 148.5)
- added D1: Status, LEDs:LED-3MM, F.Cu at (131.6, 126.4)
- added D2: CAN Ovf, LEDs:LED-3MM, F.Cu at (126.5, 134.2)
- added D3: UART Ovf, LEDs:LED-3MM, F.Cu at (127.9, 142.7)
- added P2: CONN_01X09, Pin_Headers:Pin_Header_Straight_1x04, F.Cu at (111.3, 96.3)
- added P3: USB_B, w_conn_pc:conn_usb_B, F.Cu at (117.9, 142.6)
- added P4: ISO_I2C, Pin_Headers:Pin_Header_Straight_1x04, F.Cu at (141.0, 156.1)
- added P6: CONN_01X03, Pin_Headers:Pin_Header_Straight_1x03, F.Cu at (141.0, 156.1)
- added P7: UART, Pin_Headers:Pin_Header_Straight_1x03, F.Cu at (178.6, 96.9)
- added R10, R11, R8, R9: 3k3, Resistors_SMD:R_0805_HandSoldering, F.Cu at (141.0, 156.1)
- added R12, R15: 220, Resistors_SMD:R_0805_HandSoldering, F.Cu at (141.0, 156.1)
- added R13: 0, Resistors_SMD:R_0805_HandSoldering, F.Cu at (141.0, 156.1)
- added R16, R17, R18, R19: 50, Resistors_SMD:R_0805_HandSoldering, F.Cu at (141.0, 156.1)
- added R20: 10k, Resistors_SMD:R_0603_HandSoldering, F.Cu at (141.0, 156.1)
- added R5, R6: 3k3, Resistors_SMD:R_0603_HandSoldering, F.Cu at (141.0, 156.1)
- added U1: Omega2, Onion2:Omega2, F.Cu at (159.1, 110.7)
- added Y1: 16MHz, Crystals:Crystal_HC49-U_Vertical, F.Cu at (123.4, 108.1)
- C1, C2: value 47pF -> 100nF; footprint Resistors_SMD:R_0805_HandSoldering_II -> Capacitors_SMD:C_0805_HandSoldering
- C4: value 100nF -> 22pF; footprint Resistors_SMD:R_0805_HandSoldering_II -> Capacitors_SMD:C_0805_HandSoldering
- C6: value 4.7uF -> 10uF; footprint Resistors_SMD:R_0805_HandSoldering_II -> Capacitors_ThroughHole:C_Radial_D5_L6_P2.5
- R2: value 27 -> 560; footprint Resistors_SMD:R_0805_HandSoldering_II -> Resistors_SMD:R_0805_HandSoldering
- R3: value 220 -> 4k7; footprint Resistors_SMD:R_0805_HandSoldering_II -> Resistors_SMD:R_0805_HandSoldering
- R4: value 220 -> 560; footprint Resistors_SMD:R_0805_HandSoldering_II -> Resistors_SMD:R_0805_HandSoldering
- U3: value FT230XS -> PIC18F25K80; footprint w_smd_dil:ssop-16 -> w_smd_dil:soic-28
- U4: footprint RJ45ALED_1PRIMARY -> HR911105A:RJ45ALED_1PRIMARY
- U5: value HR911105A -> SP3485CN; footprint RJ45ALED_1PRIMARY -> SO-8
- moved R4 68.2 mm to (141.0, 156.1)
- moved R2 67.8 mm to (141.0, 156.1)
- moved C2 58.2 mm to (141.0, 156.1), turned to 0 degrees
- moved R3 57.4 mm to (141.0, 156.1)
- moved C1 51.6 mm to (143.9, 142.6)
- moved U3 25.8 mm to (134.2, 105.8), turned to 270 degrees
- moved C6 8.14 mm to (124.3, 99.1), turned to 180 degrees
- moved U5 6.48 mm to (141.0, 156.1)
- moved C4 4.98 mm to (118.2, 110.6), turned to 180 degrees
- moved U4 3.17 mm to (151.6, 148.5)
Connections:
- net /CBUS3 renamed /SPI_DO
- C1 pad 1: /USBDP -> VCC
- C2 pad 1: /USBDM -> VCC
- C4 pad 1: VCC -> Net-(C4-Pad1)
- C6 pad 1: VCC -> Net-(C6-Pad1)
- R2 pad 1: Net-(R2-Pad1) -> Net-(D2-Pad1)
- R2 pad 2: /USBDP -> Net-(R2-Pad2)
- R3 pad 1: Net-(D1-Pad1) -> //MCLR
- R3 pad 2: Net-(R3-Pad2) -> VCC
- U3 pad 1: /TxD -> //MCLR
- U3 pad 10: Net-(C3-Pad1) -> Net-(C4-Pad1)
- U3 pad 11: Net-(C3-Pad1) -> /RC0
- U3 pad 12: VCC -> /RC1
- U3 pad 13: GND -> /LIGHT
- U3 pad 14: Net-(R3-Pad2) -> /I2C_SCL
- U3 pad 15: /CBUS0 -> /I2C_SDA
- U3 pad 2: /RTS -> Net-(R4-Pad2)
- U3 pad 3: Net-(C3-Pad1) -> Net-(R2-Pad2)
- U3 pad 4: /RxD -> /RTS
- U3 pad 5: GND -> Net-(R1-Pad2)
- U3 pad 6: /CTS -> Net-(C6-Pad1)
- U3 pad 7: Net-(R4-Pad2) -> /RS485_DE
- U3 pad 8: Net-(R2-Pad1) -> GND
- U4 pad 1: Net-(U4-Pad1) -> /LTDP
- U4 pad 10: Net-(U4-Pad10) -> /LLEDG
- U4 pad 11: Net-(U4-Pad11) -> /LLEDY
- U4 pad 15: Net-(U4-Pad15) -> Net-(R13-Pad1)
- U4 pad 16: Net-(U4-Pad16) -> Net-(R13-Pad1)
- U4 pad 2: Net-(U4-Pad2) -> /LTDM
- U4 pad 3: Net-(U4-Pad3) -> /LRDP
- U4 pad 4: Net-(U4-Pad4) -> /LP4
- U4 pad 5: Net-(U4-Pad5) -> /LP4
- U4 pad 6: Net-(U4-Pad6) -> /LRDM
- U4 pad 8: Net-(U4-Pad8) -> GND
- U5 pad 1: Net-(U5-Pad1) -> /RS485_R
- U5 pad 2: Net-(U5-Pad2) -> /RS485_DE
- U5 pad 3: Net-(U5-Pad3) -> /RS485_DE
- U5 pad 4: Net-(U5-Pad4) -> /RS485_T
- U5 pad 5: Net-(U5-Pad5) -> GND
- U5 pad 8: Net-(U5-Pad8) -> VCC

Commit message: wip - accurate Omega2 footprint
Parts:
- added C11: 100nF, Capacitors_SMD:C_0805_HandSoldering, F.Cu at (149.8, 126.3)
- added C12: 100nF, Capacitors_SMD:C_0805_HandSoldering, F.Cu at (147.1, 157.9)
- added C13: 100nF, Capacitors_SMD:C_0805_HandSoldering, F.Cu at (140.8, 125.5)
- added J1: S88, w_conn_pc:megb8-8, F.Cu at (126.8, 143.3)
- added J2: CAN, w_conn_pc:megb8-8, F.Cu at (142.3, 143.3)
- added P1: I2S, Pin_Headers:Pin_Header_Straight_1x06, F.Cu at (155.1, 79.5)
- added P10: PIC_SPARE, Pin_Headers:Pin_Header_Straight_1x06, F.Cu at (130.3, 100.5)
- added P11: RS485 TERM, Pin_Headers:Pin_Header_Straight_1x02, F.Cu at (117.5, 125.6)
- added P12: RS485, Pin_Headers:Pin_Header_Straight_1x03, F.Cu at (112.7, 129.4)
- added P5: USB_B, w_conn_pc:conn_usb_B, F.Cu at (108.8, 115.1)
- added P8: CAN, Pin_Headers:Pin_Header_Straight_1x04, F.Cu at (135.0, 88.1)
- added P9: PIC_I2C, Pin_Headers:Pin_Header_Straight_1x04, F.Cu at (178.9, 118.1)
- added R1: 10k, Resistors_SMD:R_0603_HandSoldering, F.Cu at (134.1, 126.5)
- added R14: 3k3, Resistors_SMD:R_0805_HandSoldering, F.Cu at (141.0, 156.1)
- added R21: 120, Resistors_SMD:R_0805_HandSoldering, F.Cu at (141.0, 156.1)
- added R7: 3k3, Resistors_SMD:R_0603_HandSoldering, F.Cu at (154.6, 122.8)
- added U2: ADuM1250CR, w_smd_dil:so-8, F.Cu at (128.9, 124.3)
- added U6: SP3485CN, Power_Integrations:SO-8, F.Cu at (142.1, 110.9)
- C3: value 4.7uF -> 22pF
- C5: value 22pF -> 10uF; footprint Capacitors_SMD:C_0805_HandSoldering -> Capacitors_ThroughHole:C_Radial_D5_L6_P2.5
- C6: value 10uF -> 100nF; footprint Capacitors_ThroughHole:C_Radial_D5_L6_P2.5 -> Capacitors_SMD:C_0805_HandSoldering
- P2: footprint Pin_Headers:Pin_Header_Straight_1x04 -> Pin_Headers:Pin_Header_Straight_1x09
- P3: value USB_B -> opt 18V; footprint w_conn_pc:conn_usb_B -> Pin_Headers:Pin_Header_Straight_1x01
- P4: value ISO_I2C -> UART; footprint Pin_Headers:Pin_Header_Straight_1x04 -> Pin_Headers:Pin_Header_Straight_1x03
- P6: value CONN_01X03 -> ISO_I2C; footprint Pin_Headers:Pin_Header_Straight_1x03 -> Pin_Headers:Pin_Header_Straight_1x04
- P7: value UART -> CAN_TERM; footprint Pin_Headers:Pin_Header_Straight_1x03 -> Pin_Headers:Pin_Header_Straight_1x02
- R11: value 3k3 -> 120
- R15: value 220 -> 3k3
- R16: value 50 -> 220
- R20: value 10k -> 50; footprint Resistors_SMD:R_0603_HandSoldering -> Resistors_SMD:R_0805_HandSoldering
- R3: value 4k7 -> 560
- R4: value 560 -> 4k7
- R5: value 3k3 -> 560; footprint Resistors_SMD:R_0603_HandSoldering -> Resistors_SMD:R_0805_HandSoldering
- R8: value 3k3 -> 0
- U3: value PIC18F25K80 -> MCP2562-I/SN; footprint w_smd_dil:soic-28 -> Power_Integrations:SO-8
- U4: value HR911105A -> PIC18F25K80; footprint HR911105A:RJ45ALED_1PRIMARY -> w_smd_dil:soic-28
- U5: value SP3485CN -> HR911105A; footprint SO-8 -> HR911105A:RJ45ALED_1PRIMARY
- moved P6 72.3 mm to (103.2, 94.5)
- moved P4 68.6 mm to (155.8, 89.1)
- moved R4 56.2 mm to (166.7, 106.0)
- moved C3 55.1 mm to (144.7, 101.1), turned to 180 degrees
- moved D3 53.8 mm to (119.7, 89.6)
- moved P7 53.4 mm to (127.4, 81.6)
- moved C6 50.3 mm to (166.7, 126.1), turned to 0 degrees
- moved D2 46.3 mm to (114.1, 89.6)
- moved C4 44.5 mm to (161.7, 101.2), turned to 0 degrees
- moved C7 43.8 mm to (173.2, 126.4)
- moved C2 41.7 mm to (158.8, 118.4)
- moved C8 39.8 mm to (128.7, 118.2), turned to 180 degrees
- moved U4 37.7 mm to (155.0, 110.9), turned to 180 degrees
- moved R6 36.0 mm to (160.4, 125.8)
- moved D1 35.8 mm to (112.2, 96.3)
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Connections:
- C10 pad 1: Net-(C10-Pad1) -> /LP4
- C3 pad 1: VCC -> Net-(C3-Pad1)
- C6 pad 1: Net-(C6-Pad1) -> GND
- C6 pad 2: GND -> VCC
- C7 pad 1: /LP4 -> GND
- C7 pad 2: GND -> VCC
- C8 pad 1: /LP4 -> Net-(C8-Pad1)
- C8 pad 2: GND -> Net-(C8-Pad2)
- C9 pad 1: Net-(C9-Pad1) -> GND
- C9 pad 2: GND -> +5V
- P3 pad 1: +5V -> Net-(J2-Pad6)
- P4 pad 1: Net-(P4-Pad1) -> GND
- P6 pad 1: GND -> Net-(C8-Pad1)
- P6 pad 2: Net-(P5-Pad2) -> Net-(P6-Pad2)
- P7 pad 1: GND -> Net-(P7-Pad1)
- P7 pad 2: Net-(P7-Pad2) -> /CANL
- R10 pad 1: /I2C_SCL -> Net-(P6-Pad2)
- R10 pad 2: VCC -> Net-(C8-Pad2)
- R11 pad 1: VCC -> Net-(P7-Pad1)
- R11 pad 2: /I2C_SDA -> /CANH
- R15 pad 2: Net-(R15-Pad2) -> /I2C_SDA
- R16 pad 1: Net-(C10-Pad1) -> VCC
- R16 pad 2: /LTDP -> Net-(R16-Pad2)
- R17 pad 1: Net-(C10-Pad1) -> Net-(C13-Pad1)
- R17 pad 2: /LTDM -> /LTDP
- R18 pad 1: Net-(C9-Pad1) -> Net-(C13-Pad1)
- R18 pad 2: /LRDP -> /LTDM
- R19 pad 1: Net-(C9-Pad1) -> Net-(C12-Pad1)
- R19 pad 2: /LRDM -> /LRDP
- R2 pad 1: Net-(D2-Pad1) -> Net-(D1-Pad1)
- R20 pad 1: VCC -> Net-(C12-Pad1)
- R20 pad 2: Net-(R20-Pad2) -> /LRDM
- R3 pad 1: //MCLR -> Net-(D2-Pad1)
- R3 pad 2: VCC -> Net-(R3-Pad2)
- R4 pad 1: Net-(D3-Pad1) -> //MCLR
- R4 pad 2: Net-(R4-Pad2) -> VCC
- R5 pad 1: Net-(R5-Pad1) -> Net-(D3-Pad1)
- R5 pad 2: VCC -> Net-(R5-Pad2)
- R8 pad 1: Net-(P4-Pad3) -> GND
- R8 pad 2: Net-(P4-Pad4) -> Net-(P5-Pad5)
- R9 pad 1: Net-(P4-Pad2) -> Net-(P6-Pad3)
- R9 pad 2: Net-(P4-Pad4) -> Net-(C8-Pad2)
- U1 pad 16: Net-(R20-Pad2) -> Net-(R1-Pad2)
- U1 pad 17: Net-(R5-Pad1) -> Net-(R6-Pad1)
- U1 pad 18: Net-(R6-Pad1) -> Net-(R7-Pad1)
- U1 pad 27: Net-(P7-Pad2) -> Net-(P4-Pad2)
- U1 pad 28: Net-(P7-Pad3) -> Net-(P4-Pad3)
- U1 pad 29: Net-(P3-Pad2) -> Net-(P5-Pad2)
- U1 pad 30: Net-(P3-Pad3) -> Net-(P5-Pad3)
- U3 pad 1: //MCLR -> /CANTX
- U3 pad 2: Net-(R4-Pad2) -> GND
- U3 pad 3: Net-(R2-Pad2) -> +5V
- U3 pad 4: /RTS -> /CANRX
- U3 pad 5: Net-(R1-Pad2) -> VCC
- U3 pad 6: Net-(C6-Pad1) -> /CANL
- U3 pad 7: /RS485_DE -> /CANH
- U4 pad 1: /LTDP -> //MCLR
- U4 pad 10: /LLEDG -> Net-(C3-Pad1)
- U4 pad 11: /LLEDY -> /RC0
- U4 pad 12: Net-(R15-Pad2) -> /RC1
- U4 pad 13: (no net) -> /LIGHT
- U4 pad 14: (no net) -> /I2C_SCL
- U4 pad 15: Net-(R13-Pad1) -> /I2C_SDA
- U4 pad 16: Net-(R13-Pad1) -> /SPI_DO
- U4 pad 2: /LTDM -> Net-(R5-Pad2)
- U4 pad 3: /LRDP -> Net-(R3-Pad2)
- U4 pad 4: /LP4 -> /RTS
- U4 pad 5: /LP4 -> Net-(R2-Pad2)
- U4 pad 6: /LRDM -> Net-(C5-Pad1)
- U4 pad 7: Net-(U4-Pad7) -> /RS485_DE
- U4 pad 9: Net-(R12-Pad1) -> Net-(C4-Pad1)
- U5 pad 1: /RS485_R -> /LTDP
- U5 pad 2: /RS485_DE -> /LTDM
- U5 pad 3: /RS485_DE -> /LRDP
- U5 pad 4: /RS485_T -> /LP4
- U5 pad 5: GND -> /LP4
- U5 pad 6: Net-(P6-Pad3) -> /LRDM
- U5 pad 7: Net-(P5-Pad2) -> Net-(U5-Pad7)
- U5 pad 8: VCC -> GND
- Y1 pad 1: Net-(C4-Pad1) -> Net-(C3-Pad1)
- Y1 pad 2: Net-(C5-Pad1) -> Net-(C4-Pad1)

Commit message: wip
Parts:
- moved P4 24.4 mm to (180.2, 88.5)
- moved C5 23.8 mm to (158.0, 100.4), turned to 90 degrees
- moved P8 15.9 mm to (120.7, 95.0), turned to 90 degrees
- moved C4 9.13 mm to (154.3, 95.8)
- moved C3 5.87 mm to (147.0, 95.7)
- moved C2 3.57 mm to (158.4, 114.8)
- moved C1 3.47 mm to (152.8, 115.0)
- moved U4 3.15 mm to (154.8, 107.8)
- moved Y1 3.04 mm to (150.8, 99.3)
- moved U6 1.86 mm to (142.2, 109.0)
- moved R4 1.86 mm to (166.8, 104.2)
- moved U1 1.86 mm to (155.8, 105.5)
Changed lines of the file:
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@@
   )
   (module Capacitors_SMD:C_0805_HandSoldering (layer F.Cu)
-    (at 153.2 118.5 180)
+    (at 152.8 115.05 180)
     (descr "Capacitor SMD 0805, hand soldering")
     (tags "capacitor 0805")
@@
   )
   (module Capacitors_SMD:C_0805_HandSoldering (layer F.Cu)
-    (at 158.8 118.4)
+    (at 158.45 114.85)
     (descr "Capacitor SMD 0805, hand soldering")
     (tags "capacitor 0805")
@@
   )
   (module Capacitors_SMD:C_0805_HandSoldering (layer F.Cu)
-    (at 144.7 101.1 180)
+    (at 147 95.7 180)
     (descr "Capacitor SMD 0805, hand soldering")
     (tags "capacitor 0805")
     (attr smd)
-    (fp_text reference C3 (at 0 -2.1 180) (layer F.SilkS)
+    (fp_text reference C3 (at 3.5 -0.25 180) (layer F.SilkS)
       (effects (font (size 1 1) (thickness 0.15)))
     )
@@
   )
   (module Capacitors_SMD:C_0805_HandSoldering (layer F.Cu)
-    (at 161.7 101.2)
+    (at 154.3 95.85)
     (descr "Capacitor SMD 0805, hand soldering")
     (tags "capacitor 0805")
     (attr smd)
-    (fp_text reference C4 (at 0 -2.1) (layer F.SilkS)
-      (effects (font (size 1 1) (thickness 0.15)))
-    )
-    (fp_text value 22pF (at 0 2.1) (layer F.Fab)
+    (fp_text reference C4 (at 3.3 0) (layer F.SilkS)
+      (effects (font (size 1 1) (thickness 0.15)))
+    )
+    (fp_text value 22pF (at 4.3 -2.2) (layer F.Fab)
       (effects (font (size 1 1) (thickness 0.15)))
     )
@@
   )
   (module Capacitors_ThroughHole:C_Radial_D5_L6_P2.5 (layer F.Cu)
-    (at 138.5 86.7)
+    (at 158 100.4 90)
     (descr "Radial Electrolytic Capacitor Diameter 5mm x Length 6mm, Pitch 2.5mm")
     (tags "Electrolytic Capacitor")
-    (fp_text reference C5 (at 1.25 -3.8) (layer F.SilkS)
-      (effects (font (size 1 1) (thickness 0.15)))
-    )
-    (fp_text value 10uF (at 1.25 3.8) (layer F.Fab)
+    (fp_text reference C5 (at 1.25 -3.8 90) (layer F.SilkS)
+      (effects (font (size 1 1) (thickness 0.15)))
+    )
+    (fp_text value 10uF (at 1.25 3.8 90) (layer F.Fab)
       (effects (font (size 1 1) (thickness 0.15)))
     )
@@
     (fp_circle (center 1.25 0) (end 1.25 -2.5375) (layer F.SilkS) (width 0.15))
     (fp_circle (center 1.25 0) (end 1.25 -2.8) (layer F.CrtYd) (width 0.05))
-    (pad 1 thru_hole rect (at 0 0) (size 1.3 1.3) (drill 0.8) (layers *.Cu *.Mask F.SilkS)
+    (pad 1 thru_hole rect (at 0 0 90) (size 1.3 1.3) (drill 0.8) (layers *.Cu *.Mask F.SilkS)
       (net 9 "Net-(C5-Pad1)"))
-    (pad 2 thru_hole circle (at 2.5 0) (size 1.3 1.3) (drill 0.8) (layers *.Cu *.Mask F.SilkS)
+    (pad 2 thru_hole circle (at 2.5 0 90) (size 1.3 1.3) (drill 0.8) (layers *.Cu *.Mask F.SilkS)
       (net 1 GND))
     (model Capacitors_ThroughHole.3dshapes/C_Radial_D5_L6_P2.5.wrl
@@
   )
   (module Pin_Headers:Pin_Header_Straight_1x03 (layer F.Cu)
-    (at 155.8 89.1)
+    (at 180.15 88.55)
     (descr "Through hole pin header")
     (tags "pin header")
@@
   )
   (module Pin_Headers:Pin_Header_Straight_1x04 (layer F.Cu)
-    (at 135 88.1)
+    (at 120.65 94.95 90)
     (descr "Through hole pin header")
     (tags "pin header")
-    (fp_text reference P8 (at 0 -5.1) (layer F.SilkS)
-      (effects (font (size 1 1) (thickness 0.15)))
-    )
-    (fp_text value CAN (at 0 -3.1) (layer F.Fab)
+    (fp_text reference P8 (at 0 -5.1 90) (layer F.SilkS)
+      (effects (font (size 1 1) (thickness 0.15)))
+    )
+    (fp_text value CAN (at 0 -3.1 90) (layer F.Fab)
       (effects (font (size 1 1) (thickness 0.15)))
     )
@@
     (fp_line (start -1.55 0) (end -1.55 -1.55) (layer F.SilkS) (width 0.15))
     (fp_line (start -1.55 -1.55) (end 1.55 -1.55) (layer F.SilkS) (width 0.15))
-    (pad 1 thru_hole rect (at 0 0) (size 2.032 1.7272) (drill 1.016) (layers *.Cu *.Mask F.SilkS)
-      (net 1 GND))
-    (pad 2 thru_hole oval (at 0 2.54) (size 2.032 1.7272) (drill 1.016) (layers *.Cu *.Mask F.SilkS)
+    (pad 1 thru_hole rect (at 0 0 90) (size 2.032 1.7272) (drill 1.016) (layers *.Cu *.Mask F.SilkS)
+      (net 1 GND))
+    (pad 2 thru_hole oval (at 0 2.54 90) (size 2.032 1.7272) (drill 1.016) (layers *.Cu *.Mask F.SilkS)
       (net 62 /CANL))
-    (pad 3 thru_hole oval (at 0 5.08) (size 2.032 1.7272) (drill 1.016) (layers *.Cu *.Mask F.SilkS)
+    (pad 3 thru_hole oval (at 0 5.08 90) (size 2.032 1.7272) (drill 1.016) (layers *.Cu *.Mask F.SilkS)
       (net 63 /CANH))
-    (pad 4 thru_hole oval (at 0 7.62) (size 2.032 1.7272) (drill 1.016) (layers *.Cu *.Mask F.SilkS)
+    (pad 4 thru_hole oval (at 0 7.62 90) (size 2.032 1.7272) (drill 1.016) (layers *.Cu *.Mask F.SilkS)
       (net 20 +5V))
     (model Pin_Headers.3dshapes/Pin_Header_Straight_1x04.wrl
@@
   )
   (module Resistors_SMD:R_0805_HandSoldering (layer F.Cu)
-    (at 166.7 106.05)
+    (at 166.85 104.2)
     (descr "Resistor SMD 0805, hand soldering")
     (tags "resistor 0805")
@@
   )
   (module Onion2:Omega2 (layer F.Cu)
-    (at 155.6 107.3 180)
+    (at 155.75 105.45 180)
     (fp_text reference U1 (at -17.3 0 270) (layer F.SilkS)
       (effects (font (size 1.2 1.2) (thickness 0.15)))
@@
   )
   (module w_smd_dil:soic-28 (layer F.Cu)
-    (at 155 110.9 180)
+    (at 154.85 107.75 180)
     (descr "SOIC Wide, 28 pins")
     (fp_text reference U4 (at 0 -1.016 180) (layer F.SilkS)
@@
   )
   (module Power_Integrations:SO-8 (layer F.Cu)
-    (at 142.05 110.9)
+    (at 142.2 109.05)
     (descr "SO-8 Surface Mount Small Outline 150mil 8pin Package")
     (tags "Power Integrations D Package")
@@
   )
   (module Crystals:Crystal_HC49-U_Vertical (layer F.Cu)
-    (at 153.2 101.1)
+    (at 150.75 99.3)
     (descr "Crystal, Quarz, HC49/U, vertical, stehend,")
     (tags "Crystal, Quarz, HC49/U, vertical, stehend,")

Commit message: wip
Parts:
- moved R13 45.8 mm to (170.2, 120.8)
- moved R14 40.4 mm to (164.9, 123.5)
- moved C12 38.9 mm to (159.6, 121.0)
- moved R16 37.9 mm to (154.3, 120.6)
- moved R15 37.4 mm to (159.6, 123.5)
- moved R18 35.6 mm to (148.2, 121.2)
- moved R17 35.3 mm to (141.5, 120.8)
- moved C10 34.9 mm to (164.6, 121.0)
- moved R12 33.1 mm to (155.4, 126.3)
- moved R20 6.56 mm to (146.6, 152.7)
- moved R19 6.35 mm to (143.9, 161.7)
- moved R7 0.81 mm to (154.4, 123.6)
Changed lines of the file:
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@@
   (general
     (links 158)
-    (no_connects 154)
-    (area 99.924999 73.924999 182.075001 146.075001)
+    (no_connects 158)
+    (area 99.924999 73.924999 182.258334 163.875)
     (thickness 1.6)
     (drawings 8)
@@
   )
   (module Capacitors_SMD:C_0805_HandSoldering (layer F.Cu)
-    (at 146.7 151)
+    (at 164.55 121.05)
     (descr "Capacitor SMD 0805, hand soldering")
     (tags "capacitor 0805")
@@
   )
   (module Capacitors_SMD:C_0805_HandSoldering (layer F.Cu)
-    (at 147.1 157.9)
+    (at 159.55 121.05)
     (descr "Capacitor SMD 0805, hand soldering")
     (tags "capacitor 0805")
@@
   )
   (module Resistors_SMD:R_0603_HandSoldering (layer F.Cu)
-    (at 154.6 122.8)
+    (at 154.45 123.6)
     (descr "Resistor SMD 0603, hand soldering")
     (tags "resistor 0603")
@@
   )
   (module Resistors_SMD:R_0805_HandSoldering (layer F.Cu)
-    (at 141 156.075001)
+    (at 155.4 126.3)
     (descr "Resistor SMD 0805, hand soldering")
     (tags "resistor 0805")
@@
   )
   (module Resistors_SMD:R_0805_HandSoldering (layer F.Cu)
-    (at 141 156.075001)
+    (at 170.2 120.85)
     (descr "Resistor SMD 0805, hand soldering")
     (tags "resistor 0805")
@@
   )
   (module Resistors_SMD:R_0805_HandSoldering (layer F.Cu)
-    (at 141 156.075001)
+    (at 164.95 123.55)
     (descr "Resistor SMD 0805, hand soldering")
     (tags "resistor 0805")
@@
   )
   (module Resistors_SMD:R_0805_HandSoldering (layer F.Cu)
-    (at 141 156.075001)
+    (at 159.55 123.55)
     (descr "Resistor SMD 0805, hand soldering")
     (tags "resistor 0805")
@@
   )
   (module Resistors_SMD:R_0805_HandSoldering (layer F.Cu)
-    (at 141 156.075001)
+    (at 154.3 120.6)
     (descr "Resistor SMD 0805, hand soldering")
     (tags "resistor 0805")
@@
   )
   (module Resistors_SMD:R_0805_HandSoldering (layer F.Cu)
-    (at 141 156.075001)
+    (at 141.5 120.75)
     (descr "Resistor SMD 0805, hand soldering")
     (tags "resistor 0805")
@@
   )
   (module Resistors_SMD:R_0805_HandSoldering (layer F.Cu)
-    (at 141 156.075001)
+    (at 148.2 121.25)
     (descr "Resistor SMD 0805, hand soldering")
     (tags "resistor 0805")
@@
   )
   (module Resistors_SMD:R_0805_HandSoldering (layer F.Cu)
-    (at 141 156.075001)
+    (at 143.95 161.7)
     (descr "Resistor SMD 0805, hand soldering")
     (tags "resistor 0805")
@@
   )
   (module Resistors_SMD:R_0805_HandSoldering (layer F.Cu)
-    (at 141 156.075001)
+    (at 146.6 152.65)
     (descr "Resistor SMD 0805, hand soldering")
     (tags "resistor 0805")

Commit message: wip
Parts:
- R1, R6, R7: footprint Resistors_SMD:R_0603_HandSoldering -> Resistors_SMD:R_0805_HandSoldering
- moved R5 77.9 mm to (121.3, 83.6)
- moved R3 69.8 mm to (114.9, 84.5)
- moved R10 65.0 mm to (175.6, 97.8)
- moved R2 57.7 mm to (113.4, 102.2)
- moved R9 56.3 mm to (171.7, 100.3), turned to 90 degrees
- moved C8 53.2 mm to (178.6, 99.8)
- moved U2 50.5 mm to (175.6, 105.2)
- moved R19 38.7 mm to (158.4, 125.8), turned to 270 degrees
- moved U3 38.6 mm to (140.1, 127.8), turned to 180 degrees
- moved R1 37.8 mm to (140.8, 89.3), turned to 270 degrees
- moved R21 33.4 mm to (116.9, 132.9), turned to 270 degrees
- moved C6 32.4 mm to (134.6, 130.4)
- moved R20 31.1 mm to (162.4, 125.9), turned to 270 degrees
- moved R11 27.6 mm to (140.5, 122.2)
- moved C13 26.2 mm to (166.9, 127.1), turned to 180 degrees
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
Commit message: wip
Parts:
- moved R4 3.24 mm to (166.8, 103.0)
- moved C5 0.18 mm to (157.8, 100.3)
Changed lines of the file:
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@@
-(kicad_pcb (version 4) (host pcbnew 4.0.4+e1-6308~48~ubuntu14.04.1-stable)
+(kicad_pcb (version 4) (host pcbnew 4.0.2+dfsg1-stable)
   (general
     (links 158)
     (no_connects 158)
-    (area 99.924999 73.924999 182.075001 146.075001)
+    (area 99.924999 73.924999 183.2245 152.923)
     (thickness 1.6)
     (drawings 8)
@@
   )
   (module Capacitors_ThroughHole:C_Radial_D5_L6_P2.5 (layer F.Cu)
-    (at 157.6705 100.457 90)
+    (at 157.75 100.3 90)
     (descr "Radial Electrolytic Capacitor Diameter 5mm x Length 6mm, Pitch 2.5mm")
     (tags "Electrolytic Capacitor")
@@
   )
   (module Resistors_SMD:R_0805_HandSoldering (layer F.Cu)
-    (at 164.465 100.711)
+    (at 166.8 102.95)
     (descr "Resistor SMD 0805, hand soldering")
     (tags "resistor 0805")

Commit message: wip
Parts:
- U2: value ADuM1250CR -> ADuM1250
- moved P6 77.4 mm to (180.3, 101.9)
- moved P4 45.3 mm to (148.9, 121.4)
- moved C6 45.3 mm to (175.2, 110.5), turned to 180 degrees
- moved P7 42.9 mm to (134.7, 123.9)
- moved R7 37.9 mm to (170.9, 111.0), turned to 270 degrees
- moved P8 33.3 mm to (128.7, 127.3), turned to 180 degrees
- moved C9 30.0 mm to (140.3, 122.9), turned to 180 degrees
- moved P9 28.9 mm to (180.1, 89.2)
- moved R15 16.5 mm to (175.8, 93.4)
- moved C13 15.0 mm to (151.9, 125.9), turned to 270 degrees
- moved R3 12.3 mm to (119.9, 95.7)
- moved R5 10.0 mm to (128.0, 91.1)
- moved R14 9.27 mm to (175.7, 95.8), turned to 180 degrees
- moved R11 8.75 mm to (131.8, 123.3), turned to 90 degrees
- moved R10 8.67 mm to (171.8, 105.6), turned to 90 degrees
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Routing:
- net /LTDM: track 0.00 -> 3.32 mm
Other:
- net class Default: trace_width 0.25 -> 0.305
