File: srse2/SRSE2.kicad_pcb (KiCad board)
At the start: 2 copper layers, 82 x 72 mm, 62 parts, among them J1 S88, J2 CAN, P1 I2S, P10 PIC_SPARE, P11 RS485 TERM, P12 RS485, P2 CONN_01X09, P3 opt 18V, P4 UART, P5 USB_B, P6 ISO_I2C, P7 CAN_TERM, P8 CAN, P9 PIC_I2C, U1 Omega2, U2 ADuM1250, U3 MCP2562-I/SN, U4 PIC18F25K80, U5 HR911105A, U6 SP3485CN, Y1 16MHz

Commit message: wip
Parts:
- moved D1 11.8 mm to (113.1, 90.5)
- moved R2 5.74 mm to (113.1, 96.4), turned to 270 degrees
- moved R5 4.37 mm to (132.4, 90.9)
- moved D2 2.96 mm to (121.1, 90.7)
- moved D3 2.77 mm to (126.5, 90.7)
- moved C5 1.00 mm to (159.3, 100.6)
- moved U5 0.80 mm to (152.7, 150.6)
- moved C2 0.80 mm to (158.3, 115.6)
- moved Y1 0.75 mm to (151.3, 99.8)
- moved C1 0.74 mm to (153.0, 115.6)
- moved C3 0.70 mm to (147.5, 96.2)
- moved U4 0.61 mm to (154.8, 108.4)
- moved C4 0.35 mm to (154.5, 96.2)
- moved R12 0.12 mm to (149.8, 130.7), turned to 0 degrees
Routing:
- net /LRDP: track 0.21 -> 22.7 mm, vias 0 -> 1
- net /LTDP: track 0.00 -> 17.5 mm, vias 0 -> 2
- net /LTDM: track 3.32 -> 14.2 mm, vias 0 -> 2
- net /CANL: track 0.00 -> 9.27 mm
- net /LP4: track 0.22 -> 8.17 mm
- net /CANH: track 0.00 -> 7.88 mm
- net /LRDM: track 0.37 -> 4.51 mm
