File: srse2/SRSE2.sch (KiCad schematic (older format))
At the start: 28 parts, among them U1 PIC18F25K80, U2 HR911105A, Y1 16MHz

Commit message: wip
Parts:
- added P1: CONN_01X06, symbol CONN_01X06
- added P2: CONN_01X09, symbol CONN_01X09
- added P3: USB_B, w_conn_pc:conn_usb_B, symbol USB_B
- added P4: ISO_I2C, Pin_Headers:Pin_Header_Straight_1x04, symbol CONN_01X04
- added P5: CONN_01X02, symbol CONN_01X02
- added P6: CONN_01X03, Pin_Headers:Pin_Header_Straight_1x03, symbol CONN_01X03
- added P7: UART, Pin_Headers:Pin_Header_Straight_1x03, symbol CONN_01X03
- added R13: 0, Resistors_SMD:R_0805_HandSoldering, symbol R
- added R14: 120, Resistors_SMD:R_0805_HandSoldering_II, symbol R
- added R20: 10k, Resistors_SMD:R_0603_HandSoldering, symbol R
- added R5, R6: 3k3, Resistors_SMD:R_0603_HandSoldering, symbol R
- added R7: 0, Resistors_SMD:R_0805_HandSoldering_II, symbol R
- added R8, R9: 3k3, Resistors_SMD:R_0805_HandSoldering, symbol R
- added U1: Omega2, Onion2:Omega2, symbol Omega2
- added U2: ADuM1250CR, w_smd_dil:so-8, symbol ADuM1201CR
- added U5: SP3485CN, SO-8, symbol SP3485CN
- C1, C10, C2, C3, C7, C8, C9: footprint Resistors_SMD:R_0805_HandSoldering_II -> Capacitors_SMD:C_0805_HandSoldering
- R10: renamed from R7; footprint Resistors_SMD:R_0805_HandSoldering_II -> Resistors_SMD:R_0805_HandSoldering
- R11: renamed from R8; footprint Resistors_SMD:R_0805_HandSoldering_II -> Resistors_SMD:R_0805_HandSoldering
- R12: renamed from R6; footprint Resistors_SMD:R_0805_HandSoldering_II -> Resistors_SMD:R_0805_HandSoldering
- R15: renamed from R9; footprint Resistors_SMD:R_0805_HandSoldering_II -> Resistors_SMD:R_0805_HandSoldering
- R16: renamed from R10; footprint Resistors_SMD:R_0805_HandSoldering_II -> Resistors_SMD:R_0805_HandSoldering
- R17: renamed from R11; footprint Resistors_SMD:R_0805_HandSoldering_II -> Resistors_SMD:R_0805_HandSoldering
- R18: renamed from R12; footprint Resistors_SMD:R_0805_HandSoldering_II -> Resistors_SMD:R_0805_HandSoldering
- R19: renamed from R13; footprint Resistors_SMD:R_0805_HandSoldering_II -> Resistors_SMD:R_0805_HandSoldering
- R2: renamed from R4; footprint Resistors_SMD:R_0805_HandSoldering_II -> Resistors_SMD:R_0805_HandSoldering
- R3: renamed from R1; footprint Resistors_SMD:R_0805_HandSoldering_II -> Resistors_SMD:R_0805_HandSoldering
- R4: renamed from R5; footprint Resistors_SMD:R_0805_HandSoldering_II -> Resistors_SMD:R_0805_HandSoldering
- renumbered D2 to D1, D3 to D2, D4 to D3, R3 to R1, U1 to U3, U2 to U4
Connections:
- net labels added: +5V, I2S_CLK, I2S_SDI, I2S_SDO, I2S_WS, RS485_R, RS485_T
- net labels removed: GNDD, RS485
- wire segments 102 -> 258
- no-connect marks 0 -> 3
Other:
- moved on the sheet: D1, D3, R1, R10, R11, R4

Commit message: wip - still missing 2 components
Parts:
- added C6, C8: 100nF, Capacitors_SMD:C_0805_HandSoldering, symbol C
- added J1, J2: CAN, symbol RJ45
- added P3: opt 18V, Pin_Headers:Pin_Header_Straight_1x01, symbol CONN_01X01
- added P7: CAN, Pin_Headers:Pin_Header_Straight_1x04, symbol CONN_01X04
- added P8: CONN_01X06, Pin_Headers:Pin_Header_Straight_1x06, symbol CONN_01X06
- added U3: MCP2561-I/SN, SO-8, symbol MCP2551-I/SN
- P10: renamed from P6; value CONN_01X03 -> RS485
- P9: renamed from P5; value CONN_01X02 -> RS485 TERM
- R15: renamed from R14; footprint Resistors_SMD:R_0805_HandSoldering_II -> Resistors_SMD:R_0805_HandSoldering
- R2: renamed from R1; footprint Resistors_SMD:R_0805_HandSoldering_II -> Resistors_SMD:R_0805_HandSoldering
- R8: renamed from R7; footprint Resistors_SMD:R_0805_HandSoldering_II -> Resistors_SMD:R_0805_HandSoldering
- renumbered C8 to C10, C9 to C11, C10 to C12, C6 to C7, C7 to C9, P7 to P4, P3 to P5, P4 to P6, R20 to R1, R9 to R10, R10 to R11, R11 to R12, R12 to R13, R13 to R14, R15 to R16, R16 to R17, R17 to R18, R18 to R19, R19 to R20, R2 to R3, R3 to R4, R4 to R5, R5 to R6, R6 to R7, R8 to R9, U3 to U4, U4 to U5, U5 to U6
Connections:
- net labels added: CANH, CANL
- wire segments 258 -> 267
- no-connect marks 3 -> 11
Other:
- moved on the sheet: P10, P6, P9, R11, R12, R15, U6

Commit message: wip - add footprints
Parts:
- removed C3: 4.7uF, Capacitors_SMD:C_0805_HandSoldering, symbol C
- added C7, C9: 100nF, Capacitors_SMD:C_0805_HandSoldering, symbol C
- added P7: CAN_TERM, Pin_Headers:Pin_Header_Straight_1x02, symbol CONN_01X02
- added P9: CAN, Pin_Headers:Pin_Header_Straight_1x04, symbol CONN_01X04
- added R11: 120, Resistors_SMD:R_0805_HandSoldering, symbol R
- J1, J2: footprint (none) -> w_conn_pc:megb8-8
- P1: footprint (none) -> Pin_Headers:Pin_Header_Straight_1x06
- P11: renamed from P9; footprint (none) -> Pin_Headers:Pin_Header_Straight_1x02
- P2: footprint (none) -> Pin_Headers:Pin_Header_Straight_1x09
- U3: value MCP2561-I/SN -> MCP2562-I/SN; footprint SO-8 -> Power_Integrations:SO-8
- U6: footprint SO-8 -> Power_Integrations:SO-8
- renumbered C9 to C10, C10 to C11, C11 to C12, C12 to C13, C4 to C3, C5 to C4, C7 to C5, P8 to P10, P10 to P12, P7 to P8, R13 to R12, R14 to R13, R11 to R14, R12 to R15, R15 to R21
Connections:
- wire segments 267 -> 284
Other:
- moved on the sheet: C3, C4, C5, C6, D1, D2, D3, P8, R14, R15, R2, R3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

Commit message: wip - accurate Omega2 footprint
Parts:
- J1: value CAN -> S88
- P1: value CONN_01X06 -> I2S
- P10: value CONN_01X06 -> PIC_SPARE
- P9: value CAN -> PIC_I2C
Changed lines of the file:
@@
 P 850 1550
 F 0 "P1" H 850 1900 50  0000 C CNN
-F 1 "CONN_01X06" V 950 1550 50  0000 C CNN
+F 1 "I2S" V 950 1550 50  0000 C CNN
 F 2 "Pin_Headers:Pin_Header_Straight_1x06" H 850 1550 50  0001 C CNN
 F 3 "" H 850 1550 50  0000 C CNN
@@
 P 1150 4400
 F 0 "J1" H 1350 4900 50  0000 C CNN
-F 1 "CAN" H 1000 4900 50  0000 C CNN
+F 1 "S88" H 1000 4900 50  0000 C CNN
 F 2 "w_conn_pc:megb8-8" H 1150 4400 50  0001 C CNN
 F 3 "" H 1150 4400 50  0000 C CNN
@@
 P 9100 4900
 F 0 "P10" H 9100 5250 50  0000 C CNN
-F 1 "CONN_01X06" V 9200 4900 50  0000 C CNN
+F 1 "PIC_SPARE" V 9200 4900 50  0000 C CNN
 F 2 "Pin_Headers:Pin_Header_Straight_1x06" V 9100 4900 50  0001 C CNN
 F 3 "" H 9100 4900 50  0000 C CNN
@@
 P 8250 5850
 F 0 "P9" H 8250 6100 50  0000 C CNN
-F 1 "CAN" V 8350 5850 50  0000 C CNN
+F 1 "PIC_I2C" V 8350 5850 50  0000 C CNN
 F 2 "Pin_Headers:Pin_Header_Straight_1x04" V 8250 5850 50  0001 C CNN
 F 3 "" H 8250 5850 50  0000 C CNN

Commit message: wip
Parts:
- R1, R6, R7: footprint Resistors_SMD:R_0603_HandSoldering -> Resistors_SMD:R_0805_HandSoldering
- U3: symbol MCP2551-I/SN -> MCP2551-I/SN-RESCUE-SRSE2
Changed lines of the file:
@@
 F 0 "R6" V 4200 2900 50  0000 C CNN
 F 1 "3k3" V 4250 2750 50  0000 C CNN
-F 2 "Resistors_SMD:R_0603_HandSoldering" H 4180 2750 50  0001 C CNN
+F 2 "Resistors_SMD:R_0805_HandSoldering" H 4180 2750 50  0001 C CNN
 F 3 "" H 4250 2750 50  0000 C CNN
 	1    4250 2750
@@
 F 0 "R7" V 4350 2900 50  0000 C CNN
 F 1 "3k3" V 4400 2750 50  0000 C CNN
-F 2 "Resistors_SMD:R_0603_HandSoldering" H 4330 2750 50  0001 C CNN
+F 2 "Resistors_SMD:R_0805_HandSoldering" H 4330 2750 50  0001 C CNN
 F 3 "" H 4400 2750 50  0000 C CNN
 	1    4400 2750
@@
 F 0 "R1" V 2000 3500 50  0000 C CNN
 F 1 "10k" V 2050 3350 50  0000 C CNN
-F 2 "Resistors_SMD:R_0603_HandSoldering" H 1980 3350 50  0001 C CNN
+F 2 "Resistors_SMD:R_0805_HandSoldering" H 1980 3350 50  0001 C CNN
 F 3 "" H 2050 3350 50  0000 C CNN
 	1    2050 3350
@@
 S88_RESET
 $Comp
-L MCP2551-I/SN U3
+L MCP2551-I/SN-RESCUE-SRSE2 U3
 U 1 1 57C0B300
 P 5250 4900

Commit message: wip
Parts:
- removed P5: USB_B, w_conn_pc:conn_usb_B, symbol USB_B
- added C14: 100nF, Capacitors_SMD:C_0805_HandSoldering, symbol C
- added C15: 4uF7, Capacitors_SMD:C_0805_HandSoldering, symbol C
- added P13: CONN_01X03, Pin_Headers:Pin_Header_Straight_1x03, symbol CONN_01X03
- added P5: Grove, w_conn_jst-ph:s4b-ph-kl, symbol CONN_01X04
- added R22, R23: 10k, Resistors_SMD:R_0805_HandSoldering, symbol R
- added U7: FT230XS, w_smd_dil:ssop-16, symbol FT230XS
- R8: value 0 -> 10k
- U3, U6: footprint Power_Integrations:SO-8 -> w_smd_dil:so-8
- Y1: footprint Crystals:Crystal_HC49-U_Vertical -> w_crystal:crystal_hc-49s
Connections:
- net labels added: +24V, RxD2, TxD2
- wire segments 284 -> 320
- no-connect marks 11 -> 17
Other:
- moved on the sheet: C1, C2, P10, P11, P12, P9, R13, R14, R15, R21, U6

Commit message: wip
Parts:
- removed P4: UART, Pin_Headers:Pin_Header_Straight_1x03, symbol CONN_01X03
- added C16, C17, C19: 100nF, Capacitors_SMD:C_0805_HandSoldering, symbol C
- added C18: 10uF, Capacitors_ThroughHole:C_Radial_D5_L6_P2.5, symbol CP
- added CON?: BARREL_JACK, symbol BARREL_JACK
- added D4: 1N4148, w_smd_diode:melf, symbol D_Small
- added J? (x3): s88-N, w_conn_pc:megb8-8, symbol RJ45
- added P14, P16: CONN_01X04, Pin_Headers:Pin_Header_Straight_1x04, symbol CONN_01X04
- added P15, P17: opt 18V, Pin_Headers:Pin_Header_Straight_1x01, symbol CONN_01X01
- added P18: CONN_01X03, Pin_Headers:Pin_Header_Angled_1x03, symbol CONN_01X03
- added P19, P?: CONN_01X02, Pin_Headers:Pin_Header_Straight_1x02, symbol CONN_01X02
- added P4: CONN_01X04, w_conn_jst-ph:b4b-ph-kl, symbol CONN_01X04
- added P?: CONN_01X06, symbol CONN_01X06
- added R24: 1k, Resistors_SMD:R_1206_HandSoldering, symbol R
- added R25, R26: 27, Resistors_SMD:R_0805_HandSoldering, symbol R
- added U8: 4504, w_smd_dil:so-16, symbol 4504
- added U9: 7812, TO_SOT_Packages_SMD:TO-252-2Lead, symbol 7805
- added VR?: VR, w_pth_resistors:RC07, symbol VR
- J1: value S88 -> s88-N
- P5: value Grove -> UART
- P6, P8, P9: footprint Pin_Headers:Pin_Header_Straight_1x04 -> w_conn_jst-ph:b4b-ph-kl
- U3: value MCP2562-I/SN -> MCP2562
Connections:
- net labels added: Vdd, _S88_CLK, _S88_DATA, _S88_LOAD, _S88_RESET, br, rt
- wire segments 320 -> 472
- no-connect marks 17 -> 14
Other:
- moved on the sheet: C10, C11, C12, C13, C8, C9, J1, J2, P10, P13, P3, P5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

Commit message: wip
Parts:
- removed CON?: BARREL_JACK, symbol BARREL_JACK
- removed P?: CONN_01X02, Pin_Headers:Pin_Header_Straight_1x02, symbol CONN_01X02
- removed VR?: VR, w_pth_resistors:RC07, symbol VR
- added P20: CONN_01X02, w_conn_pt-1,5:pt_1,5-2-3,5-h, symbol CONN_01X02
- J4, J5: renamed from J?; value s88-N -> CAN
- P21: renamed from P?; footprint (none) -> Socket_Strips:Socket_Strip_Angled_1x06
- U2: value ADuM1250CR -> ADuM1250
- gave numbers to parts that had none: 1
Connections:
- net _Vcc_: now reaches J3.1
- net _Vcc_: now also P21.6 (P6), P20.2 (P2)
- net _DATA_: now reaches J3.2, P21.1 (P1)
- net _GND_: now reaches J3.3, J3.5, P21.2 (P2)
- net _GND_: now also P20.1 (P1)
- net _CLK_: now reaches J3.4, P21.3 (P3)
- net _LOAD_: now reaches J3.6, P21.4 (P4)
- net _RESET_: now reaches J3.7, P21.5 (P5)
