File: srse2/schablone.kicad_pcb (KiCad board)
At the start: 2 copper layers, 210.1 x 107.4 mm, 32 parts

Commit message: template wip
Other:
- board text added: "49,2 mm x 13,5 mm"
- board text added: "6,8 m m ----------- 13,5 mm ----------- 6,7 mm"
Changed lines of the file:
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@@
     (area 48.600001 49.924999 260.075001 157.475001)
     (thickness 1.6)
-    (drawings 26)
+    (drawings 28)
     (tracks 0)
     (zones 0)
@@
       (outputformat 1)
       (mirror false)
-      (drillshape 1)
+      (drillshape 0)
       (scaleselection 1)
       (outputdirectory ""))
@@
     (pad 1 thru_hole circle (at 0 0) (size 6 6) (drill 1) (layers *.Cu *.Mask))
   )
+  (gr_text " 6,8 m m\n-----------\n13,5 mm\n-----------\n6,7 mm" (at 130.7 144.3) (layer F.Cu)
+    (effects (font (size 1.5 1.5) (thickness 0.3)))
+  )
+  (gr_text "49,2 mm x 13,5 mm" (at 91.9 154.6) (layer F.Cu)
+    (effects (font (size 1.5 1.5) (thickness 0.3)))
+  )
   (dimension 13.2 (width 0.3) (layer Dwgs.User)
