File: mfx-link/mfx-link.sch (KiCad schematic (older format))
At the start: 18 parts, among them P1 CONN_01X02, P2 CONN_02X03, Q1 BC547, Q2 BC547, U1 LM393

Commit message: wip
Parts:
- removed U1: LM393, w_pth_circuits:dil_8-300_socket, symbol LM393
- added RR1: RR7, symbol RR7
- added U1: LM393-1, symbol LM393-1
- C1: value C -> 100nF
- D1, D2, D3, D4: footprint Discret:D4 -> w_pth_diodes:diode_do35
- TR1: footprint Choke_Common-Mode_Wurth:CommonModeChoke_WuerthType-WE-CMB_Size-L -> Choke_Axial_ThroughHole:Choke_Horizontal_RM25mm
Connections:
- wire segments 58 -> 59
Other:
- moved on the sheet: C1, D1, D2, D3, D4, P1, P2, Q1, Q2, R1, R2, R3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

Commit message: wip
Parts:
- removed RR1: RR7, symbol RR7
- added C?: 100nF, w_capacitors:cnp_7.5mm_disc, symbol C
- added C?: CP, symbol CP
- added D?: D, symbol D
- added D? (x4): 1N4007, w_pth_diodes:diode_do35, symbol D
- added P?: CONN_02X04, symbol CONN_02X04
- added P?: CONN_01X04, symbol CONN_01X04
- added R?: 4k7, w_pth_resistors:RC03, symbol R
- added RR?: RR7, symbol RR7
- added U?: 7805, symbol 7805
- added U?: PIC16F1705, MODULE, symbol PIC16F1705
Connections:
- net labels added: GNDA, SCL, SDA, VCC, VDD
- wire segments 59 -> 85

Commit message: wip
Parts:
- added C4: 100nF, w_capacitors:cnp_3mm_disc, symbol C
- added JP?: ICSP, ICSP:ICSP, symbol ICSP
- added P3: 5V DCD, w_pth_circuits:dcdc_sil4, symbol CONN_01X04
- added Q?: BC547, w_to:to92_3, symbol BC547
- added R? (x2): 1k, w_pth_resistors:RC03, symbol R
- added U?: 6N137, DIP-8, symbol 6N136
- C1: footprint w_capacitors:cnp_7.5mm_disc -> w_capacitors:cnp_3mm_disc
- C2: renamed from C?; footprint w_capacitors:cnp_7.5mm_disc -> w_capacitors:cnp_3mm_disc
- C3: renamed from C?; footprint (none) -> w_capacitors:CP_4x7mm
- D8: renamed from D?; footprint (none) -> w_pth_diodes:diode_do35
- P4: renamed from P?; value CONN_01X04 -> I2C; footprint (none) -> Pin_Headers:Pin_Header_Angled_1x04
- P5: renamed from P?; value CONN_02X04 -> IBT-2; footprint (none) -> Pin_Headers:Pin_Header_Straight_2x04
- RR1: renamed from RR?; footprint (none) -> w_pth_resistors:r-sil_8
- TR1: footprint Choke_Axial_ThroughHole:Choke_Horizontal_RM25mm -> Choke_Toroid_ThroughHole:Murata56000C
- U1: footprint (none) -> w_smd_dil:mdip_8
- U2: renamed from U?; footprint (none) -> w_to:to220_std
- U3: renamed from U?; footprint MODULE -> w_pth_circuits:dil_16-300_socket
- gave numbers to parts that had none: 5
Connections:
- net labels added: ENABLE, MCLR, PGC, PGD, SENSE
- wire segments 85 -> 123
- no-connect marks 0 -> 1

Commit message: wip
Parts:
- removed P3: 5V DCD, w_pth_circuits:dcdc_sil4, symbol CONN_01X04
- added C5, C6: 100nF, w_capacitors:cnp_3mm_disc, symbol C
- added D10: 1N4148, w_pth_diodes:diode_do35, symbol D
- added D11: LED, LEDs:LED-3MM, symbol LED
- added P3: CONN_01X02, Pin_Headers:Pin_Header_Straight_1x02, symbol CONN_01X02
- added P6: CONN_01X02, w_conn_pt-1,5:pt_1,5-2-3,5-h, symbol CONN_01X02
- added P7: CONN_01X03, Pin_Headers:Pin_Header_Straight_1x03, symbol CONN_01X03
- added Q4: BC547, w_to:to92_3, symbol BC547
- added R12, R13, R14: 4k7, w_pth_resistors:RC03, symbol R
- added R15: 10k, w_pth_resistors:RC03, symbol R
- added R9: 1k5, w_pth_resistors:RC03, symbol R
- added U5: 7805, w_to:to220_std, symbol 7805
- P4: value I2C -> Grove I2C
- gave numbers to parts that had none: 5
Connections:
- net labels added: PULSE, boost_1, boost_2, brown, red
- wire segments 123 -> 178
- no-connect marks 1 -> 4
Other:
- moved on the sheet: C1, C2, C3, D1, D2, D3, D4, D5, D6, D7, D8, D9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

Commit message: wip
Parts:
- P4: footprint Pin_Headers:Pin_Header_Angled_1x04 -> w_conn_jst-ph:b4b-ph-kl
- U1: footprint w_smd_dil:mdip_8 -> w_pth_circuits:dil_8-300_socket
- U2, U5: footprint w_to:to220_std -> 78xx:to220
- U4: footprint DIP-8 -> w_pth_circuits:dil_8-300_socket
Changed lines of the file:
@@
 F 0 "U1" H 4550 6050 50  0000 C CNN
 F 1 "LM393-1" H 4500 5700 50  0000 C CNN
-F 2 "w_smd_dil:mdip_8" H 4400 5900 50  0001 C CNN
+F 2 "w_pth_circuits:dil_8-300_socket" H 4400 5900 50  0001 C CNN
 F 3 "" H 4400 5900 50  0000 C CNN
 	1    4400 5900
@@
 F 0 "U2" H 3000 4504 50  0000 C CNN
 F 1 "7805" H 2850 4900 50  0000 C CNN
-F 2 "w_to:to220_std" H 2850 4700 50  0001 C CNN
+F 2 "78xx:to220" H 2850 4700 50  0001 C CNN
 F 3 "" H 2850 4700 50  0000 C CNN
 	1    2850 4700
@@
 F 0 "P4" H 7350 3050 50  0000 C CNN
 F 1 "Grove I2C" V 7450 2800 50  0000 C CNN
-F 2 "Pin_Headers:Pin_Header_Angled_1x04" H 7350 2800 50  0001 C CNN
+F 2 "w_conn_jst-ph:b4b-ph-kl" H 7350 2800 50  0001 C CNN
 F 3 "" H 7350 2800 50  0000 C CNN
 	1    7350 2800
@@
 F 0 "U4" H 6300 1800 50  0000 L CNN
 F 1 "6N137" H 6500 1800 50  0000 L CNN
-F 2 "DIP-8" H 6300 1200 50  0000 L CIN
+F 2 "w_pth_circuits:dil_8-300_socket" H 6300 1200 50  0001 L CIN
 F 3 "" H 6500 1500 50  0000 L CNN
 	1    6500 1500
@@
 F 0 "U5" H 3300 1704 50  0000 C CNN
 F 1 "7805" H 3150 2100 50  0000 C CNN
-F 2 "w_to:to220_std" H 3150 1900 50  0001 C CNN
+F 2 "78xx:to220" H 3150 1900 50  0001 C CNN
 F 3 "" H 3150 1900 50  0000 C CNN
 	1    3150 1900

Commit message: wip
Parts:
- added D12: BAT43, w_pth_diodes:diode_do35, symbol D_Schottky
- added P8: Grove UART, w_conn_jst-ph:b4b-ph-kl, symbol CONN_01X04
- added SW1: SW_PUSH, Buttons_Switches_ThroughHole:SW_PUSH_SMALL, symbol SW_PUSH
Connections:
- net labels added: RxD, TxD
- wire segments 178 -> 189
- no-connect marks 4 -> 2
Other:
- moved on the sheet: C6, D10, D11, P4, Q4, R12, R13, R14, R8, R9, U4

Commit message: wip
Parts:
- R14: value 4k7 -> 1k5
Connections:
- wire segments 189 -> 188
Changed lines of the file:
@@
 	-1   0    0    1
-$EndComp
-Wire Wire Line
-	10150 1850 10150 2200
-$Comp
-L VDD #PWR023
-U 1 1 5892F635
-P 10150 1850
-F 0 "#PWR023" H 10150 1700 50  0001 C CNN
-F 1 "VDD" H 10150 2000 50  0000 C CNN
-F 2 "" H 10150 1850 50  0000 C CNN
-F 3 "" H 10150 1850 50  0000 C CNN
-	1    10150 1850
-	1    0    0    -1
 $EndComp
 Text Label 8000 2850 0    60   ~ 0
@@
 P 7700 2000
 F 0 "R14" V 7780 2000 50  0000 C CNN
-F 1 "4k7" V 7700 2000 50  0000 C CNN
+F 1 "1k5" V 7700 2000 50  0000 C CNN
 F 2 "w_pth_resistors:RC03" V 7630 2000 50  0001 C CNN
 F 3 "" H 7700 2000 50  0000 C CNN

Commit message: wip
Parts:
- removed Q4: BC547, w_to:to92_3, symbol BC547
- removed R13: 4k7, w_pth_resistors:RC03, symbol R
Connections:
- wire segments 188 -> 183
Other:
- moved on the sheet: P4
Changed lines of the file:
@@
 L CONN_01X04 P4
 U 1 1 5890E270
-P 7250 2800
-F 0 "P4" H 7250 3050 50  0000 C CNN
-F 1 "Grove I2C" V 7350 2800 50  0000 C CNN
-F 2 "w_conn_jst-ph:b4b-ph-kl" H 7250 2800 50  0001 C CNN
-F 3 "" H 7250 2800 50  0000 C CNN
-	1    7250 2800
+P 7200 2800
+F 0 "P4" H 7200 3050 50  0000 C CNN
+F 1 "Grove I2C" V 7300 2800 50  0000 C CNN
+F 2 "w_conn_jst-ph:b4b-ph-kl" H 7200 2800 50  0001 C CNN
+F 3 "" H 7200 2800 50  0000 C CNN
+	1    7200 2800
 	-1   0    0    1
 $EndComp
@@
 L GNDA #PWR06
 U 1 1 5890E3A7
-P 7550 3050
-F 0 "#PWR06" H 7550 2800 50  0001 C CNN
-F 1 "GNDA" H 7550 2900 50  0000 C CNN
-F 2 "" H 7550 3050 50  0000 C CNN
-F 3 "" H 7550 3050 50  0000 C CNN
-	1    7550 3050
+P 7450 3050
+F 0 "#PWR06" H 7450 2800 50  0001 C CNN
+F 1 "GNDA" H 7450 2900 50  0000 C CNN
+F 2 "" H 7450 3050 50  0000 C CNN
+F 3 "" H 7450 3050 50  0000 C CNN
+	1    7450 3050
 	1    0    0    -1
 $EndComp
@@
 L VDD #PWR07
 U 1 1 5890E581
-P 7550 2300
-F 0 "#PWR07" H 7550 2150 50  0001 C CNN
-F 1 "VDD" H 7550 2450 50  0000 C CNN
-F 2 "" H 7550 2300 50  0000 C CNN
-F 3 "" H 7550 2300 50  0000 C CNN
-	1    7550 2300
+P 7450 2300
+F 0 "#PWR07" H 7450 2150 50  0001 C CNN
+F 1 "VDD" H 7450 2450 50  0000 C CNN
+F 2 "" H 7450 2300 50  0000 C CNN
+F 3 "" H 7450 2300 50  0000 C CNN
+	1    7450 2300
 	1    0    0    -1
 $EndComp
@@
 Text Label 9500 5650 0    60   ~ 0
 SENSE
-Text Label 7850 3050 0    60   ~ 0
+Text Label 7900 3050 0    60   ~ 0
 ENABLE
 $Comp
@@
 	4100 6000 4000 6000
 Wire Wire Line
-	4000 6000 4000 6100
+	4000 6100 4000 6000
 Wire Wire Line
 	3900 6050 3900 6200
@@
 Connection ~ 2950 6100
 Wire Wire Line
-	4000 6100 2800 6100
+	2800 6100 4000 6100
 Wire Wire Line
 	3900 6500 5900 6500
@@
 Connection ~ 3100 5150
 Wire Wire Line
-	7450 2950 7550 2950
-Wire Wire Line
-	7550 2950 7550 3050
-Wire Wire Line
-	7550 2850 7450 2850
-Wire Wire Line
-	7550 2300 7550 2850
-Wire Wire Line
-	7450 2750 8150 2750
-Wire Wire Line
-	7450 2650 8150 2650
+	7400 2950 7450 2950
+Wire Wire Line
+	7450 2950 7450 3050
+Wire Wire Line
+	7450 2850 7400 2850
+Wire Wire Line
+	7450 2300 7450 2850
+Wire Wire Line
+	7400 2750 8150 2750
+Wire Wire Line
+	7400 2650 8150 2650
 Wire Wire Line
 	8900 3700 8900 3800
@@
 Connection ~ 6550 1400
 Wire Wire Line
-	6400 1700 6750 1700
+	6400 1700 7200 1700
 Wire Wire Line
 	6700 1700 6700 1600
@@
 	5200 4100 2700 4100
 Wire Wire Line
-	2700 4100 2700 4350
-Wire Wire Line
-	2700 4350 1900 4350
+	2700 4350 2700 4100
+Wire Wire Line
+	1900 4350 2700 4350
 Wire Wire Line
 	1900 4200 1900 4650
@@
 	6700 1250 6700 1300
 Connection ~ 6550 1250
-$Comp
-L BC547 Q4
-U 1 1 5892B631
-P 6950 1700
-F 0 "Q4" H 7150 1775 50  0000 L CNN
-F 1 "BC547" H 7150 1700 50  0000 L CNN
-F 2 "w_to:to92_3" H 7150 1625 50  0001 L CIN
-F 3 "" H 6950 1700 50  0000 L CNN
-	1    6950 1700
-	1    0    0    -1
-$EndComp
 Connection ~ 6700 1700
-$Comp
-L R R13
-U 1 1 5892BF41
-P 7050 1250
-F 0 "R13" V 7130 1250 50  0000 C CNN
-F 1 "4k7" V 7050 1250 50  0000 C CNN
-F 2 "w_pth_resistors:RC03" V 6980 1250 50  0001 C CNN
-F 3 "" H 7050 1250 50  0000 C CNN
-	1    7050 1250
-	-1   0    0    1
-$EndComp
-Wire Wire Line
-	7050 1400 7050 1500
-Wire Wire Line
-	7050 1100 7050 1050
-Wire Wire Line
-	7050 1050 6550 1050
-Connection ~ 6550 1050
-$Comp
-L GNDA #PWR022
-U 1 1 5892C228
-P 7050 2000
-F 0 "#PWR022" H 7050 1750 50  0001 C CNN
-F 1 "GNDA" H 7050 1850 50  0000 C CNN
-F 2 "" H 7050 2000 50  0000 C CNN
-F 3 "" H 7050 2000 50  0000 C CNN
-	1    7050 2000
-	1    0    0    -1
-$EndComp
-Wire Wire Line
-	7050 1900 7050 2000
-Wire Wire Line
-	7050 1450 7450 1450
-Connection ~ 7050 1450
 $Comp
 L CONN_01X03 P7
@@
 Wire Wire Line
 	9850 4650 9850 5100
-Text Label 7200 1450 0    60   ~ 0
+Text Label 6900 1700 0    60   ~ 0
 PULSE
 Text Label 8650 5100 0    60   ~ 0
@@
 $EndComp
 $Comp
-L VDD #PWR024
+L VDD #PWR022
 U 1 1 5893057F
 P 7700 1800
-F 0 "#PWR024" H 7700 1650 50  0001 C CNN
+F 0 "#PWR022" H 7700 1650 50  0001 C CNN
 F 1 "VDD" H 7700 1950 50  0000 C CNN
 F 2 "" H 7700 1800 50  0000 C CNN
@@
 	8200 5100 8150 5100
 $Comp
-L VDD #PWR025
+L VDD #PWR023
 U 1 1 589322F2
 P 10350 2550
-F 0 "#PWR025" H 10350 2400 50  0001 C CNN
+F 0 "#PWR023" H 10350 2400 50  0001 C CNN
 F 1 "VDD" H 10350 2700 50  0000 C CNN
 F 2 "" H 10350 2550 50  0000 C CNN
@@
 $EndComp
 $Comp
-L GNDA #PWR026
+L GNDA #PWR024
 U 1 1 58932648
 P 10350 3150
-F 0 "#PWR026" H 10350 2900 50  0001 C CNN
+F 0 "#PWR024" H 10350 2900 50  0001 C CNN
 F 1 "GNDA" H 10350 3000 50  0000 C CNN
 F 2 "" H 10350 3150 50  0000 C CNN
@@
 	10350 2950 10350 3150
 $Comp
-L GNDA #PWR027
+L GNDA #PWR025
 U 1 1 58932E12
 P 10150 3650
-F 0 "#PWR027" H 10150 3400 50  0001 C CNN
+F 0 "#PWR025" H 10150 3400 50  0001 C CNN
 F 1 "GNDA" H 10150 3500 50  0000 C CNN
 F 2 "" H 10150 3650 50  0000 C CNN
@@
 $EndComp
 $Comp
-L GNDA #PWR028
+L GNDA #PWR026
 U 1 1 5893744C
 P 10600 4150
-F 0 "#PWR028" H 10600 3900 50  0001 C CNN
+F 0 "#PWR026" H 10600 3900 50  0001 C CNN
 F 1 "GNDA" H 10600 4000 50  0000 C CNN
 F 2 "" H 10600 4150 50  0000 C CNN
@@
 $EndComp
 $Comp
-L VDD #PWR029
+L VDD #PWR027
 U 1 1 58937D09
 P 10600 3700
-F 0 "#PWR029" H 10600 3550 50  0001 C CNN
+F 0 "#PWR027" H 10600 3550 50  0001 C CNN
 F 1 "VDD" H 10600 3850 50  0000 C CNN
 F 2 "" H 10600 3700 50  0000 C CNN
@@
 $EndComp
 $Comp
-L GNDA #PWR030
+L GNDA #PWR028
 U 1 1 5893AE37
 P 8650 2150
-F 0 "#PWR030" H 8650 1900 50  0001 C CNN
+F 0 "#PWR028" H 8650 1900 50  0001 C CNN
 F 1 "GNDA" H 8650 2000 50  0000 C CNN
 F 2 "" H 8650 2150 50  0000 C CNN
