File: mfx-link/mfx-link.sch (KiCad schematic (older format))
At the start: 52 parts, among them P1 CONN_01X02, P2 CONN_02X03, P3 CONN_01X02, P4 Grove I2C, P5 IBT-2, P6 CONN_01X02, P7 CONN_01X03, P8 Grove UART, Q1 BC547, Q2 BC547, Q3 BC547, SW1 SW_PUSH, U1 LM393-1, U2 7805, U3 PIC16F1705, U4 6N137, U5 7805

Commit message: start routing
Parts:
- added P9: MFX, Pin_Headers:Pin_Header_Straight_1x02, symbol CONN_01X02
Connections:
- wire segments 183 -> 186
Other:
- moved on the sheet: C5, C6, D10, P6, R12, R9, U4, U5

Commit message: rework
Parts:
- U2, U5: footprint 78xx:to220 -> TO_SOT_Packages_THT:TO-220_Neutral123_Vertical_LargePads
- U3: footprint w_pth_circuits:dil_16-300_socket -> w_pth_circuits:dil_14-300_socket
Changed lines of the file:
@@
 $EndComp
 $Comp
-L GND #PWR5
+L GND #PWR01
 U 1 1 586FBEF9
 P 4300 6650
-F 0 "#PWR5" H 4300 6400 50  0001 C CNN
+F 0 "#PWR01" H 4300 6400 50  0001 C CNN
 F 1 "GND" H 4300 6500 50  0000 C CNN
 F 2 "" H 4300 6650 50  0000 C CNN
@@
 F 0 "U2" H 3000 4504 50  0000 C CNN
 F 1 "7805" H 2850 4900 50  0000 C CNN
-F 2 "78xx:to220" H 2850 4700 50  0001 C CNN
+F 2 "TO_SOT_Packages_THT:TO-220_Neutral123_Vertical_LargePads" H 2850 4700 50  0001 C CNN
 F 3 "" H 2850 4700 50  0000 C CNN
 	1    2850 4700
@@
 $EndComp
 $Comp
-L GND #PWR1
+L GND #PWR02
 U 1 1 5890D0A3
 P 2850 5300
-F 0 "#PWR1" H 2850 5050 50  0001 C CNN
+F 0 "#PWR02" H 2850 5050 50  0001 C CNN
 F 1 "GND" H 2850 5150 50  0000 C CNN
 F 2 "" H 2850 5300 50  0000 C CNN
@@
 $EndComp
 $Comp
-L VCC #PWR3
+L VCC #PWR03
 U 1 1 5890D155
 P 3350 4400
-F 0 "#PWR3" H 3350 4250 50  0001 C CNN
+F 0 "#PWR03" H 3350 4250 50  0001 C CNN
 F 1 "VCC" H 3350 4550 50  0000 C CNN
 F 2 "" H 3350 4400 50  0000 C CNN
@@
 $EndComp
 $Comp
-L PWR_FLAG #FLG2
+L PWR_FLAG #FLG04
 U 1 1 5890D427
 P 3700 4450
-F 0 "#FLG2" H 3700 4545 50  0001 C CNN
+F 0 "#FLG04" H 3700 4545 50  0001 C CNN
 F 1 "PWR_FLAG" H 3700 4630 50  0000 C CNN
 F 2 "" H 3700 4450 50  0000 C CNN
@@
 $EndComp
 $Comp
-L PWR_FLAG #FLG1
+L PWR_FLAG #FLG05
 U 1 1 5890D50F
 P 3350 5500
-F 0 "#FLG1" H 3350 5595 50  0001 C CNN
+F 0 "#FLG05" H 3350 5595 50  0001 C CNN
 F 1 "PWR_FLAG" H 3350 5680 50  0000 C CNN
 F 2 "" H 3350 5500 50  0000 C CNN
@@
 $EndComp
 $Comp
-L GNDA #PWR9
+L GNDA #PWR06
 U 1 1 5890E3A7
 P 7450 3050
-F 0 "#PWR9" H 7450 2800 50  0001 C CNN
+F 0 "#PWR06" H 7450 2800 50  0001 C CNN
 F 1 "GNDA" H 7450 2900 50  0000 C CNN
 F 2 "" H 7450 3050 50  0000 C CNN
@@
 $EndComp
 $Comp
-L VDD #PWR8
+L VDD #PWR07
 U 1 1 5890E581
 P 7450 2300
-F 0 "#PWR8" H 7450 2150 50  0001 C CNN
+F 0 "#PWR07" H 7450 2150 50  0001 C CNN
 F 1 "VDD" H 7450 2450 50  0000 C CNN
 F 2 "" H 7450 2300 50  0000 C CNN
@@
 SDA
 $Comp
-L GNDA #PWR15
+L GNDA #PWR08
 U 1 1 5890F719
 P 8900 3800
-F 0 "#PWR15" H 8900 3550 50  0001 C CNN
+F 0 "#PWR08" H 8900 3550 50  0001 C CNN
 F 1 "GNDA" H 8900 3650 50  0000 C CNN
 F 2 "" H 8900 3800 50  0000 C CNN
@@
 F 0 "U3" H 8900 2800 50  0000 C CNN
 F 1 "PIC16F1705" H 8900 2700 50  0000 C CNN
-F 2 "w_pth_circuits:dil_16-300_socket" H 8350 2300 50  0001 C CNN
+F 2 "w_pth_circuits:dil_14-300_socket" H 8350 2300 50  0001 C CNN
 F 3 "DOCUMENTATION" H 8500 2200 50  0001 C CNN
 	1    8900 2900
@@
 $EndComp
 $Comp
-L VDD #PWR14
+L VDD #PWR09
 U 1 1 58910635
 P 8900 2000
-F 0 "#PWR14" H 8900 1850 50  0001 C CNN
+F 0 "#PWR09" H 8900 1850 50  0001 C CNN
 F 1 "VDD" H 8900 2150 50  0000 C CNN
 F 2 "" H 8900 2000 50  0000 C CNN
@@
 $EndComp
 $Comp
-L VDD #PWR12
+L VDD #PWR010
 U 1 1 5891152D
 P 7950 1200
-F 0 "#PWR12" H 7950 1050 50  0001 C CNN
+F 0 "#PWR010" H 7950 1050 50  0001 C CNN
 F 1 "VDD" H 7950 1350 50  0000 C CNN
 F 2 "" H 7950 1200 50  0000 C CNN
@@
 $EndComp
 $Comp
-L VDD #PWR17
+L VDD #PWR011
 U 1 1 5891F45B
 P 9750 1850
-F 0 "#PWR17" H 9750 1700 50  0001 C CNN
+F 0 "#PWR011" H 9750 1700 50  0001 C CNN
 F 1 "VDD" H 9750 2000 50  0000 C CNN
 F 2 "" H 9750 1850 50  0000 C CNN
@@
 $EndComp
 $Comp
-L GNDA #PWR18
+L GNDA #PWR012
 U 1 1 5891F4CC
 P 9750 2300
-F 0 "#PWR18" H 9750 2050 50  0001 C CNN
+F 0 "#PWR012" H 9750 2050 50  0001 C CNN
 F 1 "GNDA" H 9750 2150 50  0000 C CNN
 F 2 "" H 9750 2300 50  0000 C CNN
@@
 $EndComp
 $Comp
-L GNDA #PWR11
+L GNDA #PWR013
 U 1 1 589209D0
 P 7850 5700
-F 0 "#PWR11" H 7850 5450 50  0001 C CNN
+F 0 "#PWR013" H 7850 5450 50  0001 C CNN
 F 1 "GNDA" H 7850 5550 50  0000 C CNN
 F 2 "" H 7850 5700 50  0000 C CNN
@@
 ENABLE
 $Comp
-L GNDA #PWR20
+L GNDA #PWR014
 U 1 1 589214FB
 P 10200 5700
-F 0 "#PWR20" H 10200 5450 50  0001 C CNN
+F 0 "#PWR014" H 10200 5450 50  0001 C CNN
 F 1 "GNDA" H 10200 5550 50  0000 C CNN
 F 2 "" H 10200 5700 50  0000 C CNN
@@
 $EndComp
 $Comp
-L VDD #PWR16
+L VDD #PWR015
 U 1 1 5892163B
 P 9000 4950
-F 0 "#PWR16" H 9000 4800 50  0001 C CNN
+F 0 "#PWR015" H 9000 4800 50  0001 C CNN
 F 1 "VDD" H 9000 5100 50  0000 C CNN
 F 2 "" H 9000 4950 50  0000 C CNN
@@
 F 0 "U5" H 5400 1404 50  0000 C CNN
 F 1 "7805" H 5250 1800 50  0000 C CNN
-F 2 "78xx:to220" H 5250 1600 50  0001 C CNN
+F 2 "TO_SOT_Packages_THT:TO-220_Neutral123_Vertical_LargePads" H 5250 1600 50  0001 C CNN
 F 3 "" H 5250 1600 50  0000 C CNN
 	1    5250 1600
@@
 $EndComp
 $Comp
-L GNDA #PWR2
+L GNDA #PWR016
 U 1 1 5892345E
 P 5250 2100
-F 0 "#PWR2" H 5250 1850 50  0001 C CNN
+F 0 "#PWR016" H 5250 1850 50  0001 C CNN
 F 1 "GNDA" H 5250 1950 50  0000 C CNN
 F 2 "" H 5250 2100 50  0000 C CNN
@@
 $EndComp
 $Comp
-L VDD #PWR4
+L VDD #PWR017
 U 1 1 589234E4
 P 5750 1400
-F 0 "#PWR4" H 5750 1250 50  0001 C CNN
+F 0 "#PWR017" H 5750 1250 50  0001 C CNN
 F 1 "VDD" H 5750 1550 50  0000 C CNN
 F 2 "" H 5750 1400 50  0000 C CNN
@@
 $EndComp
 $Comp
-L PWR_FLAG #FLG3
+L PWR_FLAG #FLG018
 U 1 1 5892374C
 P 6150 1450
-F 0 "#FLG3" H 6150 1545 50  0001 C CNN
+F 0 "#FLG018" H 6150 1545 50  0001 C CNN
 F 1 "PWR_FLAG" H 6150 1630 50  0000 C CNN
 F 2 "" H 6150 1450 50  0000 C CNN
@@
 $EndComp
 $Comp
-L PWR_FLAG #FLG4
+L PWR_FLAG #FLG019
 U 1 1 589238E7
 P 6150 1900
-F 0 "#FLG4" H 6150 1995 50  0001 C CNN
+F 0 "#FLG019" H 6150 1995 50  0001 C CNN
 F 1 "PWR_FLAG" H 6150 2080 50  0000 C CNN
 F 2 "" H 6150 1900 50  0000 C CNN
@@
 boost_1
 $Comp
-L VDD #PWR6
+L VDD #PWR020
 U 1 1 58926B3B
 P 2950 1050
-F 0 "#PWR6" H 2950 900 50  0001 C CNN
+F 0 "#PWR020" H 2950 900 50  0001 C CNN
 F 1 "VDD" H 2950 1200 50  0000 C CNN
 F 2 "" H 2950 1050 50  0000 C CNN
@@
 $EndComp
 $Comp
-L GNDA #PWR7
+L GNDA #PWR021
 U 1 1 58926BCD
 P 2950 2100
-F 0 "#PWR7" H 2950 1850 50  0001 C CNN
+F 0 "#PWR021" H 2950 1850 50  0001 C CNN
 F 1 "GNDA" H 2950 1950 50  0000 C CNN
 F 2 "" H 2950 2100 50  0000 C CNN
@@
 $EndComp
 $Comp
-L VDD #PWR10
+L VDD #PWR022
 U 1 1 5893057F
 P 7700 1800
-F 0 "#PWR10" H 7700 1650 50  0001 C CNN
+F 0 "#PWR022" H 7700 1650 50  0001 C CNN
 F 1 "VDD" H 7700 1950 50  0000 C CNN
 F 2 "" H 7700 1800 50  0000 C CNN
@@
 	8200 5100 8150 5100
 $Comp
-L VDD #PWR21
+L VDD #PWR023
 U 1 1 589322F2
 P 10350 2550
-F 0 "#PWR21" H 10350 2400 50  0001 C CNN
+F 0 "#PWR023" H 10350 2400 50  0001 C CNN
 F 1 "VDD" H 10350 2700 50  0000 C CNN
 F 2 "" H 10350 2550 50  0000 C CNN
@@
 $EndComp
 $Comp
-L GNDA #PWR22
+L GNDA #PWR024
 U 1 1 58932648
 P 10350 3150
-F 0 "#PWR22" H 10350 2900 50  0001 C CNN
+F 0 "#PWR024" H 10350 2900 50  0001 C CNN
 F 1 "GNDA" H 10350 3000 50  0000 C CNN
 F 2 "" H 10350 3150 50  0000 C CNN
@@
 	10350 2950 10350 3150
 $Comp
-L GNDA #PWR19
+L GNDA #PWR025
 U 1 1 58932E12
 P 10150 3650
-F 0 "#PWR19" H 10150 3400 50  0001 C CNN
+F 0 "#PWR025" H 10150 3400 50  0001 C CNN
 F 1 "GNDA" H 10150 3500 50  0000 C CNN
 F 2 "" H 10150 3650 50  0000 C CNN
@@
 $EndComp
 $Comp
-L GNDA #PWR24
+L GNDA #PWR026
 U 1 1 5893744C
 P 10600 4150
-F 0 "#PWR24" H 10600 3900 50  0001 C CNN
+F 0 "#PWR026" H 10600 3900 50  0001 C CNN
 F 1 "GNDA" H 10600 4000 50  0000 C CNN
 F 2 "" H 10600 4150 50  0000 C CNN
@@
 $EndComp
 $Comp
-L VDD #PWR23
+L VDD #PWR027
 U 1 1 58937D09
 P 10600 3700
-F 0 "#PWR23" H 10600 3550 50  0001 C CNN
+F 0 "#PWR027" H 10600 3550 50  0001 C CNN
 F 1 "VDD" H 10600 3850 50  0000 C CNN
 F 2 "" H 10600 3700 50  0000 C CNN
@@
 $EndComp
 $Comp
-L GNDA #PWR13
+L GNDA #PWR028
 U 1 1 5893AE37
 P 8650 2150
-F 0 "#PWR13" H 8650 1900 50  0001 C CNN
+F 0 "#PWR028" H 8650 1900 50  0001 C CNN
 F 1 "GNDA" H 8650 2000 50  0000 C CNN
 F 2 "" H 8650 2150 50  0000 C CNN

Commit message: optimize placement
Parts:
- C1, C2, C4, C5, C6: footprint w_capacitors:cnp_3mm_disc -> Capacitors_ThroughHole:C_Disc_D3_P2.5
- P3: footprint Pin_Headers:Pin_Header_Straight_1x02 -> w_conn_pt-1,5:pt_1,5-2-3,5-h
Connections:
- net labels added: VI, VO
Other:
- moved on the sheet: D6
Changed lines of the file:
@@
 F 0 "C1" H 3425 6000 50  0000 L CNN
 F 1 "100nF" H 3425 5800 50  0000 L CNN
-F 2 "w_capacitors:cnp_3mm_disc" H 3438 5750 50  0001 C CNN
+F 2 "Capacitors_ThroughHole:C_Disc_D3_P2.5" H 3438 5750 50  0001 C CNN
 F 3 "" H 3400 5900 50  0000 C CNN
 	1    3400 5900
@@
 F 0 "C2" H 2375 5050 50  0000 L CNN
 F 1 "100nF" H 2375 4850 50  0000 L CNN
-F 2 "w_capacitors:cnp_3mm_disc" H 2388 4800 50  0001 C CNN
+F 2 "Capacitors_ThroughHole:C_Disc_D3_P2.5" H 2388 4800 50  0001 C CNN
 F 3 "" H 2350 4950 50  0000 C CNN
 	1    2350 4950
@@
 U 1 1 5890D6E1
 P 1900 4050
-F 0 "D5" H 1800 4000 50  0000 C CNN
+F 0 "D5" H 2000 4000 50  0000 C CNN
 F 1 "1N4007" H 1900 4150 50  0000 C CNN
 F 2 "w_pth_diodes:diode_do35" H 1900 4050 50  0001 C CNN
@@
 L D D6
 U 1 1 5890D779
-P 2150 4050
-F 0 "D6" H 2050 4000 50  0000 C CNN
-F 1 "1N4007" H 2150 4150 50  0000 C CNN
-F 2 "w_pth_diodes:diode_do35" H 2150 4050 50  0001 C CNN
-F 3 "" H 2150 4050 50  0000 C CNN
-	1    2150 4050
+P 2100 4050
+F 0 "D6" H 2200 4075 50  0000 C CNN
+F 1 "1N4007" H 2100 3950 50  0000 C CNN
+F 2 "w_pth_diodes:diode_do35" H 2100 4050 50  0001 C CNN
+F 3 "" H 2100 4050 50  0000 C CNN
+	1    2100 4050
 	0    -1   -1   0
 $EndComp
@@
 U 1 1 5890D818
 P 1400 4050
-F 0 "D7" H 1300 4000 50  0000 C CNN
-F 1 "1N4007" H 1400 4150 50  0000 C CNN
+F 0 "D7" H 1300 4100 50  0000 C CNN
+F 1 "1N4007" H 1400 3950 50  0000 C CNN
 F 2 "w_pth_diodes:diode_do35" H 1400 4050 50  0001 C CNN
 F 3 "" H 1400 4050 50  0000 C CNN
@@
 F 0 "C4" H 9775 2150 50  0000 L CNN
 F 1 "100nF" H 9775 1950 50  0000 L CNN
-F 2 "w_capacitors:cnp_3mm_disc" H 9788 1900 50  0001 C CNN
+F 2 "Capacitors_ThroughHole:C_Disc_D3_P2.5" H 9788 1900 50  0001 C CNN
 F 3 "" H 9750 2050 50  0000 C CNN
 	1    9750 2050
@@
 F 0 "C6" H 5775 1850 50  0000 L CNN
 F 1 "100nF" H 5775 1650 50  0000 L CNN
-F 2 "w_capacitors:cnp_3mm_disc" H 5788 1600 50  0001 C CNN
+F 2 "Capacitors_ThroughHole:C_Disc_D3_P2.5" H 5788 1600 50  0001 C CNN
 F 3 "" H 5750 1750 50  0000 C CNN
 	1    5750 1750
@@
 F 0 "C5" H 4825 1850 50  0000 L CNN
 F 1 "100nF" H 4825 1650 50  0000 L CNN
-F 2 "w_capacitors:cnp_3mm_disc" H 4838 1600 50  0001 C CNN
+F 2 "Capacitors_ThroughHole:C_Disc_D3_P2.5" H 4838 1600 50  0001 C CNN
 F 3 "" H 4800 1750 50  0000 C CNN
 	1    4800 1750
@@
 P 950 3500
 F 0 "P3" H 950 3650 50  0000 C CNN
-F 1 "CONN_01X02" V 1050 3500 50  0000 C CNN
-F 2 "Pin_Headers:Pin_Header_Straight_1x02" H 950 3500 50  0001 C CNN
+F 1 "CONN_01X02" V 1050 3500 50  0001 C CNN
+F 2 "w_conn_pt-1,5:pt_1,5-2-3,5-h" H 950 3500 50  0001 C CNN
 F 3 "" H 950 3500 50  0000 C CNN
 	1    950  3500
@@
 	1350 1650 1100 1650
 Wire Wire Line
-	1150 3450 2150 3450
+	1150 3450 2100 3450
 Wire Wire Line
 	1150 3550 1900 3550
@@
 	1900 4200 1900 4650
 Wire Wire Line
-	2150 4200 2150 4350
-Connection ~ 2150 4350
+	2100 4200 2100 4350
+Connection ~ 2100 4350
 Connection ~ 1900 4350
 Wire Wire Line
@@
 	1900 3550 1900 3900
 Wire Wire Line
-	2150 3450 2150 3900
+	2100 3450 2100 3900
 Wire Wire Line
 	1600 4200 1600 5150
@@
 	4750 6400 4750 6500
 Connection ~ 4750 6500
+Text Label 4825 1550 0    60   ~ 0
+VI
+Text Label 5700 1550 2    60   ~ 0
+VO
 $EndSCHEMATC

Commit message: wip
Connections:
- net labels added: GVI, GVO
Changed lines of the file:
@@
 Text Label 5700 1550 2    60   ~ 0
 VO
+Text Label 2350 4650 0    60   ~ 0
+GVI
+Text Label 3275 4650 2    60   ~ 0
+GVO
 $EndSCHEMATC
