File: mfx-link/mfx-link.kicad_pcb (KiCad board)
At the start: 2 copper layers, 50 x 50 mm, 22 parts, among them P1 CONN_01X02, P2 CONN_02X03, Q1 BC547, Q2 BC547, U1 LM393

Commit message: wip
Parts:
- added C2, C4: 100nF, w_capacitors:cnp_3mm_disc, F.Cu at (120.0, 140.1)
- added C3: CP, w_capacitors:CP_4x5mm, F.Cu at (112.0, 98.5)
- added D5, D6, D7, D9: 1N4007, w_pth_diodes:diode_do35, F.Cu at (120.0, 140.1)
- added D8: D, w_pth_diodes:diode_do35, F.Cu at (120.0, 140.1)
- added P3: 5V DCD, w_pth_circuits:dcdc_sil4, F.Cu at (124.0, 100.5)
- added P4: I2C, Pin_Headers:Pin_Header_Angled_1x04, F.Cu at (136.0, 89.0)
- added P5: CONN_02X04, Pin_Headers:Pin_Header_Straight_2x04, F.Cu at (99.0, 99.0)
- added R8: 4k7, w_pth_resistors:RC03, F.Cu at (120.0, 140.1)
- added RR1: RR7, w_pth_resistors:r-sil_8, F.Cu at (141.5, 108.5)
- added U2: 7805, w_to:to220_std, F.Cu at (106.5, 90.0)
- added U3: PIC16F1705, w_pth_circuits:dil_16-300_socket, F.Cu at (123.5, 88.0)
- C1: value C -> 100nF; footprint w_capacitors:cnp_7.5mm_disc -> w_capacitors:cnp_3mm_disc
- D1, D2, D3, D4: footprint Discret:D4 -> w_pth_diodes:diode_do35
- TR1: footprint Choke_Common-Mode_Wurth:CommonModeChoke_WuerthType-WE-CMB_Size-L -> Choke_Toroid_ThroughHole:Murata56000C
- U1: value LM393 -> LM393-1
- moved Q2 33.0 mm to (129.5, 108.5)
- moved R1 32.7 mm to (106.0, 110.5)
- moved R2 30.0 mm to (106.0, 113.5)
- moved Q1 29.2 mm to (134.0, 114.5)
- moved TR1 23.3 mm to (121.0, 123.0)
- moved D2 23.0 mm to (101.0, 139.5), turned to 180 degrees
- moved D1 20.6 mm to (101.0, 136.0), turned to 0 degrees
- moved D4 17.4 mm to (133.0, 128.5), turned to 180 degrees
- moved U1 14.4 mm to (117.5, 111.0)
- moved C1 13.9 mm to (117.0, 104.0), turned to 0 degrees
- moved D3 13.7 mm to (133.5, 120.0), turned to 0 degrees
- moved P2 9.51 mm to (137.5, 108.5), turned to 180 degrees
- moved P1 2.50 mm to (107.0, 126.0)
Connections:
- net Net-(R2-Pad2) renamed VCC
- R1 pad 2: Net-(C1-Pad2) -> Net-(C1-Pad1)
- R2 pad 1: Net-(C1-Pad1) -> Net-(R1-Pad1)
- R3 pad 1: Net-(R1-Pad1) -> Net-(C1-Pad2)
- R3 pad 2: Net-(C1-Pad1) -> Net-(R1-Pad1)
- R4 pad 2: Net-(R1-Pad1) -> Net-(C1-Pad2)
- U1 pad 3: Net-(C1-Pad1) -> Net-(C1-Pad2)
- U1 pad 5: (no net) -> Net-(U1-Pad5)
- U1 pad 6: (no net) -> Net-(U1-Pad6)
- U1 pad 7: (no net) -> Net-(U1-Pad7)

Commit message: wip
Parts:
- added C5: 100nF, w_capacitors:cnp_3mm_disc, F.Cu at (133.9, 96.7)
- added C6: 100nF, w_capacitors:cnp_3mm_disc, F.Cu at (111.5, 87.4)
- added D10: 1N4148, w_pth_diodes:diode_do35, F.Cu at (150.4, 129.6)
- added D11: LED, LEDs:LED-3MM, F.Cu at (130.8, 137.1)
- added JP1: ICSP, ICSP:ICSP, F.Cu at (117.6, 82.5)
- added P6: CONN_01X02, w_conn_pt-1,5:pt_1,5-2-3,5-h, F.Cu at (141.4, 93.0)
- added Q3: BC547, w_to:to92_3, F.Cu at (150.1, 77.1)
- added Q4: BC547, w_to:to92_3, F.Cu at (149.7, 88.7)
- added R10: 1k, w_pth_resistors:RC03, F.Cu at (151.0, 115.4)
- added R11: 1k, w_pth_resistors:RC03, F.Cu at (150.7, 119.1)
- added R12: 4k7, w_pth_resistors:RC03, F.Cu at (150.9, 123.1)
- added R13: 4k7, w_pth_resistors:RC03, F.Cu at (158.4, 111.1)
- added R14: 4k7, w_pth_resistors:RC03, F.Cu at (158.1, 106.8)
- added R15: 10k, w_pth_resistors:RC03, F.Cu at (157.5, 102.7)
- added R9: 1k5, w_pth_resistors:RC03, F.Cu at (144.5, 136.3)
- added U5: 7805, w_to:to220_std, F.Cu at (128.1, 113.9)
- P3: value 5V DCD -> CONN_01X02; footprint w_pth_circuits:dcdc_sil4 -> Pin_Headers:Pin_Header_Straight_1x02
- P4: value I2C -> Grove I2C
- P5: value CONN_02X04 -> IBT-2
- moved C4 50.4 mm to (122.0, 89.7)
- moved D8 47.6 mm to (108.5, 93.9), turned to 90 degrees
- moved D9 47.2 mm to (113.0, 93.4), turned to 90 degrees
- moved D2 45.5 mm to (101.8, 94.1)
- moved D1 44.9 mm to (101.8, 91.1)
- moved R3 41.9 mm to (125.4, 98.5)
- moved R6 40.3 mm to (109.3, 101.3), turned to 180 degrees
- moved R4 39.3 mm to (126.7, 101.4), turned to 180 degrees
- moved R7 37.7 mm to (108.7, 104.1), turned to 180 degrees
- moved R5 36.4 mm to (126.8, 104.3)
- moved D6 35.4 mm to (96.8, 113.4), turned to 90 degrees
- moved R8 34.9 mm to (107.8, 107.4)
- moved D7 34.0 mm to (99.4, 113.1), turned to 90 degrees
- moved C2 32.1 mm to (124.6, 108.3), turned to 90 degrees
- moved P3 27.3 mm to (142.7, 120.3), turned to 270 degrees
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Connections:
- net Net-(D1-Pad1) renamed /boost_1
- net Net-(D1-Pad2) renamed /boost_2
- net Net-(R8-Pad1) renamed /MCLR
- D5 pad 2: Net-(D5-Pad2) -> /red
- D6 pad 1: Net-(D6-Pad1) -> Net-(D5-Pad1)
- D6 pad 2: Net-(D6-Pad2) -> /brown
- D7 pad 1: Net-(D7-Pad1) -> /red
- D7 pad 2: Net-(D7-Pad2) -> GND
- D8 pad 2: Net-(D8-Pad2) -> Net-(D5-Pad1)
- D9 pad 1: Net-(D9-Pad1) -> /brown
- D9 pad 2: Net-(D9-Pad2) -> GND
- P3 pad 1: GND -> /red
- P3 pad 2: VCC -> /brown
- P5 pad 1: Net-(P5-Pad1) -> /PULSE
- P5 pad 3: Net-(P5-Pad3) -> /ENABLE
- P5 pad 4: Net-(P5-Pad4) -> /ENABLE
- P5 pad 5: Net-(P5-Pad5) -> /SENSE
- P5 pad 6: Net-(P5-Pad6) -> /SENSE
- P5 pad 7: Net-(P5-Pad7) -> VDD
- P5 pad 8: Net-(P5-Pad8) -> GNDA
- RR1 pad 1: Net-(RR1-Pad1) -> Net-(D5-Pad1)
- U1 pad 7: Net-(U1-Pad7) -> Net-(U1-Pad6)
- U3 pad 10: Net-(U3-Pad10) -> /SENSE
- U3 pad 12: Net-(U3-Pad12) -> /PGC
- U3 pad 13: Net-(U3-Pad13) -> /PGD
- U3 pad 6: Net-(U3-Pad6) -> /ENABLE
- U3 pad 7: Net-(U3-Pad7) -> /PULSE

Commit message: wip
Parts:
- added P7: CONN_01X03, Pin_Headers:Pin_Header_Straight_1x03, F.Cu at (136.0, 87.0)
- added U4: 6N137, w_pth_circuits:dil_8-300_socket, F.Cu at (119.4, 100.4)
- C3: footprint w_capacitors:CP_4x5mm -> w_capacitors:CP_4x7mm
- P4: footprint Pin_Headers:Pin_Header_Angled_1x04 -> w_conn_jst-ph:b4b-ph-kl
- U2, U5: footprint w_to:to220_std -> 78xx:to220
- moved R14 55.6 mm to (102.7, 101.9)
- moved D11 49.9 mm to (97.1, 100.3), turned to 90 degrees
- moved R13 49.5 mm to (111.6, 94.9)
- moved D10 48.2 mm to (106.3, 110.0), turned to 180 degrees
- moved R12 47.1 mm to (111.2, 97.6)
- moved Q3 45.9 mm to (111.0, 101.2)
- moved P6 44.5 mm to (96.9, 92.6), turned to 270 degrees
- moved R11 44.3 mm to (109.1, 104.1)
- moved Q4 38.7 mm to (111.1, 92.4)
- moved U5 37.0 mm to (107.4, 83.2)
- moved U2 36.0 mm to (128.0, 114.0)
- moved D1 35.1 mm to (113.1, 124.3), turned to 270 degrees
- moved R9 33.3 mm to (116.9, 117.7), turned to 180 degrees
- moved D2 33.3 mm to (115.3, 124.5), turned to 90 degrees
- moved R15 31.6 mm to (134.2, 81.3), turned to 180 degrees
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
Commit message: wip
Parts:
- added D12: BAT43, w_pth_diodes:diode_do35, F.Cu at (133.5, 81.3)
- added P8: Grove UART, w_conn_jst-ph:b4b-ph-kl, F.Cu at (135.8, 93.0)
- added SW1: SW_PUSH, Buttons_Switches_ThroughHole:SW_PUSH_SMALL, F.Cu at (117.6, 83.8)
- moved P3 45.7 mm to (97.0, 119.1), turned to 0 degrees
- moved R15 34.9 mm to (104.6, 100.1), turned to 270 degrees
- moved R8 33.6 mm to (127.8, 86.6), turned to 0 degrees
- moved R3 26.9 mm to (110.0, 116.8), turned to 180 degrees
- moved R10 23.2 mm to (106.8, 100.1), turned to 270 degrees
- moved D9 13.4 mm to (110.0, 110.6), turned to 180 degrees
- moved P7 13.1 mm to (137.7, 100.0), turned to 90 degrees
- moved R4 12.8 mm to (130.3, 113.8), turned to 270 degrees
- moved U2 12.5 mm to (129.3, 101.6)
- moved D11 12.2 mm to (103.1, 89.7), turned to 270 degrees
- moved D5 9.56 mm to (97.0, 112.3), turned to 90 degrees
- moved C3 9.52 mm to (132.3, 106.7), turned to 270 degrees
- moved JP1 9.16 mm to (123.2, 83.9)
- moved P5 8.45 mm to (97.0, 98.0)
- moved R14 8.41 mm to (106.3, 94.2)
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Connections:
- R8 pad 2: VDD -> Net-(D12-Pad1)
- U3 pad 8: Net-(U3-Pad8) -> /TxD
- U3 pad 9: Net-(U3-Pad9) -> /RxD
Other:
- board text added: "1"

Commit message: wip
Parts:
- moved U2 31.5 mm to (103.8, 120.0)
- moved R1 28.9 mm to (132.3, 111.4), turned to 270 degrees
- moved C2 27.5 mm to (102.0, 116.7)
- moved R2 27.3 mm to (130.2, 112.1), turned to 270 degrees
- moved C3 26.7 mm to (106.9, 115.1)
- moved D4 16.1 mm to (117.7, 124.5)
- moved D3 16.1 mm to (120.1, 124.5)
- moved R6 13.6 mm to (128.9, 103.0)
- moved R4 12.2 mm to (124.6, 103.0)
- moved R5 8.64 mm to (126.7, 103.0), turned to 270 degrees
- moved TR1 4.84 mm to (129.4, 123.3)
- moved Q1 4.79 mm to (133.5, 104.1)
- moved R3 3.95 mm to (113.9, 117.1)
- moved R9 3.95 mm to (113.9, 115.1)
- moved D10 3.94 mm to (113.9, 112.9)
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
Commit message: wip
Parts:
- removed Q4: BC547, w_to:to92_3
- removed R13: 4k7, w_pth_resistors:RC03
- R14: value 4k7 -> 1k5
- moved Q3 16.7 mm to (108.5, 89.9)
- moved C4 8.73 mm to (109.6, 94.1), turned to 180 degrees
- moved R14 8.07 mm to (111.1, 100.3), turned to 270 degrees
- moved D8 3.79 mm to (106.7, 106.7)
- moved C2 3.45 mm to (102.4, 113.3)
- moved D7 3.22 mm to (104.8, 108.8)
- moved C3 1.53 mm to (106.8, 113.5)
- moved U2 0.64 mm to (103.8, 119.4)
- moved R10 0.38 mm to (106.8, 100.2)
- moved R11 0.38 mm to (104.6, 100.2)
- moved R12 0.38 mm to (109.0, 100.2)
- moved R15 0.38 mm to (102.5, 100.2)
- moved D1 0.13 mm to (112.9, 124.5)
- moved D2 0.13 mm to (115.3, 124.5)
- turned R3 to 0 degrees
Connections:
- R12 pad 1: Net-(Q4-Pad2) -> /PULSE
- U4 pad 6: Net-(Q4-Pad2) -> /PULSE

Commit message: start routing
Parts:
- added P9: MFX, Pin_Headers:Pin_Header_Straight_1x02, F.Cu at (139.7, 118.1)
- moved P2 2.05 mm to (139.7, 115.1)
- moved Q2 1.97 mm to (139.0, 105.1)
- moved Q1 1.35 mm to (133.3, 102.8)
- moved P1 0.71 mm to (107.2, 127.5)
- moved P7 0.43 mm to (137.9, 100.3)
- moved RR1 0.40 mm to (143.0, 112.5)
Routing:
- net /boost_1: track 0.00 -> 35.5 mm
- net /boost_2: track 0.00 -> 30.7 mm
- net Net-(C1-Pad2): track 0.00 -> 17.7 mm
Other:
- net class Boost added: clearance 0.4, trace_width 2, via_dia 2.5, via_drill 1.5
- net class Default: trace_width 0.25 -> 0.3048
- net class GB added: clearance 0.2, trace_width 0.508, via_dia 0.8, via_drill 0.6

Commit message: wip
Parts:
- U1: value LM393-1 -> LM393
- moved D3 11.2 mm to (113.9, 115.2), turned to 180 degrees
- moved R9 10.6 mm to (104.3, 110.6)
- moved R3 10.6 mm to (104.3, 112.7)
- moved P1 9.94 mm to (117.1, 127.9)
- moved C1 8.74 mm to (119.0, 120.3), turned to 180 degrees
- moved D2 8.45 mm to (107.6, 127.8), turned to 180 degrees
- moved D4 8.05 mm to (113.8, 117.4), turned to 0 degrees
- moved D1 5.31 mm to (107.6, 124.7), turned to 0 degrees
- moved C2 4.01 mm to (101.9, 117.3)
- moved D7 2.57 mm to (107.3, 108.3)
- moved C3 2.51 mm to (107.1, 116.0), turned to 0 degrees
- moved U2 2.02 mm to (105.3, 120.7)
- moved D8 0.78 mm to (107.3, 106.3)
Routing:
- net /boost_1: track 35.5 -> 0.00 mm
- net /boost_2: track 30.7 -> 0.00 mm
- net Net-(C1-Pad2): track 17.7 -> 0.00 mm
Other:
- net class Boost: trace_width 2 -> 2.8
