File: dsPIC33-Arduino/dsPIC33-Arduino.sch (KiCad schematic (older format))
At the start: 10 parts, among them P1 Power, P2 Analog, P3 Digital, P4 Digital, P5 CONN_1, P6 CONN_1, P7 CONN_1, P8 CONN_1

Commit message: wip
Parts:
- added C1, C14, C15, C6, C7, C8: 100nF, Capacitors_SMD:C_0805_HandSoldering, symbol C
- added C10, C9: 100nF, Capacitors_ThroughHole:C_Disc_D3_P2.5, symbol C
- added C11: CP, w_capacitors:CP_5x5mm, symbol CP
- added C12, C13: 22pF, Capacitors_ThroughHole:C_Disc_D3_P2.5, symbol C
- added C2: 4,7uF, Capacitors_SMD:C_0805_HandSoldering, symbol C
- added C3: 10nF, Capacitors_SMD:C_0805_HandSoldering, symbol C
- added C4, C5: 47pF, Capacitors_SMD:C_0805_HandSoldering, symbol C
- added CON1: BARREL_JACK, symbol BARREL_JACK
- added D1: RX LED, LEDs:LED_0805, symbol LED
- added D2: TX LED, LEDs:LED_0805, symbol LED
- added D3: Power LED, LEDs:LED-5MM, symbol LED
- added D4: BAT43, w_pth_diodes:diode_do15, symbol D
- added D5: LED, LEDs:LED-5MM, symbol LED
- added F1: Ferrit, Resistors_SMD:R_0805_HandSoldering, symbol R
- added JP1: ICSP, MODULE, symbol ICSP
- added P10, P11: CONN_01X03, Pin_Headers:Pin_Header_Straight_1x03, symbol CONN_01X03
- added P?: Power Select, symbol CONN_01X03
- added P?: CONN_01X02, symbol CONN_01X02
- added P?: CONN_01X04, symbol CONN_01X04
- added R1, R2: 27, Resistors_SMD:R_0805_HandSoldering, symbol R
- added R10: 0, Resistors_SMD:R_0805_HandSoldering, symbol R
- added R3, R4: 270, Resistors_SMD:R_0805_HandSoldering, symbol R
- added R5, R9: 1k5, Resistors_ThroughHole:Resistor_Horizontal_RM7mm, symbol R
- added R6: 470, Resistors_ThroughHole:Resistor_Horizontal_RM7mm, symbol R
- added R7: 4k7, Resistors_ThroughHole:Resistor_Horizontal_RM7mm, symbol R
- added R8: 4k7, Resistors_SMD:R_0805_HandSoldering, symbol R
- added SW1: SW_PUSH, Buttons_Switches_ThroughHole:SW_PUSH_SMALL, symbol SW_PUSH
- added U2: AP1117D33, symbol AP1117D33
- added U3: dsPIC33EVxxxGM102-I/SP, SPDIP28, symbol dsPIC33EVxxxGM102-I/SP
- added U4: 74LVC1G32, TO_SOT_Packages_SMD:SOT-23_Handsoldering, symbol 74AHC1G32
- added U5: AP1117D5, symbol AP1117D33
- added Y1: Crystal, w_crystal:crystal_hc-49s, symbol Crystal
- P9: renamed from P?; footprint (none) -> Connect:USB_B
- gave numbers to parts that had none: 1
Connections:
- net labels added: +3V3, CBUS0, CTS, PrgEn, RTS, RX, RxD, SCL, SDA, TX, TxD, VCC, VDD, VSS, ~MCLR~, ~RESET~
- net labels removed: 0(Rx), 1(Tx), A4(SDA), A5(SCL), Reset
- wire segments 37 -> 198
- no-connect marks 5 -> 6
Other:
- moved on the sheet: P9, U1

Commit message: wip
Parts:
- gave numbers to parts that had none: 3
Connections:
- net labels removed: RxD, TxD
- wire segments 198 -> 237
- no-connect marks 6 -> 8
Other:
- moved on the sheet: R8

Commit message: wip
Connections:
- wire segments 237 -> 199
Changed lines of the file:
@@
 Text Label 3750 1850 0    60   ~ 0
 TX
-Text Label 3650 2050 0    60   ~ 0
-CTS
-Text Label 3650 1950 0    60   ~ 0
+Text Label 3700 1950 0    60   ~ 0
 RTS
 Text Label 3550 2550 0    60   ~ 0
@@
 	9050 1925 9375 1925
 Wire Wire Line
-	9300 2025 9300 2125
-Wire Wire Line
-	9300 2125 9300 3100
+	9300 2025 9300 3100
 Wire Wire Line
 	8600 1725 9375 1725
@@
 	9925 825  9925 475
 Wire Wire Line
-	1150 2050 1400 2050
-Wire Wire Line
-	1400 2050 1750 2050
+	1150 2050 1750 2050
 Wire Wire Line
 	2050 2050 2150 2050
@@
 	2150 2150 2050 2150
 Wire Wire Line
-	1150 2150 1650 2150
-Wire Wire Line
-	1650 2150 1750 2150
+	1150 2150 1750 2150
 Wire Wire Line
 	1400 2450 1400 2050
@@
 Connection ~ 1650 2150
 Wire Wire Line
-	1150 2250 1200 2250
-Wire Wire Line
-	1200 2250 1300 2250
+	1150 2250 1300 2250
 Wire Wire Line
 	1200 2250 1200 2950
 Wire Wire Line
-	1200 2950 1400 2950
-Wire Wire Line
-	1400 2950 1650 2950
-Wire Wire Line
-	1650 2950 2100 2950
-Wire Wire Line
-	2100 2950 2750 2950
-Wire Wire Line
-	2750 2950 2950 2950
-Wire Wire Line
-	2950 2950 3200 2950
-Wire Wire Line
-	2950 2850 2950 2950
-Wire Wire Line
-	2950 2950 2950 3100
+	1200 2950 3200 2950
+Wire Wire Line
+	2950 2850 2950 3100
 Connection ~ 2950 2950
 Wire Wire Line
@@
 Connection ~ 1200 2250
 Wire Wire Line
-	1150 1300 1150 1600
-Wire Wire Line
-	1150 1600 1150 1950
+	1150 1300 1150 1950
 Wire Wire Line
 	1150 1600 1300 1600
@@
 	2750 1300 2750 1450
 Wire Wire Line
-	1650 1300 1750 1300
-Wire Wire Line
-	1750 1300 2750 1300
-Wire Wire Line
-	2750 1300 4100 1300
-Wire Wire Line
-	4100 1300 4350 1300
+	1650 1300 4350 1300
 Wire Wire Line
 	2950 1450 2950 1200
 Wire Wire Line
-	2100 1200 2100 1750
-Wire Wire Line
-	2100 1750 2100 2350
-Wire Wire Line
-	2100 2350 2100 2550
+	2100 1200 2100 2550
 Wire Wire Line
 	2100 2350 2150 2350
@@
 Connection ~ 2100 2950
 Wire Wire Line
-	700  1200 850  1200
-Wire Wire Line
-	850  1200 1000 1200
+	700  1200 1000 1200
 Wire Wire Line
 	850  1200 850  1300
@@
 	1000 800  1000 900
 Wire Wire Line
-	700  800  850  800
-Wire Wire Line
-	850  800  1000 800
+	700  800  1000 800
 Wire Wire Line
 	700  800  700  900
@@
 	3550 2550 3800 2550
 Wire Wire Line
-	1750 1100 1750 1200
-Wire Wire Line
-	1750 1200 1750 1300
+	1750 1100 1750 1300
 Connection ~ 1750 1300
 Wire Wire Line
@@
 	5500 3100 5500 3150
 Wire Wire Line
-	5500 3150 5950 3150
-Wire Wire Line
-	5950 3150 6400 3150
+	5500 3150 6400 3150
 Wire Wire Line
 	6400 3150 6400 3100
 Wire Wire Line
-	5950 2950 5950 3150
-Wire Wire Line
-	5950 3150 5950 3250
+	5950 2950 5950 3250
 Connection ~ 5950 3150
 Wire Wire Line
 	5500 2800 5500 2650
 Wire Wire Line
-	5150 2650 5500 2650
-Wire Wire Line
-	5500 2650 5650 2650
+	5150 2650 5650 2650
 Wire Wire Line
 	6400 2650 6400 2800
@@
 	4150 7050 4150 7150
 Wire Wire Line
-	4150 7150 4300 7150
-Wire Wire Line
-	4300 7150 4450 7150
+	4150 7150 4450 7150
 Wire Wire Line
 	4450 7150 4450 7050
 Wire Wire Line
-	4300 7050 4300 7150
-Wire Wire Line
-	4300 7150 4300 7250
+	4300 7050 4300 7250
 Connection ~ 4300 7150
 Wire Wire Line
 	4200 4500 4200 4450
 Wire Wire Line
-	4200 4450 4300 4450
-Wire Wire Line
-	4300 4450 4400 4450
+	4200 4450 4400 4450
 Wire Wire Line
 	4400 4450 4400 4500
 Wire Wire Line
-	4300 4250 4300 4300
-Wire Wire Line
-	4300 4300 4300 4450
+	4300 4250 4300 4450
 Connection ~ 4300 4450
 Wire Wire Line
@@
 	3600 4100 3600 4000
 Wire Wire Line
-	3600 4000 3700 4000
-Wire Wire Line
-	3700 4000 3800 4000
+	3600 4000 3800 4000
 Wire Wire Line
 	3800 4000 3800 4100
@@
 $EndComp
 Wire Wire Line
-	2450 5650 2750 5650
-Wire Wire Line
-	2750 5650 3100 5650
-Wire Wire Line
-	2450 6000 2750 6000
-Wire Wire Line
-	2750 6000 3100 6000
+	2450 5650 3100 5650
+Wire Wire Line
+	2450 6000 3100 6000
 $Comp
 L C C13
@@
 	2150 5650 1950 5650
 Wire Wire Line
-	1950 5650 1950 6000
-Wire Wire Line
-	1950 6000 1950 6150
+	1950 5650 1950 6150
 Wire Wire Line
 	2150 6000 1950 6000
@@
 	5650 1700 5650 1750
 Wire Wire Line
-	5500 1750 5650 1750
-Wire Wire Line
-	5650 1750 6100 1750
-Wire Wire Line
-	6100 1750 6550 1750
+	5500 1750 6550 1750
 Wire Wire Line
 	6550 1750 6550 1700
 Wire Wire Line
-	6100 1550 6100 1750
-Wire Wire Line
-	6100 1750 6100 1850
+	6100 1550 6100 1850
 Connection ~ 6100 1750
 Wire Wire Line
 	5650 1400 5650 1250
 Wire Wire Line
-	5450 1250 5650 1250
-Wire Wire Line
-	5650 1250 5800 1250
-Wire Wire Line
-	6400 1250 6550 1250
-Wire Wire Line
-	6550 1250 6800 1250
+	5450 1250 5800 1250
+Wire Wire Line
+	6400 1250 6800 1250
 Wire Wire Line
 	6550 1250 6550 1400
@@
 	5450 1350 5500 1350
 Wire Wire Line
-	5500 1350 5500 1450
-Wire Wire Line
-	5500 1450 5500 1750
+	5500 1350 5500 1750
 Connection ~ 5650 1750
 Wire Wire Line
@@
 	4550 3100 4800 3100
 Wire Wire Line
-	4000 3150 3650 3150
-Wire Wire Line
-	3650 3150 3400 3150
+	3400 3150 4000 3150
 Wire Wire Line
 	3800 3050 4000 3050
-Text Label 3400 3150 0    60   ~ 0
-CTS
 $Comp
 L R R8
@@
 	5200 2450 5150 2450
 NoConn ~ 3850 1950
+NoConn ~ 3850 2250
+Wire Wire Line
+	3650 2750 3650 2800
+Wire Wire Line
+	3650 3100 3650 3150
+Connection ~ 3650 3150
+Wire Wire Line
+	6250 2650 6600 2650
+Wire Wire Line
+	4650 4300 4300 4300
+Connection ~ 4300 4300
+Wire Wire Line
+	4650 4250 4650 4300
+Text Label 3400 3150 0    60   ~ 0
+RTS
+Text Label 3700 2050 0    60   ~ 0
+CTS
 Text Label 6000 4400 0    60   ~ 0
 CTS
-NoConn ~ 3850 2250
-Wire Wire Line
-	3650 2750 3650 2800
-Wire Wire Line
-	3650 3100 3650 3150
-Connection ~ 3650 3150
-Wire Wire Line
-	6250 2650 6400 2650
-Wire Wire Line
-	6400 2650 6600 2650
-Wire Wire Line
-	4650 4300 4300 4300
-Connection ~ 4300 4300
-Wire Wire Line
-	4650 4250 4650 4300
 $EndSCHEMATC

Commit message: wip
Parts:
- removed P12: CONN_01X04, symbol CONN_01X04
- added D6: D, w_pth_diodes:diode_do35, symbol D
- added P12: CONN_01X03, Pin_Headers:Pin_Header_Straight_1x03, symbol CONN_01X03
- added P15: Grove I2C, w_conn_jst-ph:s4b-ph-kl, symbol CONN_01X04
- C11: footprint w_capacitors:CP_5x5mm -> w_capacitors:CP_4x5mm
- CON1: footprint (none) -> Connect:BARREL_JACK
- D3, D5: footprint LEDs:LED-5MM -> LEDs:LED-3MM
- D4: footprint w_pth_diodes:diode_do15 -> w_pth_diodes:diode_do35
- JP1: footprint MODULE -> ICSP:ICSP
- P13: footprint (none) -> Socket_Strips:Socket_Strip_Straight_2x01
- P14: footprint (none) -> Socket_Strips:Socket_Strip_Straight_1x03
- R5, R6, R7, R9: footprint Resistors_ThroughHole:Resistor_Horizontal_RM7mm -> w_pth_resistors:RC03
- U1: footprint SSOP-16 -> w_smd_dil:ssop-16
- U2: value AP1117D33 -> LM1117 3V3; footprint (none) -> TO_SOT_Packages_SMD:SOT-223
- U3: footprint SPDIP28 -> w_pth_circuits:dil_28-300_socket
- U4: footprint TO_SOT_Packages_SMD:SOT-23_Handsoldering -> TO_SOT_Packages_SMD:SOT-353
- U5: value AP1117D5 -> LM1117 5V; footprint (none) -> TO_SOT_Packages_SMD:SOT-223
Connections:
- wire segments 199 -> 206
Other:
- moved on the sheet: C7, C8, D3, JP1, P14, R5, R6, U2

Commit message: wip
Parts:
- added P16: PIN19, Pin_Headers:Pin_Header_Straight_1x03, symbol CONN_01X03
- added P17: UART/CAN, w_conn_jst-ph:s4b-ph-kl, symbol CONN_01X04
- P10: value CONN_01X03 -> PIN20
- P11: value CONN_01X03 -> PIN5
- P12: value CONN_01X03 -> PWR_IN
- P13: value CONN_01X02 -> PIN2
Connections:
- wire segments 206 -> 258
Other:
- moved on the sheet: D5, JP1, P13, P15, R9

Commit message: wip
Parts:
- removed D4: BAT43, w_pth_diodes:diode_do35, symbol D
- removed D6: D, w_pth_diodes:diode_do35, symbol D
- added D4, D6: BAT43, w_pth_diodes:diode_do35, symbol ZENER
- P13: footprint Socket_Strips:Socket_Strip_Straight_2x01 -> Pin_Headers:Pin_Header_Straight_1x02
- P14: footprint Socket_Strips:Socket_Strip_Straight_1x03 -> Pin_Headers:Pin_Header_Straight_1x03
- P15: value Grove I2C -> I2C
Connections:
- wire segments 258 -> 217
Other:
- moved on the sheet: R7
Changed lines of the file:
@@
 A3
-$Comp
-L D D4
-U 1 1 588DD0A8
-P 2850 4550
-F 0 "D4" H 2850 4650 50  0000 C CNN
-F 1 "BAT43" H 3000 4450 50  0000 C CNN
-F 2 "w_pth_diodes:diode_do35" H 2850 4550 50  0001 C CNN
-F 3 "" H 2850 4550 50  0000 C CNN
-	1    2850 4550
-	0    -1   -1   0
-$EndComp
 $Comp
 L R R7
 U 1 1 588DD141
-P 2850 4200
-F 0 "R7" V 2930 4200 50  0000 C CNN
-F 1 "4k7" V 2850 4200 50  0000 C CNN
-F 2 "w_pth_resistors:RC03" V 2780 4200 50  0001 C CNN
-F 3 "" H 2850 4200 50  0000 C CNN
-	1    2850 4200
+P 2850 3950
+F 0 "R7" V 2930 3950 50  0000 C CNN
+F 1 "4k7" V 2850 3950 50  0000 C CNN
+F 2 "w_pth_resistors:RC03" V 2780 3950 50  0001 C CNN
+F 3 "" H 2850 3950 50  0000 C CNN
+	1    2850 3950
 	1    0    0    -1
 $EndComp
@@
 L VDD #PWR021
 U 1 1 588DD1FB
-P 2850 3950
-F 0 "#PWR021" H 2850 3800 50  0001 C CNN
-F 1 "VDD" H 2850 4100 50  0000 C CNN
-F 2 "" H 2850 3950 50  0000 C CNN
-F 3 "" H 2850 3950 50  0000 C CNN
-	1    2850 3950
+P 2850 3700
+F 0 "#PWR021" H 2850 3550 50  0001 C CNN
+F 1 "VDD" H 2850 3850 50  0000 C CNN
+F 2 "" H 2850 3700 50  0000 C CNN
+F 3 "" H 2850 3700 50  0000 C CNN
+	1    2850 3700
 	1    0    0    -1
 $EndComp
@@
 F 0 "P14" H 8000 2650 50  0000 C CNN
 F 1 "Power Select" V 8100 2450 50  0000 C CNN
-F 2 "Socket_Strips:Socket_Strip_Straight_1x03" H 8000 2450 50  0001 C CNN
+F 2 "Pin_Headers:Pin_Header_Straight_1x03" H 8000 2450 50  0001 C CNN
 F 3 "" H 8000 2450 50  0000 C CNN
 	1    8000 2450
@@
 F 0 "P13" H 5500 4600 50  0000 C CNN
 F 1 "PIN2" V 5600 4450 50  0000 C CNN
-F 2 "Socket_Strips:Socket_Strip_Straight_2x01" H 5500 4450 50  0001 C CNN
+F 2 "Pin_Headers:Pin_Header_Straight_1x02" H 5500 4450 50  0001 C CNN
 F 3 "" H 5500 4450 50  0000 C CNN
 	1    5500 4450
@@
 	1    0    0    -1
 $EndComp
-Text Label 4950 3100 0    60   ~ 0
+Text Label 5050 3100 0    60   ~ 0
 ~MCLR~
 $Comp
@@
 $EndComp
 $Comp
-L D D6
-U 1 1 589A18F3
-P 4775 3100
-F 0 "D6" H 4775 3200 50  0000 C CNN
-F 1 "D" H 4775 3000 50  0000 C CNN
-F 2 "w_pth_diodes:diode_do35" H 4775 3100 50  0001 C CNN
-F 3 "" H 4775 3100 50  0000 C CNN
-	1    4775 3100
-	-1   0    0    1
-$EndComp
-$Comp
 L CONN_01X04 P15
 U 1 1 589A6EC0
 P 1225 3550
 F 0 "P15" H 1225 3800 50  0000 C CNN
-F 1 "Grove I2C" V 1325 3550 50  0000 C CNN
+F 1 "I2C" V 1325 3550 50  0000 C CNN
 F 2 "w_conn_jst-ph:s4b-ph-kl" V 1225 3550 50  0001 C CNN
 F 3 "" H 1225 3550 50  0000 C CNN
@@
 	9050 1925 9375 1925
 Wire Wire Line
-	9300 2025 9300 2125
-Wire Wire Line
-	9300 2125 9300 3100
+	9300 2025 9300 3100
 Wire Wire Line
 	8600 1725 9375 1725
@@
 	9925 825  9925 475
 Wire Wire Line
-	1150 2050 1400 2050
-Wire Wire Line
-	1400 2050 1750 2050
+	1150 2050 1750 2050
 Wire Wire Line
 	2050 2050 2150 2050
@@
 	2150 2150 2050 2150
 Wire Wire Line
-	1150 2150 1650 2150
-Wire Wire Line
-	1650 2150 1750 2150
+	1150 2150 1750 2150
 Wire Wire Line
 	1400 2450 1400 2050
@@
 Connection ~ 1650 2150
 Wire Wire Line
-	1150 2250 1200 2250
-Wire Wire Line
-	1200 2250 1300 2250
+	1150 2250 1300 2250
 Wire Wire Line
 	1200 2250 1200 2950
 Wire Wire Line
-	1200 2950 1400 2950
-Wire Wire Line
-	1400 2950 1650 2950
-Wire Wire Line
-	1650 2950 2100 2950
-Wire Wire Line
-	2100 2950 2750 2950
-Wire Wire Line
-	2750 2950 2950 2950
-Wire Wire Line
-	2950 2950 3200 2950
-Wire Wire Line
-	2950 2850 2950 2950
-Wire Wire Line
-	2950 2950 2950 3100
+	1200 2950 3200 2950
+Wire Wire Line
+	2950 2850 2950 3100
 Connection ~ 2950 2950
 Wire Wire Line
@@
 Connection ~ 1200 2250
 Wire Wire Line
-	1150 1300 1150 1600
-Wire Wire Line
-	1150 1600 1150 1950
+	1150 1300 1150 1950
 Wire Wire Line
 	1150 1600 1300 1600
@@
 	2950 1450 2950 1200
 Wire Wire Line
-	2100 1200 2100 1750
-Wire Wire Line
-	2100 1750 2100 2350
-Wire Wire Line
-	2100 2350 2100 2550
+	2100 1200 2100 2550
 Wire Wire Line
 	2100 2350 2150 2350
@@
 Connection ~ 2100 2950
 Wire Wire Line
-	700  1200 850  1200
-Wire Wire Line
-	850  1200 1000 1200
+	700  1200 1000 1200
 Wire Wire Line
 	850  1200 850  1300
@@
 	1000 800  1000 900
 Wire Wire Line
-	700  800  850  800
-Wire Wire Line
-	850  800  1000 800
+	700  800  1000 800
 Wire Wire Line
 	700  800  700  900
@@
 	3550 2550 3800 2550
 Wire Wire Line
-	1750 1100 1750 1200
-Wire Wire Line
-	1750 1200 1750 1300
+	1750 1100 1750 1300
 Connection ~ 1750 1300
 Wire Wire Line
@@
 	750  2450 750  2450
 Wire Wire Line
-	2100 1200 2950 1200
-Wire Wire Line
-	2950 1200 4100 1200
-Wire Wire Line
-	4100 1200 4350 1200
+	2100 1200 4350 1200
 Wire Wire Line
 	4100 1200 4100 1800
@@
 	5650 2850 5650 2900
 Wire Wire Line
-	5650 2900 6100 2900
-Wire Wire Line
-	6100 2900 6550 2900
+	5650 2900 6550 2900
 Wire Wire Line
 	6550 2900 6550 2850
 Wire Wire Line
-	6100 2700 6100 2900
-Wire Wire Line
-	6100 2900 6100 3000
+	6100 2700 6100 3000
 Connection ~ 6100 2900
 Wire Wire Line
 	5650 2550 5650 2400
 Wire Wire Line
-	5300 2400 5650 2400
-Wire Wire Line
-	5650 2400 5800 2400
+	5300 2400 5800 2400
 Wire Wire Line
 	6550 2400 6550 2550
@@
 	4150 7050 4150 7325
 Wire Wire Line
-	4150 7325 4300 7325
-Wire Wire Line
-	4300 7325 4450 7325
-Wire Wire Line
-	4450 7325 4775 7325
+	4150 7325 4775 7325
 Wire Wire Line
 	4450 7325 4450 7050
@@
 	4200 4500 4200 4450
 Wire Wire Line
-	4200 4450 4300 4450
-Wire Wire Line
-	4300 4450 4400 4450
+	4200 4450 4400 4450
 Wire Wire Line
 	4400 4450 4400 4500
 Wire Wire Line
-	4300 4250 4300 4300
-Wire Wire Line
-	4300 4300 4300 4450
+	4300 4250 4300 4450
 Connection ~ 4300 4450
 Wire Wire Line
@@
 	3600 4100 3600 4000
 Wire Wire Line
-	3600 4000 3700 4000
-Wire Wire Line
-	3700 4000 3800 4000
+	3600 4000 3800 4000
 Wire Wire Line
 	3800 4000 3800 4100
@@
 	2100 5300 3100 5300
 Wire Wire Line
-	2800 4800 2850 4800
-Wire Wire Line
-	2850 4800 3050 4800
-Wire Wire Line
-	3050 4800 3100 4800
-Wire Wire Line
-	2850 4800 2850 4700
-Wire Wire Line
-	2850 4400 2850 4350
-Wire Wire Line
-	2850 4050 2850 3950
+	2800 4800 3100 4800
+Wire Wire Line
+	2850 4800 2850 4550
 Connection ~ 2850 4800
 Wire Wire Line
@@
 	3100 5500 2850 5500
 Wire Wire Line
-	2450 5650 2750 5650
-Wire Wire Line
-	2750 5650 3100 5650
-Wire Wire Line
-	2450 6000 2750 6000
-Wire Wire Line
-	2750 6000 3100 6000
+	2450 5650 3100 5650
+Wire Wire Line
+	2450 6000 3100 6000
 Wire Wire Line
 	2150 5650 1950 5650
 Wire Wire Line
-	1950 5650 1950 6000
-Wire Wire Line
-	1950 6000 1950 6150
+	1950 5650 1950 6150
 Wire Wire Line
 	2150 6000 1950 6000
@@
 	5650 1700 5650 1750
 Wire Wire Line
-	5500 1750 5650 1750
-Wire Wire Line
-	5650 1750 6100 1750
-Wire Wire Line
-	6100 1750 6550 1750
+	5500 1750 6550 1750
 Wire Wire Line
 	6550 1750 6550 1700
 Wire Wire Line
-	6100 1550 6100 1750
-Wire Wire Line
-	6100 1750 6100 1850
+	6100 1550 6100 1850
 Connection ~ 6100 1750
 Wire Wire Line
 	5650 1400 5650 1250
 Wire Wire Line
-	5450 1250 5650 1250
-Wire Wire Line
-	5650 1250 5800 1250
-Wire Wire Line
-	6400 1250 6550 1250
-Wire Wire Line
-	6550 1250 6800 1250
+	5450 1250 5800 1250
+Wire Wire Line
+	6400 1250 6800 1250
 Wire Wire Line
 	6550 1250 6550 1400
@@
 	5450 1350 5500 1350
 Wire Wire Line
-	5500 1350 5500 1450
-Wire Wire Line
-	5500 1450 5500 1750
+	5500 1350 5500 1750
 Connection ~ 5650 1750
 Wire Wire Line
@@
 	3800 2550 3800 3050
 Wire Wire Line
-	3400 3150 3650 3150
-Wire Wire Line
-	3650 3150 4000 3150
+	3400 3150 4000 3150
 Wire Wire Line
 	3800 3050 4000 3050
@@
 Connection ~ 3650 3150
 Wire Wire Line
-	6400 2400 6550 2400
-Wire Wire Line
-	6550 2400 6750 2400
+	6400 2400 6750 2400
 Wire Wire Line
 	4650 4300 4300 4300
@@
 Connection ~ 3050 4800
 Wire Wire Line
-	4625 3100 4550 3100
-Wire Wire Line
-	4925 3100 5200 3100
-Wire Wire Line
-	1650 1300 1750 1300
-Wire Wire Line
-	1750 1300 2750 1300
+	1650 1300 2750 1300
 Connection ~ 2950 1200
 Connection ~ 4100 1200
@@
 	4300 7050 4300 7225
 Wire Wire Line
-	4300 7225 4675 7225
-Wire Wire Line
-	4675 7225 4775 7225
+	4300 7225 4775 7225
 Connection ~ 4450 7325
 Wire Wire Line
@@
 Text Label 800  4250 0    60   ~ 0
 6(**)
+$Comp
+L ZENER D4
+U 1 1 589B6E76
+P 2850 4350
+F 0 "D4" H 2850 4450 50  0000 C CNN
+F 1 "BAT43" H 2850 4250 50  0000 C CNN
+F 2 "w_pth_diodes:diode_do35" H 2850 4350 50  0001 C CNN
+F 3 "" H 2850 4350 50  0000 C CNN
+	1    2850 4350
+	0    -1   -1   0
+$EndComp
+Wire Wire Line
+	2850 4100 2850 4150
+Wire Wire Line
+	2850 3700 2850 3800
+$Comp
+L ZENER D6
+U 1 1 589B7FB8
+P 4850 3100
+F 0 "D6" H 4850 3200 50  0000 C CNN
+F 1 "BAT43" H 4850 3000 50  0000 C CNN
+F 2 "w_pth_diodes:diode_do35" H 4850 3100 50  0001 C CNN
+F 3 "" H 4850 3100 50  0000 C CNN
+	1    4850 3100
+	-1   0    0    1
+$EndComp
+Wire Wire Line
+	4550 3100 4650 3100
+Wire Wire Line
+	5050 3100 5300 3100
 $EndSCHEMATC
