File: dsPIC33-Arduino/dsPIC33-Arduino.sch (KiCad schematic (older format))
At the start: 58 parts, among them CON1 BARREL_JACK, P1 Power, P10 PIN20, P11 PIN5, P12 PWR_IN, P13 PIN2, P14 Power Select, P15 I2C, P16 PIN19, P17 UART/CAN, P2 Analog, P3 Digital, P4 Digital, P5 CONN_1, P6 CONN_1, P7 CONN_1, P8 CONN_1, P9 USB_B, SW1 SW_PUSH, U1 FT230XS, U2 LM1117 3V3, U3 dsPIC33EVxxxGM102-I/SP, U4 74LVC1G32, U5 LM1117 5V, Y1 Crystal

Commit message: wip
Parts:
- removed D4, D6: BAT43, w_pth_diodes:diode_do35, symbol ZENER
- removed U5: LM1117 5V, TO_SOT_Packages_SMD:SOT-223, symbol AP1117D33
- added D4, D6: BAT43, w_pth_diodes:diode_do35, symbol D_Schottky
- added U5: 7805, TO_SOT_Packages_SMD:TO-252-2Lead, symbol 7805
- C14, C15, C7, C8: footprint Capacitors_SMD:C_0805_HandSoldering -> Capacitors_ThroughHole:C_Disc_D3_P2.5
- P17: value UART/CAN -> UART
- SW1: footprint Buttons_Switches_ThroughHole:SW_PUSH_SMALL -> w_switch:PCB_PUSH
Connections:
- net labels added: VI, VO
Other:
- moved on the sheet: R7
Changed lines of the file:
@@
 F 0 "C7" H 5675 2800 50  0000 L CNN
 F 1 "100nF" H 5675 2600 50  0000 L CNN
-F 2 "Capacitors_SMD:C_0805_HandSoldering" H 5688 2550 50  0001 C CNN
+F 2 "Capacitors_ThroughHole:C_Disc_D3_P2.5" H 5688 2550 50  0001 C CNN
 F 3 "" H 5650 2700 50  0000 C CNN
 	1    5650 2700
@@
 F 0 "C8" H 6575 2800 50  0000 L CNN
 F 1 "100nF" H 6575 2600 50  0000 L CNN
-F 2 "Capacitors_SMD:C_0805_HandSoldering" H 6588 2550 50  0001 C CNN
+F 2 "Capacitors_ThroughHole:C_Disc_D3_P2.5" H 6588 2550 50  0001 C CNN
 F 3 "" H 6550 2700 50  0000 C CNN
 	1    6550 2700
@@
 L R R7
 U 1 1 588DD141
-P 2850 3950
-F 0 "R7" V 2930 3950 50  0000 C CNN
-F 1 "4k7" V 2850 3950 50  0000 C CNN
-F 2 "w_pth_resistors:RC03" V 2780 3950 50  0001 C CNN
-F 3 "" H 2850 3950 50  0000 C CNN
-	1    2850 3950
+P 2850 4050
+F 0 "R7" V 2930 4050 50  0000 C CNN
+F 1 "4k7" V 2850 4050 50  0000 C CNN
+F 2 "w_pth_resistors:RC03" V 2780 4050 50  0001 C CNN
+F 3 "" H 2850 4050 50  0000 C CNN
+	1    2850 4050
 	1    0    0    -1
 $EndComp
@@
 L VDD #PWR021
 U 1 1 588DD1FB
-P 2850 3700
-F 0 "#PWR021" H 2850 3550 50  0001 C CNN
-F 1 "VDD" H 2850 3850 50  0000 C CNN
-F 2 "" H 2850 3700 50  0000 C CNN
-F 3 "" H 2850 3700 50  0000 C CNN
-	1    2850 3700
+P 2850 3850
+F 0 "#PWR021" H 2850 3700 50  0001 C CNN
+F 1 "VDD" H 2850 4000 50  0000 C CNN
+F 2 "" H 2850 3850 50  0000 C CNN
+F 3 "" H 2850 3850 50  0000 C CNN
+	1    2850 3850
 	1    0    0    -1
 $EndComp
@@
 F 0 "SW1" H 2100 4910 50  0000 C CNN
 F 1 "SW_PUSH" H 1950 4720 50  0000 C CNN
-F 2 "Buttons_Switches_ThroughHole:SW_PUSH_SMALL" H 1950 4800 50  0001 C CNN
+F 2 "w_switch:PCB_PUSH" H 1950 4800 50  0001 C CNN
 F 3 "" H 1950 4800 50  0000 C CNN
 	1    1950 4800
@@
 TX
 $Comp
-L AP1117D33 U5
-U 1 1 588E4306
-P 6100 1250
-F 0 "U5" H 6200 1000 50  0000 C CNN
-F 1 "LM1117 5V" H 6100 1500 50  0000 C CNN
-F 2 "TO_SOT_Packages_SMD:SOT-223" H 6100 1250 50  0001 C CNN
-F 3 "" H 6100 1250 50  0000 C CNN
-	1    6100 1250
-	1    0    0    -1
-$EndComp
-$Comp
 L GND #PWR025
 U 1 1 588E430C
@@
 F 0 "C14" H 5675 1650 50  0000 L CNN
 F 1 "100nF" H 5675 1450 50  0000 L CNN
-F 2 "Capacitors_SMD:C_0805_HandSoldering" H 5688 1400 50  0001 C CNN
+F 2 "Capacitors_ThroughHole:C_Disc_D3_P2.5" H 5688 1400 50  0001 C CNN
 F 3 "" H 5650 1550 50  0000 C CNN
 	1    5650 1550
@@
 F 0 "C15" H 6575 1650 50  0000 L CNN
 F 1 "100nF" H 6575 1450 50  0000 L CNN
-F 2 "Capacitors_SMD:C_0805_HandSoldering" H 6588 1400 50  0001 C CNN
+F 2 "Capacitors_ThroughHole:C_Disc_D3_P2.5" H 6588 1400 50  0001 C CNN
 F 3 "" H 6550 1550 50  0000 C CNN
 	1    6550 1550
@@
 	1    0    0    -1
 $EndComp
-Text Label 5050 3100 0    60   ~ 0
+Text Label 4950 3100 0    60   ~ 0
 ~MCLR~
 $Comp
@@
 P 1225 4300
 F 0 "P17" H 1225 4550 50  0000 C CNN
-F 1 "UART/CAN" V 1325 4300 50  0000 C CNN
+F 1 "UART" V 1325 4300 50  0000 C CNN
 F 2 "w_conn_jst-ph:s4b-ph-kl" V 1225 4300 50  0001 C CNN
 F 3 "" H 1225 4300 50  0000 C CNN
@@
 	5650 1400 5650 1250
 Wire Wire Line
-	5450 1250 5800 1250
-Wire Wire Line
-	6400 1250 6800 1250
-Wire Wire Line
 	6550 1250 6550 1400
 Connection ~ 6550 1250
@@
 Text Label 800  4250 0    60   ~ 0
 6(**)
-$Comp
-L ZENER D4
-U 1 1 589B6E76
-P 2850 4350
-F 0 "D4" H 2850 4450 50  0000 C CNN
-F 1 "BAT43" H 2850 4250 50  0000 C CNN
-F 2 "w_pth_diodes:diode_do35" H 2850 4350 50  0001 C CNN
-F 3 "" H 2850 4350 50  0000 C CNN
-	1    2850 4350
+Wire Wire Line
+	2850 4200 2850 4250
+Wire Wire Line
+	2850 3850 2850 3900
+Wire Wire Line
+	4550 3100 4650 3100
+$Comp
+L 7805 U5
+U 1 1 589C50BD
+P 6100 1300
+F 0 "U5" H 6250 1104 50  0000 C CNN
+F 1 "7805" H 6100 1500 50  0000 C CNN
+F 2 "TO_SOT_Packages_SMD:TO-252-2Lead" H 6100 1300 50  0001 C CNN
+F 3 "" H 6100 1300 50  0000 C CNN
+	1    6100 1300
+	1    0    0    -1
+$EndComp
+Wire Wire Line
+	5450 1250 5700 1250
+Wire Wire Line
+	6500 1250 6800 1250
+Text Label 6600 1250 0    60   ~ 0
+VO
+Text Label 5500 1250 0    60   ~ 0
+VI
+$Comp
+L D_Schottky D6
+U 1 1 589CD03F
+P 4800 3100
+F 0 "D6" H 4800 3200 50  0000 C CNN
+F 1 "BAT43" H 4800 3000 50  0000 C CNN
+F 2 "w_pth_diodes:diode_do35" H 4800 3100 50  0001 C CNN
+F 3 "" H 4800 3100 50  0000 C CNN
+	1    4800 3100
+	-1   0    0    1
+$EndComp
+Wire Wire Line
+	4950 3100 5200 3100
+$Comp
+L D_Schottky D4
+U 1 1 589CD86C
+P 2850 4400
+F 0 "D4" H 2850 4500 50  0000 C CNN
+F 1 "BAT43" H 2850 4300 50  0000 C CNN
+F 2 "w_pth_diodes:diode_do35" H 2850 4400 50  0001 C CNN
+F 3 "" H 2850 4400 50  0000 C CNN
+	1    2850 4400
 	0    -1   -1   0
 $EndComp
-Wire Wire Line
-	2850 4100 2850 4150
-Wire Wire Line
-	2850 3700 2850 3800
-$Comp
-L ZENER D6
-U 1 1 589B7FB8
-P 4850 3100
-F 0 "D6" H 4850 3200 50  0000 C CNN
-F 1 "BAT43" H 4850 3000 50  0000 C CNN
-F 2 "w_pth_diodes:diode_do35" H 4850 3100 50  0001 C CNN
-F 3 "" H 4850 3100 50  0000 C CNN
-	1    4850 3100
-	-1   0    0    1
-$EndComp
-Wire Wire Line
-	4550 3100 4650 3100
-Wire Wire Line
-	5050 3100 5300 3100
 $EndSCHEMATC
