File: mfx-link2/mfx-link2.kicad_pcb (KiCad board)
At the start: 2 copper layers, 51 parts, among them P1 Rail, P2 Gleisbox, P3 18V, P4 UART, P5 I2C, P6 CONN_02X03, P7 POTI, P8 IBT-2, Q1 BC817-40, T1 53040C, U1 6N137, U2 7805, U3 LM393, U4 7805, U5 PIC16F1709

Commit message: wip
Parts:
- removed D11: BAT43, w_smd_diode:sod323
- removed D12: LED, LEDs:LED_0805
- D10: value 1N4148 -> LED; footprint w_smd_diode:sod323 -> LEDs:LED_0805
- D6, D7: value 1N4007 -> 1N4148
- D9: value 1N4148 -> BAT43
- moved R10 82.1 mm to (90.4, 124.4)
- moved R11 82.1 mm to (90.4, 121.7)
- moved R12 82.1 mm to (90.4, 119.1)
- moved R13 82.1 mm to (90.4, 116.4)
- moved R14 82.1 mm to (90.4, 113.9)
- moved R8 82.1 mm to (90.4, 129.9)
- moved R9 82.1 mm to (90.4, 127.1)
- moved P6 63.8 mm to (101.0, 123.5)
- moved U2 63.0 mm to (157.5, 118.0), turned to 270 degrees
- moved R7 62.9 mm to (101.5, 117.5)
- moved Q1 62.1 mm to (101.0, 110.8)
- moved C5 59.9 mm to (153.5, 120.0)
- moved P3 52.8 mm to (147.5, 119.5), turned to 0 degrees
- moved C3 51.7 mm to (153.5, 115.5), turned to 180 degrees
- moved D9 46.7 mm to (142.0, 64.5), turned to 180 degrees
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Connections:
- D10 pad 1: /brown -> Net-(D10-Pad1)
- D10 pad 2: Net-(D10-Pad2) -> VCC
- D6 pad 1: Net-(D6-Pad1) -> Net-(C1-Pad1)
- D6 pad 2: Net-(D6-Pad2) -> Net-(C1-Pad2)
- D7 pad 1: Net-(D6-Pad2) -> Net-(C1-Pad2)
- D7 pad 2: Net-(D6-Pad1) -> Net-(C1-Pad1)
- D8 pad 1: Net-(C1-Pad1) -> /brown
- D8 pad 2: Net-(C1-Pad2) -> Net-(D8-Pad2)
- D9 pad 1: Net-(C1-Pad2) -> Net-(D9-Pad1)
- D9 pad 2: Net-(C1-Pad1) -> VCC
- P1 pad 1: Net-(D6-Pad1) -> Net-(P1-Pad1)
- R1 pad 1: Net-(D10-Pad2) -> Net-(D8-Pad2)
- R15 pad 2: Net-(D12-Pad1) -> Net-(D10-Pad1)
- R16 pad 2: Net-(D11-Pad1) -> Net-(D9-Pad1)
- T1 pad 7: Net-(D6-Pad1) -> Net-(P1-Pad1)
- T1 pad 8: Net-(D6-Pad2) -> Net-(P1-Pad2)
- U1 pad 2: Net-(D10-Pad2) -> Net-(D8-Pad2)
Other:
- board outline added: 50 x 50 mm

Commit message: wip
Parts:
- added REF**: 1pin, Connect:1pin, F.Cu at (163.0, 83.5)
- added REF**: 1pin, Connect:1pin, F.Cu at (123.0, 83.5)
- added REF**: 1pin, Connect:1pin, F.Cu at (163.0, 123.5)
- added REF**: 1pin, Connect:1pin, F.Cu at (123.0, 123.5)
- P8: footprint Pin_Headers:Pin_Header_Straight_2x04 -> Socket_Strips:Socket_Strip_Straight_2x04; moved to B.Cu
- moved P8 4.50 mm to (131.0, 85.5), turned to 0 degrees
- moved C1 0.50 mm to (139.5, 104.0)
- moved C2 0.50 mm to (120.5, 110.5)
- moved C3 0.50 mm to (154.0, 115.5)
- moved C4 0.50 mm to (128.0, 110.5)
- moved C5 0.50 mm to (154.0, 120.0)
- moved D1 0.50 mm to (127.8, 103.3)
- moved D2 0.50 mm to (127.8, 99.7)
- moved D3 0.50 mm to (127.8, 101.5)
- moved D4 0.50 mm to (127.8, 98.0)
- moved D5 0.50 mm to (122.5, 110.5)
- moved D6 0.50 mm to (135.5, 103.0)
- moved D7 0.50 mm to (133.0, 103.5)
- moved D8 0.50 mm to (134.0, 96.6)
- moved P1 0.50 mm to (137.0, 119.0)
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Other:
- outline, holes or cut-outs redrawn

Commit message: wip
Parts:
- U1: footprint w_smd_dil:mdip_8 -> w_pth_circuits:dil_8-300_socket
- moved U5 22.1 mm to (141.6, 93.3)
- moved P4 15.6 mm to (151.8, 85.7)
- moved P5 15.6 mm to (158.8, 85.7)
- moved D7 11.9 mm to (144.8, 105.4), turned to 180 degrees
- moved R6 11.0 mm to (155.6, 111.1)
- moved D6 9.29 mm to (144.8, 103.5), turned to 0 degrees
- moved C1 8.37 mm to (144.8, 110.5)
- moved R3 8.34 mm to (144.8, 108.0)
- moved R4 7.71 mm to (156.2, 103.5)
- moved U3 7.08 mm to (155.6, 107.3)
- moved R5 5.64 mm to (148.6, 109.2)
- moved T1 4.19 mm to (137.2, 107.3)
- moved C5 3.18 mm to (153.7, 116.8)
- moved P3 2.86 mm to (146.6, 117.0)
- moved P1 2.80 mm to (137.2, 116.2)
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
Commit message: wip
Parts:
- moved D5 19.4 mm to (126.5, 91.5)
- moved U4 9.55 mm to (122.0, 111.0), turned to 180 degrees
- moved R1 6.80 mm to (128.5, 95.5)
- moved P8 3.04 mm to (128.0, 85.0)
- moved C2 2.55 mm to (121.0, 108.0), turned to 0 degrees
- moved D8 2.41 mm to (132.5, 98.5), turned to 90 degrees
- moved C4 1.50 mm to (128.0, 109.0), turned to 270 degrees
- moved U2 0.85 mm to (158.0, 116.0)
Other:
- outline, holes or cut-outs redrawn
Changed lines of the file:
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@@
     (area 117.924999 79.924999 168.075001 130.075001)
     (thickness 1.6)
-    (drawings 19)
+    (drawings 20)
     (tracks 0)
     (zones 0)
@@
   )
   (module Capacitors_SMD:C_0805_HandSoldering (layer F.Cu)
-    (at 120.5 110.5 270)
+    (at 121 108)
     (descr "Capacitor SMD 0805, hand soldering")
     (tags "capacitor 0805")
     (attr smd)
-    (fp_text reference C2 (at 0 -2.1 270) (layer F.SilkS)
-      (effects (font (size 1 1) (thickness 0.15)))
-    )
-    (fp_text value 100nF (at -0.127 0.0508 270) (layer F.Fab)
+    (fp_text reference C2 (at 0 -2.1) (layer F.SilkS)
+      (effects (font (size 1 1) (thickness 0.15)))
+    )
+    (fp_text value 100nF (at -0.127 0.0508) (layer F.Fab)
       (effects (font (size 1 1) (thickness 0.15)))
     )
@@
     (fp_line (start 0.5 -0.85) (end -0.5 -0.85) (layer F.SilkS) (width 0.15))
     (fp_line (start -0.5 0.85) (end 0.5 0.85) (layer F.SilkS) (width 0.15))
-    (pad 1 smd rect (at -1.25 0 270) (size 1.5 1.25) (layers F.Cu F.Paste F.Mask)
+    (pad 1 smd rect (at -1.25 0) (size 1.5 1.25) (layers F.Cu F.Paste F.Mask)
       (net 3 "Net-(C2-Pad1)"))
-    (pad 2 smd rect (at 1.25 0 270) (size 1.5 1.25) (layers F.Cu F.Paste F.Mask)
+    (pad 2 smd rect (at 1.25 0) (size 1.5 1.25) (layers F.Cu F.Paste F.Mask)
       (net 4 GNDA))
     (model Capacitors_SMD.3dshapes/C_0805_HandSoldering.wrl
@@
   )
   (module Capacitors_SMD:c_elec_4x5.3 (layer F.Cu)
-    (at 128 110.5 180)
+    (at 128 109 270)
     (descr "SMT capacitor, aluminium electrolytic, 4x5.3")
     (attr smd)
-    (fp_text reference C4 (at 5.0292 0.6604 180) (layer F.SilkS)
-      (effects (font (size 1 1) (thickness 0.15)))
-    )
-    (fp_text value 47uF (at 0.1524 -0.2286 180) (layer F.Fab)
+    (fp_text reference C4 (at 5.0292 0.6604 270) (layer F.SilkS)
+      (effects (font (size 1 1) (thickness 0.15)))
+    )
+    (fp_text value 47uF (at 0.1524 -0.2286 270) (layer F.Fab)
       (effects (font (size 1 1) (thickness 0.15)))
     )
@@
     (fp_line (start -2.286 -2.286) (end -2.286 2.286) (layer F.SilkS) (width 0.15))
     (fp_circle (center 0 0) (end -2.032 0) (layer F.SilkS) (width 0.15))
-    (pad 1 smd rect (at 1.80086 0 180) (size 2.60096 1.6002) (layers F.Cu F.Paste F.Mask)
+    (pad 1 smd rect (at 1.80086 0 270) (size 2.60096 1.6002) (layers F.Cu F.Paste F.Mask)
       (net 7 +5V))
-    (pad 2 smd rect (at -1.80086 0 180) (size 2.60096 1.6002) (layers F.Cu F.Paste F.Mask)
+    (pad 2 smd rect (at -1.80086 0 270) (size 2.60096 1.6002) (layers F.Cu F.Paste F.Mask)
       (net 4 GNDA))
     (model Capacitors_SMD.3dshapes/c_elec_4x5.3.wrl
@@
   )
   (module w_smd_diode:sod323 (layer F.Cu)
-    (at 122.5 110.5 90)
+    (at 126.5 91.5 90)
     (descr SOD323)
     (fp_text reference D5 (at -0.0762 1.143 90) (layer F.SilkS)
@@
   )
   (module Resistors_SMD:R_0805_HandSoldering (layer F.Cu)
-    (at 134 99.5 180)
+    (at 128.5 95.5 180)
     (descr "Resistor SMD 0805, hand soldering")
     (tags "resistor 0805")
@@
   )
   (module 78xx:TO-252-2Lead (layer F.Cu)
-    (at 158.115 116.84 270)
+    (at 158 116 270)
     (descr "DPAK / TO-252 2-lead smd package")
     (tags "dpak TO-252")
@@
   )
   (module 78xx:TO-252-2Lead (layer F.Cu)
-    (at 129 117.5 90)
+    (at 122 111 180)
     (descr "DPAK / TO-252 2-lead smd package")
     (tags "dpak TO-252")
     (attr smd)
-    (fp_text reference U4 (at 0 -10.414 90) (layer F.SilkS)
-      (effects (font (size 1 1) (thickness 0.15)))
-    )
-    (fp_text value 7805 (at 0 -2.413 90) (layer F.Fab)
+    (fp_text reference U4 (at 2.5 -10.5 180) (layer F.SilkS)
+      (effects (font (size 1 1) (thickness 0.15)))
+    )
+    (fp_text value 7805 (at 0 -2.413 180) (layer F.Fab)
       (effects (font (size 1 1) (thickness 0.15)))
     )
@@
     (fp_line (start -3.429 -9.525) (end 3.429 -9.525) (layer F.SilkS) (width 0.15))
     (fp_line (start 3.429 -9.398) (end 3.429 -7.62) (layer F.SilkS) (width 0.15))
-    (pad VI smd rect (at -2.286 0 90) (size 1.651 3.048) (layers F.Cu F.Paste F.Mask)
+    (pad VI smd rect (at -2.286 0 180) (size 1.651 3.048) (layers F.Cu F.Paste F.Mask)
       (net 3 "Net-(C2-Pad1)"))
-    (pad 1 smd rect (at 0 -6.35 90) (size 6.096 6.096) (layers F.Cu F.Paste F.Mask))
-    (pad VO smd rect (at 2.286 0 90) (size 1.651 3.048) (layers F.Cu F.Paste F.Mask)
+    (pad 1 smd rect (at 0 -6.35 180) (size 6.096 6.096) (layers F.Cu F.Paste F.Mask))
+    (pad VO smd rect (at 2.286 0 180) (size 1.651 3.048) (layers F.Cu F.Paste F.Mask)
       (net 7 +5V))
     (model TO_SOT_Packages_SMD.3dshapes/TO-252-2Lead.wrl
@@
   )
   (module w_smd_diode:sod323 (layer F.Cu)
-    (at 134.0405 96.647)
+    (at 132.5 98.5 90)
     (descr SOD323)
-    (fp_text reference D8 (at 0 -1.09982) (layer F.SilkS)
+    (fp_text reference D8 (at 0 -1.09982 90) (layer F.SilkS)
       (effects (font (size 0.39878 0.39878) (thickness 0.09906)))
     )
-    (fp_text value 1N4148 (at 0 1.19888) (layer F.SilkS) hide
+    (fp_text value 1N4148 (at 0 1.19888 90) (layer F.SilkS) hide
       (effects (font (size 0.39878 0.39878) (thickness 0.09906)))
     )
@@
     (fp_line (start -0.89916 0.70104) (end 0.89916 0.70104) (layer F.SilkS) (width 0.127))
     (fp_line (start 0.89916 0.70104) (end 0.89916 -0.70104) (layer F.SilkS) (width 0.127))
-    (pad 2 smd rect (at 1.09982 0) (size 1.7 1) (layers F.Cu F.Paste F.Mask)
+    (pad 2 smd rect (at 1.09982 0 90) (size 1.7 1) (layers F.Cu F.Paste F.Mask)
       (net 38 "Net-(D8-Pad2)"))
-    (pad 1 smd rect (at -1.09982 0) (size 1.7 1) (layers F.Cu F.Paste F.Mask)
+    (pad 1 smd rect (at -1.09982 0 90) (size 1.7 1) (layers F.Cu F.Paste F.Mask)
       (net 10 /brown))
     (model walter/smd_diode/sod323.wrl
@@
   )
   (module Socket_Strips:Socket_Strip_Straight_2x04 (layer B.Cu)
-    (at 131 85.5)
+    (at 128 85)
     (descr "Through hole socket strip")
     (tags "socket strip")
@@
     )
   )
-  (dimension 9.5 (width 0.3) (layer Dwgs.User)
-    (gr_text "9,500 mm" (at 133.35 125.25 270) (layer Dwgs.User)
+  (dimension 10.5 (width 0.3) (layer Dwgs.User)
+    (gr_text "10.500 mm" (at 135.85 124.75 90) (layer Dwgs.User)
       (effects (font (size 1.5 1.5) (thickness 0.3)))
     )
-    (feature1 (pts (xy 128 130) (xy 134.7 130)))
-    (feature2 (pts (xy 128 120.5) (xy 134.7 120.5)))
-    (crossbar (pts (xy 132 120.5) (xy 132 130)))
-    (arrow1a (pts (xy 132 130) (xy 131.413579 128.873496)))
-    (arrow1b (pts (xy 132 130) (xy 132.586421 128.873496)))
-    (arrow2a (pts (xy 132 120.5) (xy 131.413579 121.626504)))
-    (arrow2b (pts (xy 132 120.5) (xy 132.586421 121.626504)))
+    (feature1 (pts (xy 129.5 119.5) (xy 137.2 119.5)))
+    (feature2 (pts (xy 129.5 130) (xy 137.2 130)))
+    (crossbar (pts (xy 134.5 130) (xy 134.5 119.5)))
+    (arrow1a (pts (xy 134.5 119.5) (xy 135.086421 120.626504)))
+    (arrow1b (pts (xy 134.5 119.5) (xy 133.913579 120.626504)))
+    (arrow2a (pts (xy 134.5 130) (xy 135.086421 128.873496)))
+    (arrow2b (pts (xy 134.5 130) (xy 133.913579 128.873496)))
+  )
+  (gr_line (start 126.5 128.5) (end 126.5 120.5) (angle 90) (layer Edge.Cuts) (width 0.15))
+  (gr_line (start 119.5 130) (end 125 130) (angle 90) (layer Edge.Cuts) (width 0.15))
+  (gr_line (start 161 130) (end 166.5 130) (angle 90) (layer Edge.Cuts) (width 0.15))
+  (gr_line (start 159.5 120.5) (end 159.5 128.5) (angle 90) (layer Edge.Cuts) (width 0.15))
+  (gr_line (start 127.5 119.5) (end 158.5 119.5) (angle 90) (layer Edge.Cuts) (width 0.15))
+  (dimension 8.5 (width 0.3) (layer Dwgs.User)
+    (gr_text "8.500 mm" (at 122.25 133.85) (layer Dwgs.User)
+      (effects (font (size 1.5 1.5) (thickness 0.3)))
+    )
+    (feature1 (pts (xy 126.5 127.5) (xy 126.5 135.2)))
+    (feature2 (pts (xy 118 127.5) (xy 118 135.2)))
+    (crossbar (pts (xy 118 132.5) (xy 126.5 132.5)))
+    (arrow1a (pts (xy 126.5 132.5) (xy 125.373496 133.086421)))
+    (arrow1b (pts (xy 126.5 132.5) (xy 125.373496 131.913579)))
+    (arrow2a (pts (xy 118 132.5) (xy 119.126504 133.086421)))
+    (arrow2b (pts (xy 118 132.5) (xy 119.126504 131.913579)))
   )
   (dimension 50 (width 0.3) (layer Dwgs.User)
@@
     (arrow2b (pts (xy 118 138.5) (xy 119.126504 137.913579)))
   )
-  (gr_line (start 159.5 130) (end 166.5 130) (angle 90) (layer Edge.Cuts) (width 0.15))
-  (gr_line (start 158 121.5) (end 158 128.5) (angle 90) (layer Edge.Cuts) (width 0.15))
-  (gr_line (start 129 120.5) (end 157 120.5) (angle 90) (layer Edge.Cuts) (width 0.15))
-  (gr_line (start 128 128.5) (end 128 121.5) (angle 90) (layer Edge.Cuts) (width 0.15))
-  (gr_line (start 119.5 130) (end 126.5 130) (angle 90) (layer Edge.Cuts) (width 0.15))
-  (gr_arc (start 129 121.5) (end 128 121.5) (angle 90) (layer Edge.Cuts) (width 0.15))
-  (gr_arc (start 157 121.5) (end 157 120.5) (angle 90) (layer Edge.Cuts) (width 0.15))
-  (gr_arc (start 159.5 128.5) (end 159.5 130) (angle 90) (layer Edge.Cuts) (width 0.15))
-  (gr_arc (start 126.5 128.5) (end 128 128.5) (angle 90) (layer Edge.Cuts) (width 0.15))
+  (gr_arc (start 127.5 120.5) (end 126.5 120.5) (angle 90) (layer Edge.Cuts) (width 0.15))
+  (gr_arc (start 158.5 120.5) (end 158.5 119.5) (angle 90) (layer Edge.Cuts) (width 0.15))
+  (gr_arc (start 161 128.5) (end 161 130) (angle 90) (layer Edge.Cuts) (width 0.15))
+  (gr_arc (start 125 128.5) (end 126.5 128.5) (angle 90) (layer Edge.Cuts) (width 0.15))
   (gr_line (start 168 128.5) (end 168 81.5) (angle 90) (layer Edge.Cuts) (width 0.15))
   (gr_line (start 118 81.5) (end 118 128.5) (angle 90) (layer Edge.Cuts) (width 0.15))

Commit message: wip
Parts:
- removed P3: 18V, w_conn_pt-1,5:pt_1,5-2-3,5-h
- P1: value Rail -> CONN_01X04; footprint Wire_Pads:SolderWirePad_2x_1-5mmDrill -> w_conn_mkds:akl0711,5-4
- U4: value 7805 -> 78L05; footprint 78xx:TO-252-2Lead -> TO_SOT_Packages_SMD:SOT89-3_Housing_Handsoldering
- moved R8 19.4 mm to (90.6, 110.5), turned to 180 degrees
- moved C2 14.8 mm to (123.1, 93.3)
- moved R9 14.0 mm to (90.6, 113.1), turned to 180 degrees
- moved R14 12.4 mm to (90.6, 126.3), turned to 180 degrees
- moved R7 9.96 mm to (100.4, 107.6)
- moved R10 8.67 mm to (90.6, 115.7), turned to 180 degrees
- moved U4 7.40 mm to (122.2, 118.4), turned to 90 degrees
- moved R13 7.34 mm to (90.6, 123.7), turned to 180 degrees
- moved C4 6.76 mm to (122.7, 113.2), turned to 0 degrees
- moved C1 5.47 mm to (148.7, 114.3), turned to 90 degrees
- moved R6 5.28 mm to (150.7, 109.1), turned to 90 degrees
- moved P2 3.57 mm to (120.9, 104.0)
- moved R11 3.34 mm to (90.6, 118.4), turned to 180 degrees
- moved C3 3.31 mm to (152.6, 112.5)
- moved R1 3.24 mm to (127.9, 98.7)
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Connections:
- C2 pad 1: Net-(C2-Pad1) -> /VI
- C3 pad 1: Net-(C3-Pad1) -> /18V+
- D5 pad 2: Net-(C2-Pad1) -> /VI
- U2 pad VI: Net-(C3-Pad1) -> /18V+

Commit message: wip
Parts:
- C1: value 1nF -> 100nF
- D1, D2, D3, D4, D5: value 1N4007 -> US1M; footprint w_smd_diode:sod323 -> w_smd_diode:do214ac
- moved R10 74.1 mm to (164.3, 108.6), turned to 0 degrees
- moved R11 74.1 mm to (164.3, 111.3), turned to 0 degrees
- moved R12 74.1 mm to (164.3, 114.0), turned to 0 degrees
- moved R9 74.1 mm to (164.3, 106.0), turned to 0 degrees
- moved R13 74.1 mm to (164.3, 116.6), turned to 0 degrees
- moved R14 74.1 mm to (164.3, 119.3), turned to 0 degrees
- moved R8 74.1 mm to (164.3, 103.5), turned to 0 degrees
- moved P6 58.6 mm to (158.5, 117.7)
- moved R7 53.4 mm to (153.0, 116.6), turned to 270 degrees
- moved Q1 49.2 mm to (149.9, 116.5)
- moved D10 33.4 mm to (145.7, 100.6), turned to 0 degrees
- moved U1 30.4 mm to (124.2, 91.9)
- moved C6 28.1 mm to (131.8, 87.8), turned to 180 degrees
- moved R15 27.1 mm to (148.7, 97.8), turned to 270 degrees
- moved D9 26.5 mm to (157.6, 86.0)
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
Commit message: wip
Parts:
- C4, C5: footprint Capacitors_SMD:c_elec_4x5.3 -> Capacitors_SMD:c_elec_5x5.3
- R1: value 1k8 -> 1k5; footprint Resistors_SMD:R_0805_HandSoldering -> Resistors_SMD:R_1206_HandSoldering
- moved C2 32.9 mm to (119.5, 122.0), turned to 90 degrees
- moved C3 13.3 mm to (158.2, 102.6)
- moved R4 9.48 mm to (151.1, 112.8)
- moved R1 6.09 mm to (130.5, 92.5)
- moved D8 2.59 mm to (133.0, 96.5)
- moved R17 2.22 mm to (133.0, 91.0)
- moved C4 1.39 mm to (122.0, 112.0)
- moved U4 0.92 mm to (122.0, 117.5)
- moved C5 0.71 mm to (153.0, 99.0)
- moved C6 0.31 mm to (132.0, 87.5)

Commit message: wip
Parts:
- moved C1 14.9 mm to (149.4, 104.1)
- moved C3 9.02 mm to (159.8, 93.7), turned to 0 degrees
- moved R4 1.02 mm to (150.1, 112.8)
- moved U3 0.65 mm to (156.7, 108.0)
- moved R7 0.28 mm to (153.2, 116.8)
- moved U2 0.25 mm to (157.7, 98.3)
- moved R6 0.21 mm to (150.9, 109.2)
- moved R5 0.12 mm to (148.6, 109.2)
- moved C5 0.11 mm to (152.9, 99.1), turned to 270 degrees
Changed lines of the file:
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@@
   )
   (module Capacitors_SMD:C_0805_HandSoldering (layer F.Cu)
-    (at 160.147 93.853)
+    (at 149.352 104.14)
     (descr "Capacitor SMD 0805, hand soldering")
     (tags "capacitor 0805")
@@
   )
   (module Capacitors_SMD:C_0805_HandSoldering (layer F.Cu)
-    (at 158.242 102.616 180)
+    (at 159.766 93.726)
     (descr "Capacitor SMD 0805, hand soldering")
     (tags "capacitor 0805")
     (attr smd)
-    (fp_text reference C3 (at -3.302 0.127 180) (layer F.SilkS)
-      (effects (font (size 1 1) (thickness 0.15)))
-    )
-    (fp_text value 100nF (at 0.0508 0.2794 180) (layer F.Fab)
+    (fp_text reference C3 (at 3.556 0.254) (layer F.SilkS)
+      (effects (font (size 1 1) (thickness 0.15)))
+    )
+    (fp_text value 100nF (at 0.0508 0.2794) (layer F.Fab)
       (effects (font (size 1 1) (thickness 0.15)))
     )
@@
     (fp_line (start 0.5 -0.85) (end -0.5 -0.85) (layer F.SilkS) (width 0.15))
     (fp_line (start -0.5 0.85) (end 0.5 0.85) (layer F.SilkS) (width 0.15))
-    (pad 1 smd rect (at -1.25 0 180) (size 1.5 1.25) (layers F.Cu F.Paste F.Mask)
+    (pad 1 smd rect (at -1.25 0) (size 1.5 1.25) (layers F.Cu F.Paste F.Mask)
       (net 41 /18V+))
-    (pad 2 smd rect (at 1.25 0 180) (size 1.5 1.25) (layers F.Cu F.Paste F.Mask)
+    (pad 2 smd rect (at 1.25 0) (size 1.5 1.25) (layers F.Cu F.Paste F.Mask)
       (net 4 GND))
     (model Capacitors_SMD.3dshapes/C_0805_HandSoldering.wrl
@@
     (tags SOT-23)
     (attr smd)
-    (fp_text reference Q1 (at 0 -2.25 90) (layer F.SilkS)
+    (fp_text reference Q1 (at 1.651 -1.778 90) (layer F.SilkS)
       (effects (font (size 1 1) (thickness 0.15)))
     )
@@
   )
   (module Resistors_SMD:R_0805_HandSoldering (layer F.Cu)
-    (at 151.13 112.776)
+    (at 150.114 112.776)
     (descr "Resistor SMD 0805, hand soldering")
     (tags "resistor 0805")
     (attr smd)
-    (fp_text reference R4 (at 3.39 -0.005) (layer F.SilkS)
+    (fp_text reference R4 (at 3.556 -0.762) (layer F.SilkS)
       (effects (font (size 1 1) (thickness 0.15)))
     )
@@
   )
   (module Resistors_SMD:R_0805_HandSoldering (layer F.Cu)
-    (at 148.6 109.1 270)
+    (at 148.59 109.22 270)
     (descr "Resistor SMD 0805, hand soldering")
     (tags "resistor 0805")
@@
   )
   (module Resistors_SMD:R_0805_HandSoldering (layer F.Cu)
-    (at 150.7 109.1 90)
+    (at 150.876 109.22 90)
     (descr "Resistor SMD 0805, hand soldering")
     (tags "resistor 0805")
@@
   )
   (module Resistors_SMD:R_0805_HandSoldering (layer F.Cu)
-    (at 153.035 116.586 270)
+    (at 153.162 116.84 270)
     (descr "Resistor SMD 0805, hand soldering")
     (tags "resistor 0805")
     (attr smd)
-    (fp_text reference R7 (at 2.414 2.035 360) (layer F.SilkS)
+    (fp_text reference R7 (at -3.302 -0.508 450) (layer F.SilkS)
       (effects (font (size 1 1) (thickness 0.15)))
     )
@@
   )
   (module 78xx:TO-252-2Lead (layer F.Cu)
-    (at 157.48 98.298 270)
+    (at 157.734 98.298 270)
     (descr "DPAK / TO-252 2-lead smd package")
     (tags "dpak TO-252")
@@
   )
   (module w_smd_dil:so-8 (layer F.Cu)
-    (at 156.7 108.6 270)
+    (at 156.718 107.95 270)
     (descr SO-8)
     (fp_text reference U3 (at -0.2186 -0.5704 270) (layer F.SilkS)
@@
   )
   (module Capacitors_SMD:c_elec_5x5.3 (layer F.Cu)
-    (at 153 99 90)
+    (at 152.908 99.06 270)
     (descr "SMT capacitor, aluminium electrolytic, 5x5.3")
     (attr smd)
-    (fp_text reference C5 (at 0 2 90) (layer F.SilkS)
-      (effects (font (size 1 1) (thickness 0.15)))
-    )
-    (fp_text value 47uF (at 0 3.81 90) (layer F.Fab)
+    (fp_text reference C5 (at 0 2 270) (layer F.SilkS)
+      (effects (font (size 1 1) (thickness 0.15)))
+    )
+    (fp_text value 47uF (at 0 3.81 270) (layer F.Fab)
       (effects (font (size 1 1) (thickness 0.15)))
     )
@@
     (fp_line (start 1.778 -0.381) (end 1.778 0.381) (layer F.SilkS) (width 0.15))
     (fp_circle (center 0 0) (end -2.413 0) (layer F.SilkS) (width 0.15))
-    (pad 1 smd rect (at 2.19964 0 90) (size 2.99974 1.6002) (layers F.Cu F.Paste F.Mask)
+    (pad 1 smd rect (at 2.19964 0 270) (size 2.99974 1.6002) (layers F.Cu F.Paste F.Mask)
       (net 6 VCC))
-    (pad 2 smd rect (at -2.19964 0 90) (size 2.99974 1.6002) (layers F.Cu F.Paste F.Mask)
+    (pad 2 smd rect (at -2.19964 0 270) (size 2.99974 1.6002) (layers F.Cu F.Paste F.Mask)
       (net 4 GND))
     (model Capacitors_SMD.3dshapes/c_elec_5x5.3.wrl
