File: mfx-link2/mfx-link2.sch (KiCad schematic (older format))
At the start: 24 parts

Commit message: wip
Parts:
- removed Q?: BC817-40, SOT-23, symbol BC817-40
- added D? (x4): D, w_smd_diode:sod323, symbol D
- added P?: POTI, Pin_Headers:Pin_Header_Straight_1x03, symbol CONN_01X03
- added P?: CONN_02X03, symbol CONN_02X03
- added P?: CONN_01X02, symbol CONN_01X02
- added Q?: BC817-40, SOT-23, symbol BC817-40
- added R? (x7): 1K5, Resistors_SMD:R_1206_HandSoldering, symbol R
- added R?: 1k, Resistors_SMD:R_0805_HandSoldering, symbol R
- added U?: 7805, 78xx:TO-252-2Lead, symbol 7805
- P?: footprint (none) -> w_conn_pt-1,5:pt_1,5-2-3,5-h
- P? (x2): footprint (none) -> w_conn_jst-ph:b4b-ph-kl
- U?: footprint (none) -> 78xx:TO-252-2Lead
Connections:
- net +5V: now also P?.2 (P2), P?.2 (P2), P?.3 (P3)
- net GND: now also P?.1 (P1), P?.1 (P1), P?.1 (P1)
- net GB_OUT: now reaches U?.12 (RB5)
- net GB_IN: now reaches U?.13 (RB4)
- net at U?.19 (IDAT/RA0): now also P?.2 (P2)
- net LED: now reaches R?.1, U?.5 (RC5)
- net RxD: now reaches U?.6 (RC4)
- net RxD: now also P?.4 (P4)
- net TxD: now reaches U?.7 (RC3)
- net TxD: now also P?.3 (P3)
- net SDA: now reaches U?.8 (RC6)
- net SDA: now also P?.4 (P4)
- net SCL: now reaches U?.9 (RC7)
- net SCL: now also P?.3 (P3)
- new net: Q?.1 (B), R?.2
- new net: Q?.3 (C), R?.2, R?.2, R?.2, R?.2, R?.2, R?.2, R?.2
- new net: P?.2 (P2), R?.1, R?.1, R?.1
- new net: P?.4 (P4), R?.1, R?.1
- new net: P?.6 (P6), R?.1
- new net GNDA: Q?.2 (E)
- new net _GB_OUT: R?.1
- no-connect marks 0 -> 2
Other:
- moved on the sheet: C?, D?, P?, R?, T?, U?

Commit message: wip
Parts:
- removed C?: C, Capacitors_SMD:C_0805_HandSoldering, symbol C
- added C2: 100nF, Capacitors_SMD:C_0805_HandSoldering, symbol C
- added C4, C5: 47uF, Capacitors_SMD:c_elec_4x5.3, symbol CP
- added D10: 1N4148, w_smd_diode:sod323, symbol D
- added D5, D6, D7: 1N4007, w_smd_diode:sod323, symbol D
- added JP1: ICSP, ICSP:ICSP, symbol ICSP
- added R1: 1k8, Resistors_SMD:R_0805_HandSoldering, symbol R
- added R2: 390, Resistors_SMD:R_0805_HandSoldering, symbol R
- added U1: 6N137, w_smd_dil:mdip_8, symbol 6N135
- added U3: LM393, w_smd_dil:so-8, symbol LM393
- C3: renamed from C?; value C -> 100nF
- D1, D2, D3, D4: renamed from D?; value D -> 1N4007
- D12: renamed from D?; value Led_Small -> LED; footprint (none) -> LEDs:LED_0805
- P1: renamed from P?; footprint (none) -> Wire_Pads:SolderWirePad_2x_1-5mmDrill
- P2: renamed from P?; value CONN_01X02 -> Gleisbox; footprint (none) -> w_conn_pt-1,5:pt_1,5-2-3,5-h
- P6: renamed from P?; footprint (none) -> Pin_Headers:Pin_Header_Straight_2x03
- Q1: renamed from Q?; footprint SOT-23 -> TO_SOT_Packages_SMD:SOT-23
- gave numbers to parts that had none: 29
Connections:
- net GB_IN is gone; now on net ENABLE: U5.13 (RB4)
- net GB_OUT is gone; now on net RPWM: U5.12 (RB5)
- net +5V: now also U4.VO, C4.1, U3.8 (V+); no longer C6.1, D11.2 (A), D12.2 (A), P4.2 (P2), P5.2 (P2), P7.3 (P3), P8.7 (P7), R17.1, U2.VO, U5.1 (Vdd)
- net ENABLE: no longer U5.16 (RC0)
- net GND: now also C5.2, JP1.3 (Vss), U1.5; no longer R6.1
- net GNDA: now also D1.1 (A), D2.1 (A), R6.1, U4.GND, C2.2, C4.2, U3.4 (V-)
- net LPWM: now also U5.11 (RB6); no longer U5.14 (RC2)
- net MCLR: now also JP1.1 (VPP/~MCLR)
- net RPWM: no longer U5.15 (RC1)
- net RxD: now also U5.15 (RC1); no longer U5.6 (RC4)
- net SCL: now also U5.2 (RA5); no longer U5.9 (RC7)
- net SDA: now also U5.3 (RA4); no longer U5.8 (RC6)
- net SENSE: now also U5.16 (RC0); no longer U5.17 (RA2)
- net TxD: now also U5.14 (RC2); no longer U5.7 (RC3)
- net _GB_OUT: now also U3.1
- net PGC: now reaches U5.18 (ICLK/RA1)
- net PGC: now also JP1.5 (PGC)
- net at P7.2 (P2): now also U5.17 (RA2); no longer U5.19 (IDAT/RA0)
- net at R3.1, R4.1, R5.1: now also U3.2 (-); no longer U5.2 (RA5)
- net at C1.2, D8.2 (K), D9.1 (A)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: now also U3.3 (+); no longer U5.3 (RA4)
- net at P1.1 (P1), T1.7 (SA): now also D6.1 (A), D7.2 (K)
- net at P1.2 (P2), T1.8 (SB): now also D6.2 (K), D7.1 (A)
- net at P6.2 (P2), R11.1, R12.1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: now also R13.1
- net at P6.1 (P1): now also D3.2 (K), D4.2 (K), P6.3 (P3), P6.5 (P5), D5.1 (A)
- net brown: now reaches D4.1 (A)
- net brown: now also D2.2 (K), P2.2 (P2), D10.1 (A), U1.3
- net red: now reaches D3.1 (A)
- net red: now also D1.2 (K), P2.1 (P1), R1.2
- net at U4.VI: now also C2.1, D5.2 (K)
- new net: D10.2 (K), R1.1, U1.2
- new net PGD: JP1.4 (PGD), U5.19 (IDAT/RA0)
- new net PULSE: R2.2, U1.6, U5.7 (RC3)
- new net VCC: C5.1, C6.1, D11.2 (A), D12.2 (A), JP1.2 (Vdd), P4.2 (P2), P5.2 (P2), P7.3 (P3), P8.7 (P7), R17.1, R2.1, U1.7, U1.8, U2.VO, U5.1 (Vdd)
- no-connect marks 2 -> 5
Other:
- moved on the sheet: C1, C3, C6, D1, D11, D12, D2, D3, D4, D8, D9, P1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

Commit message: wip
Parts:
- removed D6, D7: 1N4007, w_smd_diode:sod323, symbol D
- D1, D2, D3, D4, D5: symbol D -> D-RESCUE-mfx-link2
- D6: renamed from D8; symbol D -> D-RESCUE-mfx-link2
- D7: renamed from D9; symbol D -> D-RESCUE-mfx-link2
- D8: renamed from D10; symbol D -> D-RESCUE-mfx-link2
- U3: symbol LM393 -> LM393-RESCUE-mfx-link2
- renumbered D12 to D10, D11 to D9
Other:
- moved on the sheet: D1, D2, D3, D4, D5, P1, P2
Changed lines of the file:
@@
 EESchema Schematic File Version 2
+LIBS:mfx-link2-rescue
 LIBS:power
 LIBS:device
@@
 L CONN_01X02 P1
 U 1 1 58FE254A
-P 850 6750
-F 0 "P1" H 850 6900 50  0000 C CNN
-F 1 "Rail" V 950 6750 50  0000 C CNN
-F 2 "Wire_Pads:SolderWirePad_2x_1-5mmDrill" H 850 6750 50  0001 C CNN
-F 3 "" H 850 6750 50  0000 C CNN
-	1    850  6750
+P 1450 6750
+F 0 "P1" H 1450 6900 50  0000 C CNN
+F 1 "Rail" V 1550 6750 50  0000 C CNN
+F 2 "Wire_Pads:SolderWirePad_2x_1-5mmDrill" H 1450 6750 50  0001 C CNN
+F 3 "" H 1450 6750 50  0000 C CNN
+	1    1450 6750
 	-1   0    0    1
 $EndComp
 $Comp
-L D D8
+L D-RESCUE-mfx-link2 D6
 U 1 1 58FE266D
 P 2425 6750
-F 0 "D8" H 2425 6850 50  0000 C CNN
+F 0 "D6" H 2425 6850 50  0000 C CNN
 F 1 "1N4148" H 2425 6650 50  0000 C CNN
 F 2 "w_smd_diode:sod323" H 2425 6750 50  0001 C CNN
@@
 $EndComp
 $Comp
-L D D9
+L D-RESCUE-mfx-link2 D7
 U 1 1 58FE27B5
 P 2700 6750
-F 0 "D9" H 2700 6650 50  0000 C CNN
+F 0 "D7" H 2700 6650 50  0000 C CNN
 F 1 "1N4148" H 2700 6875 50  0000 C CNN
 F 2 "w_smd_diode:sod323" H 2700 6750 50  0001 C CNN
@@
 $EndComp
 $Comp
-L D_Schottky D11
+L D_Schottky D9
 U 1 1 58FE485B
 P 6450 1425
-F 0 "D11" H 6450 1300 50  0000 C CNN
+F 0 "D9" H 6450 1300 50  0000 C CNN
 F 1 "BAT43" H 6625 1375 50  0000 C CNN
 F 2 "w_smd_diode:sod323" H 6450 1425 50  0001 C CNN
@@
 $EndComp
 $Comp
-L Led_Small D12
+L Led_Small D10
 U 1 1 58FE78BA
 P 6250 1425
-F 0 "D12" H 6200 1550 50  0000 L CNN
+F 0 "D10" H 6200 1550 50  0000 L CNN
 F 1 "LED" H 6300 1375 50  0000 L CNN
 F 2 "LEDs:LED_0805" V 6250 1425 50  0001 C CNN
@@
 $EndComp
 $Comp
-L D D4
+L D-RESCUE-mfx-link2 D4
 U 1 1 58FFE9CD
-P 2375 4700
-F 0 "D4" H 2200 4650 50  0000 C CNN
-F 1 "1N4007" H 2375 4600 50  0000 C CNN
-F 2 "w_smd_diode:sod323" H 2375 4700 50  0001 C CNN
-F 3 "" H 2375 4700 50  0000 C CNN
-	1    2375 4700
+P 2700 4700
+F 0 "D4" H 2525 4650 50  0000 C CNN
+F 1 "1N4007" H 2700 4600 50  0000 C CNN
+F 2 "w_smd_diode:sod323" H 2700 4700 50  0001 C CNN
+F 3 "" H 2700 4700 50  0000 C CNN
+	1    2700 4700
 	0    -1   -1   0
 $EndComp
 $Comp
-L D D3
+L D-RESCUE-mfx-link2 D3
 U 1 1 58FFEBB8
-P 2175 4700
-F 0 "D3" H 2000 4650 50  0000 C CNN
-F 1 "1N4007" H 2175 4600 50  0000 C CNN
-F 2 "w_smd_diode:sod323" H 2175 4700 50  0001 C CNN
-F 3 "" H 2175 4700 50  0000 C CNN
-	1    2175 4700
+P 2500 4700
+F 0 "D3" H 2325 4650 50  0000 C CNN
+F 1 "1N4007" H 2500 4600 50  0000 C CNN
+F 2 "w_smd_diode:sod323" H 2500 4700 50  0001 C CNN
+F 3 "" H 2500 4700 50  0000 C CNN
+	1    2500 4700
 	0    -1   -1   0
 $EndComp
 $Comp
-L D D2
+L D-RESCUE-mfx-link2 D2
 U 1 1 58FFEC40
-P 1925 4700
-F 0 "D2" H 2100 4750 50  0000 C CNN
-F 1 "1N4007" H 1925 4800 50  0000 C CNN
-F 2 "w_smd_diode:sod323" H 1925 4700 50  0001 C CNN
-F 3 "" H 1925 4700 50  0000 C CNN
-	1    1925 4700
+P 2250 4700
+F 0 "D2" H 2425 4750 50  0000 C CNN
+F 1 "1N4007" H 2250 4800 50  0000 C CNN
+F 2 "w_smd_diode:sod323" H 2250 4700 50  0001 C CNN
+F 3 "" H 2250 4700 50  0000 C CNN
+	1    2250 4700
 	0    1    1    0
 $EndComp
 $Comp
-L D D1
+L D-RESCUE-mfx-link2 D1
 U 1 1 58FFECE5
-P 1700 4700
-F 0 "D1" H 1875 4750 50  0000 C CNN
-F 1 "1N4007" H 1700 4800 50  0000 C CNN
-F 2 "w_smd_diode:sod323" H 1700 4700 50  0001 C CNN
-F 3 "" H 1700 4700 50  0000 C CNN
-	1    1700 4700
+P 2025 4700
+F 0 "D1" H 2200 4750 50  0000 C CNN
+F 1 "1N4007" H 2025 4800 50  0000 C CNN
+F 2 "w_smd_diode:sod323" H 2025 4700 50  0001 C CNN
+F 3 "" H 2025 4700 50  0000 C CNN
+	1    2025 4700
 	0    1    1    0
 $EndComp
@@
 $EndComp
 $Comp
-L D D10
+L D-RESCUE-mfx-link2 D8
 U 1 1 590921A7
 P 2200 3000
-F 0 "D10" H 2200 3100 50  0000 C CNN
+F 0 "D8" H 2200 3100 50  0000 C CNN
 F 1 "1N4148" H 2200 2900 50  0000 C CNN
 F 2 "w_smd_diode:sod323" H 2200 3000 50  0001 C CNN
@@
 $EndComp
 $Comp
-L D D5
+L D-RESCUE-mfx-link2 D5
 U 1 1 5909499E
-P 2525 5150
-F 0 "D5" H 2525 5050 50  0000 C CNN
-F 1 "1N4007" H 2525 5250 50  0000 C CNN
-F 2 "w_smd_diode:sod323" H 2525 5150 50  0001 C CNN
-F 3 "" H 2525 5150 50  0000 C CNN
-	1    2525 5150
+P 2850 5150
+F 0 "D5" H 2850 5050 50  0000 C CNN
+F 1 "1N4007" H 2850 5250 50  0000 C CNN
+F 2 "w_smd_diode:sod323" H 2850 5150 50  0001 C CNN
+F 3 "" H 2850 5150 50  0000 C CNN
+	1    2850 5150
 	-1   0    0    1
 $EndComp
@@
 L CONN_01X02 P2
 U 1 1 59002303
-P 1175 4450
-F 0 "P2" H 1175 4600 50  0000 C CNN
-F 1 "Gleisbox" V 1275 4450 50  0000 C CNN
-F 2 "w_conn_pt-1,5:pt_1,5-2-3,5-h" H 1175 4450 50  0001 C CNN
-F 3 "" H 1175 4450 50  0000 C CNN
-	1    1175 4450
+P 1500 4450
+F 0 "P2" H 1500 4600 50  0000 C CNN
+F 1 "Gleisbox" V 1600 4450 50  0000 C CNN
+F 2 "w_conn_pt-1,5:pt_1,5-2-3,5-h" H 1500 4450 50  0001 C CNN
+F 3 "" H 1500 4450 50  0000 C CNN
+	1    1500 4450
 	-1   0    0    1
 $EndComp
@@
 	1    0    0    -1
 $EndComp
-Text Label 1400 4500 0    60   ~ 0
+Text Label 1725 4500 0    60   ~ 0
 red
-Text Label 1400 4400 0    60   ~ 0
+Text Label 1725 4400 0    60   ~ 0
 brown
 Text Label 1400 3150 0    60   ~ 0
@@
 $EndComp
 $Comp
-L LM393 U3
+L LM393-RESCUE-mfx-link2 U3
 U 1 1 5908B602
 P 4050 6750
@@
 	1    4050 6750
 	1    0    0    -1
-$EndComp
-$Comp
-L D D6
-U 1 1 590937E6
-P 1350 6750
-F 0 "D6" H 1475 6700 50  0000 C CNN
-F 1 "1N4007" H 1350 6850 50  0000 C CNN
-F 2 "w_smd_diode:sod323" H 1350 6750 50  0001 C CNN
-F 3 "" H 1350 6750 50  0000 C CNN
-	1    1350 6750
-	0    1    1    0
-$EndComp
-$Comp
-L D D7
-U 1 1 590938DF
-P 1600 6750
-F 0 "D7" H 1475 6800 50  0000 C CNN
-F 1 "1N4007" H 1600 6650 50  0000 C CNN
-F 2 "w_smd_diode:sod323" H 1600 6750 50  0001 C CNN
-F 3 "" H 1600 6750 50  0000 C CNN
-	1    1600 6750
-	0    -1   -1   0
 $EndComp
 $Comp
@@
 	3525 6450 3525 6600
 Wire Wire Line
-	1050 6700 1200 6700
-Wire Wire Line
-	1200 6700 1200 6550
-Wire Wire Line
-	1200 6550 1750 6550
-Wire Wire Line
-	1750 6950 1200 6950
-Wire Wire Line
-	1200 6950 1200 6800
-Wire Wire Line
-	1200 6800 1050 6800
+	1650 6700 1700 6700
+Wire Wire Line
+	1700 6700 1700 6550
+Wire Wire Line
+	1700 6550 1750 6550
+Wire Wire Line
+	1750 6950 1700 6950
+Wire Wire Line
+	1700 6950 1700 6800
+Wire Wire Line
+	1700 6800 1650 6800
 Connection ~ 3525 6550
 Connection ~ 3525 6950
@@
 	5475 5625 5475 5825
 Wire Wire Line
-	1375 4500 2175 4500
-Wire Wire Line
-	1700 4500 1700 4550
-Wire Wire Line
-	2175 4500 2175 4550
-Connection ~ 1700 4500
-Wire Wire Line
-	1375 4400 2375 4400
-Wire Wire Line
-	2375 4400 2375 4550
-Wire Wire Line
-	1925 4550 1925 4400
-Connection ~ 1925 4400
+	1700 4500 2500 4500
+Wire Wire Line
+	2025 4500 2025 4550
+Wire Wire Line
+	2500 4500 2500 4550
+Connection ~ 2025 4500
+Wire Wire Line
+	1700 4400 2700 4400
+Wire Wire Line
+	2700 4400 2700 4550
+Wire Wire Line
+	2250 4550 2250 4400
+Connection ~ 2250 4400
 Wire Wire Line
 	4150 5450 4150 5750
 Wire Wire Line
-	1800 5600 1800 4950
-Wire Wire Line
-	1700 4850 1700 4950
-Wire Wire Line
-	1700 4950 1925 4950
-Wire Wire Line
-	1925 4950 1925 4850
-Connection ~ 1800 4950
-Wire Wire Line
-	2175 4850 2175 4950
-Wire Wire Line
-	2375 4850 2375 5150
-Connection ~ 2375 4950
+	2125 5600 2125 4950
+Wire Wire Line
+	2025 4850 2025 4950
+Wire Wire Line
+	2025 4950 2250 4950
+Wire Wire Line
+	2250 4950 2250 4850
+Connection ~ 2125 4950
+Wire Wire Line
+	2500 4850 2500 4950
+Wire Wire Line
+	2700 4850 2700 5150
+Connection ~ 2700 4950
 Wire Wire Line
 	5475 5050 5675 5050
 Wire Wire Line
-	2575 4950 2575 4400
-Wire Wire Line
-	2175 4950 2575 4950
+	2900 4950 2900 4400
+Wire Wire Line
+	2500 4950 2900 4950
 Wire Wire Line
 	3700 5600 3700 5550
@@
 	1750 2850 1400 2850
 Wire Wire Line
-	2675 5150 3750 5150
-Wire Wire Line
-	2575 4400 5575 4400
-Wire Wire Line
-	1800 5600 4650 5600
+	3000 5150 3750 5150
+Wire Wire Line
+	2125 5600 4650 5600
 Wire Wire Line
 	3000 3200 3100 3200
@@
 Wire Wire Line
 	3175 2600 3175 2700
-Wire Wire Line
-	1350 6600 1350 6550
-Connection ~ 1350 6550
-Wire Wire Line
-	1600 6550 1600 6600
-Connection ~ 1600 6550
-Wire Wire Line
-	1600 6900 1600 6950
-Connection ~ 1600 6950
-Wire Wire Line
-	1350 6900 1350 6950
-Connection ~ 1350 6950
 Wire Wire Line
 	5925 5900 5925 5975
@@
 	1    0    0    -1
 $EndComp
+Wire Wire Line
+	2900 4400 5575 4400
 $EndSCHEMATC

Commit message: wip
Parts:
- P8: footprint Pin_Headers:Pin_Header_Straight_2x04 -> Socket_Strips:Socket_Strip_Straight_2x04
Changed lines of the file:
@@
 EESchema Schematic File Version 2
-LIBS:mfx-link2-rescue
 LIBS:power
 LIBS:device
@@
 F 0 "P8" H 9975 2950 50  0000 C CNN
 F 1 "IBT-2" H 9975 2450 50  0000 C CNN
-F 2 "Pin_Headers:Pin_Header_Straight_2x04" H 9975 1500 50  0001 C CNN
+F 2 "Socket_Strips:Socket_Strip_Straight_2x04" H 9975 1500 50  0001 C CNN
 F 3 "" H 9975 1500 50  0000 C CNN
 	1    9975 2700

Commit message: wip
Parts:
- removed P1: Rail, Wire_Pads:SolderWirePad_2x_1-5mmDrill, symbol CONN_01X02
- removed P3: 18V, w_conn_pt-1,5:pt_1,5-2-3,5-h, symbol CONN_01X02
- added P1: CONN_01X04, w_conn_mkds:akl0711,5-4, symbol CONN_01X04
- U1: footprint w_smd_dil:mdip_8 -> w_pth_circuits:dil_8-300_socket
- U4: value 7805 -> 78L05; footprint 78xx:TO-252-2Lead -> TO_SOT_Packages_SMD:SOT89-3_Housing_Handsoldering
Connections:
- net GND: now also P1.4 (P4)
- net at T1.7 (SA): now also P1.1 (P1)
- net at T1.8 (SB): now also P1.2 (P2)
- net 18V+: now reaches C3.1, U2.VI
- net 18V+: now also P1.3 (P3)
- net VI: now reaches C2.1, D5.2 (K), U4.VI
Other:
- note added: "Rail"
Changed lines of the file:
@@
-$EndComp
-$Comp
-L CONN_01X02 P1
-U 1 1 58FE254A
-P 1450 6750
-F 0 "P1" H 1450 6900 50  0000 C CNN
-F 1 "Rail" V 1550 6750 50  0000 C CNN
-F 2 "Wire_Pads:SolderWirePad_2x_1-5mmDrill" H 1450 6750 50  0001 C CNN
-F 3 "" H 1450 6750 50  0000 C CNN
-	1    1450 6750
-	-1   0    0    1
 $EndComp
 $Comp
@@
 	1    3550 1600
 	1    0    0    -1
-$EndComp
-$Comp
-L CONN_01X02 P3
-U 1 1 58FE3599
-P 2950 1350
-F 0 "P3" H 2950 1500 50  0000 C CNN
-F 1 "18V" V 3050 1350 50  0000 C CNN
-F 2 "w_conn_pt-1,5:pt_1,5-2-3,5-h" V 2950 1350 50  0001 C CNN
-F 3 "" H 2950 1350 50  0000 C CNN
-	1    2950 1350
-	-1   0    0    1
 $EndComp
 $Comp
@@
 P 4150 5200
 F 0 "U4" H 4300 5004 50  0000 C CNN
-F 1 "7805" H 4150 5400 50  0000 C CNN
-F 2 "78xx:TO-252-2Lead" H 4150 5200 50  0001 C CNN
+F 1 "78L05" H 4150 5400 50  0000 C CNN
+F 2 "TO_SOT_Packages_SMD:SOT89-3_Housing_Handsoldering" H 4150 5200 50  0001 C CNN
 F 3 "" H 4150 5200 50  0000 C CNN
 	1    4150 5200
@@
 F 0 "U1" H 2500 3300 50  0000 L CNN
 F 1 "6N137" H 2700 3300 50  0001 L CNN
-F 2 "w_smd_dil:mdip_8" H 2500 2700 50  0001 L CIN
+F 2 "w_pth_circuits:dil_8-300_socket" H 2500 2700 50  0001 L CIN
 F 3 "" H 2700 3000 50  0000 L CNN
 	1    2700 3000
@@
 F 3 "" H 2850 5150 50  0000 C CNN
 	1    2850 5150
-	-1   0    0    1
-$EndComp
-$Comp
-L CONN_01X02 P2
-U 1 1 59002303
-P 1500 4450
-F 0 "P2" H 1500 4600 50  0000 C CNN
-F 1 "Gleisbox" V 1600 4450 50  0000 C CNN
-F 2 "w_conn_pt-1,5:pt_1,5-2-3,5-h" H 1500 4450 50  0001 C CNN
-F 3 "" H 1500 4450 50  0000 C CNN
-	1    1500 4450
 	-1   0    0    1
 $EndComp
@@
 	3525 6450 3525 6600
 Wire Wire Line
-	1650 6700 1700 6700
+	1375 6700 1700 6700
 Wire Wire Line
 	1700 6700 1700 6550
@@
 	1700 6950 1700 6800
 Wire Wire Line
-	1700 6800 1650 6800
+	1700 6800 1375 6800
 Connection ~ 3525 6550
 Connection ~ 3525 6950
@@
 Connection ~ 4100 1825
 Wire Wire Line
-	3150 1300 3700 1300
+	2975 1300 3700 1300
 Wire Wire Line
 	3550 1300 3550 1450
 Connection ~ 3550 1300
 Wire Wire Line
-	3150 1400 3300 1400
+	2975 1400 3300 1400
 Wire Wire Line
 	3300 1400 3300 1825
@@
 Wire Wire Line
 	5925 5900 5925 5975
-Wire Bus Line
-	600  3800 7000 3800
 Wire Bus Line
 	7000 3800 7000 6350
@@
 Wire Wire Line
 	2900 4400 5575 4400
+Wire Bus Line
+	7000 3800 1625 3800
+$Comp
+L CONN_01X04 P1
+U 1 1 592D9A8D
+P 1175 6650
+F 0 "P1" H 1175 6900 50  0000 C CNN
+F 1 "CONN_01X04" V 1275 6650 50  0001 C CNN
+F 2 "w_conn_mkds:akl0711,5-4" V 1175 6650 50  0001 C CNN
+F 3 "" H 1175 6650 50  0000 C CNN
+	1    1175 6650
+	-1   0    0    1
+$EndComp
+Wire Wire Line
+	1375 6500 1500 6500
+Wire Wire Line
+	1500 6500 1500 6225
+Wire Wire Line
+	1500 6225 1875 6225
+Wire Wire Line
+	1375 6600 1600 6600
+Wire Wire Line
+	1600 6600 1600 6325
+Wire Wire Line
+	1600 6325 1875 6325
+Text Label 1625 6325 0    60   ~ 0
+18V+
+Text Label 1625 6225 0    60   ~ 0
+18V-
+Text Label 2975 1300 0    60   ~ 0
+18V+
+Text Label 2975 1400 0    60   ~ 0
+18V-
+$Comp
+L CONN_01X02 P2
+U 1 1 592E55CE
+P 1500 4450
+F 0 "P2" H 1500 4600 50  0000 C CNN
+F 1 "Gleisbox" V 1600 4450 50  0000 C CNN
+F 2 "w_conn_pt-1,5:pt_1,5-2-3,5-h" V 1500 4450 50  0001 C CNN
+F 3 "" H 1500 4450 50  0000 C CNN
+	1    1500 4450
+	-1   0    0    1
+$EndComp
+Text Notes 1375 6800 0    60   ~ 0
+Rail
+Text Label 3700 5150 0    60   ~ 0
+VI
+Text Label 4575 5150 2    60   ~ 0
+VO
 $EndSCHEMATC

Commit message: wip
Parts:
- C1: value 1nF -> 100nF
- D1, D2, D3, D4, D5: value 1N4007 -> US1M; footprint w_smd_diode:sod323 -> w_smd_diode:do214ac
Changed lines of the file:
@@
 P 3025 6750
 F 0 "C1" H 3050 6850 50  0000 L CNN
-F 1 "1nF" H 3050 6650 50  0000 L CNN
+F 1 "100nF" H 3050 6650 50  0000 L CNN
 F 2 "Capacitors_SMD:C_0805_HandSoldering" H 3063 6600 50  0001 C CNN
 F 3 "" H 3025 6750 50  0000 C CNN
@@
 P 2700 4700
 F 0 "D4" H 2525 4650 50  0000 C CNN
-F 1 "1N4007" H 2700 4600 50  0000 C CNN
-F 2 "w_smd_diode:sod323" H 2700 4700 50  0001 C CNN
+F 1 "US1M" H 2700 4600 50  0000 C CNN
+F 2 "w_smd_diode:do214ac" H 2700 4700 50  0001 C CNN
 F 3 "" H 2700 4700 50  0000 C CNN
 	1    2700 4700
@@
 P 2500 4700
 F 0 "D3" H 2325 4650 50  0000 C CNN
-F 1 "1N4007" H 2500 4600 50  0000 C CNN
-F 2 "w_smd_diode:sod323" H 2500 4700 50  0001 C CNN
+F 1 "US1M" H 2500 4600 50  0000 C CNN
+F 2 "w_smd_diode:do214ac" H 2500 4700 50  0001 C CNN
 F 3 "" H 2500 4700 50  0000 C CNN
 	1    2500 4700
@@
 P 2250 4700
 F 0 "D2" H 2425 4750 50  0000 C CNN
-F 1 "1N4007" H 2250 4800 50  0000 C CNN
-F 2 "w_smd_diode:sod323" H 2250 4700 50  0001 C CNN
+F 1 "US1M" H 2250 4800 50  0000 C CNN
+F 2 "w_smd_diode:do214ac" H 2250 4700 50  0001 C CNN
 F 3 "" H 2250 4700 50  0000 C CNN
 	1    2250 4700
@@
 P 2025 4700
 F 0 "D1" H 2200 4750 50  0000 C CNN
-F 1 "1N4007" H 2025 4800 50  0000 C CNN
-F 2 "w_smd_diode:sod323" H 2025 4700 50  0001 C CNN
+F 1 "US1M" H 2025 4800 50  0000 C CNN
+F 2 "w_smd_diode:do214ac" H 2025 4700 50  0001 C CNN
 F 3 "" H 2025 4700 50  0000 C CNN
 	1    2025 4700
@@
 P 2850 5150
 F 0 "D5" H 2850 5050 50  0000 C CNN
-F 1 "1N4007" H 2850 5250 50  0000 C CNN
-F 2 "w_smd_diode:sod323" H 2850 5150 50  0001 C CNN
+F 1 "US1M" H 2850 5250 50  0000 C CNN
+F 2 "w_smd_diode:do214ac" H 2850 5150 50  0001 C CNN
 F 3 "" H 2850 5150 50  0000 C CNN
 	1    2850 5150

Commit message: wip
Parts:
- C4, C5: footprint Capacitors_SMD:c_elec_4x5.3 -> Capacitors_SMD:c_elec_5x5.3
- R1: value 1k8 -> 1k5; footprint Resistors_SMD:R_0805_HandSoldering -> Resistors_SMD:R_1206_HandSoldering
Changed lines of the file:
@@
 P 1900 2850
 F 0 "R1" V 1980 2850 50  0000 C CNN
-F 1 "1k8" V 1900 2850 50  0000 C CNN
-F 2 "Resistors_SMD:R_0805_HandSoldering" V 1830 2850 50  0001 C CNN
+F 1 "1k5" V 1900 2850 50  0000 C CNN
+F 2 "Resistors_SMD:R_1206_HandSoldering" V 1830 2850 50  0001 C CNN
 F 3 "" H 1900 2850 50  0000 C CNN
 	1    1900 2850
@@
 F 0 "C4" H 4675 5475 50  0000 L CNN
 F 1 "47uF" H 4675 5275 50  0000 L CNN
-F 2 "Capacitors_SMD:c_elec_4x5.3" H 4688 5225 50  0001 C CNN
+F 2 "Capacitors_SMD:c_elec_5x5.3" H 4688 5225 50  0001 C CNN
 F 3 "" H 4650 5375 50  0000 C CNN
 	1    4650 5375
@@
 F 0 "C5" H 4675 1700 50  0000 L CNN
 F 1 "47uF" H 4675 1500 50  0000 L CNN
-F 2 "Capacitors_SMD:c_elec_4x5.3" H 4688 1450 50  0001 C CNN
+F 2 "Capacitors_SMD:c_elec_5x5.3" H 4688 1450 50  0001 C CNN
 F 3 "" H 4650 1600 50  0000 C CNN
 	1    4650 1600
