File: mfx-link2/mfx-link2.sch (KiCad schematic (older format))
At the start: 55 parts, among them P1 CONN_01X04, P2 Gleisbox, P4 UART, P5 I2C, P6 CONN_02X03, P7 POTI, P8 IBT-2, Q1 BC817-40, SW1 SW_PUSH, T1 53040C, U1 6N137, U2 7805, U3 LM393, U4 78L05, U5 PIC16F1709

Commit message: wip
Connections:
- wire segments 196 -> 250
Changed lines of the file:
@@
 U 1 1 58FFCD58
 P 5625 6125
-F 0 "R11" V 5675 6275 50  0000 C CNN
+F 0 "R11" V 5675 6300 50  0000 C CNN
 F 1 "1K5" V 5625 6125 50  0000 C CNN
 F 2 "Resistors_SMD:R_1206_HandSolderingII" V 5555 6125 50  0001 C CNN
@@
 U 1 1 58FFD390
 P 5775 6125
-F 0 "R12" V 5825 6275 50  0000 C CNN
+F 0 "R12" V 5825 6300 50  0000 C CNN
 F 1 "1K5" V 5775 6125 50  0000 C CNN
 F 2 "Resistors_SMD:R_1206_HandSolderingII" V 5705 6125 50  0001 C CNN
@@
 U 1 1 58FFD424
 P 5925 6125
-F 0 "R13" V 5975 6275 50  0000 C CNN
+F 0 "R13" V 5975 6300 50  0000 C CNN
 F 1 "1K5" V 5925 6125 50  0000 C CNN
 F 2 "Resistors_SMD:R_1206_HandSolderingII" V 5855 6125 50  0001 C CNN
@@
 U 1 1 58FFD74D
 P 6075 6125
-F 0 "R14" V 6125 6275 50  0000 C CNN
+F 0 "R14" V 6125 6300 50  0000 C CNN
 F 1 "1K5" V 6075 6125 50  0000 C CNN
 F 2 "Resistors_SMD:R_1206_HandSolderingII" V 6005 6125 50  0001 C CNN
@@
 U 1 1 58FFDD14
 P 5475 6125
-F 0 "R10" V 5525 6275 50  0000 C CNN
+F 0 "R10" V 5525 6300 50  0000 C CNN
 F 1 "1K5" V 5475 6125 50  0000 C CNN
 F 2 "Resistors_SMD:R_1206_HandSolderingII" V 5405 6125 50  0001 C CNN
@@
 MCLR
 Wire Wire Line
-	2350 6550 3150 6550
-Wire Wire Line
-	3525 6900 3525 7050
+	2350 6550 2425 6550
+Wire Wire Line
+	2425 6550 2700 6550
+Wire Wire Line
+	2700 6550 3025 6550
+Wire Wire Line
+	3025 6550 3150 6550
+Wire Wire Line
+	3525 6900 3525 6950
+Wire Wire Line
+	3525 6950 3525 7050
 Wire Wire Line
 	2425 6900 2425 6950
@@
 Connection ~ 3025 6950
 Wire Wire Line
-	3525 6450 3525 6600
-Wire Wire Line
-	1050 6700 1700 6700
+	3525 6450 3525 6550
+Wire Wire Line
+	3525 6550 3525 6600
+Wire Wire Line
+	1050 6700 1475 6700
+Wire Wire Line
+	1475 6700 1700 6700
 Wire Wire Line
 	1700 6700 1700 6550
@@
 	1700 6950 1700 6800
 Wire Wire Line
-	1700 6800 1050 6800
+	1700 6800 1200 6800
+Wire Wire Line
+	1200 6800 1050 6800
 Connection ~ 3525 6550
 Connection ~ 3525 6950
@@
 	6675 2100 6675 1875
 Wire Wire Line
-	4500 1300 4975 1300
-Wire Wire Line
-	4100 1600 4100 1925
-Wire Wire Line
-	3300 1825 4950 1825
+	4500 1300 4650 1300
+Wire Wire Line
+	4650 1300 4975 1300
+Wire Wire Line
+	4100 1600 4100 1825
+Wire Wire Line
+	4100 1825 4100 1925
+Wire Wire Line
+	3300 1825 3550 1825
+Wire Wire Line
+	3550 1825 4100 1825
+Wire Wire Line
+	4100 1825 4650 1825
+Wire Wire Line
+	4650 1825 4950 1825
 Wire Wire Line
 	4650 1825 4650 1750
@@
 Connection ~ 4100 1825
 Wire Wire Line
-	2975 1300 3700 1300
+	2975 1300 3550 1300
+Wire Wire Line
+	3550 1300 3700 1300
 Wire Wire Line
 	3550 1300 3550 1450
@@
 	6450 2400 6700 2400
 Wire Wire Line
-	6450 1925 6450 2400
+	6450 1925 6450 2025
+Wire Wire Line
+	6450 2025 6450 2400
 Wire Wire Line
 	6450 1625 6450 1575
@@
 	9550 2750 9550 2225
 Wire Wire Line
-	9550 2225 10425 2225
+	9550 2225 10200 2225
+Wire Wire Line
+	10200 2225 10425 2225
 Wire Wire Line
 	10425 2225 10425 2750
@@
 	5250 6750 5325 6750
 Wire Wire Line
-	6075 5900 6075 5975
-Wire Wire Line
-	5625 5900 6075 5900
-Wire Wire Line
-	5675 5625 5675 5900
-Wire Wire Line
-	5625 5975 5625 5900
-Connection ~ 5675 5900
-Wire Wire Line
-	5775 5900 5775 5975
-Connection ~ 5775 5900
-Connection ~ 5925 5900
-Wire Wire Line
-	5325 5975 5325 5900
-Wire Wire Line
-	5325 5900 5575 5900
-Wire Wire Line
-	5475 5900 5475 5975
-Wire Wire Line
-	5575 5900 5575 5625
-Connection ~ 5475 5900
-Wire Wire Line
-	5475 5825 5175 5825
-Wire Wire Line
-	5175 5825 5175 5975
+	6075 5850 6075 5975
+Wire Wire Line
+	5625 5850 5675 5850
+Wire Wire Line
+	5675 5850 5775 5850
+Wire Wire Line
+	5775 5850 5925 5850
+Wire Wire Line
+	5925 5850 6075 5850
+Wire Wire Line
+	5675 5625 5675 5850
+Wire Wire Line
+	5625 5975 5625 5850
+Connection ~ 5675 5850
+Wire Wire Line
+	5775 5850 5775 5975
+Connection ~ 5775 5850
+Connection ~ 5925 5850
+Wire Wire Line
+	5325 5975 5325 5850
+Wire Wire Line
+	5325 5850 5475 5850
+Wire Wire Line
+	5475 5850 5575 5850
+Wire Wire Line
+	5475 5850 5475 5975
+Wire Wire Line
+	5575 5850 5575 5625
+Connection ~ 5475 5850
+Wire Wire Line
+	5475 5775 5175 5775
+Wire Wire Line
+	5175 5775 5175 5975
 Wire Wire Line
 	5175 6275 5175 6400
 Wire Wire Line
-	5175 6400 6075 6400
+	5175 6400 5325 6400
+Wire Wire Line
+	5325 6400 5475 6400
+Wire Wire Line
+	5475 6400 5625 6400
+Wire Wire Line
+	5625 6400 5775 6400
+Wire Wire Line
+	5775 6400 5925 6400
+Wire Wire Line
+	5925 6400 6075 6400
 Wire Wire Line
 	6075 6400 6075 6275
@@
 Connection ~ 5475 6400
 Wire Wire Line
-	5625 6275 5625 6550
+	5625 6275 5625 6400
+Wire Wire Line
+	5625 6400 5625 6550
 Connection ~ 5625 6400
 Wire Wire Line
@@
 	10600 3000 10600 2550
 Wire Wire Line
-	2350 6950 3700 6950
-Wire Wire Line
-	3450 6550 3700 6550
+	2350 6950 2425 6950
+Wire Wire Line
+	2425 6950 2700 6950
+Wire Wire Line
+	2700 6950 3025 6950
+Wire Wire Line
+	3025 6950 3525 6950
+Wire Wire Line
+	3525 6950 3700 6950
+Wire Wire Line
+	3450 6550 3525 6550
+Wire Wire Line
+	3525 6550 3700 6550
 Wire Wire Line
 	5675 5050 5675 5125
@@
 	5475 5125 5475 5050
 Wire Wire Line
-	5575 4400 5575 5125
+	5575 4400 5575 5050
+Wire Wire Line
+	5575 5050 5575 5125
 Connection ~ 5575 5050
 Wire Wire Line
-	5475 5625 5475 5825
-Wire Wire Line
-	1700 4500 2500 4500
+	5475 5625 5475 5775
+Wire Wire Line
+	1700 4500 2025 4500
+Wire Wire Line
+	2025 4500 2500 4500
 Wire Wire Line
 	2025 4500 2025 4550
@@
 Connection ~ 2025 4500
 Wire Wire Line
-	1700 4400 2700 4400
+	1700 4400 2250 4400
+Wire Wire Line
+	2250 4400 2700 4400
 Wire Wire Line
 	2700 4400 2700 4550
@@
 Connection ~ 2250 4400
 Wire Wire Line
-	4150 5450 4150 5750
+	4150 5450 4150 5600
+Wire Wire Line
+	4150 5600 4150 5750
 Wire Wire Line
 	2125 5600 2125 4950
@@
 	2025 4850 2025 4950
 Wire Wire Line
-	2025 4950 2250 4950
+	2025 4950 2125 4950
+Wire Wire Line
+	2125 4950 2250 4950
 Wire Wire Line
 	2250 4950 2250 4850
@@
 	2500 4850 2500 4950
 Wire Wire Line
-	2700 4850 2700 5150
+	2700 4850 2700 4950
+Wire Wire Line
+	2700 4950 2700 5150
 Connection ~ 2700 4950
 Wire Wire Line
-	5475 5050 5675 5050
+	5475 5050 5575 5050
+Wire Wire Line
+	5575 5050 5675 5050
 Wire Wire Line
 	2900 4950 2900 4400
 Wire Wire Line
-	2500 4950 2900 4950
+	2500 4950 2700 4950
+Wire Wire Line
+	2700 4950 2900 4950
 Wire Wire Line
 	3700 5600 3700 5550
@@
 Connection ~ 4150 5600
 Wire Wire Line
-	4650 4725 4650 5225
+	4650 4725 4650 4750
+Wire Wire Line
+	4650 4750 4650 5150
+Wire Wire Line
+	4650 5150 4650 5225
 Wire Wire Line
 	4550 5150 4650 5150
@@
 	2400 2850 2400 2900
 Wire Wire Line
-	2050 2850 2400 2850
+	2050 2850 2200 2850
+Wire Wire Line
+	2200 2850 2400 2850
 Connection ~ 2200 2850
 Wire Wire Line
-	1400 3150 2400 3150
+	1400 3150 2200 3150
+Wire Wire Line
+	2200 3150 2400 3150
 Wire Wire Line
 	2400 3150 2400 3100
@@
 	1750 2850 1400 2850
 Wire Wire Line
-	3000 5150 3750 5150
-Wire Wire Line
-	2125 5600 5000 5600
+	3000 5150 3700 5150
+Wire Wire Line
+	3700 5150 3750 5150
+Wire Wire Line
+	2125 5600 3200 5600
+Wire Wire Line
+	3200 5600 3700 5600
+Wire Wire Line
+	3700 5600 4150 5600
+Wire Wire Line
+	4150 5600 4650 5600
+Wire Wire Line
+	4650 5600 5000 5600
 Wire Wire Line
 	3000 3200 3100 3200
@@
 	8475 2600 8200 2600
 Wire Wire Line
-	3000 2425 3000 2900
+	3000 2425 3000 2600
+Wire Wire Line
+	3000 2600 3000 2800
+Wire Wire Line
+	3000 2800 3000 2900
 Connection ~ 3000 2600
 Connection ~ 3000 2800
 Wire Wire Line
-	3000 3100 3550 3100
+	3000 3100 3175 3100
+Wire Wire Line
+	3175 3100 3550 3100
 Wire Wire Line
 	3175 3100 3175 3000
@@
 	3175 2600 3175 2700
 Wire Wire Line
-	5925 5900 5925 5975
+	5925 5850 5925 5975
 Wire Bus Line
 	7000 3800 7000 6350
@@
 	1200 6800 1200 7050
 Wire Wire Line
-	1100 7050 1325 7050
+	1100 7050 1200 7050
+Wire Wire Line
+	1200 7050 1325 7050
 Connection ~ 1200 6800
 Connection ~ 1200 7050
 Wire Wire Line
-	1100 7350 1325 7350
+	1100 7350 1225 7350
+Wire Wire Line
+	1225 7350 1325 7350
 Wire Wire Line
 	1225 7350 1225 7450
@@
 	5750 2625 5750 2575
 Wire Wire Line
-	5750 2575 5900 2575
+	5750 2575 5825 2575
+Wire Wire Line
+	5825 2575 5900 2575
 Wire Wire Line
 	5900 2575 5900 2625
@@
 	1050 5575 950  5575
 Wire Wire Line
-	950  5375 950  5775
+	950  5375 950  5575
+Wire Wire Line
+	950  5575 950  5775
 $Comp
 L LM393-RESCUE-mfx-link2-RESCUE-mfx-link2 U3

Commit message: wip
Parts:
- removed D11, D12: US1M, w_smd_diode:do214ac, symbol D-RESCUE-mfx-link2
- removed P1: CONN_01X04, w_conn_mkds:akl0711,5-4, symbol CONN_01X04
- added R19: 4k7, Resistors_SMD:R_0805_HandSolderingII, symbol R
Connections:
- wire segments 250 -> 183

Commit message: wip
Parts:
- R4, R6: value 4k7 -> 100k
Changed lines of the file:
@@
 EESchema Schematic File Version 2
-LIBS:mfx-link2-rescue
 LIBS:power
 LIBS:device
@@
 $EndComp
 $Comp
-L PWR_FLAG #FLG2
+L PWR_FLAG #FLG01
 U 1 1 58FE3ABA
 P 4950 1775
-F 0 "#FLG2" H 4950 1870 50  0001 C CNN
+F 0 "#FLG01" H 4950 1870 50  0001 C CNN
 F 1 "PWR_FLAG" H 4950 1955 50  0000 C CNN
 F 2 "" H 4950 1775 50  0000 C CNN
@@
 P 3525 7200
 F 0 "R6" V 3605 7200 50  0000 C CNN
-F 1 "4k7" V 3525 7200 50  0000 C CNN
+F 1 "100k" V 3525 7200 50  0000 C CNN
 F 2 "Resistors_SMD:R_0805_HandSolderingII" V 3455 7200 50  0001 C CNN
 F 3 "" H 3525 7200 50  0000 C CNN
@@
 P 3525 6300
 F 0 "R4" V 3605 6300 50  0000 C CNN
-F 1 "4k7" V 3525 6300 50  0000 C CNN
+F 1 "100k" V 3525 6300 50  0000 C CNN
 F 2 "Resistors_SMD:R_0805_HandSolderingII" V 3455 6300 50  0001 C CNN
 F 3 "" H 3525 6300 50  0000 C CNN
@@
 $EndComp
 $Comp
-L +5V #PWR8
+L +5V #PWR02
 U 1 1 58FE4D35
 P 3950 6350
-F 0 "#PWR8" H 3950 6200 50  0001 C CNN
+F 0 "#PWR02" H 3950 6200 50  0001 C CNN
 F 1 "+5V" H 3950 6490 50  0000 C CNN
 F 2 "" H 3950 6350 50  0000 C CNN
@@
 ENABLE
 $Comp
-L GND #PWR32
+L GND #PWR03
 U 1 1 58FE66BD
 P 10325 3075
-F 0 "#PWR32" H 10325 2825 50  0001 C CNN
+F 0 "#PWR03" H 10325 2825 50  0001 C CNN
 F 1 "GND" H 10325 2925 50  0000 C CNN
 F 2 "" H 10325 3075 50  0000 C CNN
@@
 SENSE
 $Comp
-L GND #PWR27
+L GND #PWR04
 U 1 1 58FE942D
 P 8475 2200
-F 0 "#PWR27" H 8475 1950 50  0001 C CNN
+F 0 "#PWR04" H 8475 1950 50  0001 C CNN
 F 1 "GND" H 8475 2050 50  0000 C CNN
 F 2 "" H 8475 2200 50  0000 C CNN
@@
 $EndComp
 $Comp
-L GND #PWR29
+L GND #PWR05
 U 1 1 58FFB153
 P 8750 1925
-F 0 "#PWR29" H 8750 1675 50  0001 C CNN
+F 0 "#PWR05" H 8750 1675 50  0001 C CNN
 F 1 "GND" H 8750 1775 50  0000 C CNN
 F 2 "" H 8750 1925 50  0000 C CNN
@@
 _GB_OUT
 $Comp
-L GNDA #PWR20
+L GNDA #PWR06
 U 1 1 59001DF4
 P 5625 7000
-F 0 "#PWR20" H 5625 6750 50  0001 C CNN
+F 0 "#PWR06" H 5625 6750 50  0001 C CNN
 F 1 "GNDA" H 5625 6850 50  0000 C CNN
 F 2 "" H 5625 7000 50  0000 C CNN
@@
 $EndComp
 $Comp
-L +5V #PWR15
+L +5V #PWR07
 U 1 1 5909C148
 P 4650 4725
-F 0 "#PWR15" H 4650 4575 50  0001 C CNN
+F 0 "#PWR07" H 4650 4575 50  0001 C CNN
 F 1 "+5V" H 4650 4865 50  0000 C CNN
 F 2 "" H 4650 4725 50  0000 C CNN
@@
 red
 $Comp
-L +5V #PWR6
+L +5V #PWR08
 U 1 1 5908A86E
 P 3525 6075
-F 0 "#PWR6" H 3525 5925 50  0001 C CNN
+F 0 "#PWR08" H 3525 5925 50  0001 C CNN
 F 1 "+5V" H 3525 6215 50  0000 C CNN
 F 2 "" H 3525 6075 50  0000 C CNN
@@
 $EndComp
 $Comp
-L GND #PWR10
+L GND #PWR09
 U 1 1 58FE372A
 P 4100 1925
-F 0 "#PWR10" H 4100 1675 50  0001 C CNN
+F 0 "#PWR09" H 4100 1675 50  0001 C CNN
 F 1 "GND" H 4100 1775 50  0000 C CNN
 F 2 "" H 4100 1925 50  0000 C CNN
@@
 $EndComp
 $Comp
-L GND #PWR26
+L GND #PWR010
 U 1 1 58FE38A1
 P 7200 1575
-F 0 "#PWR26" H 7200 1325 50  0001 C CNN
+F 0 "#PWR010" H 7200 1325 50  0001 C CNN
 F 1 "GND" H 7200 1425 50  0000 C CNN
 F 2 "" H 7200 1575 50  0000 C CNN
@@
 $EndComp
 $Comp
-L GND #PWR19
+L GND #PWR011
 U 1 1 58FF775E
 P 5450 3275
-F 0 "#PWR19" H 5450 3025 50  0001 C CNN
+F 0 "#PWR011" H 5450 3025 50  0001 C CNN
 F 1 "GND" H 5450 3125 50  0000 C CNN
 F 2 "" H 5450 3275 50  0000 C CNN
@@
 $EndComp
 $Comp
-L GND #PWR13
+L GND #PWR012
 U 1 1 58FF8516
 P 4450 3275
-F 0 "#PWR13" H 4450 3025 50  0001 C CNN
+F 0 "#PWR012" H 4450 3025 50  0001 C CNN
 F 1 "GND" H 4450 3125 50  0000 C CNN
 F 2 "" H 4450 3275 50  0000 C CNN
@@
 $EndComp
 $Comp
-L GND #PWR5
+L GND #PWR013
 U 1 1 5909205E
 P 3100 3300
-F 0 "#PWR5" H 3100 3050 50  0001 C CNN
+F 0 "#PWR013" H 3100 3050 50  0001 C CNN
 F 1 "GND" H 3100 3150 50  0000 C CNN
 F 2 "" H 3100 3300 50  0000 C CNN
@@
 $EndComp
 $Comp
-L GNDA #PWR9
+L GNDA #PWR014
 U 1 1 59092D00
 P 3950 7150
-F 0 "#PWR9" H 3950 6900 50  0001 C CNN
+F 0 "#PWR014" H 3950 6900 50  0001 C CNN
 F 1 "GNDA" H 3950 7000 50  0000 C CNN
 F 2 "" H 3950 7150 50  0000 C CNN
@@
 $EndComp
 $Comp
-L GNDA #PWR7
+L GNDA #PWR015
 U 1 1 59092E5B
 P 3525 7425
-F 0 "#PWR7" H 3525 7175 50  0001 C CNN
+F 0 "#PWR015" H 3525 7175 50  0001 C CNN
 F 1 "GNDA" H 3525 7275 50  0000 C CNN
 F 2 "" H 3525 7425 50  0000 C CNN
@@
 $EndComp
 $Comp
-L VCC #PWR16
+L VCC #PWR016
 U 1 1 59094284
 P 4975 1200
-F 0 "#PWR16" H 4975 1050 50  0001 C CNN
+F 0 "#PWR016" H 4975 1050 50  0001 C CNN
 F 1 "VCC" H 4975 1350 50  0000 C CNN
 F 2 "" H 4975 1200 50  0000 C CNN
@@
 $EndComp
 $Comp
-L VCC #PWR25
+L VCC #PWR017
 U 1 1 590943B0
 P 7200 1075
-F 0 "#PWR25" H 7200 925 50  0001 C CNN
+F 0 "#PWR017" H 7200 925 50  0001 C CNN
 F 1 "VCC" H 7200 1225 50  0000 C CNN
 F 2 "" H 7200 1075 50  0000 C CNN
@@
 $EndComp
 $Comp
-L VCC #PWR22
+L VCC #PWR018
 U 1 1 590944D7
 P 6250 1175
-F 0 "#PWR22" H 6250 1025 50  0001 C CNN
+F 0 "#PWR018" H 6250 1025 50  0001 C CNN
 F 1 "VCC" H 6250 1325 50  0000 C CNN
 F 2 "" H 6250 1175 50  0000 C CNN
@@
 $EndComp
 $Comp
-L VCC #PWR23
+L VCC #PWR019
 U 1 1 5909459E
 P 6450 1175
-F 0 "#PWR23" H 6450 1025 50  0001 C CNN
+F 0 "#PWR019" H 6450 1025 50  0001 C CNN
 F 1 "VCC" H 6450 1325 50  0000 C CNN
 F 2 "" H 6450 1175 50  0000 C CNN
@@
 $EndComp
 $Comp
-L VCC #PWR24
+L VCC #PWR020
 U 1 1 5909516C
 P 6675 1875
-F 0 "#PWR24" H 6675 1725 50  0001 C CNN
+F 0 "#PWR020" H 6675 1725 50  0001 C CNN
 F 1 "VCC" H 6675 2025 50  0000 C CNN
 F 2 "" H 6675 1875 50  0000 C CNN
@@
 $EndComp
 $Comp
-L VCC #PWR4
+L VCC #PWR021
 U 1 1 5909A87E
 P 3000 2425
-F 0 "#PWR4" H 3000 2275 50  0001 C CNN
+F 0 "#PWR021" H 3000 2275 50  0001 C CNN
 F 1 "VCC" H 3000 2575 50  0000 C CNN
 F 2 "" H 3000 2425 50  0000 C CNN
@@
 $EndComp
 $Comp
-L VCC #PWR18
+L VCC #PWR022
 U 1 1 5909D6E9
 P 5450 2800
-F 0 "#PWR18" H 5450 2650 50  0001 C CNN
+F 0 "#PWR022" H 5450 2650 50  0001 C CNN
 F 1 "VCC" H 5450 2950 50  0000 C CNN
 F 2 "" H 5450 2800 50  0000 C CNN
@@
 $EndComp
 $Comp
-L VCC #PWR12
+L VCC #PWR023
 U 1 1 5909D844
 P 4450 2775
-F 0 "#PWR12" H 4450 2625 50  0001 C CNN
+F 0 "#PWR023" H 4450 2625 50  0001 C CNN
 F 1 "VCC" H 4450 2925 50  0000 C CNN
 F 2 "" H 4450 2775 50  0000 C CNN
@@
 	4650 1450 4650 1300
 $Comp
-L VCC #PWR28
+L VCC #PWR024
 U 1 1 590A14EA
 P 8750 1425
-F 0 "#PWR28" H 8750 1275 50  0001 C CNN
+F 0 "#PWR024" H 8750 1275 50  0001 C CNN
 F 1 "VCC" H 8750 1575 50  0000 C CNN
 F 2 "" H 8750 1425 50  0000 C CNN
@@
 $EndComp
 $Comp
-L VCC #PWR31
+L VCC #PWR025
 U 1 1 590A1627
 P 10200 1775
-F 0 "#PWR31" H 10200 1625 50  0001 C CNN
+F 0 "#PWR025" H 10200 1625 50  0001 C CNN
 F 1 "VCC" H 10200 1925 50  0000 C CNN
 F 2 "" H 10200 1775 50  0000 C CNN
@@
 $EndComp
 $Comp
-L VCC #PWR30
+L VCC #PWR026
 U 1 1 590A3FCB
 P 9400 2250
-F 0 "#PWR30" H 9400 2100 50  0001 C CNN
+F 0 "#PWR026" H 9400 2100 50  0001 C CNN
 F 1 "VCC" H 9400 2400 50  0000 C CNN
 F 2 "" H 9400 2250 50  0000 C CNN
@@
 	5325 2025 5325 2325
 $Comp
-L GND #PWR17
+L GND #PWR027
 U 1 1 59358A73
 P 5325 2325
-F 0 "#PWR17" H 5325 2075 50  0001 C CNN
+F 0 "#PWR027" H 5325 2075 50  0001 C CNN
 F 1 "GND" H 5325 2175 50  0000 C CNN
 F 2 "" H 5325 2325 50  0000 C CNN
@@
 $EndComp
 $Comp
-L VCC #PWR21
+L VCC #PWR028
 U 1 1 593A49AD
 P 5825 2575
-F 0 "#PWR21" H 5825 2425 50  0001 C CNN
+F 0 "#PWR028" H 5825 2425 50  0001 C CNN
 F 1 "VCC" H 5825 2725 50  0000 C CNN
 F 2 "" H 5825 2575 50  0000 C CNN
@@
 	950  5375 1050 5375
 $Comp
-L +5V #PWR2
+L +5V #PWR029
 U 1 1 593A5D98
 P 1250 5175
-F 0 "#PWR2" H 1250 5025 50  0001 C CNN
+F 0 "#PWR029" H 1250 5025 50  0001 C CNN
 F 1 "+5V" H 1250 5315 50  0000 C CNN
 F 2 "" H 1250 5175 50  0000 C CNN
@@
 $EndComp
 $Comp
-L GNDA #PWR3
+L GNDA #PWR030
 U 1 1 593A5FA4
 P 1250 5775
-F 0 "#PWR3" H 1250 5525 50  0001 C CNN
+F 0 "#PWR030" H 1250 5525 50  0001 C CNN
 F 1 "GNDA" H 1250 5625 50  0000 C CNN
 F 2 "" H 1250 5775 50  0000 C CNN
@@
 $EndComp
 $Comp
-L GNDA #PWR1
+L GNDA #PWR031
 U 1 1 593A61E9
 P 950 5775
-F 0 "#PWR1" H 950 5525 50  0001 C CNN
+F 0 "#PWR031" H 950 5525 50  0001 C CNN
 F 1 "GNDA" H 950 5625 50  0000 C CNN
 F 2 "" H 950 5775 50  0000 C CNN
@@
 $EndComp
 $Comp
-L PWR_FLAG #FLG1
+L PWR_FLAG #FLG032
 U 1 1 593A5E46
 P 3200 5550
-F 0 "#FLG1" H 3200 5645 50  0001 C CNN
+F 0 "#FLG032" H 3200 5645 50  0001 C CNN
 F 1 "PWR_FLAG" H 3200 5730 50  0000 C CNN
 F 2 "" H 3200 5550 50  0000 C CNN
@@
 $EndComp
 $Comp
-L +5V #PWR14
+L +5V #PWR033
 U 1 1 5965C0C7
 P 4450 6225
-F 0 "#PWR14" H 4450 6075 50  0001 C CNN
+F 0 "#PWR033" H 4450 6075 50  0001 C CNN
 F 1 "+5V" H 4450 6365 50  0000 C CNN
 F 2 "" H 4450 6225 50  0000 C CNN

Commit message: evenif the schematic is not working, fix the layout ...
Parts:
- added D11, D12: US1M, w_smd_diode:do214ac, symbol D-RESCUE-mfx-link2
- added P1: Conn_01x04, w_conn_mkds:akl0711,5-4, symbol Conn_01x04
- D13: symbol LED -> LED-RESCUE-mfx-link2
- U3: footprint (none) -> w_smd_dil:so-8
Connections:
- net labels added: rail1, rail2
- wire segments 183 -> 193
Other:
- moved on the sheet: U4
Changed lines of the file:
@@
 EESchema Schematic File Version 2
+LIBS:mfx-link2-rescue
 LIBS:power
 LIBS:device
@@
 L 7805 U4
 U 1 1 5900103C
-P 4150 5200
-F 0 "U4" H 4300 5004 50  0000 C CNN
-F 1 "78L05" H 4150 5400 50  0000 C CNN
-F 2 "TO_SOT_Packages_SMD:SOT89-3_Housing_Handsoldering" H 4150 5200 50  0001 C CNN
-F 3 "" H 4150 5200 50  0000 C CNN
-	1    4150 5200
+P 4175 5200
+F 0 "U4" H 4325 5004 50  0000 C CNN
+F 1 "78L05" H 4175 5400 50  0000 C CNN
+F 2 "TO_SOT_Packages_SMD:SOT89-3_Housing_Handsoldering" H 4175 5200 50  0001 C CNN
+F 3 "" H 4175 5200 50  0000 C CNN
+	1    4175 5200
 	1    0    0    -1
 $EndComp
@@
 Wire Wire Line
 	4650 5600 4650 5525
-Connection ~ 4150 5600
 Wire Wire Line
 	4650 4725 4650 5225
 Wire Wire Line
-	4550 5150 4650 5150
+	4575 5150 4650 5150
 Connection ~ 4650 5150
 Wire Wire Line
@@
 	1750 2850 1400 2850
 Wire Wire Line
-	3000 5150 3750 5150
+	3000 5150 3775 5150
 Wire Wire Line
 	2125 5600 5000 5600
@@
 	-1   0    0    1
 $EndComp
-Text Notes 1375 6800 0    60   ~ 0
+Text Notes 1250 6800 0    60   ~ 0
 Rail
 Text Label 3700 5150 0    60   ~ 0
@@
 $EndComp
 $Comp
-L LED D13
+L LED-RESCUE-mfx-link2 D13
 U 1 1 59389A4F
 P 5000 5350
@@
 F 0 "U3" H 1500 5625 50  0000 C CNN
 F 1 "LM393" H 1600 5325 50  0000 C CNN
-F 2 "" H 1350 5475 50  0000 C CNN
+F 2 "w_smd_dil:so-8" H 1350 5475 50  0001 C CNN
 F 3 "" H 1350 5475 50  0000 C CNN
 	2    1350 5475
@@
 	1    0    0    -1
 $EndComp
+$Comp
+L Conn_01x04 P1
+U 1 1 5A11BCEB
+P 1050 1950
+F 0 "P1" H 1050 2150 50  0000 C CNN
+F 1 "Conn_01x04" V 1050 1650 50  0001 C CNN
+F 2 "w_conn_mkds:akl0711,5-4" H 1050 1950 50  0001 C CNN
+F 3 "" H 1050 1950 50  0001 C CNN
+	1    1050 1950
+	-1   0    0    1
+$EndComp
+Wire Wire Line
+	1250 1750 1450 1750
+Wire Wire Line
+	1250 1850 1450 1850
+Text Label 1450 1850 2    60   ~ 0
+18V+
+Text Label 1450 1750 2    60   ~ 0
+18V-
+Wire Wire Line
+	1450 6700 1700 6700
+Wire Wire Line
+	1700 6800 1450 6800
+Text Label 1450 6800 0    60   ~ 0
+rail1
+Text Label 1450 6700 0    60   ~ 0
+rail2
+Text Label 1450 2050 2    60   ~ 0
+rail1
+Text Label 1450 1950 2    60   ~ 0
+rail2
+Wire Wire Line
+	1250 1950 1450 1950
+Wire Wire Line
+	1250 2050 1450 2050
+Connection ~ 4175 5600
+Wire Wire Line
+	4175 5450 4175 5600
+$Comp
+L PWR_FLAG #FLG034
+U 1 1 5A11FF2E
+P 700 5725
+F 0 "#FLG034" H 700 5800 50  0001 C CNN
+F 1 "PWR_FLAG" H 700 5875 50  0000 C CNN
+F 2 "" H 700 5725 50  0001 C CNN
+F 3 "" H 700 5725 50  0001 C CNN
+	1    700  5725
+	1    0    0    -1
+$EndComp
+Wire Wire Line
+	700  5725 950  5725
+Connection ~ 950  5725
+$Comp
+L D-RESCUE-mfx-link2 D12
+U 1 1 5A122364
+P 2400 6075
+F 0 "D12" H 2575 6125 50  0000 C CNN
+F 1 "US1M" H 2400 6175 50  0000 C CNN
+F 2 "w_smd_diode:do214ac" H 2400 6075 50  0001 C CNN
+F 3 "" H 2400 6075 50  0000 C CNN
+	1    2400 6075
+	0    1    1    0
+$EndComp
+$Comp
+L D-RESCUE-mfx-link2 D11
+U 1 1 5A1227E6
+P 2250 6075
+F 0 "D11" H 2425 6125 50  0000 C CNN
+F 1 "US1M" H 2250 6175 50  0000 C CNN
+F 2 "w_smd_diode:do214ac" H 2250 6075 50  0001 C CNN
+F 3 "" H 2250 6075 50  0000 C CNN
+	1    2250 6075
+	0    -1   -1   0
+$EndComp
+Wire Wire Line
+	1900 5925 2400 5925
+Connection ~ 2250 5925
+Wire Wire Line
+	1900 6225 2400 6225
+Connection ~ 2250 6225
+Text Label 1900 5925 0    60   ~ 0
+rail2
+Text Label 1900 6225 0    60   ~ 0
+rail1
 $EndSCHEMATC
