File: RPi-MCP2517/RPi-MCP2517.sch (KiCad schematic (older format))
At the start: 32 parts, among them P1 CONN_02X20, P10 CONN_02X08, P11 CONN_02X08, P12 CONN_01X08, P13 CONN_02X08, P14 CONN_02X08, P15 CONN_01X06, P17 PWR, P2 CONN_01X02, P3 CONN_01X03, P4 CONN_01X09, P5 CONN_01X04, P8 CONN_01X02, P9 CONN_01X04, U1 MCP2517FD, U2 MCP2562FD, U3 P82B715, Y1 20MHz

Commit message: wip
Parts:
- removed P10, P11, P13, P14: CONN_02X08, Socket_Strips:Socket_Strip_Straight_2x08, symbol CONN_02X08
- removed P12: CONN_01X08, Socket_Strips:Socket_Strip_Straight_1x08, symbol CONN_01X08
- removed P15: CONN_01X06, Socket_Strips:Socket_Strip_Straight_1x06, symbol CONN_01X06
- removed P17: PWR, Pin_Headers:Pin_Header_Straight_1x02, symbol CONN_01X02
- removed P4: CONN_01X09, Pin_Headers:Pin_Header_Straight_1x09, symbol CONN_01X09
- removed P5: CONN_01X04, w_conn_jst-ph:s4b-ph-kl, symbol CONN_01X04
- P2, P8: footprint Pin_Headers:Pin_Header_Straight_1x02 -> Pin_Headers:Pin_Header_Angled_1x02
- Y1: value 20MHz -> 4MHz
Connections:
- no-connect marks 34 -> 22

Commit message: QA
Parts:
- removed P3: CONN_01X03, Pin_Headers:Pin_Header_Angled_1x03, symbol CONN_01X03
- added C6, C7, C8: 100nF, Capacitors_SMD:C_0805_HandSoldering, symbol C
- added J1: Conn_01x06, Pin_Headers:Pin_Header_Angled_1x06_Pitch2.54mm, symbol Conn_01x06
- added J2: Conn_01x02, Pin_Headers:Pin_Header_Straight_1x02_Pitch2.54mm, symbol Conn_01x02
- added J3: DB9_Female_MountingHoles, w_conn_d-sub:DB_9M, symbol DB9_Female_MountingHoles
- added P3, P4: CONN_01X04, w_conn_jst-ph:s4b-ph-kl, symbol CONN_01X04
- added R5, R6, R8: 0, Resistors_SMD:R_0805_HandSolderingII, symbol R
- added R9: 50, Resistors_SMD:R_0805_HandSolderingII, symbol R
- added U4: SI8641-SOIC, w_smd_dil:so-16, symbol SI8641-SOIC
- renumbered R24 to R10, R25 to R11, R14 to R12, R15 to R13, R5 to R7
Connections:
- net +3V3: now also C6.1, C8.1, P4.2 (P2), U4.1 (VDD1)
- net +5V: now also P3.2 (P2)
- net GND: now also C6.2, C8.2, J3.3, J3.6, P3.1 (P1), P4.1 (P1), U4.2 (GND1), U4.8 (GND1)
- net GPIO17: now also U4.5
- net GPIO22: now also U4.3
- net GPIO27: now also U4.4
- net GPIO4: now also U4.6
- net INT0: now also R5.2; no longer P1.16 (P16), R3.2
- net INT1: now also R6.2; no longer P1.18 (P18), R4.2
- net RxD: now also P4.4 (P4)
- net TxD: now also P4.3 (P3)
- net CANL: now reaches P2.2 (P2), U2.6 (CANL)
- net CANL: now also J3.2, P3.4 (P4)
- net CANH: now reaches R7.2, U2.7 (CANH)
- net CANH: now also J3.7, P3.3 (P3)
- new net: R9.1, U4.11
- new net: R8.1, U4.12
- new net: J1.3 (Pin_3), U4.13
- new net: J1.2 (Pin_2), U4.14
- new net: J1.6 (Pin_6), R9.2
- new net: J1.4 (Pin_4), R8.2
- new net GNDA: C7.2, J1.5 (Pin_5), J2.2 (Pin_2), U4.15 (GND2), U4.9 (GND2)
- new net INT0_: P1.16 (P16), R3.2, R5.1
- new net INT1_: P1.18 (P18), R4.2, R6.1
- new net VDDA: C7.1, J1.1 (Pin_1), J2.1 (Pin_1), U4.16 (VDD2)
- no-connect marks 22 -> 30
Other:
- note added: "GPIO Option"
- note added: "I2C Option"
- note added: "UART Option"
- moved on the sheet: P8, P9, R10, R11, R12, R13, U3
