File: RPi-Rail/RPi-Rail.sch (KiCad schematic (older format))
At the start: 35 parts, among them J1 Conn_01x06, J2 Conn_01x02, P1 CONN_02X20, P2 CONN_01X02, P3 CONN_01X04, P4 CONN_01X04, P8 CONN_01X02, P9 CONN_01X04, SW1 SW_PUSH, U1 MCP2517FD, U2 ISO1050, U3 P82B715, U4 SI8641-SOIC, U5 DSPIC33EP128GM604, Y1 4MHz

Commit message: wip
Parts:
- added D? (x2): LED, symbol LED
- added P?: IBT-2 Interface, symbol CONN_02X04
- added Q?: BC817-40, SOT-23, symbol BC817-40
- added R?: 10k, Resistors_SMD:R_0805_HandSolderingII, symbol R
- added R?: 22k, Resistors_SMD:R_0805_HandSolderingII, symbol R
- added R?: 150k, Resistors_SMD:R_0805_HandSolderingII, symbol R
- added R?: 47k, Resistors_SMD:R_0805_HandSolderingII, symbol R
- added R?: 220k, Resistors_SMD:R_0805_HandSolderingII, symbol R
- added R? (x3): 4k7, Resistors_SMD:R_0805_HandSolderingII, symbol R
- added R? (x2): 3k3, Resistors_SMD:R_0805_HandSolderingII, symbol R
- added R? (x2): 0, Resistors_SMD:R_0805_HandSolderingII, symbol R
- added U?: LM311N, w_smd_dil:so-8, symbol LM311N
- added U?: Si8605, symbol Si8605
Connections:
- net +3V3: no longer C8.1
- net +5VA: now also P?.7 (P7)
- net GNDD: now also P?.8 (P8), Q?.2 (E), R?.2, R?.2, U?.1 (GND), U?.4 (V-)
- net TXCAN_: now reaches P1.16 (P16)
- net TXCAN_: now also R?.1
- net RXCAN_: now reaches P1.18 (P18)
- net RXCAN_: now also R?.2
- net TXCAN: now reaches U1.1 (TXCAN), U2.3 (TXD)
- net TXCAN: now also R?.2
- net RXCAN: now reaches U1.2 (RXCAN), U2.2 (RXD)
- net RXCAN: now also R?.1
- net S88_RESET: now reaches U4.3
- net S88_PS: now reaches U4.4
- net S88_CLOCK: now reaches U4.5
- net S88_DATA: now reaches U4.6
- net at U5.21 (PGED3/AN2/SS1/RPI32/CTED2/RB0): now also R?.2, U?.3 (A1)
- net at U5.22 (PGEC3/AN3/RPI33/CTED1/RB1): now also U?.4 (A2)
- net TxD_: now reaches U5.23 (PGEC1/OA1IN+/AN4/RPI34/RB2)
- net TxD_: now also U?.5 (A3)
- net RxD_: now reaches U5.24 (PGED1/OA1IN-/AN5/CTMUC/RP35/RB3)
- net RxD_: now also R?.2, U?.6 (A4)
- new net: R?.1, R?.1, R?.2, U?.2 (+)
- new net: R?.1, R?.2, U?.3 (-)
- new net: Q?.1 (B), R?.1
- new net: D?.2 (A), R?.2 (x2)
- new net: R?.1, R?.1
- new net +12V: C8.1, R?.1, R?.1, R?.1
- new net ENA: P?.3 (P3), P?.4 (P4)
- new net LN_DATA: D?.1 (K), Q?.3 (C), R?.2
- new net LN_IN: R?.1, U?.7
- new net LN_OUT: D?.1 (K), R?.2
- new net LPWM: P?.2 (P2)
- new net RPWM: P?.1 (P1)
- new net SENSE: P?.5 (P5), P?.6 (P6)
- no-connect marks 27 -> 25
Other:
- note added: "TODO\n"
- moved on the sheet: C1, C2, C3, C4, C5, C6, C7, C8, J1, J2, P1, P2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

Commit message: wip
Parts:
- added C? (x6): 100nF, Capacitors_SMD:C_0805_HandSoldering, symbol C
- added C?: 2.2uF, symbol CP_Small
- added C?: 22pf, Capacitors_SMD:C_0805_HandSoldering, symbol C
- added C?: 22pF, Capacitors_SMD:C_0805_HandSoldering, symbol C
- added JP?: ICSP, ICSP:ICSP, symbol ICSP
- added P?: L*conet, symbol CONN_01X06
- added P?: CONN_01X04, w_conn_jst-ph:s4b-ph-kl, symbol CONN_01X04
- added P?: CONN_01X02, Pin_Headers:Pin_Header_Angled_1x02, symbol CONN_01X02
- added R? (x4): 3k3, Resistors_SMD:R_0805_HandSolderingII, symbol R
- added U?: LC72725, MODULE, symbol LC72725
- added U?: P82B715, w_smd_dil:so-8, symbol P82B715
- added Y?: 4MHz, w_crystal:crystal_hc-49s, symbol Crystal
Connections:
- net +3V3: now also C?.1
- net +5VA: now also R?.1, R?.1
- net GND: now also C?.2
- net GNDD: now also C?.1, C?.1, C?.2, C?.2, C?.2, C?.2, JP?.3 (Vss), P?.1 (P1), U?.11 (Vssd), U?.4 (GND), U?.6 (Vssa)
- net RxD_: now also JP?.5 (PGC)
- net SCL: now also R?.2, U?.3 (SX)
- net SDA: now also R?.2, U?.6 (SY)
- net SENSE: now also C?.2
- net TxD_: now also JP?.4 (PGD)
- net VDD: now also C?.2, C?.2, R?.1, R?.1, U?.12 (Vddd), U?.5 (Vdda), U?.8 (VCC)
- net MCLR: now reaches D1.1 (K), R3.2, SW1.1
- net MCLR: now also JP?.1 (VPP/~MCLR)
- new net: C?.1, U?.13 (XIN), Y?.2
- new net: C?.1, U?.14 (XOUT), Y?.1
- new net: C?.1, U?.3 (Vref)
- new net: C?.1, U?.4 (MPXIN)
- new net: C?.2, U?.7 (FLOUT)
- new net: C?.1, U?.8 (CIN)
- new net: P?.4 (P4), R?.2, U?.2 (LX)
- new net: P?.3 (P3), R?.2, U?.7 (LY)
- new net: P?.2 (P2), P?.2 (P2)
- new net RDS_CL: U?.16 (RDCL)
- new net RDS_DA: U?.2 (RDDA)
- new net RDS_ID: U?.1 (RDS-ID)
- new net RDS_MODE: U?.10 (MODE)
- new net RDS_RST: U?.15 (RST)
- new net RDS_TEST: U?.9 (TEST)
- no-connect marks 25 -> 27
