File: USB2CAN-CAN/USB2-CAN-CAN.kicad_pcb (KiCad board)
At the start: 2 copper layers, 50 x 50 mm, 37 parts, among them P1 USB_A, P2 Prog, P3 Term, P4 CONN_01X03, P5 CONN_01X12, P6 CONN_01X12, U1 FT230XS, U2 PIC18F25K80_I/SS, U3 MCP2562

Commit message: wip
Parts:
- D5: footprint Diodes_SMD:Diode-MELF_Handsoldering -> Diodes_SMD:MiniMELF_Standard
- P4: value CONN_01X03 -> CAN
- U2: value PIC18F25K80_I/SS -> PIC18F25K80
- moved HLU 73.7 mm to (148.0, 131.0), turned to 180 degrees
- moved HLD 68.7 mm to (148.0, 87.0), turned to 180 degrees
- moved HRU 58.9 mm to (104.0, 131.0), turned to 180 degrees
- moved HRD 52.6 mm to (104.0, 87.0), turned to 180 degrees
- moved JP1 51.7 mm to (147.7, 101.3)
- moved P5 48.8 mm to (115.3, 130.8), turned to 90 degrees
- moved P2 44.2 mm to (147.7, 91.7), turned to 0 degrees
- moved P6 42.8 mm to (114.8, 87.1)
- moved R6 42.7 mm to (142.9, 93.1), turned to 90 degrees
- moved D5 42.7 mm to (144.3, 98.6), turned to 90 degrees
- moved P4 39.7 mm to (147.7, 123.4), turned to 180 degrees
- moved R7 38.7 mm to (133.5, 94.5)
- moved U3 38.2 mm to (142.1, 116.0)
- moved R5 35.9 mm to (136.5, 117.0), turned to 180 degrees
- moved P1 34.9 mm to (103.3, 109.0), turned to 270 degrees
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
Commit message: V1.1 wip
Parts:
- added D6: LED, LEDs:LED-0805, F.Cu at (136.0, 90.5)
- added R9: 270, Resistors_SMD:R_0805_HandSoldering, F.Cu at (136.0, 95.0)
- P4: value CAN -> CONN_01X03
- P5: value CONN_01X12 -> CON1; footprint Pin_Headers:Pin_Header_Straight_1x12 -> Pin_Headers:Pin_Header_Straight_1x10
- P6: value CONN_01X12 -> CON2; footprint Pin_Headers:Pin_Header_Straight_1x12 -> Pin_Headers:Pin_Header_Straight_1x10
- R5: value 270 -> 120
- U2: value PIC18F25K80 -> PIC18F25K80_I/SS
- moved D1 10.7 mm to (114.8, 97.8), turned to 0 degrees
- moved D2 10.6 mm to (114.8, 95.2), turned to 0 degrees
- moved HRD 10.0 mm to (114.0, 87.0)
- moved HRU 10.0 mm to (114.0, 131.0)
- moved R8 7.20 mm to (140.0, 95.0), turned to 90 degrees
- moved C8 6.75 mm to (120.0, 92.2)
- moved Ferrit1 6.46 mm to (120.0, 112.5)
- moved C4 6.27 mm to (120.0, 105.7)
- moved C5 6.27 mm to (120.0, 107.7)
- moved R1 6.27 mm to (120.0, 103.6)
- moved R2 6.27 mm to (120.0, 109.7)
- moved R4 5.86 mm to (114.2, 93.0)
- moved R3 5.61 mm to (114.8, 100.0)
- moved P1 5.46 mm to (108.8, 108.5)
- moved P4 4.95 mm to (148.0, 118.5)
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Connections:
- P5 pad 10: /RA5 -> /CLKOUT
- P5 pad 9: /RA3 -> /RA5
- P6 pad 1: VCOM -> VCC

Commit message: house keeping
Connections:
- U1 pad 2: Net-(U1-Pad2) -> Net-(P2-Pad1)
- U1 pad 6: Net-(P2-Pad1) -> Net-(U1-Pad6)
- U2 pad 2: Net-(U1-Pad2) -> Net-(U1-Pad6)
Changed lines of the file:
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@@
-(kicad_pcb (version 4) (host pcbnew 4.0.1-3.201512221402+6198~38~ubuntu14.04.1-stable)
+(kicad_pcb (version 4) (host pcbnew 4.0.1-stable)
   (general
     (links 88)
@@
   (net 46 "Net-(R8-Pad1)")
   (net 47 "Net-(U1-Pad16)")
-  (net 48 "Net-(U1-Pad2)")
-  (net 49 "Net-(U1-Pad15)")
-  (net 50 "Net-(D6-Pad1)")
+  (net 48 "Net-(U1-Pad15)")
+  (net 49 "Net-(D6-Pad1)")
+  (net 50 "Net-(U1-Pad6)")
   (net_class Default "This is the default net class."
     (clearance 0.2)
@@
     (add_net "Net-(U1-Pad15)")
     (add_net "Net-(U1-Pad16)")
-    (add_net "Net-(U1-Pad2)")
+    (add_net "Net-(U1-Pad6)")
     (add_net VCC)
     (add_net VCOM)
@@
       (net 2 GND))
     (pad 6 smd rect (at 0.9525 2.667 180) (size 0.4064 1.651) (layers F.Cu F.Paste F.Mask)
-      (net 20 "Net-(P2-Pad1)"))
+      (net 50 "Net-(U1-Pad6)"))
     (pad 7 smd rect (at 1.5875 2.667 180) (size 0.4064 1.651) (layers F.Cu F.Paste F.Mask)
       (net 44 "Net-(R4-Pad1)"))
@@
       (net 17 /PGD))
     (pad 2 smd rect (at -1.5875 2.667 180) (size 0.4064 1.651) (layers F.Cu F.Paste F.Mask)
-      (net 48 "Net-(U1-Pad2)"))
+      (net 20 "Net-(P2-Pad1)"))
     (pad 3 smd rect (at -0.9525 2.667 180) (size 0.4064 1.651) (layers F.Cu F.Paste F.Mask)
       (net 7 VCOM))
@@
       (net 42 "Net-(R2-Pad1)"))
     (pad 15 smd rect (at -1.5875 -2.667 180) (size 0.4064 1.651) (layers F.Cu F.Paste F.Mask)
-      (net 49 "Net-(U1-Pad15)"))
+      (net 48 "Net-(U1-Pad15)"))
     (model walter/smd_dil/ssop-16.wrl
       (at (xyz 0 0 0))
@@
       (net 13 //MCLR))
     (pad 2 smd rect (at -6.985 4.81076 180) (size 0.55118 1.43002) (layers F.Cu F.Paste F.Mask)
-      (net 48 "Net-(U1-Pad2)"))
+      (net 50 "Net-(U1-Pad6)"))
     (pad 3 smd rect (at -5.715 4.81076 180) (size 0.55118 1.43002) (layers F.Cu F.Paste F.Mask)
       (net 46 "Net-(R8-Pad1)"))
@@
       (net 7 VCOM))
     (pad 1 smd rect (at -1.04902 0 270) (size 1.19888 1.19888) (layers F.Cu F.Paste F.Mask)
-      (net 50 "Net-(D6-Pad1)"))
+      (net 49 "Net-(D6-Pad1)"))
   )
   (module Pin_Headers:Pin_Header_Straight_1x10 (layer F.Cu)
@@
       (net 30 /RA3))
     (pad 2 smd rect (at 1.35 0 90) (size 1.5 1.3) (layers F.Cu F.Paste F.Mask)
-      (net 50 "Net-(D6-Pad1)"))
+      (net 49 "Net-(D6-Pad1)"))
     (model Resistors_SMD.3dshapes/R_0805_HandSoldering.wrl
       (at (xyz 0 0 0))

Commit message: some work done
Parts:
- moved P1 1.82 mm to (106.9, 108.5)
- moved R1 0.10 mm to (120.1, 103.6), turned to 180 degrees
- turned C4 to 0 degrees
Routing:
- net VCC: track 0.00 -> 33.8 mm
- net /PGD: track 0.00 -> 28.0 mm, vias 0 -> 2
- net /PGC: track 0.00 -> 27.7 mm, vias 0 -> 2
- net Net-(R2-Pad1): track 0.00 -> 16.6 mm, vias 0 -> 2
- net VCOM: track 0.00 -> 15.6 mm
- net GND: track 0.00 -> 15.6 mm, vias 0 -> 1
- net Net-(C1-Pad1): track 0.00 -> 11.5 mm
- net Net-(C5-Pad1): track 0.00 -> 9.86 mm
- net Net-(C4-Pad1): track 0.00 -> 7.54 mm
- net Net-(R3-Pad1): track 0.00 -> 6.84 mm, vias 0 -> 2
- net Net-(R1-Pad1): track 0.00 -> 6.31 mm
- net Net-(R4-Pad1): track 0.00 -> 4.03 mm
- net Net-(D2-Pad1): track 0.00 -> 2.58 mm
- net Net-(D1-Pad1): track 0.00 -> 2.37 mm
Other:
- board size 50 x 50 mm -> 45 x 50 mm
- net class Power added: clearance 0.2, trace_width 0.4, via_dia 0.6, via_drill 0.4

Commit message: wip
Parts:
- moved P6 0.73 mm to (119.4, 87.6)
- moved P5 0.65 mm to (119.4, 130.8)
- moved U2 0.63 mm to (133.3, 104.1)
- moved R8 0.26 mm to (140.1, 95.2)
- moved R7 0.25 mm to (138.0, 95.2)
- moved R9 0.25 mm to (136.0, 95.2)
Routing:
- net /PGD: track 28.0 -> 18.6 mm
- net /PGC: track 27.7 -> 18.9 mm
- net (no net): track 0.00 -> 1.57 mm
Changed lines of the file:
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@@
-(kicad_pcb (version 4) (host pcbnew 4.0.7-e2-6376~58~ubuntu16.04.1)
+(kicad_pcb (version 4) (host pcbnew 4.0.2+dfsg1-stable)
   (general
     (links 88)
-    (no_connects 65)
-    (area 98.580599 79.8 160.6 138.950001)
+    (no_connects 67)
+    (area 98.580599 74.15 175 138.950001)
     (thickness 1.6)
     (drawings 9)
-    (tracks 127)
+    (tracks 125)
     (zones 0)
     (modules 39)
@@
       (effects (font (size 1 1) (thickness 0.15)))
     )
-    (fp_text value 47pF (at 0 2.1) (layer F.Fab)
+    (fp_text value 47pF (at 0 0.0635) (layer F.Fab)
       (effects (font (size 1 1) (thickness 0.15)))
     )
@@
       (effects (font (size 1 1) (thickness 0.15)))
     )
-    (fp_text value 10uH (at 0 2.1 180) (layer F.Fab)
+    (fp_text value 10uH (at 0.0485 -0.0855 180) (layer F.Fab)
       (effects (font (size 1 1) (thickness 0.15)))
     )
@@
   )
   (module Resistors_SMD:R_0805_HandSoldering (layer F.Cu)
-    (at 138 95 90)
+    (at 138.049 95.25 90)
     (descr "Resistor SMD 0805, hand soldering")
     (tags "resistor 0805")
@@
   )
   (module Resistors_SMD:R_0805_HandSoldering (layer F.Cu)
-    (at 140 95 90)
+    (at 140.081 95.25 90)
     (descr "Resistor SMD 0805, hand soldering")
     (tags "resistor 0805")
@@
   )
   (module w_smd_dil:soic-28 (layer F.Cu)
-    (at 132.969 103.632 180)
+    (at 133.35 104.14 180)
     (descr "SOIC Wide, 28 pins")
     (fp_text reference U2 (at 0 -1.016 180) (layer F.SilkS)
@@
       (effects (font (size 0.7493 0.7493) (thickness 0.14986)))
     )
-    (fp_text value MCP2562 (at 0 1.016 180) (layer F.SilkS)
+    (fp_text value MCP2562 (at -0.0495 0.081 180) (layer F.SilkS)
       (effects (font (size 0.7493 0.7493) (thickness 0.14986)))
     )
@@
   )
   (module Pin_Headers:Pin_Header_Straight_1x10 (layer F.Cu)
-    (at 120 131 90)
+    (at 119.38 130.81 90)
     (descr "Through hole pin header")
     (tags "pin header")
@@
   )
   (module Pin_Headers:Pin_Header_Straight_1x10 (layer F.Cu)
-    (at 119.75 87 90)
+    (at 119.38 87.63 90)
     (descr "Through hole pin header")
     (tags "pin header")
@@
   )
   (module Resistors_SMD:R_0805_HandSoldering (layer F.Cu)
-    (at 136 95 90)
+    (at 136.017 95.25 90)
     (descr "Resistor SMD 0805, hand soldering")
     (tags "resistor 0805")
@@
   (gr_line (start 105.9825 83.995) (end 105.9825 133.995) (angle 90) (layer Edge.Cuts) (width 0.15))
   (gr_line (start 150.9825 83.995) (end 105.9825 83.995) (angle 90) (layer Edge.Cuts) (width 0.15))
+  (segment (start 141.224 108.44276) (end 141.224 107.315) (width 0.25) (layer F.Cu) (net 0))
+  (segment (start 139.954 108.44276) (end 139.954 108.00334) (width 0.25) (layer F.Cu) (net 0))
   (segment (start 115.478 117.356) (end 115.478 114.348) (width 0.25) (layer F.Cu) (net 1))
   (segment (start 115.478 114.348) (end 117.326 112.5) (width 0.25) (layer F.Cu) (net 1))
@@
   (via (at 124.079 97.409) (size 0.6) (drill 0.4) (layers F.Cu B.Cu) (net 17))
   (segment (start 126.492 101.473) (end 125.476 101.473) (width 0.25) (layer F.Cu) (net 17))
-  (segment (start 141.224 108.44276) (end 141.224 107.315) (width 0.25) (layer F.Cu) (net 17))
   (segment (start 135.382 101.473) (end 126.492 101.473) (width 0.25) (layer F.Cu) (net 17))
-  (segment (start 141.224 107.315) (end 135.382 101.473) (width 0.25) (layer F.Cu) (net 17))
-  (segment (start 139.954 108.44276) (end 139.954 108.00334) (width 0.25) (layer F.Cu) (net 18))
   (segment (start 120.015 96.266) (end 121.641449 97.892449) (width 0.25) (layer B.Cu) (net 18))
   (segment (start 121.641449 97.892449) (end 122.369596 97.892449) (width 0.25) (layer B.Cu) (net 18))
   (segment (start 125.47459 102.108) (end 122.79386 99.42727) (width 0.25) (layer F.Cu) (net 18))
-  (segment (start 139.954 108.00334) (end 134.05866 102.108) (width 0.25) (layer F.Cu) (net 18))
   (segment (start 122.79386 99.42727) (end 122.79386 98.316713) (width 0.25) (layer F.Cu) (net 18))
   (segment (start 134.05866 102.108) (end 125.47459 102.108) (width 0.25) (layer F.Cu) (net 18))
