File: USB2CAN-CAN/USB2-CAN-CAN.sch (KiCad schematic (older format))
At the start: 28 parts, among them P1 USB_A, P2 Prog, P3 Prog, P4 CONN_01X03, U1 FT230XS, U2 PIC18F25K80_I/SS, U3 MCP2551-I/SN

Commit message: wip
Parts:
- added P? (x2): CONN_01X10, symbol CONN_01X10
Connections:
- net labels added: CANRX, CANTX, RA3, RA5, RB0, RB1, RB4, RB5, RC0, RC1, RC2, RC3, RC4, RC5, RC6, RC7
- wire segments 96 -> 128
- no-connect marks 17 -> 3
Changed lines of the file:
@@
-$EndComp
-$Comp
-L PIC18F25K80_I/SS U2
-U 1 1 56991EA1
-P 6850 3400
-F 0 "U2" H 6150 4350 50  0000 L CNN
-F 1 "PIC18F25K80_I/SS" H 7550 4350 50  0000 R CNN
-F 2 "SSOP28" H 6850 3150 50  0000 C CNN
-F 3 "" H 6850 3350 50  0000 C CNN
-	1    6850 3400
-	1    0    0    -1
 $EndComp
 $Comp
@@
 	0    -1   -1   0
 $EndComp
-NoConn ~ 6050 2900
-NoConn ~ 6050 3000
 NoConn ~ 6050 3400
 NoConn ~ 6050 3800
-NoConn ~ 7650 2600
-NoConn ~ 7650 2700
-NoConn ~ 7650 3000
-NoConn ~ 7650 3100
-NoConn ~ 7650 3500
-NoConn ~ 7650 3600
-NoConn ~ 7650 3700
-NoConn ~ 7650 3800
-NoConn ~ 7650 3900
-NoConn ~ 7650 4000
-NoConn ~ 7650 4100
-NoConn ~ 7650 4200
 $Comp
 L GND #PWR015
@@
 	1    0    0    -1
 $EndComp
+$Comp
+L CONN_01X10 P?
+U 1 1 5699117D
+P 8600 4300
+F 0 "P?" H 8600 4850 50  0000 C CNN
+F 1 "CONN_01X10" V 8700 4300 50  0000 C CNN
+F 2 "" H 8600 4300 50  0000 C CNN
+F 3 "" H 8600 4300 50  0000 C CNN
+	1    8600 4300
+	-1   0    0    1
+$EndComp
+$Comp
+L VCOM #PWR?
+U 1 1 56991391
+P 9100 3800
+F 0 "#PWR?" H 9100 3650 50  0001 C CNN
+F 1 "VCOM" H 9100 3950 50  0000 C CNN
+F 2 "" H 9100 3800 50  0000 C CNN
+F 3 "" H 9100 3800 50  0000 C CNN
+	1    9100 3800
+	1    0    0    -1
+$EndComp
+$Comp
+L GND #PWR?
+U 1 1 569913F3
+P 9150 4800
+F 0 "#PWR?" H 9150 4550 50  0001 C CNN
+F 1 "GND" H 9150 4650 50  0000 C CNN
+F 2 "" H 9150 4800 50  0000 C CNN
+F 3 "" H 9150 4800 50  0000 C CNN
+	1    9150 4800
+	1    0    0    -1
+$EndComp
+$Comp
+L GND #PWR?
+U 1 1 56991455
+P 9500 3950
+F 0 "#PWR?" H 9500 3700 50  0001 C CNN
+F 1 "GND" H 9500 3800 50  0000 C CNN
+F 2 "" H 9500 3950 50  0000 C CNN
+F 3 "" H 9500 3950 50  0000 C CNN
+	1    9500 3950
+	1    0    0    -1
+$EndComp
+Text Label 9150 4050 0    60   ~ 0
+RC0
+Text Label 9150 4150 0    60   ~ 0
+RC1
+Text Label 9150 4250 0    60   ~ 0
+RC2
+Text Label 9150 4450 0    60   ~ 0
+RC4
+Text Label 9150 4350 0    60   ~ 0
+RC3
+Text Label 9150 4550 0    60   ~ 0
+RC5
+Text Label 9150 4650 0    60   ~ 0
+RC6
+Text Label 9150 4750 0    60   ~ 0
+RC7
+Text Label 7750 3500 0    60   ~ 0
+RC0
+Text Label 7750 3600 0    60   ~ 0
+RC1
+Text Label 7750 3700 0    60   ~ 0
+RC2
+Text Label 7750 3800 0    60   ~ 0
+RC3
+Text Label 7750 3900 0    60   ~ 0
+RC4
+Text Label 7750 4000 0    60   ~ 0
+RC5
+Text Label 7750 4100 0    60   ~ 0
+RC6
+Text Label 7750 4200 0    60   ~ 0
+RC7
+$Comp
+L CONN_01X10 P?
+U 1 1 56993502
+P 8250 1400
+F 0 "P?" H 8250 1950 50  0000 C CNN
+F 1 "CONN_01X10" V 8350 1400 50  0000 C CNN
+F 2 "" H 8250 1400 50  0000 C CNN
+F 3 "" H 8250 1400 50  0000 C CNN
+	1    8250 1400
+	-1   0    0    1
+$EndComp
 Wire Wire Line
 	2950 3150 3150 3150
@@
 	4550 3150 5250 3150
 Wire Wire Line
-	5900 1450 5700 1450
+	5700 1450 5900 1450
 Wire Wire Line
 	5800 1350 5800 1450
@@
 Wire Wire Line
 	5900 2700 5900 2150
+Wire Wire Line
+	8800 3850 9100 3850
+Wire Wire Line
+	9100 3850 9100 3800
+Wire Wire Line
+	9500 3950 8800 3950
+Wire Wire Line
+	8800 4050 9300 4050
+Wire Wire Line
+	8800 4150 9300 4150
+Wire Wire Line
+	8800 4250 9300 4250
+Wire Wire Line
+	8800 4350 9300 4350
+Wire Wire Line
+	8800 4450 9300 4450
+Wire Wire Line
+	8800 4550 9300 4550
+Wire Wire Line
+	9300 4650 8800 4650
+Wire Wire Line
+	8800 4750 9300 4750
+Wire Wire Line
+	7650 3500 7900 3500
+Wire Wire Line
+	7650 3600 7900 3600
+Wire Wire Line
+	7650 3700 7900 3700
+Wire Wire Line
+	7650 3800 7900 3800
+Wire Wire Line
+	7650 3900 7900 3900
+Wire Wire Line
+	7650 4000 7900 4000
+Wire Wire Line
+	7650 4100 7900 4100
+Wire Wire Line
+	7650 4200 7900 4200
+Wire Wire Line
+	8450 1150 8750 1150
+Wire Wire Line
+	8450 1250 8750 1250
+Wire Wire Line
+	8450 1350 8750 1350
+Wire Wire Line
+	8450 1450 8750 1450
+Wire Wire Line
+	8450 1550 8750 1550
+Wire Wire Line
+	8450 1650 8750 1650
+Wire Wire Line
+	8450 1750 8750 1750
+Wire Wire Line
+	8450 1850 8750 1850
+$Comp
+L VCOM #PWR?
+U 1 1 56993D99
+P 8550 900
+F 0 "#PWR?" H 8550 750 50  0001 C CNN
+F 1 "VCOM" H 8550 1050 50  0000 C CNN
+F 2 "" H 8550 900 50  0000 C CNN
+F 3 "" H 8550 900 50  0000 C CNN
+	1    8550 900
+	1    0    0    -1
+$EndComp
+$Comp
+L GND #PWR?
+U 1 1 56993EB2
+P 9000 1050
+F 0 "#PWR?" H 9000 800 50  0001 C CNN
+F 1 "GND" H 9000 900 50  0000 C CNN
+F 2 "" H 9000 1050 50  0000 C CNN
+F 3 "" H 9000 1050 50  0000 C CNN
+	1    9000 1050
+	1    0    0    -1
+$EndComp
+Wire Wire Line
+	8450 950  8550 950
+Wire Wire Line
+	8550 950  8550 900
+Wire Wire Line
+	8450 1050 9000 1050
+Text Label 8600 1150 0    60   ~ 0
+RB0
+Text Label 8600 1250 0    60   ~ 0
+RB1
+Text Label 8600 1550 0    60   ~ 0
+RB4
+Text Label 8500 1350 0    60   ~ 0
+CANTX
+Text Label 8500 1450 0    60   ~ 0
+CANRX
+Text Label 8600 1650 0    60   ~ 0
+RB5
+Text Label 8600 1750 0    60   ~ 0
+RA3
+Text Label 8600 1850 0    60   ~ 0
+RA5
+$Comp
+L PIC18F25K80_I/SS U2
+U 1 1 56991EA1
+P 6850 3400
+F 0 "U2" H 6150 4350 50  0000 L CNN
+F 1 "PIC18F25K80_I/SS" H 7550 4350 50  0000 R CNN
+F 2 "SSOP28" H 6850 3150 50  0000 C CNN
+F 3 "" H 6850 3350 50  0000 C CNN
+	1    6850 3400
+	1    0    0    -1
+$EndComp
+Wire Wire Line
+	6050 2900 5900 2900
+Wire Wire Line
+	6050 3000 5900 3000
+Text Label 5900 2900 0    60   ~ 0
+RA3
+Text Label 5900 3000 0    60   ~ 0
+RA5
 $EndSCHEMATC

Commit message: wip
Parts:
- removed P? (x2): CONN_01X10, symbol CONN_01X10
- added C9: CP, Capacitors_SMD:C_0805_HandSoldering, symbol CP
- added D5: BAT43, Diodes_SMD:Diode-MELF_Handsoldering, symbol D_Schottky
- added JP1: ICSP, ICSP:ICSP, symbol ICSP
- added P5, P6: CONN_01X12, Pin_Headers:Pin_Header_Straight_1x12, symbol CONN_01X12
- C1, C2, C3, C4, C5, C6, C7, C8: footprint (none) -> Capacitors_SMD:C_0805_HandSoldering
- D1, D2, D3, D4: footprint (none) -> LEDs:LED-0805
- Ferrit1, R1, R2, R3, R4, R5, R7, R8: footprint (none) -> Resistors_SMD:R_0805_HandSoldering
- P1: footprint (none) -> w_conn_pc:conn_usb_B
- P2: footprint (none) -> Pin_Headers:Pin_Header_Straight_1x02
- P3: value Prog -> Term; footprint (none) -> Pin_Headers:Pin_Header_Straight_1x02
- P4: footprint (none) -> Pin_Headers:Pin_Header_Straight_1x03
- R6: value 10k -> 4k7; footprint (none) -> Resistors_SMD:R_0805_HandSoldering
- U1: footprint SSOP-16 -> w_smd_dil:ssop-16
- U2: footprint SSOP28 -> w_smd_dil:soic-28
- U3: value MCP2551-I/SN -> MCP2562; footprint SO-8 -> w_smd_dil:so-8
Connections:
- net labels added: /MCLR, CLKOUT, PGC, PGD
- wire segments 128 -> 148
Other:
- moved on the sheet: C1, C2, C3, C4, C5, C6, C7, C8, D1, D2, D3, D4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

Commit message: wip
Parts:
- R5: value 270 -> 120
Changed lines of the file:
@@
 LIBS:ftdi
 LIBS:microchip_pic18mcu
-LIBS:ICSP
 LIBS:USB2-CAN-CAN-cache
 EELAYER 25 0
@@
 P 9350 3550
 F 0 "R5" V 9430 3550 50  0000 C CNN
-F 1 "270" V 9350 3550 50  0000 C CNN
+F 1 "120" V 9350 3550 50  0000 C CNN
 F 2 "Resistors_SMD:R_0805_HandSoldering" V 9280 3550 50  0001 C CNN
 F 3 "" H 9350 3550 50  0000 C CNN

Commit message: V1.1 wip
Parts:
- removed P5, P6: CONN_01X12, Pin_Headers:Pin_Header_Straight_1x12, symbol CONN_01X12
- added D6: LED, LEDs:LED-0805, symbol LED
- added P5: CON1, Pin_Headers:Pin_Header_Straight_1x10, symbol CONN_01X10
- added P6: CON2, Pin_Headers:Pin_Header_Straight_1x10, symbol CONN_01X10
- added R9: 270, Resistors_SMD:R_0805_HandSoldering, symbol R
Connections:
- wire segments 148 -> 144
Changed lines of the file:
@@
 F 0 "U1" H 3050 4850 50  0000 L CNN
 F 1 "FT230XS" H 3900 4850 50  0001 L CNN
-F 2 "w_smd_dil:ssop-16" H 3600 4250 50  0000 C CNN
+F 2 "w_smd_dil:ssop-16" H 3600 4250 50  0001 C CNN
 F 3 "" H 3600 4250 50  0000 C CNN
 	1    3600 4250
@@
 L VCOM #PWR017
 U 1 1 56995501
-P 7900 3650
-F 0 "#PWR017" H 7900 3500 50  0001 C CNN
-F 1 "VCOM" H 7900 3800 50  0000 C CNN
-F 2 "" H 7900 3650 50  0000 C CNN
-F 3 "" H 7900 3650 50  0000 C CNN
-	1    7900 3650
+P 8000 3650
+F 0 "#PWR017" H 8000 3500 50  0001 C CNN
+F 1 "VCOM" H 8000 3800 50  0000 C CNN
+F 2 "" H 8000 3650 50  0000 C CNN
+F 3 "" H 8000 3650 50  0000 C CNN
+	1    8000 3650
 	1    0    0    -1
 $EndComp
@@
 $EndComp
 $Comp
-L VCOM #PWR020
-U 1 1 56991391
-P 8850 4800
-F 0 "#PWR020" H 8850 4650 50  0001 C CNN
-F 1 "VCOM" H 8850 4950 50  0000 C CNN
-F 2 "" H 8850 4800 50  0000 C CNN
-F 3 "" H 8850 4800 50  0000 C CNN
-	1    8850 4800
-	1    0    0    -1
-$EndComp
-$Comp
-L GND #PWR021
+L GND #PWR020
 U 1 1 56991455
 P 9250 4950
-F 0 "#PWR021" H 9250 4700 50  0001 C CNN
+F 0 "#PWR020" H 9250 4700 50  0001 C CNN
 F 1 "GND" H 9250 4800 50  0000 C CNN
 F 2 "" H 9250 4950 50  0000 C CNN
@@
 	7800 3900 7400 3900
 Wire Wire Line
-	8050 3900 7850 3900
-Wire Wire Line
-	7850 3900 7850 3850
-Wire Wire Line
-	7850 3850 7750 3850
+	8050 3900 7900 3900
+Wire Wire Line
+	7900 3900 7900 3850
+Wire Wire Line
+	7900 3850 7750 3850
 Wire Wire Line
 	7750 3850 7750 3800
@@
 Connection ~ 6500 6050
 Wire Wire Line
-	8050 4100 7900 4100
-Wire Wire Line
-	7900 4100 7900 3650
-Wire Wire Line
-	8050 4200 7900 4200
-Wire Wire Line
-	7900 4200 7900 4400
-Wire Wire Line
-	7900 4400 8550 4400
+	8050 4100 8000 4100
+Wire Wire Line
+	8000 4100 8000 3650
+Wire Wire Line
+	8050 4200 8000 4200
+Wire Wire Line
+	8000 4200 8000 4400
+Wire Wire Line
+	8000 4400 8550 4400
 Wire Wire Line
 	8550 4400 8550 4450
@@
 	7400 5200 7650 5200
 Wire Wire Line
-	8200 2150 8500 2150
-Wire Wire Line
-	8200 2250 8500 2250
-Wire Wire Line
-	8200 2350 8500 2350
-Wire Wire Line
-	8200 2450 8500 2450
-Wire Wire Line
-	8200 2550 8500 2550
-Wire Wire Line
-	8200 2750 8500 2750
-Wire Wire Line
-	8200 2850 8500 2850
-$Comp
-L VCOM #PWR022
+	9950 5100 10250 5100
+Wire Wire Line
+	9950 5200 10250 5200
+Wire Wire Line
+	9950 5300 10250 5300
+Wire Wire Line
+	9950 5400 10250 5400
+Wire Wire Line
+	9950 5500 10250 5500
+Wire Wire Line
+	9950 5700 10250 5700
+Wire Wire Line
+	9950 5800 10250 5800
+$Comp
+L VCOM #PWR021
 U 1 1 56993D99
-P 8300 1900
-F 0 "#PWR022" H 8300 1750 50  0001 C CNN
-F 1 "VCOM" H 8300 2050 50  0000 C CNN
-F 2 "" H 8300 1900 50  0000 C CNN
-F 3 "" H 8300 1900 50  0000 C CNN
-	1    8300 1900
-	1    0    0    -1
-$EndComp
-$Comp
-L GND #PWR023
+P 10050 4850
+F 0 "#PWR021" H 10050 4700 50  0001 C CNN
+F 1 "VCOM" H 10050 5000 50  0000 C CNN
+F 2 "" H 10050 4850 50  0000 C CNN
+F 3 "" H 10050 4850 50  0000 C CNN
+	1    10050 4850
+	1    0    0    -1
+$EndComp
+$Comp
+L GND #PWR022
 U 1 1 56993EB2
-P 8750 2050
-F 0 "#PWR023" H 8750 1800 50  0001 C CNN
-F 1 "GND" H 8750 1900 50  0000 C CNN
-F 2 "" H 8750 2050 50  0000 C CNN
-F 3 "" H 8750 2050 50  0000 C CNN
-	1    8750 2050
-	1    0    0    -1
-$EndComp
-Wire Wire Line
-	8200 1950 8300 1950
-Wire Wire Line
-	8300 1950 8300 1900
-Wire Wire Line
-	8200 2050 8750 2050
-Text Label 8350 2150 0    60   ~ 0
+P 10500 5000
+F 0 "#PWR022" H 10500 4750 50  0001 C CNN
+F 1 "GND" H 10500 4850 50  0000 C CNN
+F 2 "" H 10500 5000 50  0000 C CNN
+F 3 "" H 10500 5000 50  0000 C CNN
+	1    10500 5000
+	1    0    0    -1
+$EndComp
+Wire Wire Line
+	9950 4900 10050 4900
+Wire Wire Line
+	10050 4900 10050 4850
+Wire Wire Line
+	9950 5000 10500 5000
+Text Label 10100 5100 0    60   ~ 0
 RB0
-Text Label 8350 2250 0    60   ~ 0
+Text Label 10100 5200 0    60   ~ 0
 RB1
-Text Label 8350 2550 0    60   ~ 0
+Text Label 10100 5500 0    60   ~ 0
 RB4
-Text Label 8250 2350 0    60   ~ 0
+Text Label 10000 5300 0    60   ~ 0
 CANTX
-Text Label 8250 2450 0    60   ~ 0
+Text Label 10000 5400 0    60   ~ 0
 CANRX
-Text Label 8350 2650 0    60   ~ 0
+Text Label 10100 5600 0    60   ~ 0
 RB5
-Text Label 8350 2750 0    60   ~ 0
-RA3
-Text Label 8350 2850 0    60   ~ 0
+Text Label 10100 5700 0    60   ~ 0
 RA5
 $Comp
@@
 F 0 "U2" H 5900 5350 50  0000 L CNN
 F 1 "PIC18F25K80_I/SS" H 7300 5350 50  0001 R CNN
-F 2 "w_smd_dil:soic-28" H 6600 4150 50  0000 C CNN
+F 2 "w_smd_dil:soic-28" H 6600 4150 50  0001 C CNN
 F 3 "" H 6600 4350 50  0000 C CNN
 	1    6600 4400
@@
 Text Label 5650 4000 0    60   ~ 0
 RA5
-$Comp
-L CONN_01X12 P6
-U 1 1 569933BD
-P 8350 5400
-F 0 "P6" H 8350 6050 50  0000 C CNN
-F 1 "CONN_01X12" V 8450 5400 50  0000 C CNN
-F 2 "Pin_Headers:Pin_Header_Straight_1x12" H 8350 5400 50  0001 C CNN
-F 3 "" H 8350 5400 50  0000 C CNN
-	1    8350 5400
-	-1   0    0    -1
-$EndComp
-$Comp
-L CONN_01X12 P5
-U 1 1 56993A95
-P 8000 2500
-F 0 "P5" H 8000 3150 50  0000 C CNN
-F 1 "CONN_01X12" V 8100 2500 50  0000 C CNN
-F 2 "Pin_Headers:Pin_Header_Straight_1x12" H 8000 2500 50  0001 C CNN
-F 3 "" H 8000 2500 50  0000 C CNN
-	1    8000 2500
-	-1   0    0    -1
-$EndComp
-Wire Wire Line
-	8200 2950 8500 2950
-Wire Wire Line
-	8200 3050 8500 3050
-Text Label 8200 2950 0    60   ~ 0
+Text Label 9950 5800 0    60   ~ 0
 CLKOUT
-Wire Wire Line
-	8550 5850 9100 5850
-Wire Wire Line
-	8550 5950 8800 5950
-Wire Wire Line
-	8800 5950 8800 6100
-$Comp
-L GND #PWR024
-U 1 1 56995A47
-P 8500 3050
-F 0 "#PWR024" H 8500 2800 50  0001 C CNN
-F 1 "GND" H 8500 2900 50  0000 C CNN
-F 2 "" H 8500 3050 50  0000 C CNN
-F 3 "" H 8500 3050 50  0000 C CNN
-	1    8500 3050
-	1    0    0    -1
-$EndComp
-$Comp
-L GND #PWR025
-U 1 1 56995B6A
-P 8800 6100
-F 0 "#PWR025" H 8800 5850 50  0001 C CNN
-F 1 "GND" H 8800 5950 50  0000 C CNN
-F 2 "" H 8800 6100 50  0000 C CNN
-F 3 "" H 8800 6100 50  0000 C CNN
-	1    8800 6100
-	1    0    0    -1
-$EndComp
-Wire Wire Line
-	9100 5850 9100 5800
-$Comp
-L VCC #PWR026
-U 1 1 56996E1B
-P 9100 5800
-F 0 "#PWR026" H 9100 5650 50  0001 C CNN
-F 1 "VCC" H 9100 5950 50  0000 C CNN
-F 2 "" H 9100 5800 50  0000 C CNN
-F 3 "" H 9100 5800 50  0000 C CNN
-	1    9100 5800
-	1    0    0    -1
-$EndComp
 Wire Wire Line
 	5800 4400 5400 4400
@@
 	5250 4800 5250 4850
 $Comp
-L GND #PWR027
+L GND #PWR023
 U 1 1 56998F39
 P 5250 5150
-F 0 "#PWR027" H 5250 4900 50  0001 C CNN
+F 0 "#PWR023" H 5250 4900 50  0001 C CNN
 F 1 "GND" H 5250 5000 50  0000 C CNN
 F 2 "" H 5250 5150 50  0000 C CNN
@@
 	5250 3050 5050 3050
 $Comp
-L VCOM #PWR028
+L VCOM #PWR024
 U 1 1 5699B4D4
 P 5050 2350
-F 0 "#PWR028" H 5050 2200 50  0001 C CNN
+F 0 "#PWR024" H 5050 2200 50  0001 C CNN
 F 1 "VCOM" H 5050 2500 50  0000 C CNN
 F 2 "" H 5050 2350 50  0000 C CNN
@@
 NoConn ~ 6400 2750
 Wire Wire Line
-	8200 2650 8500 2650
-$Comp
-L PWR_FLAG #FLG029
+	9950 5600 10250 5600
+$Comp
+L PWR_FLAG #FLG025
 U 1 1 5699E549
 P 4900 4900
-F 0 "#FLG029" H 4900 4995 50  0001 C CNN
+F 0 "#FLG025" H 4900 4995 50  0001 C CNN
 F 1 "PWR_FLAG" H 4900 5080 50  0000 C CNN
 F 2 "" H 4900 4900 50  0000 C CNN
@@
 	5050 4900 4900 4900
 Connection ~ 5250 4800
+$Comp
+L LED D6
+U 1 1 569EBA4B
+P 4200 2500
+F 0 "D6" H 4350 2400 50  0000 C CNN
+F 1 "LED" H 4200 2400 50  0000 C CNN
+F 2 "LEDs:LED-0805" H 4200 2500 50  0001 C CNN
+F 3 "" H 4200 2500 50  0000 C CNN
+	1    4200 2500
+	0    -1   -1   0
+$EndComp
+$Comp
+L R R9
+U 1 1 569EBA51
+P 4200 2850
+F 0 "R9" V 4280 2850 50  0000 C CNN
+F 1 "270" V 4200 2850 50  0000 C CNN
+F 2 "Resistors_SMD:R_0805_HandSoldering" V 4130 2850 50  0001 C CNN
+F 3 "" H 4200 2850 50  0000 C CNN
+	1    4200 2850
+	-1   0    0    1
+$EndComp
+$Comp
+L VCOM #PWR026
+U 1 1 569EBAC4
+P 4200 2300
+F 0 "#PWR026" H 4200 2150 50  0001 C CNN
+F 1 "VCOM" H 4200 2450 50  0000 C CNN
+F 2 "" H 4200 2300 50  0000 C CNN
+F 3 "" H 4200 2300 50  0000 C CNN
+	1    4200 2300
+	1    0    0    -1
+$EndComp
+Wire Wire Line
+	4200 3000 4200 3150
+Wire Wire Line
+	4200 3150 4500 3150
+Text Label 4350 3150 0    60   ~ 0
+RA3
+$Comp
+L VCC #PWR027
+U 1 1 569EF150
+P 8850 4800
+F 0 "#PWR027" H 8850 4650 50  0001 C CNN
+F 1 "VCC" H 8850 4950 50  0000 C CNN
+F 2 "" H 8850 4800 50  0000 C CNN
+F 3 "" H 8850 4800 50  0000 C CNN
+	1    8850 4800
+	1    0    0    -1
+$EndComp
+$Comp
+L CONN_01X10 P5
+U 1 1 569EF55C
+P 9750 5350
+F 0 "P5" H 9750 5900 50  0000 C CNN
+F 1 "CON1" V 9850 5350 50  0000 C CNN
+F 2 "Pin_Headers:Pin_Header_Straight_1x10" H 9750 5350 50  0001 C CNN
+F 3 "" H 9750 5350 50  0000 C CNN
+	1    9750 5350
+	-1   0    0    -1
+$EndComp
+$Comp
+L CONN_01X10 P6
+U 1 1 569EF733
+P 8350 5300
+F 0 "P6" H 8350 5850 50  0000 C CNN
+F 1 "CON2" V 8450 5300 50  0000 C CNN
+F 2 "Pin_Headers:Pin_Header_Straight_1x10" H 8350 5300 50  0001 C CNN
+F 3 "" H 8350 5300 50  0000 C CNN
+	1    8350 5300
+	-1   0    0    -1
+$EndComp
 $EndSCHEMATC

Commit message: house keeping
Connections:
- wire segments 144 -> 143
Other:
- moved on the sheet: D1, D2, P2
Changed lines of the file:
@@
 L LED D1
 U 1 1 5698FA8C
-P 4550 3950
-F 0 "D1" H 4700 3850 50  0000 C CNN
-F 1 "LED" H 4550 3850 50  0000 C CNN
-F 2 "LEDs:LED-0805" H 4550 3950 50  0001 C CNN
-F 3 "" H 4550 3950 50  0000 C CNN
-	1    4550 3950
+P 4550 3750
+F 0 "D1" H 4700 3650 50  0000 C CNN
+F 1 "LED" H 4550 3650 50  0000 C CNN
+F 2 "LEDs:LED-0805" H 4550 3750 50  0001 C CNN
+F 3 "" H 4550 3750 50  0000 C CNN
+	1    4550 3750
 	0    -1   -1   0
 $EndComp
@@
 L LED D2
 U 1 1 5698FAFE
-P 4800 3950
-F 0 "D2" H 4950 3850 50  0000 C CNN
-F 1 "LED" H 4800 3850 50  0000 C CNN
-F 2 "LEDs:LED-0805" H 4800 3950 50  0001 C CNN
-F 3 "" H 4800 3950 50  0000 C CNN
-	1    4800 3950
+P 4800 3750
+F 0 "D2" H 4950 3650 50  0000 C CNN
+F 1 "LED" H 4800 3650 50  0000 C CNN
+F 2 "LEDs:LED-0805" H 4800 3750 50  0001 C CNN
+F 3 "" H 4800 3750 50  0000 C CNN
+	1    4800 3750
 	0    -1   -1   0
 $EndComp
@@
 L CONN_01X02 P2
 U 1 1 56993CB7
-P 5150 4000
-F 0 "P2" H 5150 4150 50  0000 C CNN
-F 1 "Prog" V 5250 4000 50  0000 C CNN
-F 2 "Pin_Headers:Pin_Header_Straight_1x02" H 5150 4000 50  0001 C CNN
-F 3 "" H 5150 4000 50  0000 C CNN
-	1    5150 4000
+P 5100 3850
+F 0 "P2" H 5100 4000 50  0000 C CNN
+F 1 "Prog" V 5200 3850 50  0000 C CNN
+F 2 "Pin_Headers:Pin_Header_Straight_1x02" H 5100 3850 50  0001 C CNN
+F 3 "" H 5100 3850 50  0000 C CNN
+	1    5100 3850
 	0    -1   -1   0
 $EndComp
@@
 	2800 3300 4800 3300
 Wire Wire Line
-	4550 3300 4550 3750
-Wire Wire Line
-	4800 3300 4800 3750
+	4550 3300 4550 3550
 Connection ~ 4550 3300
 Wire Wire Line
@@
 	2550 3500 2550 4050
 Wire Wire Line
-	4300 4050 4400 4050
-Wire Wire Line
-	4400 4050 4400 3700
-Wire Wire Line
-	4400 3700 5200 3700
-Wire Wire Line
-	4300 3850 4300 3600
-Wire Wire Line
-	4300 3600 5000 3600
+	4400 3600 4400 4150
+Wire Wire Line
+	4400 3600 5800 3600
+Wire Wire Line
+	4300 3850 4300 3400
+Wire Wire Line
+	4300 3400 5000 3400
 Wire Wire Line
 	4300 3950 4350 3950
 Wire Wire Line
-	4350 3950 4350 3650
+	4350 3950 4350 3500
 Wire Wire Line
 	4300 4650 5200 4650
@@
 	5200 4500 5800 4500
 Wire Wire Line
-	4350 3650 5100 3650
-Wire Wire Line
-	5100 3650 5100 3300
+	4350 3500 5100 3500
+Wire Wire Line
+	5100 3500 5100 3300
 Wire Wire Line
 	5100 3300 7650 3300
@@
 	7700 3250 5000 3250
 Wire Wire Line
-	5000 3250 5000 3600
-Wire Wire Line
-	5200 3700 5200 3600
-Wire Wire Line
-	5200 3600 5800 3600
+	5000 3250 5000 3400
 Wire Wire Line
 	8050 3800 7800 3800
@@
 Connection ~ 5600 5100
 Wire Wire Line
-	5200 4200 5800 4200
-Wire Wire Line
-	5000 4150 5000 4200
-Wire Wire Line
-	5000 4200 5100 4200
+	5150 4200 5800 4200
 Wire Wire Line
 	6250 6050 6700 6050
@@
 Wire Wire Line
 	4300 4550 4800 4550
-Wire Wire Line
-	4300 4150 5000 4150
 Wire Wire Line
 	5450 2450 5650 2450
@@
 	-1   0    0    -1
 $EndComp
+Wire Wire Line
+	4400 4150 4300 4150
+Wire Wire Line
+	4300 4050 5050 4050
+Wire Wire Line
+	4800 3300 4800 3550
+Wire Wire Line
+	5150 4200 5150 4050
+Wire Wire Line
+	4550 4150 4550 3950
+Wire Wire Line
+	4800 4150 4800 3950
 $EndSCHEMATC

Commit message: some work done
Connections:
- wire segments 143 -> 149
Changed lines of the file:
@@
 LIBS:ftdi
 LIBS:microchip_pic18mcu
+LIBS:microchip_dspic33dsc
 LIBS:USB2-CAN-CAN-cache
 EELAYER 25 0
@@
 Text Label 7400 3900 0    60   ~ 0
 CANRX
-Text Label 6400 2550 0    60   ~ 0
+Text Label 6200 2550 0    60   ~ 0
 PGD
-Text Label 6400 2650 0    60   ~ 0
+Text Label 6200 2650 0    60   ~ 0
 PGC
-Text Label 6400 2450 0    60   ~ 0
+Text Label 6200 2450 0    60   ~ 0
 GND
-Text Label 6400 2250 0    60   ~ 0
+Text Label 6200 2250 0    60   ~ 0
 /MCLR
-NoConn ~ 6400 2350
-NoConn ~ 6400 2750
 Wire Wire Line
 	9950 5600 10250 5600
@@
 Wire Wire Line
 	4800 4150 4800 3950
+Wire Wire Line
+	6200 2250 6400 2250
+Wire Wire Line
+	6400 2350 6200 2350
+Wire Wire Line
+	6400 2450 6200 2450
+Wire Wire Line
+	6400 2550 6200 2550
+Wire Wire Line
+	6400 2650 6200 2650
+Wire Wire Line
+	6400 2750 6200 2750
+NoConn ~ 6200 2750
+NoConn ~ 6200 2350
 $EndSCHEMATC

Commit message: wip
Parts:
- D1, D2, D3, D4, D6: symbol LED -> LED-RESCUE-USB2-CAN-CAN
- P1: symbol USB_A -> USB_A-RESCUE-USB2-CAN-CAN
- U2: symbol PIC18F25K80_I/SS -> PIC18F25K80_I/SS-RESCUE-USB2-CAN-CAN
- U3: symbol MCP2551-I/SN -> MCP2551-I/SN-RESCUE-USB2-CAN-CAN
Changed lines of the file:
@@
 EESchema Schematic File Version 2
+LIBS:USB2-CAN-CAN-rescue
 LIBS:power
 LIBS:device
@@
 $EndDescr
 $Comp
-L USB_A P1
+L USB_A-RESCUE-USB2-CAN-CAN P1
 U 1 1 5698F020
 P 1400 4250
@@
 $EndComp
 $Comp
-L LED D1
+L LED-RESCUE-USB2-CAN-CAN D1
 U 1 1 5698FA8C
 P 4550 3750
@@
 $EndComp
 $Comp
-L LED D2
+L LED-RESCUE-USB2-CAN-CAN D2
 U 1 1 5698FAFE
 P 4800 3750
@@
 $EndComp
 $Comp
-L MCP2551-I/SN U3
+L MCP2551-I/SN-RESCUE-USB2-CAN-CAN U3
 U 1 1 569928B5
 P 8550 4000
@@
 $EndComp
 $Comp
-L LED D3
+L LED-RESCUE-USB2-CAN-CAN D3
 U 1 1 56996B07
 P 5450 2650
@@
 $EndComp
 $Comp
-L LED D4
+L LED-RESCUE-USB2-CAN-CAN D4
 U 1 1 56996CE0
 P 5650 2650
@@
 RA5
 $Comp
-L PIC18F25K80_I/SS U2
+L PIC18F25K80_I/SS-RESCUE-USB2-CAN-CAN U2
 U 1 1 56991EA1
 P 6600 4400
@@
 Connection ~ 5250 4800
 $Comp
-L LED D6
+L LED-RESCUE-USB2-CAN-CAN D6
 U 1 1 569EBA4B
 P 4200 2500

Commit message: wip
Parts:
- removed U3: MCP2562, w_smd_dil:so-8, symbol MCP2551-I/SN-RESCUE-USB2-CAN-CAN
- C1, C2, C3, C4, C5, C6, C7, C8: symbol C -> USB2-CAN-CAN-rescue:C
- C9: symbol CP -> USB2-CAN-CAN-rescue:CP
- D1, D2, D3, D4, D6: symbol LED-RESCUE-USB2-CAN-CAN -> USB2-CAN-CAN-rescue:LED-RESCUE-USB2-CAN-CAN
- D5: symbol D_Schottky -> USB2-CAN-CAN-rescue:D_Schottky
- Ferrit1, R1, R2, R3, R4, R5, R6, R7, R8, R9: symbol R -> USB2-CAN-CAN-rescue:R
- JP1: symbol ICSP -> USB2-CAN-CAN-rescue:ICSP
- P1: symbol USB_A-RESCUE-USB2-CAN-CAN -> USB2-CAN-CAN-rescue:USB_A-RESCUE-USB2-CAN-CAN
- P2, P3: symbol CONN_01X02 -> USB2-CAN-CAN-rescue:CONN_01X02
- P4: symbol CONN_01X03 -> USB2-CAN-CAN-rescue:CONN_01X03
- P5, P6: symbol CONN_01X10 -> USB2-CAN-CAN-rescue:CONN_01X10
- U1: symbol FT230XS -> USB2-CAN-CAN-rescue:FT230XS
- U2: value PIC18F25K80_I/SS -> PIC18F26K80_I/SS; footprint w_smd_dil:soic-28 -> Package_SO:SSOP-28_5.3x10.2mm_P0.65mm; symbol PIC18F25K80_I/SS-RESCUE-USB2-CAN-CAN -> MCU_Microchip_PIC18:PIC18F26K80_ISS
Connections:
- wire segments 149 -> 173
