File: RS485/rs232-rs485/rs232-rs485.sch (KiCad schematic (older format))
At the start: 8 parts, among them J1 Conn_02x04_Counter_Clockwise, J2 Conn_01x03, U1 PIC10F322, U2 MAX3072E

Commit message: use 2.00mm pin header
Parts:
- J2: footprint Connector_PinHeader_1.27mm:PinHeader_1x03_P1.27mm_Vertical -> Connector_PinHeader_2.00mm:PinHeader_1x03_P2.00mm_Vertical
Changed lines of the file:
@@
 EESchema Schematic File Version 4
+LIBS:rs232-rs485-cache
 EELAYER 29 0
 EELAYER END
@@
 F 0 "J2" V 4825 3550 50  0000 R CNN
 F 1 "Conn_01x03" V 4900 3725 50  0001 R CNN
-F 2 "Connector_PinHeader_1.27mm:PinHeader_1x03_P1.27mm_Vertical" H 4725 3500 50  0001 C CNN
+F 2 "Connector_PinHeader_2.00mm:PinHeader_1x03_P2.00mm_Vertical" H 4725 3500 50  0001 C CNN
 F 3 "~" H 4725 3500 50  0001 C CNN
 	1    4725 3500
