File: c6021light/bluepill/hardware/c6021light.sch (KiCad schematic (older format))
At the start: 69 parts, among them J1 Barrel_Jack_Switch, J10 Conn_01x02, J11 Conn_01x02, J12 XpressNet, J3 Conn_02x16_Row_Letter_First, J30 Loconet, J4 Conn_01x02, J5 Grove I2C, J50 USB_B_Micro, J51 Conn_01x06, J52 Debug UART, J6 Conn_01x02, J7 Conn_01x02, J8 RJ45, Q30 BC337, SW1 SW_Push, U1 L7805, U10 SN75176, U2 L7808, U3 MCP2562, U30 LM393, U4 ISO1050DUB, U50 CH340C

Commit message: wip
Parts:
- removed R5: 0, Resistor_THT:R_Axial_DIN0207_L6.3mm_D2.5mm_P7.62mm_Horizontal, symbol Device:R
- added J2: Conn_02x03_Odd_Even, Connector_PinHeader_2.54mm:PinHeader_2x03_P2.54mm_Vertical, symbol Connector_Generic:Conn_02x03_Odd_Even
- R4: footprint Resistor_THT:R_Axial_DIN0207_L6.3mm_D2.5mm_P7.62mm_Horizontal -> Resistor_THT:R_AXIAL_0_WIRE
- renumbered R6 to R5
Connections:
- net +3V3: now also U3.5 (Vio), J2.6 (Pin_6); no longer R4.2
- net GND: now also R4.2, U3.8 (STBY), J2.5 (Pin_5)
- net GNDD: now also R4.1
- net at BP1.29 (PA4): now also J2.3 (Pin_3)
- net at BP1.30 (PA5): now also J2.1 (Pin_1)
- net at BP1.31 (PA6): now also J2.2 (Pin_2)
- net at BP1.32 (PA7): now also J2.4 (Pin_4)
- no-connect marks 32 -> 28
Other:
- moved on the sheet: D1, R3, R4
Changed lines of the file:
@@
 $EndDescr
-$Comp
-L YAAJ_STM32:BluePill_1 BP1
-U 1 1 5ED69C35
-P 4000 2475
-F 0 "BP1" H 4575 2650 50  0000 C CNN
-F 1 "BluePill_1" H 4575 2559 50  0000 C CNN
-F 2 "YAAJ_STM32:YAAJ_BluePill" H 5250 525 50  0001 C CNN
-F 3 "" H 5250 525 50  0001 C CNN
-	1    4000 2475
-	1    0    0    -1
-$EndComp
 $Comp
 L Regulator_Linear:L7805 U1
@@
 NoConn ~ 5350 4325
 NoConn ~ 5350 3125
-NoConn ~ 5350 3225
-NoConn ~ 5350 3325
-NoConn ~ 5350 3425
-NoConn ~ 5350 3525
-NoConn ~ 5350 3625
 NoConn ~ 3800 3225
 NoConn ~ 3800 3325
@@
 L power:+3V3 #PWR0108
 U 1 1 5ED9A0AB
-P 6650 1450
-F 0 "#PWR0108" H 6650 1300 50  0001 C CNN
-F 1 "+3V3" H 6665 1623 50  0000 C CNN
-F 2 "" H 6650 1450 50  0001 C CNN
-F 3 "" H 6650 1450 50  0001 C CNN
-	1    6650 1450
-	1    0    0    -1
-$EndComp
-Wire Wire Line
-	6650 1500 6650 1450
+P 7000 1450
+F 0 "#PWR0108" H 7000 1300 50  0001 C CNN
+F 1 "+3V3" H 6875 1450 50  0000 C CNN
+F 2 "" H 7000 1450 50  0001 C CNN
+F 3 "" H 7000 1450 50  0001 C CNN
+	1    7000 1450
+	1    0    0    -1
+$EndComp
+Wire Wire Line
+	7000 1500 7000 1450
 Wire Wire Line
 	7225 1200 6975 1200
@@
 Wire Wire Line
 	7725 900  7725 1000
-Wire Wire Line
-	7225 1600 7225 1825
 $Comp
 L Connector:RJ45 J8
@@
 $EndComp
 $Comp
-L Device:R R6
+L Device:R R5
 U 1 1 5F087407
 P 8425 1075
-F 0 "R6" H 8495 1121 50  0000 L CNN
+F 0 "R5" H 8495 1121 50  0000 L CNN
 F 1 "120" V 8425 1000 50  0000 L CNN
 F 2 "Resistor_THT:R_Axial_DIN0207_L6.3mm_D2.5mm_P7.62mm_Horizontal" V 8355 1075 50  0001 C CNN
@@
 L Device:LED D1
 U 1 1 5F293D84
-P 5950 3875
-F 0 "D1" V 5989 3757 50  0000 R CNN
-F 1 "LED" V 5898 3757 50  0000 R CNN
-F 2 "LED_THT:LED_D3.0mm" H 5950 3875 50  0001 C CNN
-F 3 "~" H 5950 3875 50  0001 C CNN
-	1    5950 3875
+P 6650 3875
+F 0 "D1" V 6689 3757 50  0000 R CNN
+F 1 "LED" V 6598 3757 50  0000 R CNN
+F 2 "LED_THT:LED_D3.0mm" H 6650 3875 50  0001 C CNN
+F 3 "~" H 6650 3875 50  0001 C CNN
+	1    6650 3875
 	0    -1   -1   0
 $EndComp
 Wire Wire Line
-	5950 3400 5950 3425
+	6650 3275 6650 3325
 $Comp
 L Device:R R3
 U 1 1 5F2B5CB8
-P 5950 3575
-F 0 "R3" H 6020 3621 50  0000 L CNN
-F 1 "680" H 6020 3530 50  0000 L CNN
-F 2 "Resistor_THT:R_Axial_DIN0207_L6.3mm_D2.5mm_P7.62mm_Horizontal" V 5880 3575 50  0001 C CNN
-F 3 "~" H 5950 3575 50  0001 C CNN
-	1    5950 3575
+P 6650 3575
+F 0 "R3" H 6720 3621 50  0000 L CNN
+F 1 "680" H 6720 3530 50  0000 L CNN
+F 2 "Resistor_THT:R_Axial_DIN0207_L6.3mm_D2.5mm_P7.62mm_Horizontal" V 6580 3575 50  0001 C CNN
+F 3 "~" H 6650 3575 50  0001 C CNN
+	1    6650 3575
 	1    0    0    -1
 $EndComp
@@
 L power:GNDD #PWR0138
 U 1 1 5FC035F6
-P 9025 1800
-F 0 "#PWR0138" H 9025 1550 50  0001 C CNN
-F 1 "GNDD" H 9029 1645 50  0000 C CNN
-F 2 "" H 9025 1800 50  0001 C CNN
-F 3 "" H 9025 1800 50  0001 C CNN
-	1    9025 1800
+P 9025 1900
+F 0 "#PWR0138" H 9025 1650 50  0001 C CNN
+F 1 "GNDD" H 9150 1900 50  0000 C CNN
+F 2 "" H 9025 1900 50  0001 C CNN
+F 3 "" H 9025 1900 50  0001 C CNN
+	1    9025 1900
 	1    0    0    -1
 $EndComp
@@
 	8925 1400 8925 1000
 Wire Wire Line
-	9025 1300 9025 1800
+	9025 1300 9025 1900
 Wire Wire Line
 	8325 1500 9175 1500
@@
 $EndComp
 $Comp
-L Device:R R5
-U 1 1 5EE9C389
-P 7075 1825
-F 0 "R5" V 7150 1775 50  0000 L CNN
-F 1 "0" V 7075 1800 50  0000 L CNN
-F 2 "Resistor_THT:R_Axial_DIN0207_L6.3mm_D2.5mm_P7.62mm_Horizontal" V 7005 1825 50  0001 C CNN
-F 3 "~" H 7075 1825 50  0001 C CNN
-	1    7075 1825
-	0    1    1    0
-$EndComp
-$Comp
 L power:GND #PWR0159
 U 1 1 5EE9FC93
 P 7725 1900
 F 0 "#PWR0159" H 7725 1650 50  0001 C CNN
-F 1 "GND" H 7800 1900 50  0000 C CNN
+F 1 "GND" H 7625 1900 50  0000 C CNN
 F 2 "" H 7725 1900 50  0001 C CNN
 F 3 "" H 7725 1900 50  0001 C CNN
@@
 $EndComp
 Wire Wire Line
-	6925 1825 6875 1825
-Wire Wire Line
-	6875 1825 6875 1875
-$Comp
-L Device:R R4
-U 1 1 5EEBE05E
-P 6850 1500
-F 0 "R4" V 6925 1450 50  0000 L CNN
-F 1 "0" V 6850 1475 50  0000 L CNN
-F 2 "Resistor_THT:R_Axial_DIN0207_L6.3mm_D2.5mm_P7.62mm_Horizontal" V 6780 1500 50  0001 C CNN
-F 3 "~" H 6850 1500 50  0001 C CNN
-	1    6850 1500
-	0    1    1    0
-$EndComp
-Wire Wire Line
-	6650 1500 6700 1500
-Wire Wire Line
 	7725 1800 7725 1900
-$Comp
-L power:GND #PWR0109
-U 1 1 5EF564D3
-P 6875 1875
-F 0 "#PWR0109" H 6875 1625 50  0001 C CNN
-F 1 "GND" H 6775 1875 50  0000 C CNN
-F 2 "" H 6875 1875 50  0001 C CNN
-F 3 "" H 6875 1875 50  0001 C CNN
-	1    6875 1875
-	1    0    0    -1
-$EndComp
 $Comp
 L Interface_CAN_LIN:MCP2562-E-P U3
@@
 L power:+3V3 #PWR0130
 U 1 1 5F296192
-P 5950 3400
-F 0 "#PWR0130" H 5950 3250 50  0001 C CNN
-F 1 "+3V3" H 5965 3573 50  0000 C CNN
-F 2 "" H 5950 3400 50  0001 C CNN
-F 3 "" H 5950 3400 50  0001 C CNN
-	1    5950 3400
-	1    0    0    -1
-$EndComp
-Wire Wire Line
-	5350 4025 5950 4025
+P 6650 3275
+F 0 "#PWR0130" H 6650 3125 50  0001 C CNN
+F 1 "+3V3" H 6665 3448 50  0000 C CNN
+F 2 "" H 6650 3275 50  0001 C CNN
+F 3 "" H 6650 3275 50  0001 C CNN
+	1    6650 3275
+	1    0    0    -1
+$EndComp
+Wire Wire Line
+	5350 4025 6650 4025
 NoConn ~ 5350 4125
 Wire Wire Line
 	5350 4225 5400 4225
 Wire Wire Line
-	5800 4225 5950 4225
-Wire Wire Line
-	5950 4225 5950 4275
+	5800 4225 5850 4225
+Wire Wire Line
+	5850 4225 5850 4275
 $Comp
 L power:GND #PWR0160
 U 1 1 5EDECAE2
-P 5950 4275
-F 0 "#PWR0160" H 5950 4025 50  0001 C CNN
-F 1 "GND" H 5955 4102 50  0000 C CNN
-F 2 "" H 5950 4275 50  0001 C CNN
-F 3 "" H 5950 4275 50  0001 C CNN
-	1    5950 4275
-	1    0    0    -1
-$EndComp
-Wire Wire Line
-	7000 1500 7225 1500
+P 5850 4275
+F 0 "#PWR0160" H 5850 4025 50  0001 C CNN
+F 1 "GND" H 5855 4102 50  0000 C CNN
+F 2 "" H 5850 4275 50  0001 C CNN
+F 3 "" H 5850 4275 50  0001 C CNN
+	1    5850 4275
+	1    0    0    -1
+$EndComp
 Wire Wire Line
 	1425 4250 1225 4250
@@
 Wire Wire Line
 	2175 1425 2525 1425
+$Comp
+L Device:R R4
+U 1 1 5EEBE05E
+P 8350 1800
+F 0 "R4" V 8275 1900 50  0000 L CNN
+F 1 "0" V 8350 1775 50  0000 L CNN
+F 2 "Resistor_THT:R_AXIAL_0_WIRE" V 8280 1800 50  0001 C CNN
+F 3 "~" H 8350 1800 50  0001 C CNN
+	1    8350 1800
+	0    1    1    0
+$EndComp
+$Comp
+L power:GND #PWR0161
+U 1 1 5EE35E26
+P 8150 1900
+F 0 "#PWR0161" H 8150 1650 50  0001 C CNN
+F 1 "GND" H 8050 1900 50  0000 C CNN
+F 2 "" H 8150 1900 50  0001 C CNN
+F 3 "" H 8150 1900 50  0001 C CNN
+	1    8150 1900
+	1    0    0    -1
+$EndComp
+$Comp
+L power:GNDD #PWR0162
+U 1 1 5EE39E34
+P 8550 1900
+F 0 "#PWR0162" H 8550 1650 50  0001 C CNN
+F 1 "GNDD" H 8675 1900 50  0000 C CNN
+F 2 "" H 8550 1900 50  0001 C CNN
+F 3 "" H 8550 1900 50  0001 C CNN
+	1    8550 1900
+	1    0    0    -1
+$EndComp
+Wire Wire Line
+	8500 1800 8550 1800
+Wire Wire Line
+	8550 1800 8550 1900
+Wire Wire Line
+	8200 1800 8150 1800
+Wire Wire Line
+	8150 1800 8150 1900
+Wire Wire Line
+	7000 1500 7225 1500
+$Comp
+L power:GND #PWR0109
+U 1 1 5EFFB0D6
+P 7225 1900
+F 0 "#PWR0109" H 7225 1650 50  0001 C CNN
+F 1 "GND" H 7125 1900 50  0000 C CNN
+F 2 "" H 7225 1900 50  0001 C CNN
+F 3 "" H 7225 1900 50  0001 C CNN
+	1    7225 1900
+	1    0    0    -1
+$EndComp
+Wire Wire Line
+	7225 1600 7225 1900
+$Comp
+L Connector_Generic:Conn_02x03_Odd_Even J2
+U 1 1 5F033C47
+P 6050 3625
+F 0 "J2" H 6100 3425 50  0000 C CNN
+F 1 "Conn_02x03_Odd_Even" H 6100 3851 50  0001 C CNN
+F 2 "Connector_PinHeader_2.54mm:PinHeader_2x03_P2.54mm_Vertical" H 6050 3625 50  0001 C CNN
+F 3 "~" H 6050 3625 50  0001 C CNN
+	1    6050 3625
+	1    0    0    -1
+$EndComp
+Wire Wire Line
+	6450 3325 6450 3625
+Wire Wire Line
+	6450 3625 6350 3625
+Wire Wire Line
+	6350 3425 6350 3525
+$Comp
+L YAAJ_STM32:BluePill_1 BP1
+U 1 1 5ED69C35
+P 4000 2475
+F 0 "BP1" H 4575 2650 50  0000 C CNN
+F 1 "BluePill_1" H 4575 2559 50  0000 C CNN
+F 2 "YAAJ_STM32:YAAJ_BluePill" H 5250 525 50  0001 C CNN
+F 3 "" H 5250 525 50  0001 C CNN
+	1    4000 2475
+	1    0    0    -1
+$EndComp
+NoConn ~ 5350 3225
+Wire Wire Line
+	5350 3525 5850 3525
+Wire Wire Line
+	5350 3625 5850 3625
+Wire Wire Line
+	5350 3425 6350 3425
+Wire Wire Line
+	5350 3325 6450 3325
+Wire Wire Line
+	6550 3725 6550 3325
+Wire Wire Line
+	6350 3725 6550 3725
+Wire Wire Line
+	6550 3325 6650 3325
+Connection ~ 6650 3325
+Wire Wire Line
+	6650 3325 6650 3425
+Wire Wire Line
+	5850 3725 5850 4225
+Connection ~ 5850 4225
 $EndSCHEMATC

Commit message: close to first release
Parts:
- removed J2: Conn_02x03_Odd_Even, Connector_PinHeader_2.54mm:PinHeader_2x03_P2.54mm_Vertical, symbol Connector_Generic:Conn_02x03_Odd_Even
- added J2: Conn_02x04_Odd_Even, Connector_PinHeader_2.54mm:PinHeader_2x04_P2.54mm_Vertical, symbol Connector_Generic:Conn_02x04_Odd_Even
- added TP1, TP2: Conn_01x01, TestPoint:Test_Point_NA, symbol Connector_Generic:Conn_01x01
- C1, C2, C30, C31, C32: footprint Capacitor_THT:C_Disc_D5.0mm_W2.5mm_P2.50mm -> Capacitor_THT:C_Disc_D3.0mm_W1.6mm_P2.50mm
- C10: footprint Capacitor_THT:C_Disc_D5.0mm_W2.5mm_P2.50mm -> Capacitor_THT:C_Disc_D3.0mm_W2.0mm_P2.50mm
- J8: footprint w_conn_misc:8p8c -> w_conn_pc:mebp8
Connections:
- net +12V: now also TP1.1 (Pin_1), TP2.1 (Pin_1)
- net +3V3: now also J2.8 (Pin_8)
- net GND: now also J2.7 (Pin_7)
- net at BP1.29 (PA4): now also J2.5 (Pin_5)
- net at BP1.30 (PA5): now also J2.3 (Pin_3)
- net at BP1.31 (PA6): now also J2.1 (Pin_1)
- net at BP1.32 (PA7): now also J2.2 (Pin_2)
- net at BP1.33 (PB0): now also J2.4 (Pin_4)
- net at BP1.34 (PB1): now also J2.6 (Pin_6)
- no-connect marks 28 -> 26
Changed lines of the file:
@@
 NoConn ~ 5350 4425
 NoConn ~ 5350 4325
-NoConn ~ 5350 3125
 NoConn ~ 3800 3225
 NoConn ~ 3800 3325
@@
 F 0 "J8" H 9245 1204 50  0000 R CNN
 F 1 "RJ45" H 9245 1295 50  0000 R CNN
-F 2 "w_conn_misc:8p8c" V 9575 1225 50  0001 C CNN
+F 2 "w_conn_pc:mebp8" V 9575 1225 50  0001 C CNN
 F 3 "~" V 9575 1225 50  0001 C CNN
 	1    9575 1200
@@
 F 0 "C10" H 1415 7321 50  0000 L CNN
 F 1 "100nF" H 1415 7230 50  0000 L CNN
-F 2 "Capacitor_THT:C_Disc_D5.0mm_W2.5mm_P2.50mm" H 1338 7125 50  0001 C CNN
+F 2 "Capacitor_THT:C_Disc_D3.0mm_W2.0mm_P2.50mm" H 1338 7125 50  0001 C CNN
 F 3 "~" H 1300 7275 50  0001 C CNN
 	1    1300 7275
@@
 F 0 "C2" H 2225 1700 50  0000 L CNN
 F 1 "100n" H 2200 1550 50  0000 L CNN
-F 2 "Capacitor_THT:C_Disc_D5.0mm_W2.5mm_P2.50mm" H 2213 1475 50  0001 C CNN
+F 2 "Capacitor_THT:C_Disc_D3.0mm_W1.6mm_P2.50mm" H 2213 1475 50  0001 C CNN
 F 3 "~" H 2175 1625 50  0001 C CNN
 	1    2175 1625
@@
 F 0 "C30" H 9800 5550 50  0000 L CNN
 F 1 "47p" H 9800 5375 50  0000 L CNN
-F 2 "Capacitor_THT:C_Disc_D5.0mm_W2.5mm_P2.50mm" H 9813 5325 50  0001 C CNN
+F 2 "Capacitor_THT:C_Disc_D3.0mm_W1.6mm_P2.50mm" H 9813 5325 50  0001 C CNN
 F 3 "~" H 9775 5475 50  0001 C CNN
 	1    9775 5475
@@
 F 0 "C31" V 8525 5425 50  0000 L CNN
 F 1 "100n" V 8625 5375 50  0000 L CNN
-F 2 "Capacitor_THT:C_Disc_D5.0mm_W2.5mm_P2.50mm" H 8613 5475 50  0001 C CNN
+F 2 "Capacitor_THT:C_Disc_D3.0mm_W1.6mm_P2.50mm" H 8613 5475 50  0001 C CNN
 F 3 "~" H 8575 5625 50  0001 C CNN
 	1    8575 5625
@@
 F 0 "C32" V 8750 6450 50  0000 L CNN
 F 1 "1n" V 8875 6475 50  0000 L CNN
-F 2 "Capacitor_THT:C_Disc_D5.0mm_W2.5mm_P2.50mm" H 8863 6250 50  0001 C CNN
+F 2 "Capacitor_THT:C_Disc_D3.0mm_W1.6mm_P2.50mm" H 8863 6250 50  0001 C CNN
 F 3 "~" H 8825 6400 50  0001 C CNN
 	1    8825 6400
@@
 	1150 1425 1200 1425
 Wire Wire Line
-	1200 1425 1200 2400
+	1200 1425 1200 2050
 Wire Wire Line
 	1200 2400 1500 2400
@@
 F 0 "C1" H 1525 1700 50  0000 L CNN
 F 1 "100n" H 1525 1550 50  0000 L CNN
-F 2 "Capacitor_THT:C_Disc_D5.0mm_W2.5mm_P2.50mm" H 1538 1475 50  0001 C CNN
+F 2 "Capacitor_THT:C_Disc_D3.0mm_W1.6mm_P2.50mm" H 1538 1475 50  0001 C CNN
 F 3 "~" H 1500 1625 50  0001 C CNN
 	1    1500 1625
@@
 	7225 1600 7225 1900
 $Comp
-L Connector_Generic:Conn_02x03_Odd_Even J2
-U 1 1 5F033C47
-P 6050 3625
-F 0 "J2" H 6100 3425 50  0000 C CNN
-F 1 "Conn_02x03_Odd_Even" H 6100 3851 50  0001 C CNN
-F 2 "Connector_PinHeader_2.54mm:PinHeader_2x03_P2.54mm_Vertical" H 6050 3625 50  0001 C CNN
-F 3 "~" H 6050 3625 50  0001 C CNN
-	1    6050 3625
-	1    0    0    -1
-$EndComp
-Wire Wire Line
-	6450 3325 6450 3625
-Wire Wire Line
-	6450 3625 6350 3625
-Wire Wire Line
-	6350 3425 6350 3525
-$Comp
 L YAAJ_STM32:BluePill_1 BP1
 U 1 1 5ED69C35
@@
 	1    0    0    -1
 $EndComp
-NoConn ~ 5350 3225
 Wire Wire Line
 	5350 3525 5850 3525
 Wire Wire Line
 	5350 3625 5850 3625
-Wire Wire Line
-	5350 3425 6350 3425
-Wire Wire Line
-	5350 3325 6450 3325
 Wire Wire Line
 	6550 3725 6550 3325
@@
 	5850 3725 5850 4225
 Connection ~ 5850 4225
+$Comp
+L Connector_Generic:Conn_01x01 TP1
+U 1 1 5EE1214D
+P 1000 2050
+F 0 "TP1" H 918 1917 50  0000 C CNN
+F 1 "Conn_01x01" H 918 1916 50  0001 C CNN
+F 2 "TestPoint:Test_Point_NA" H 1000 2050 50  0001 C CNN
+F 3 "~" H 1000 2050 50  0001 C CNN
+	1    1000 2050
+	-1   0    0    1
+$EndComp
+Connection ~ 1200 2050
+Wire Wire Line
+	1200 2050 1200 2300
+$Comp
+L Connector_Generic:Conn_01x01 TP2
+U 1 1 5EE12B1B
+P 1000 2300
+F 0 "TP2" H 918 2167 50  0000 C CNN
+F 1 "Conn_01x01" H 918 2166 50  0001 C CNN
+F 2 "TestPoint:Test_Point_NA" H 1000 2300 50  0001 C CNN
+F 3 "~" H 1000 2300 50  0001 C CNN
+	1    1000 2300
+	-1   0    0    1
+$EndComp
+Connection ~ 1200 2300
+Wire Wire Line
+	1200 2300 1200 2400
+$Comp
+L Connector_Generic:Conn_02x04_Odd_Even J2
+U 1 1 5EE2DFC1
+P 6050 3525
+F 0 "J2" H 6100 3750 50  0000 C CNN
+F 1 "Conn_02x04_Odd_Even" H 6100 3751 50  0001 C CNN
+F 2 "Connector_PinHeader_2.54mm:PinHeader_2x04_P2.54mm_Vertical" H 6050 3525 50  0001 C CNN
+F 3 "~" H 6050 3525 50  0001 C CNN
+	1    6050 3525
+	1    0    0    -1
+$EndComp
+Wire Wire Line
+	5350 3425 5850 3425
+Wire Wire Line
+	5350 3325 6400 3325
+Wire Wire Line
+	6400 3325 6400 3425
+Wire Wire Line
+	6400 3425 6350 3425
+Wire Wire Line
+	5350 3225 6450 3225
+Wire Wire Line
+	6450 3225 6450 3525
+Wire Wire Line
+	6450 3525 6350 3525
+Wire Wire Line
+	5350 3125 6500 3125
+Wire Wire Line
+	6500 3125 6500 3625
+Wire Wire Line
+	6500 3625 6350 3625
 $EndSCHEMATC
