File: c6021light/bluepill/hardware/c6021light.kicad_pcb (KiCad board)
At the start: 2 copper layers, 100 x 50 mm, 82 parts, among them J1 Barrel_Jack_Switch, J10 Conn_01x02, J11 Conn_01x02, J12 XpressNet, J2 Conn_02x04_Odd_Even, J3 Conn_02x16_Row_Letter_First, J30 Loconet, J31 Conn_01x02, J32 Conn_01x02, J4 Conn_01x02, J5 Grove I2C, J50 USB_B_Micro, J51 Conn_01x06, J52 Debug UART, J6 Conn_01x02, J7 Conn_01x02, J8 RJ45, Q30 BC337, Q31 BC547, Q32 BC547, SW1 SW_Push, U1 L7805, U10 SN75176, U2 L7808, U3 MCP2562, U30 LM393, U4 ISO1050DUB, U50 CH340C

Commit message: work on new revision
Parts:
- moved U2 2.72 mm to (113.7, 90.3)
- moved TP2 2.72 mm to (113.7, 87.8)
- moved C3 2.32 mm to (118.3, 88.9)
- moved C4 2.21 mm to (118.3, 96.3)
- moved J1 2.10 mm to (103.8, 87.0)
- moved J11 0.70 mm to (113.1, 85.0)
- moved J3 0.19 mm to (166.9, 94.3)
Connections:
- J8 pad 5: GNDD -> Net-(J8-Pad5)
- TP1 pad 1: +12V -> Net-(TP1-Pad1)
- TP2 pad 1: +12V -> Net-(TP2-Pad1)
Routing:
- net GND: track 223.2 -> 242.1 mm
- net Net-(J11-Pad2): track 100.7 -> 97.3 mm, vias 4 -> 3
- net +12V: track 175.0 -> 173.1 mm
- net Net-(J6-Pad1): track 32.0 -> 31.2 mm
- net +8V: track 62.1 -> 61.5 mm
Other:
- board text added: "Damian Philipp 2020/08 Gerhard Bertelsmann"
- board text removed: "Damian Philipp 2020/06 Gerhard Bertelsmann"
