File: s88isolated/s88iso/s88iso.kicad_pcb (KiCad board)
At the start: 2 copper layers, 70 x 50 mm, 30 parts, among them J1 Barrel_Jack_Switch_MountingPin, J2 5V Bypass, J3 12V 5V, J4 Conn_01x04, U1 L7805, U2 4504, U3 Si8641BB-B-IS1

Commit message: update
Parts:
- U3: value Si8641BB-B-IS1 -> Si8641BB-B
- renumbered InputS88 to Input_S88, ZentraleS88 to Zentrale_S88
