File: s88isolated/s88iso/s88iso.sch (KiCad schematic (older format))
At the start: 12 parts

Commit message: wip
Parts:
- removed J?: Barrel_Jack_MountingPin, symbol Connector:Barrel_Jack_MountingPin
- added C1, C2, C3, C4, C6: 100nF, Capacitor_SMD:C_0805_2012Metric, symbol Device:C
- added J1: Barrel_Jack_Switch_MountingPin, w_conn_misc:dc_socket, symbol Connector:Barrel_Jack_Switch_MountingPin
- added J2: 5V Bypass, Connector_PinHeader_2.54mm:PinHeader_1x02_P2.54mm_Vertical, symbol Connector_Generic:Conn_01x02
- added R1, R2, R3: 47, Resistor_SMD:R_0805_2012Metric, symbol Device:R
- added R5: 10k, Resistor_SMD:R_0805_2012Metric, symbol Device:R
- added S88: Conn_01x06, Connector_PinSocket_2.54mm:PinSocket_1x06_P2.54mm_Horizontal, symbol Connector_Generic:Conn_01x06
- added U1: L7805, Package_TO_SOT_SMD:TO-252-2, symbol Regulator_Linear:L7805
- C5: renamed from C?; value C -> 1nF; footprint (none) -> Capacitor_SMD:C_0805_2012Metric
- C7: renamed from C?; value C -> 100nF; footprint (none) -> Capacitor_SMD:C_0805_2012Metric
- InputS88, ZentraleS88: renamed from J?; footprint (none) -> w_conn_pc:megb8-8-Uni
- R4, R6, R7, R8, R9: renamed from R?; footprint (none) -> Resistor_SMD:R_0805_2012Metric
- U2: renamed from U?; footprint (none) -> w_smd_dil:so-16
- U3: renamed from U?; footprint Package_SO:SOIC-16_3.9x9.9mm_P1.27mm -> w_smd_dil:so-16
Connections:
- net labels added: +5V, Clock', Data, Data', PSLoad', Reset', VDD
- wire segments 44 -> 108
- no-connect marks 2 -> 5
Other:
- moved on the sheet: C5, C7, InputS88, R4, R6, R7, R8, R9, U2, U3, ZentraleS88

Commit message: first production version
Parts:
- added J3: 12V 5V, Connector_PinHeader_2.54mm:PinHeader_1x03_P2.54mm_Vertical, symbol Connector_Generic:Conn_01x03
- added J4: Conn_01x04, Connector_PinSocket_2.54mm:PinSocket_1x04_P2.54mm_Vertical, symbol Connector_Generic:Conn_01x04
Connections:
- net +5VD: now also J3.3 (Pin_3), J4.4 (Pin_4)
- net Clock': now also R1.1; no longer R3.1
- net GNDD: now also J4.3 (Pin_3)
- net Reset': now also R3.1; no longer R1.1
- net VDD: now also J3.2 (Pin_2); no longer C1.1, J1.3, J2.1 (Pin_1), U1.1 (IN)
- net at U2.3 (Ain): now also U3.14 (B1); no longer U3.12 (B3)
- net at U2.7 (Cin): now also U3.12 (B3); no longer U3.14 (B1)
- new net Input: C1.1, J1.3, J2.1 (Pin_1), J3.1 (Pin_1), J4.2 (Pin_2), U1.1 (IN)
- no-connect marks 5 -> 7
Other:
- moved on the sheet: C1, C2, C3, C4, C5, C6, C7, InputS88, J1, J2, R1, R2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

Commit message: update
Parts:
- U3: value Si8641BB-B-IS1 -> Si8641BB-B
- renumbered InputS88 to Input_S88, ZentraleS88 to Zentrale_S88
Changed lines of the file:
@@
 $EndDescr
 $Comp
-L Connector:RJ45 ZentraleS88
+L Connector:RJ45 Zentrale_S88
 U 1 1 5DEC0ABC
 P 9050 4275
-F 0 "ZentraleS88" H 8721 4279 50  0000 R CNN
+F 0 "Zentrale_S88" H 8721 4279 50  0000 R CNN
 F 1 "RJ45" H 8721 4370 50  0000 R CNN
 F 2 "w_conn_pc:megb8-8-Uni" V 9050 4300 50  0001 C CNN
@@
 $EndComp
 $Comp
-L Connector:RJ45 InputS88
+L Connector:RJ45 Input_S88
 U 1 1 5DEC1D69
 P 2950 4175
-F 0 "InputS88" H 2620 4179 50  0000 R CNN
+F 0 "Input_S88" H 2620 4179 50  0000 R CNN
 F 1 "RJ45" H 2620 4270 50  0000 R CNN
 F 2 "w_conn_pc:megb8-8-Uni" V 2950 4200 50  0001 C CNN
@@
 P 6875 4250
 F 0 "U3" H 6875 4917 50  0000 C CNN
-F 1 "Si8641BB-B-IS1" H 6875 4826 50  0000 C CNN
+F 1 "Si8641BB-B" H 6875 4826 50  0000 C CNN
 F 2 "w_smd_dil:so-16" H 6875 3700 50  0001 C CIN
 F 3 "https://www.silabs.com/documents/public/data-sheets/si864x-datasheet.pdf" H 6875 4650 50  0001 C CNN
